File: hardware/require.kicad_pcb (KiCad board)
At the start: 6 copper layers, 70 x 25.4 mm, 67 parts, among them J1 Conn_01x02, J9100 microSD-13p, U1 SY8088AAC, U1000 RK3308, U13 SY8088AAC, U3 EMMC_BGA_153, U3000 DDR3_FBGA96, U6000 ap6255

Commit message: wip
Parts:
- removed C1: 1u, Resistors_SMD:R_0402_NoSilk
- removed C11, C6: C, Capacitors_SMD:C_0603
- removed C15, C17, C3, C4, C5: C, Capacitors_SMD:C_0402
- removed C2: C, Capacitors_SMD:C_0402_NoSilk
- removed C2200: 10uF,10V,X5R, Capacitors_SMD:C_0805
- removed C2201: 22u, Resistors_SMD:R_0603
- removed C2202: 0.1u, Resistors_SMD:R_0402_NoSilk
- removed J9100: microSD-13p, require:xunpu_microSD_tf_115
- removed L1: 22uH, Inductors_SMD:L_Taiyo-Yuden_MD-4040
- removed L2: L, Inductors_SMD:L_Taiyo-Yuden_MD-4040
- removed R1, R2, R3, R4, R5, R6: R, Resistors_SMD:R_0402
- removed R1712: 22R, Resistors_SMD:R_0402
- removed R2200: 10k, Resistors_SMD:R_0402_NoSilk
- removed REF**: USB_C_Receptacle_Amphenol_12401610E4-2A, Connectors_USB:USB_C_Receptacle_Amphenol_12401610E4-2A
- removed U1, U13: SY8088AAC, TO_SOT_Packages_SMD:SOT-23-5
- added C100: 0.1u,10V, Capacitors_SMD:C_0402, B.Cu at (67.9, 57.2)
- added C101: 10u,10V, Capacitors_SMD:C_0805, B.Cu at (69.2, 57.2)
- added C102: 1n, Capacitors_SMD:C_0402, B.Cu at (76.0, 57.5)
- added C103: 22p, Capacitors_SMD:C_0402, F.Cu at (69.9, 55.9)
- added C104: 22u, Capacitors_SMD:C_0603, B.Cu at (69.9, 62.7)
- added C105: 0.1u, Capacitors_SMD:C_0402, B.Cu at (68.2, 60.5)
- added C106: 0.1u, Capacitors_SMD:C_0402, B.Cu at (67.3, 60.5)
- added C107: 0.1u, Capacitors_SMD:C_0402, B.Cu at (66.3, 60.5)
- added C108: 0.1u, Capacitors_SMD:C_0402, B.Cu at (69.2, 60.5)
- added C110: 0.1u, Capacitors_SMD:C_0402, F.Cu at (67.0, 55.9)
- added C1102: 0.1u, Capacitors_SMD:C_0402, F.Cu at (59.1, 72.9)
- added C122: C, Capacitors_SMD:C_0402, F.Cu at (40.2, 60.8)
- added C123: C, Capacitors_SMD:C_0402, F.Cu at (37.8, 60.8)
- added C20: 22p, Resistors_SMD:R_0402_NoSilk, B.Cu at (140.0, 47.6)
- added C200: 0.1u,10V, Capacitors_SMD:C_0402, B.Cu at (54.3, 57.2)
- added C201: 10u,10V, Capacitors_SMD:C_0805, B.Cu at (55.6, 57.2)
- added C202: 1n, Capacitors_SMD:C_0402, F.Cu at (26.1, 30.5)
- added C203: 22p, Capacitors_SMD:C_0402, F.Cu at (21.5, 35.0)
- added C204: 22u, Capacitors_SMD:C_0603, B.Cu at (58.2, 62.4)
- added C205: 0.1u, Capacitors_SMD:C_0402, B.Cu at (58.2, 63.4)
- added C206: 10u, Capacitors_SMD:C_0603, B.Cu at (63.4, 65.3)
- added C207: 0.1u, Capacitors_SMD:C_0402, B.Cu at (64.3, 65.3)
- added C208: 0.1u, Capacitors_SMD:C_0402, B.Cu at (65.2, 65.3)
- added C22: 22u, Resistors_SMD:R_0603, B.Cu at (131.6, 53.7)
- added C24: 0.1u, Resistors_SMD:R_0402_NoSilk, B.Cu at (141.6, 47.6)
- added C300: 0.1u,10V, Capacitors_SMD:C_0402, F.Cu at (46.8, 30.6)
- added C301: 10u,10V, Capacitors_SMD:C_0805, F.Cu at (44.0, 29.9)
- added C302: 1n, Capacitors_SMD:C_0402, F.Cu at (49.9, 27.2)
- added C303: 22p, Capacitors_SMD:C_0402, F.Cu at (50.0, 25.9)
- added C304: 22u, Capacitors_SMD:C_0603, F.Cu at (47.5, 26.0)
- added C305: 0.1u, Capacitors_SMD:C_0402, F.Cu at (46.8, 29.5)
- added C6008: 4.7u, Capacitors_SMD:C_0603, B.Cu at (56.0, 68.0)
- added L100: 2.2u, require:L_murata_2520, B.Cu at (71.8, 60.5)
- added L123: L, Inductors_SMD:L_0402, F.Cu at (39.0, 61.4)
- added L200: 2.2u, require:L_murata_2520, B.Cu at (58.2, 60.5)
- added L3: 3.3u, require:L_murata_2520, B.Cu at (90.4, 58.8)
- added L300: 2.2u, require:L_murata_2520, F.Cu at (47.5, 27.8)
- added L6002: 3.3u, require:L_murata_2520, B.Cu at (53.0, 74.0)
- added R10: 10, Resistors_SMD:R_0402_NoSilk, B.Cu at (141.4, 49.5)
- added R100: 10k, Resistors_SMD:R_0402, B.Cu at (76.0, 56.5)
- added R101: 100R,1%, Resistors_SMD:R_0402, F.Cu at (72.8, 55.9)
- added R102: 100k,1%, Resistors_SMD:R_0402, F.Cu at (70.8, 55.9)
- added R103: 150k,1%, Resistors_SMD:R_0402, F.Cu at (68.9, 55.9)
- added R110: 10k, Resistors_SMD:R_0402, F.Cu at (67.9, 55.9)
- added R113: 12k,1%, Resistors_SMD:R_0402, F.Cu at (64.0, 55.9)
- added R200: 10k, Resistors_SMD:R_0402, F.Cu at (37.5, 40.5)
- added R202: 110k,1%, Resistors_SMD:R_0402, F.Cu at (25.6, 36.2)
- added R203: 150k,1%, Resistors_SMD:R_0402, F.Cu at (51.5, 43.5)
- added R300: 10k, Resistors_SMD:R_0402, F.Cu at (51.8, 27.1)
- added R302: 110k,1%, Resistors_SMD:R_0402, F.Cu at (51.8, 25.9)
- added R303: 150k,1%, Resistors_SMD:R_0402, F.Cu at (48.7, 29.4)
- added R7: 10k, Resistors_SMD:R_0402_NoSilk, B.Cu at (141.6, 48.5)
- added R9: 100,5%, Resistors_SMD:R_0402_NoSilk, B.Cu at (137.0, 53.4)
- added U100: SY8089AAC, TO_SOT_Packages_SMD:SOT-23-5, B.Cu at (71.8, 57.2)
- added U15: SY8088AAC, TO_SOT_Packages_SMD:SOT-23-5, B.Cu at (90.3, 55.8)
- added U200: SY8089AAC, TO_SOT_Packages_SMD:SOT-23-5, B.Cu at (58.2, 57.2)
- added U300: SY8089AAC, TO_SOT_Packages_SMD:SOT-23-5, F.Cu at (44.2, 27.2)
- added Y1: Crystal_GND24, Crystals:Crystal_SMD_3225-4pin_3.2x2.5mm, B.Cu at (59.0, 71.4)
- C150, C151, C1700, U3: moved to B.Cu
- C16: value C -> 10uF,10V,X5R; footprint Capacitors_SMD:C_0402 -> Capacitors_SMD:C_0805
- C18: value C -> 1u; footprint Capacitors_SMD:C_0402 -> Resistors_SMD:R_0402_NoSilk
- R111: value 100,5% -> 10k,1%; footprint Resistors_SMD:R_0402_NoSilk -> Resistors_SMD:R_0402
- R112: value 10 -> 27k,1%; footprint Resistors_SMD:R_0402_NoSilk -> Resistors_SMD:R_0402
- moved R112 101.0 mm to (65.0, 55.9), turned to 90 degrees
- moved R111 100.0 mm to (66.0, 55.9), turned to 90 degrees
- moved C1701 55.6 mm to (68.0, 82.0)
- moved C1700 41.7 mm to (61.1, 65.0), turned to 180 degrees
- moved U6000 10.0 mm to (48.0, 65.0)
- moved U3 3.00 mm to (48.0, 65.0)
Connections:
- net /test/SDMMC_PWREN renamed Net-(U1000-PadB14)
- C16 pad 1: VCC_DDR -> VCC5V0_SYS
- R111 pad 1: VDD_CORE -> Net-(C110-Pad1)
- R111 pad 2: Net-(R111-Pad2) -> GND
- R112 pad 1: Net-(R111-Pad2) -> Net-(C110-Pad1)
- R112 pad 2: GND -> /rk3308-power/CORE_DVS
- U1000 pad A15: /test/SDMMC_D3 -> Net-(U1000-PadA15)
- U1000 pad A17: /test/SDMMC_D1 -> Net-(U1000-PadA17)
- U1000 pad B15: /test/SDMMC_D2 -> Net-(U1000-PadB15)
- U1000 pad B17: /test/SDMMC_D0 -> Net-(U1000-PadB17)
- U1000 pad B20: (no net) -> /rk3308-power/RESET
- U1000 pad C16: /test/SDMMC_CMD -> Net-(U1000-PadC16)
- U1000 pad C19: (no net) -> GND
- U1000 pad C20: (no net) -> Net-(U1000-PadC20)
- U1000 pad D19: (no net) -> GND
- U1000 pad E15: (no net) -> Net-(U1000-PadE15)
- U1000 pad E17: (no net) -> Net-(U1000-PadE17)
- U1000 pad E19: (no net) -> Net-(U1000-PadE19)
- U1000 pad E20: (no net) -> Net-(U1000-PadE20)
- U1000 pad F10: Net-(U1000-PadF10) -> VDD_LOG
- U1000 pad F11: Net-(U1000-PadF11) -> VDD_LOG
- U1000 pad F12: Net-(U1000-PadF12) -> VDD_LOG
- U1000 pad G10: Net-(U1000-PadG10) -> VDD_LOG
- U1000 pad G11: Net-(U1000-PadG11) -> VDD_LOG
- U1000 pad G12: Net-(U1000-PadG12) -> VDD_LOG
- U1000 pad G15: (no net) -> Net-(U1000-PadG15)
- U1000 pad N6: Net-(U1000-PadN6) -> VDD_CORE
- U1000 pad N7: Net-(U1000-PadN7) -> VDD_CORE
- U1000 pad N8: Net-(U1000-PadN8) -> VDD_CORE
- U1000 pad P5: Net-(U1000-PadP5) -> VDD_CORE
- U1000 pad P6: Net-(U1000-PadP6) -> VDD_CORE
- U1000 pad P7: Net-(U1000-PadP7) -> VDD_CORE
- U1000 pad R5: Net-(U1000-PadR5) -> VDD_CORE
- U1000 pad R6: Net-(U1000-PadR6) -> VDD_CORE
- U1000 pad R8: Net-(U1000-PadR8) -> VDD_CORE
- U6000 pad 1: Net-(U6000-Pad1) -> GND
- U6000 pad 20: Net-(U6000-Pad20) -> GND
- U6000 pad 22: Net-(U6000-Pad22) -> VCCIO_SDIO
- U6000 pad 3: Net-(U6000-Pad3) -> GND
- U6000 pad 31: Net-(U6000-Pad31) -> GND
- U6000 pad 33: Net-(U6000-Pad33) -> GND
Routing:
- net GND: track 97.6 -> 125.6 mm, vias 142 -> 109
- net /test/SDMMC_D1: track 26.8 -> 0.00 mm, vias 1 -> 0
- net /ddr/DDR_DQS0P: track 24.8 -> 0.00 mm
- net /ddr/DDR_DQS0N: track 24.8 -> 0.00 mm
- net VDD_CORE: track 0.00 -> 24.7 mm, vias 0 -> 13
- net /test/SDMMC_D0: track 24.0 -> 0.00 mm, vias 1 -> 0
- net /emmc/FLASH_D7: track 26.5 -> 6.43 mm, vias 2 -> 1
- net /test/SDMMC_CMD: track 18.9 -> 0.00 mm, vias 1 -> 0
- net /test/SDMMC_CLK: track 17.5 -> 0.00 mm
- net /test/SDMMC_D3: track 15.4 -> 0.00 mm, vias 1 -> 0
- net /emmc/FLASH_CLK: track 20.6 -> 5.66 mm, vias 2 -> 1
- net /test/SDMMC_D2: track 13.1 -> 0.00 mm, vias 1 -> 0
- net /emmc/FLASH_D2: track 18.7 -> 6.26 mm
- net /emmc/FLASH_D5: track 15.1 -> 2.73 mm
- net /emmc/FLASH_D3: track 12.9 -> 0.98 mm
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- added copper zone on B.Cu, net GND
- added copper zone on F.Cu, net GND
- added copper zone on B.Cu, net VDD_CORE
- added copper zone on In3.Cu, net VDD_CORE
- added copper zone on B.Cu, net VDD_LOG
Other:
- net class 2A added: clearance 0.1, trace_width 0.8, via_dia 0.6, via_drill 0.4
- net class Default: trace_width 0.15 -> 0.2
- net class GND3: trace_width 0.15 -> 0.2

Commit message: wip
Parts:
- removed C10: C, Capacitors_SMD:C_0402
- removed C102, C202, C302: 1n, Capacitors_SMD:C_0402
- removed C16: 10uF,10V,X5R, Capacitors_SMD:C_0805
- removed C18: 1u, Resistors_SMD:R_0402_NoSilk
- removed C20: 22p, Resistors_SMD:R_0402_NoSilk
- removed C205, C305: 0.1u, Capacitors_SMD:C_0402
- removed C22: 22u, Resistors_SMD:R_0603
- removed C24: 0.1u, Resistors_SMD:R_0402_NoSilk
- removed L3: 3.3u, require:L_murata_2520
- removed R10: 10, Resistors_SMD:R_0402_NoSilk
- removed R7: 10k, Resistors_SMD:R_0402_NoSilk
- removed R9: 100,5%, Resistors_SMD:R_0402_NoSilk
- removed U15: SY8088AAC, TO_SOT_Packages_SMD:SOT-23-5
- added C400: 0.1u,10V, Capacitors_SMD:C_0402, F.Cu at (95.5, 72.5)
- added C401: 10u,10V, Capacitors_SMD:C_0805, F.Cu at (93.0, 75.0)
- added C403: 22p, Capacitors_SMD:C_0402, F.Cu at (92.5, 70.0)
- added C404: 22u, Capacitors_SMD:C_0603, F.Cu at (88.0, 72.5)
- added C5123: 0.1u, Capacitors_SMD:C_0402, B.Cu at (64.5, 61.5)
- added C5124: 0.1u, Capacitors_SMD:C_0402, B.Cu at (70.5, 63.0)
- added L400: 2.2u, require:L_murata_2520, F.Cu at (90.0, 72.5)
- added R400: 10k, Resistors_SMD:R_0402, F.Cu at (91.5, 70.0)
- added R402: 110k,1%, Resistors_SMD:R_0402, F.Cu at (93.5, 70.0)
- added R403: 150k,1%, Resistors_SMD:R_0402, F.Cu at (94.5, 70.0)
- added U400: SY8089AAC, TO_SOT_Packages_SMD:SOT-23-5, F.Cu at (93.0, 72.5)
- C103, C110, C1984, C203, R101, R102, R103, R110, R111, R112, R113, R200, R202, R203: moved to B.Cu
- C107: value 0.1u -> 2.2u
- C108: value 0.1u -> 22u; footprint Capacitors_SMD:C_0402 -> Capacitors_SMD:C_0603
- C310: renamed from C7; value C -> 10u; moved to B.Cu
- C311: renamed from C8; value C -> 0.1u; moved to B.Cu
- C312: renamed from C9; value C -> 0.1u; moved to B.Cu
- moved C203 79.2 mm to (92.5, 70.0), turned to 90 degrees
- moved R202 75.8 mm to (93.5, 70.0), turned to 90 degrees
- moved R200 61.5 mm to (91.5, 70.0), turned to 270 degrees
- moved U300 60.3 mm to (93.0, 62.5)
- moved C301 60.2 mm to (93.0, 65.0), turned to 180 degrees
- moved C300 58.2 mm to (95.5, 62.5), turned to 90 degrees
- moved R303 55.1 mm to (94.5, 60.0), turned to 90 degrees
- moved L300 54.9 mm to (90.0, 62.5), turned to 90 degrees
- moved C303 54.5 mm to (92.5, 60.0), turned to 270 degrees
- moved C304 54.5 mm to (88.0, 62.5), turned to 270 degrees
- moved R302 53.8 mm to (93.5, 60.0), turned to 270 degrees
- moved R300 51.6 mm to (91.5, 60.0), turned to 90 degrees
- moved R203 50.5 mm to (94.5, 70.0), turned to 270 degrees
- moved C311 45.8 mm to (66.8, 65.7), turned to 90 degrees
- moved C200 42.5 mm to (95.5, 67.5), turned to 270 degrees
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Connections:
- C303 pad 1: VDD_CORE -> VCC_DDR
- C304 pad 1: VDD_CORE -> VCC_DDR
- L300 pad 2: VDD_CORE -> VCC_DDR
- R302 pad 1: VDD_CORE -> VCC_DDR
- U1000 pad G15: Net-(U1000-PadG15) -> GND
- U1000 pad N2: (no net) -> Net-(U1000-PadN2)
- U1000 pad N3: (no net) -> /rk3308-lcdc-mac-i2s1-jtag/WIFI_WAKE_HOST
- U1000 pad N4: (no net) -> Net-(U1000-PadN4)
- U1000 pad N5: (no net) -> VCC_IO
- U1000 pad P3: (no net) -> /rk3308-lcdc-mac-i2s1-jtag/WIFI_REG_ON
- U1000 pad P4: (no net) -> Net-(U1000-PadP4)
- U1000 pad R11: (no net) -> VCC_IO
- U1000 pad R3: (no net) -> Net-(U1000-PadR3)
- U1000 pad R4: (no net) -> Net-(U1000-PadR4)
- U1000 pad R9: (no net) -> Net-(U1000-PadR9)
- U1000 pad T1: (no net) -> Net-(U1000-PadT1)
- U1000 pad T10: (no net) -> /rk3308-lcdc-mac-i2s1-jtag/SPI2_CS
- U1000 pad T2: (no net) -> Net-(U1000-PadT2)
- U1000 pad T3: (no net) -> Net-(U1000-PadT3)
- U1000 pad T4: (no net) -> Net-(U1000-PadT4)
- U1000 pad T5: (no net) -> Net-(U1000-PadT5)
- U1000 pad T6: (no net) -> Net-(U1000-PadT6)
- U1000 pad T8: (no net) -> Net-(U1000-PadT8)
- U1000 pad T9: (no net) -> /rk3308-lcdc-mac-i2s1-jtag/SPI2_TX_UART2_TX_M0
- U1000 pad U2: (no net) -> Net-(U1000-PadU2)
- U1000 pad U3: (no net) -> Net-(U1000-PadU3)
- U1000 pad U4: (no net) -> Net-(U1000-PadU4)
- U1000 pad U5: (no net) -> Net-(U1000-PadU5)
- U1000 pad U6: (no net) -> Net-(U1000-PadU6)
- U1000 pad U7: (no net) -> Net-(U1000-PadU7)
- U1000 pad U8: (no net) -> Net-(U1000-PadU8)
- U1000 pad U9: (no net) -> Net-(U1000-PadU9)
- U1000 pad V1: (no net) -> Net-(U1000-PadV1)
- U1000 pad V10: (no net) -> /rk3308-lcdc-mac-i2s1-jtag/SPI2_CLK
- U1000 pad V2: (no net) -> Net-(U1000-PadV2)
- U1000 pad V3: (no net) -> Net-(U1000-PadV3)
- U1000 pad V4: (no net) -> Net-(U1000-PadV4)
- U1000 pad V5: (no net) -> Net-(U1000-PadV5)
- U1000 pad V6: (no net) -> Net-(U1000-PadV6)
- U1000 pad V7: (no net) -> Net-(U1000-PadV7)
- U1000 pad V8: (no net) -> Net-(U1000-PadV8)
- U1000 pad V9: (no net) -> Net-(U1000-PadV9)
- U1000 pad W1: (no net) -> Net-(U1000-PadW1)
- U1000 pad W2: (no net) -> Net-(U1000-PadW2)
- U1000 pad W3: (no net) -> Net-(U1000-PadW3)
- U1000 pad W4: (no net) -> Net-(U1000-PadW4)
- U1000 pad W5: (no net) -> Net-(U1000-PadW5)
- U1000 pad W6: (no net) -> Net-(U1000-PadW6)
- U1000 pad W7: (no net) -> Net-(U1000-PadW7)
- U1000 pad W9: (no net) -> /rk3308-lcdc-mac-i2s1-jtag/SPI2_RX_UART2_RX_M0
- U1000 pad Y2: (no net) -> Net-(U1000-PadY2)
- U1000 pad Y3: (no net) -> Net-(U1000-PadY3)
- U1000 pad Y5: (no net) -> Net-(U1000-PadY5)
- U1000 pad Y7: (no net) -> Net-(U1000-PadY7)
- U1000 pad Y9: (no net) -> Net-(U1000-PadY9)
Routing:
- net GND: track 125.6 -> 195.7 mm, vias 109 -> 126
- net VCC_DDR: track 32.8 -> 52.3 mm, vias 23 -> 25
- net VCC5V0_SYS: track 1.84 -> 17.0 mm, vias 0 -> 5
- net VCC_IO: track 0.00 -> 14.4 mm, vias 0 -> 1
- net VDD_CORE: track 24.7 -> 38.1 mm
- net VDD_LOG: track 10.6 -> 19.0 mm, vias 6 -> 7
- net /ddr/DDR_CASN: track 16.0 -> 11.9 mm
- net Net-(C403-Pad2): track 0.00 -> 3.54 mm
- net Net-(C203-Pad2): track 0.00 -> 3.51 mm
- net Net-(C303-Pad2): track 0.00 -> 3.31 mm
- net Net-(R400-Pad1): track 0.00 -> 1.50 mm
- net Net-(R200-Pad1): track 0.00 -> 1.47 mm
- net /ddr/DDR_DQS0N: track 0.00 -> 1.33 mm, vias 0 -> 2
- net /ddr/DDR_DQS0P: track 0.00 -> 1.27 mm, vias 0 -> 2
- net Net-(R300-Pad1): track 0.00 -> 1.27 mm
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- added copper zone on In4.Cu, net VCC5V0_SYS
- added copper zone on B.Cu, net VCC_DDR
- added copper zone on In3.Cu, net VDD_LOG

Commit message: wip
Parts:
- removed C1102: 0.1u, Capacitors_SMD:C_0402
- removed Y1: Crystal_GND24, Crystals:Crystal_SMD_3225-4pin_3.2x2.5mm
- added C220: 15p, Capacitors_SMD:C_0402, B.Cu at (57.2, 74.1)
- added C221: 15p, Capacitors_SMD:C_0402, B.Cu at (59.1, 74.1)
- added C225: 0.1u, Capacitors_SMD:C_0402, F.Cu at (59.2, 72.6)
- added C230: 0.1u, Capacitors_SMD:C_0402, B.Cu at (61.1, 68.9)
- added C231: 0.1u, Capacitors_SMD:C_0402, B.Cu at (59.1, 67.6)
- added C410: 1u, Capacitors_SMD:C_0402, B.Cu at (90.0, 73.5)
- added C413: 1u, Capacitors_SMD:C_0402, B.Cu at (95.5, 72.5)
- added FB400: L, Inductors_SMD:L_0603, B.Cu at (63.4, 68.9)
- added R220: 22R, Resistors_SMD:R_0402, B.Cu at (56.9, 68.9)
- added R230: 1R, Resistors_SMD:R_0402, B.Cu at (62.4, 68.9)
- added R410: 10k, Resistors_SMD:R_0402, B.Cu at (90.0, 71.5)
- added R420: 0R, Resistors_SMD:R_0402, F.Cu at (62.3, 91.6)
- added R421: 0R, Resistors_SMD:R_0402, F.Cu at (62.3, 92.8)
- added R422: 0R, Resistors_SMD:R_0402, F.Cu at (64.0, 91.6)
- added R423: 1R, Resistors_SMD:R_0402, F.Cu at (64.0, 92.8)
- added R425: 0R, Resistors_SMD:R_0402, F.Cu at (63.5, 83.0)
- added R426: 0R, Resistors_SMD:R_0402, F.Cu at (58.3, 93.8)
- added R429: 1R, Resistors_SMD:R_0402, F.Cu at (60.0, 92.6)
- added U410: LDO_1.8V_SOT_23_5, TO_SOT_Packages_SMD:SOT-23-5, B.Cu at (93.0, 72.5)
- added Y220: Crystal_GND24, Crystals:Crystal_SMD_3225-4pin_3.2x2.5mm, B.Cu at (58.2, 71.5)
- C208: moved to F.Cu
- moved C208 16.9 mm to (57.0, 84.5), turned to 0 degrees
- moved C6008 6.02 mm to (51.5, 72.0), turned to 180 degrees
- moved C1701 4.81 mm to (72.8, 82.2)
- moved L6002 4.27 mm to (51.5, 70.0)
- moved U3 4.24 mm to (51.0, 62.0)
- moved R1700 0.98 mm to (59.1, 67.0)
- moved C5123 0.54 mm to (64.0, 61.8)
Connections:
- C1701 pad 1: VCCIO_SDMMC -> VCC_IO
- C1984 pad 1: VCCIO_FLASH -> VCC_1V8
- U1000 pad D14: VCCIO_SDMMC -> VCC_IO
- U1000 pad E17: Net-(U1000-PadE17) -> VCC_1V8
- U1000 pad R12: VCCIO_FLASH -> VCC_1V8
- U3 pad A1: /emmc/FLASH_D4 -> /emmc/FLASH_D3
- U3 pad A8: Net-(U3-PadA8) -> /emmc/FLASH_D7
- U3 pad B1: /emmc/FLASH_D3 -> Net-(U3-PadB1)
- U3 pad B7: Net-(U3-PadB7) -> /emmc/FLASH_D7
- U3 pad C6: VCCIO_FLASH -> VCC_1V8
- U3 pad C7: /emmc/FLASH_D7 -> Net-(U3-PadC7)
- U3 pad D3: Net-(U3-PadD3) -> GND
- U3 pad D4: GND -> /emmc/FLASH_D6
- U3 pad E2: Net-(U3-PadE2) -> GND
- U3 pad E3: Net-(U3-PadE3) -> /emmc/FLASH_D6
- U3 pad F1: Net-(U3-PadF1) -> GND
- U3 pad F2: Net-(U3-PadF2) -> /emmc/FLASH_D6
- U3 pad G1: Net-(U3-PadG1) -> /emmc/FLASH_D6
- U3 pad J1: Net-(U3-PadJ1) -> /emmc/EMMC_RST
- U3 pad J2: Net-(U3-PadJ2) -> /emmc/EMMC_RST
- U3 pad J3: Net-(U3-PadJ3) -> /emmc/EMMC_RST
- U3 pad K1: Net-(U3-PadK1) -> /emmc/FLASH_CLK
- U3 pad K2: Net-(U3-PadK2) -> /emmc/FLASH_CLK
- U3 pad K3: Net-(U3-PadK3) -> /emmc/FLASH_CLK
- U3 pad L1: Net-(U3-PadL1) -> /emmc/FLASH_CMD
- U3 pad L2: Net-(U3-PadL2) -> /emmc/FLASH_CMD
- U3 pad L3: Net-(U3-PadL3) -> /emmc/FLASH_CMD
- U3 pad M4: VCCIO_FLASH -> VCC_1V8
- U3 pad N4: VCCIO_FLASH -> VCC_1V8
- U3 pad N5: Net-(U3-PadN5) -> GND
- U3 pad P1: Net-(U3-PadP1) -> GND
- U3 pad P3: VCCIO_FLASH -> VCC_1V8
- U3 pad P5: VCCIO_FLASH -> VCC_1V8
- U6000 pad 36: Net-(U6000-Pad36) -> GND
Routing:
- net /test/UART4_TXD: track 0.46 -> 26.6 mm, vias 1 -> 2
- net /test/UART4_RXD: track 0.00 -> 25.7 mm, vias 0 -> 2
- net /test/UART4_RTS: track 2.08 -> 26.2 mm
- net /emmc/FLASH_D3: track 0.98 -> 20.8 mm, vias 0 -> 1
- net /test/UART4_CTS: track 1.62 -> 21.5 mm
- net /emmc/FLASH_D4: track 1.43 -> 20.8 mm, vias 0 -> 1
- net /emmc/FLASH_D5: track 2.73 -> 20.8 mm, vias 0 -> 1
- net VCC_IO: track 14.4 -> 32.0 mm, vias 1 -> 3
- net /emmc/FLASH_D1: track 4.93 -> 20.8 mm, vias 2 -> 1
- net /emmc/EMMC_RST: track 0.46 -> 16.1 mm, vias 1 -> 2
- net /emmc/FLASH_D0: track 5.54 -> 20.8 mm
- net /emmc/FLASH_CLK: track 5.66 -> 20.9 mm, vias 1 -> 2
- net /test/BT_REG_ON: track 0.00 -> 14.8 mm, vias 0 -> 2
- net /emmc/FLASH_D2: track 6.26 -> 20.8 mm, vias 2 -> 1
- net /emmc/FLASH_D7: track 6.43 -> 20.8 mm
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- added copper zone on In3.Cu, net VCC_1V8
- added copper zone on In2.Cu, net VCC_IO
- added copper zone on B.Cu, net VDD_1V0

Commit message: wip
Parts:
- added C901: 10u, Capacitors_SMD:C_0603, F.Cu at (39.6, 67.0)
- added C902: 0.1u, Capacitors_SMD:C_0402, F.Cu at (40.5, 67.0)
- added C910: 22p, Capacitors_SMD:C_0402, B.Cu at (42.2, 72.5)
- added C911: 22p, Capacitors_SMD:C_0402, B.Cu at (44.0, 70.8)
- added Y123: Crystal_GND24, require:EPSON_FA_128, B.Cu at (42.2, 70.8)
- moved R1700 1.62 mm to (60.1, 65.7)
Connections:
- U6000 pad 6: Net-(U6000-Pad6) -> /test/HOST_WAKE_BT
- U6000 pad 7: Net-(U6000-Pad7) -> /test/BT_WAKE_HOST
- U6000 pad 9: Net-(U6000-Pad9) -> VCC_IO
Routing:
- net /test/HOST_WAKE_BT: track 0.46 -> 18.0 mm, vias 1 -> 2
- net /test/BT_WAKE_HOST: track 2.11 -> 17.7 mm, vias 1 -> 2
- net /emmc/FLASH_CMD: track 15.9 -> 21.6 mm, vias 1 -> 2
- net Net-(C910-Pad1): track 0.00 -> 5.53 mm, vias 0 -> 1
- net Net-(C911-Pad1): track 0.00 -> 4.63 mm, vias 0 -> 1
- net GND: track 207.5 -> 209.0 mm, vias 131 -> 132
- net /emmc/EMMC_RST: track 16.1 -> 17.2 mm
- net /test/UART4_RTS: track 26.2 -> 25.1 mm
- net /test/UART4_TXD: track 26.6 -> 25.7 mm
- net /emmc/FLASH_D4: track 20.8 -> 21.6 mm
- net /emmc/FLASH_D5: track 20.8 -> 21.6 mm
- net /emmc/FLASH_D1: track 20.8 -> 21.6 mm
- net /emmc/FLASH_D0: track 20.8 -> 21.6 mm
- net /test/UART4_RXD: track 25.7 -> 24.9 mm
- net /emmc/FLASH_D7: track 20.8 -> 21.6 mm
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