File: hardware/require.kicad_pcb (KiCad board)
At the start: 6 copper layers, 70 x 25.4 mm, 117 parts, among them J1 Conn_01x02, U100 SY8089AAC, U1000 RK3308, U200 SY8089AAC, U3 EMMC_BGA_153, U300 SY8089AAC, U3000 DDR3_FBGA96, U400 SY8089AAC, U410 LDO_1.8V_SOT_23_5, U6000 ap6255, Y123 Crystal_GND24, Y220 Crystal_GND24

Commit message: wip
Parts:
- removed C100, C300: 0.1u,10V, Capacitors_SMD:C_0402
- removed C162, C167, C1701, C1984, C207, C208, C225, C230, C231, C311, C5123, C5124: 0.1u, Capacitors_SMD:C_0402
- removed C220: 15p, Capacitors_SMD:C_0402
- removed C301: 10u,10V, Capacitors_SMD:C_0805
- removed C310: 10u, Capacitors_SMD:C_0603
- removed C413: 1u, Capacitors_SMD:C_0402
- removed C6008: 4.7u, Capacitors_SMD:C_0603
- removed FB400: L, Inductors_SMD:L_0603
- removed J1: Conn_01x02, Connectors_JST:JST_EH_B02B-EH-A_02x2.50mm_Straight
- removed L6002: 3.3u, require:L_murata_2520
- removed R180: R, Resistors_SMD:R_0402
- removed R220: 22R, Resistors_SMD:R_0402
- removed R230, R423, R429: 1R, Resistors_SMD:R_0402
- removed R420, R421, R422, R425, R426: 0R, Resistors_SMD:R_0402
- removed the U3 at (51.0, 62.0)
- removed Y220: Crystal_GND24, Crystals:Crystal_SMD_3225-4pin_3.2x2.5mm
- added ANT1: ANT12, require:YAIYO_YUDEN_AH104N, F.Cu at (32.5, 61.5)
- added C12: 0.1u,10V, Capacitors_SMD:C_0402, F.Cu at (96.5, 62.5)
- added C13: 10u,10V, Capacitors_SMD:C_0805, F.Cu at (94.0, 65.0)
- added C30: 0.1u,10V, Capacitors_SMD:C_0402, B.Cu at (96.5, 57.5)
- added C46: 1u, Capacitors_SMD:C_0402, B.Cu at (96.5, 72.5)
- added C54: 0.1u, Capacitors_SMD:C_0402, B.Cu at (86.0, 62.6)
- added C59: 0.1u, Capacitors_SMD:C_0402, B.Cu at (76.0, 58.6)
- added C7: 1u, Capacitors_SMD:C_0402, B.Cu at (51.0, 69.5)
- added C74: 0.1u, Capacitors_SMD:C_0402, B.Cu at (70.0, 60.6)
- added C75: 0.1u, Capacitors_SMD:C_0402, B.Cu at (65.7, 60.6)
- added C77: 0.1u, Capacitors_SMD:C_0402, B.Cu at (63.7, 65.1)
- added C8: 4.7u, Capacitors_SMD:C_0603, B.Cu at (53.0, 71.5)
- added C80: 10u, Capacitors_SMD:C_0603, B.Cu at (65.8, 65.3)
- added C81: 0.1u, Capacitors_SMD:C_0402, B.Cu at (66.8, 65.1)
- added C84: 0.1u, Capacitors_SMD:C_0402, B.Cu at (60.6, 70.2)
- added C85: 0.1u, Capacitors_SMD:C_0402, B.Cu at (61.4, 70.2)
- added C86: 0.1u, Capacitors_SMD:C_0402, B.Cu at (63.0, 70.2)
- added C87: 0.1u, Capacitors_SMD:C_0402, B.Cu at (63.9, 70.2)
- added C88: 0.1u, Capacitors_SMD:C_0402, B.Cu at (59.8, 70.2)
- added C9: 0.1u, Capacitors_SMD:C_0402, B.Cu at (46.5, 74.0)
- added C91: 15p, Capacitors_SMD:C_0402, B.Cu at (55.0, 74.5)
- added FB1: 180R,1.5A, Inductors_SMD:L_0402, B.Cu at (63.2, 68.2)
- added FB2: 180R,1.5A, Inductors_SMD:L_0402, B.Cu at (61.4, 68.2)
- added H1: MountingHole_Pad, require:PTH_MTG320_380, F.Cu at (38.7, 54.7)
- added H2: MountingHole_Pad, require:PTH_MTG320_380, F.Cu at (38.7, 75.3)
- added H3: MountingHole_Pad, require:PTH_MTG320_380, F.Cu at (102.3, 75.3)
- added H4: MountingHole_Pad, require:PTH_MTG320_380, F.Cu at (102.3, 54.7)
- added J10: USB_B_Micro, Connectors_USB:USB_Micro-B_Molex_47346-0001, F.Cu at (103.7, 65.0)
- added L2: 3.3u, require:L_murata_2520, B.Cu at (51.0, 71.5)
- added R1: 2.2R, Resistors_SMD:R_0402, F.Cu at (98.4, 65.2)
- added R2: 2.2R, Resistors_SMD:R_0402, F.Cu at (98.4, 64.0)
- added R51: R, Resistors_SMD:R_0402, B.Cu at (81.0, 63.0)
- added R91: 22R, Resistors_SMD:R_0402, B.Cu at (58.0, 68.2)
- added R92: 10k, Resistors_SMD:R_0402, B.Cu at (59.8, 68.2)
- added R93: 133R,1%, Resistors_SMD:R_0402, B.Cu at (62.2, 70.2)
- added R987: 10k, Resistors_SMD:R_0402, F.Cu at (90.5, 54.8)
- added SW1: SW_Push, require:HYP_1TS003A_SIDE_PUSH, F.Cu at (94.0, 53.5)
- added U4: EMMC_BGA_153, require:BGA-153_14x14_11.5x13.0mm, B.Cu at (51.0, 62.0)
- added Y2: Crystal_GND24, Crystals:Crystal_SMD_3225-4pin_3.2x2.5mm, B.Cu at (56.5, 71.5)
- added Y4: SG-3030CM, Oscillators:Oscillator_SMD_SeikoEpson_SG3030CM, B.Cu at (46.5, 71.5)
- moved C23 5.59 mm to (98.0, 72.5), turned to 90 degrees
- moved C31 5.39 mm to (98.0, 57.0), turned to 270 degrees
- moved C6 3.01 mm to (42.0, 73.0), turned to 180 degrees
- moved C5 2.51 mm to (42.0, 70.0)
- moved C76 1.79 mm to (62.9, 65.1), turned to 90 degrees
- moved C1 1.76 mm to (36.2, 61.0)
- moved C2 1.75 mm to (38.9, 61.0)
- moved L1 1.65 mm to (37.5, 61.5)
- moved C45 1.58 mm to (91.5, 73.0), turned to 90 degrees
- moved C90 1.22 mm to (58.0, 74.5)
- moved C10 1.00 mm to (89.0, 62.5)
- moved C11 1.00 mm to (93.5, 60.0)
- moved C20 1.00 mm to (89.0, 72.5)
- moved C21 1.00 mm to (93.5, 70.0)
- moved C22 1.00 mm to (96.5, 72.5)
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- renumbered C123 to C1, C304 to C10, C303 to C11, C122 to C2, C404 to C20, C403 to C21, C400 to C22, C401 to C23, C901 to C3, C101 to C31, C104 to C32, C103 to C33, C110 to C34, C902 to C4, C200 to C40, C201 to C41, C204 to C42, C203 to C43, C410 to C45, C910 to C5, C150 to C50, C151 to C51, C160 to C52, C161 to C53, C163 to C55, C164 to C56, C165 to C57, C166 to C58, C911 to C6, C168 to C60, C169 to C61, C170 to C62, C171 to C63, C172 to C64, C173 to C65, C181 to C66, C180 to C67, C190 to C68, C108 to C70, C105 to C71, C106 to C72, C107 to C73, C1700 to C76, C206 to C78, C312 to C82, C221 to C90, L123 to L1, L300 to L10, L400 to L20, L100 to L30, L200 to L40, R300 to R10, R302 to R11, R303 to R12, R400 to R20, R402 to R21, R403 to R22, R101 to R30, R100 to R31, R102 to R32, R103 to R33, R110 to R34, R111 to R35, R112 to R36, R113 to R37, R200 to R40, R202 to R41, R203 to R42, R410 to R45, R150 to R50, R181 to R52, R190 to R53, R191 to R54, R1700 to R90, U6000 to U1, U300 to U10, U400 to U20, U3000 to U3, U100 to U30, U200 to U40, U410 to U45, Y123 to Y1
Connections:
- net /rk3308-power/CORE_DVS renamed /power/CORE_DVS
- C76 pad 1: VCCIO_SDIO -> VCC_IO
- U1 pad 12: Net-(U6000-Pad12) -> /test/WIFI_REG_ON
- U1 pad 13: Net-(U6000-Pad13) -> /test/WIFI_WAKE_HOST
- U1 pad 22: VCCIO_SDIO -> VCC_IO
- U1 pad 24: Net-(U6000-Pad24) -> /test/LPO
- U1 pad 29: Net-(U6000-Pad29) -> GND
- U1000 pad A12: (no net) -> /usb/USB_HOST_DM
- U1000 pad A13: (no net) -> /usb/USB_OTG_DM
- U1000 pad A18: (no net) -> /rk3308-power/A3
- U1000 pad A19: (no net) -> /rk3308-power/A0
- U1000 pad B12: (no net) -> /usb/USB_HOST_DP
- U1000 pad B13: (no net) -> /usb/USB_OTG_DP
- U1000 pad B18: (no net) -> /rk3308-power/A4
- U1000 pad B19: (no net) -> /rk3308-power/A1
- U1000 pad C12: (no net) -> Net-(U1000-PadC12)
- U1000 pad C14: (no net) -> VCC_IO
- U1000 pad C15: (no net) -> Net-(R1400-Pad2)
- U1000 pad C18: (no net) -> /rk3308-power/A2
- U1000 pad D13: (no net) -> VCC_IO
- U1000 pad D15: (no net) -> VDD_1V0
- U1000 pad D16: (no net) -> AVDD_1V8
- U1000 pad D17: (no net) -> VCC_1V8
- U1000 pad D18: (no net) -> /rk3308-power/A5
- U1000 pad E14: (no net) -> VCC_IO
- U1000 pad E15: Net-(C230-Pad1) -> VDD_1V0
- U1000 pad E16: (no net) -> VCC_1V8
- U1000 pad J14: VCCIO_SDIO -> VCC_IO
- U1000 pad N3: /rk3308-lcdc-mac-i2s1-jtag/WIFI_WAKE_HOST -> /test/WIFI_WAKE_HOST
- U1000 pad P3: /rk3308-lcdc-mac-i2s1-jtag/WIFI_REG_ON -> /test/WIFI_REG_ON
- U1000 pad R12: VCC_1V8 -> VCC_IO
- U1000 pad R15: (no net) -> Net-(U1000-PadR15)
- U1000 pad R16: (no net) -> Net-(U1000-PadR16)
- U1000 pad T11: (no net) -> VCC_IO
- U1000 pad T14: (no net) -> Net-(U1000-PadT14)
- U1000 pad T15: (no net) -> Net-(U1000-PadT15)
- U1000 pad T16: (no net) -> Net-(U1000-PadT16)
- U1000 pad T17: (no net) -> Net-(U1000-PadT17)
- U1000 pad U14: (no net) -> Net-(U1000-PadU14)
- U1000 pad U15: (no net) -> Net-(U1000-PadU15)
- U1000 pad U16: (no net) -> Net-(U1000-PadU16)
- U1000 pad V14: (no net) -> Net-(U1000-PadV14)
- U1000 pad V15: (no net) -> Net-(U1000-PadV15)
- U1000 pad V16: (no net) -> Net-(U1000-PadV16)
- U1000 pad V17: (no net) -> Net-(U1000-PadV17)
- U1000 pad W14: (no net) -> Net-(U1000-PadW14)
- U1000 pad W16: (no net) -> Net-(U1000-PadW16)
- U1000 pad Y14: (no net) -> Net-(U1000-PadY14)
- U1000 pad Y16: (no net) -> Net-(U1000-PadY16)
Routing:
- net VDD_CORE: track 40.2 -> 16.6 mm
- net /test/HOST_WAKE_BT: track 18.0 -> 0.46 mm
- net /test/BT_WAKE_HOST: track 17.7 -> 0.46 mm
- net VCC_IO: track 32.0 -> 46.9 mm, vias 3 -> 13
- net Net-(C91-Pad1): track 0.00 -> 9.63 mm
- net Net-(C220-Pad1): track 8.43 -> 0.00 mm
- net /test/LPO: track 0.00 -> 7.83 mm, vias 0 -> 1
- net /test/SDIO_D1: track 24.1 -> 16.3 mm
- net VCC_DDR: track 54.2 -> 48.9 mm
- net GND: track 209.0 -> 213.4 mm, vias 132 -> 161
- net Net-(C2-Pad1): track 0.00 -> 4.35 mm
- net Net-(C8-Pad1): track 4.48 -> 0.91 mm
- net /rk3308-power/RESET: track 0.00 -> 3.13 mm, vias 0 -> 1
- net Net-(ANT1-Pad1): track 5.45 -> 2.60 mm
- net VDD_1V0: track 0.00 -> 2.74 mm, vias 0 -> 1
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- added copper zone on In3.Cu, net VCC5V0_SYS
- added copper zone on In3.Cu, net VCC_DDR
- added copper zone on In4.Cu, net VCC_IO
- added copper zone on In2.Cu, net VDD_CORE
- added copper zone on In2.Cu, net VDD_LOG
- removed copper zone on In4.Cu, net VCC5V0_SYS
- removed copper zone on In3.Cu, net VCC_1V8
- removed copper zone on In4.Cu, net VCC_DDR
- removed copper zone on In2.Cu, net VCC_IO
- removed copper zone on B.Cu, net VDD_1V0
- removed copper zone on In3.Cu, net VDD_CORE
- removed copper zone on In3.Cu, net VDD_LOG
Other:
- board size 70 x 25.4 mm -> 76 x 26 mm
- rule pad_to_mask_clearance: 0.2 -> 0.05
- rule solder_mask_min_width: 0.25 -> 0.2

Commit message: wip
Parts:
- removed R987: 10k, Resistors_SMD:R_0402
- added C14: 1u, Capacitors_SMD:C_0402, F.Cu at (101.0, 59.9)
- added D9: LED_GBAR_0603X2, require:LED_RGB_0603X2, F.Cu at (40.3, 65.0)
- added LP1: GND, require:OVAL_PIN, F.Cu at (44.1, 76.4)
- added LP10: TX2, require:OVAL_PIN, F.Cu at (67.0, 76.4)
- added LP11: DM, require:OVAL_PIN, F.Cu at (69.5, 76.4)
- added LP12: DP, require:OVAL_PIN, F.Cu at (72.1, 76.4)
- added LP13: DNC, require:OVAL_PIN, F.Cu at (74.6, 76.4)
- added LP14: RST, require:OVAL_PIN, F.Cu at (77.2, 76.4)
- added LP15: 3V3, require:OVAL_PIN, F.Cu at (79.7, 76.4)
- added LP16: 3V3, require:OVAL_PIN, F.Cu at (82.2, 76.4)
- added LP17: 5V, require:OVAL_PIN, F.Cu at (84.8, 76.4)
- added LP18: GND, require:OVAL_PIN, F.Cu at (87.3, 76.4)
- added LP2: A0, require:OVAL_PIN, F.Cu at (46.7, 76.4)
- added LP3: A1, require:OVAL_PIN, F.Cu at (49.2, 76.4)
- added LP4: A2, require:OVAL_PIN, F.Cu at (51.8, 76.4)
- added LP5: A3, require:OVAL_PIN, F.Cu at (54.3, 76.4)
- added LP6: A4, require:OVAL_PIN, F.Cu at (56.8, 76.4)
- added LP7: A5, require:OVAL_PIN, F.Cu at (59.4, 76.4)
- added LP8: GND, require:OVAL_PIN, F.Cu at (61.9, 76.4)
- added LP9: RX2, require:OVAL_PIN, F.Cu at (64.5, 76.4)
- added P10: 16, require:OVAL_PIN, F.Cu at (84.8, 53.6)
- added P11: 17, require:OVAL_PIN, F.Cu at (87.3, 53.6)
- added P12: 18, require:OVAL_PIN, F.Cu at (89.9, 53.6)
- added P13: 1, require:OVAL_PIN, F.Cu at (46.7, 53.6)
- added P14: 2, require:OVAL_PIN, F.Cu at (49.2, 53.6)
- added P15: 7, require:OVAL_PIN, F.Cu at (61.9, 53.6)
- added P16: 8, require:OVAL_PIN, F.Cu at (64.5, 53.6)
- added P17: 9, require:OVAL_PIN, F.Cu at (67.0, 53.6)
- added P18: 10, require:OVAL_PIN, F.Cu at (69.5, 53.6)
- added P19: 3, require:OVAL_PIN, F.Cu at (51.7, 53.6)
- added P20: 4, require:OVAL_PIN, F.Cu at (54.3, 53.6)
- added P21: 5, require:OVAL_PIN, F.Cu at (56.8, 53.6)
- added P22: 6, require:OVAL_PIN, F.Cu at (59.4, 53.6)
- added P23: 11, require:OVAL_PIN, F.Cu at (72.1, 53.6)
- added P24: 12, require:OVAL_PIN, F.Cu at (74.6, 53.6)
- added P25: 13, require:OVAL_PIN, F.Cu at (77.2, 53.6)
- added P26: 14, require:OVAL_PIN, F.Cu at (79.7, 53.6)
- added P7: 15, require:OVAL_PIN, F.Cu at (82.2, 53.6)
- added Q1: BSS138, TO_SOT_Packages_SMD:SOT-23, B.Cu at (94.0, 76.0)
- added R3: 30k, Resistors_SMD:R_0402, F.Cu at (110.7, 70.6)
- added R4: 22R, Resistors_SMD:R_0402, F.Cu at (107.6, 68.0)
- added R435: 10k, Resistors_SMD:R_0402, B.Cu at (91.5, 76.0)
- added R5: 22R, Resistors_SMD:R_0402, F.Cu at (108.7, 69.6)
- added RP1: GND, require:OVAL_PIN, F.Cu at (44.1, 53.6)
- added RP20: GND, require:OVAL_PIN, F.Cu at (92.4, 53.6)
- added U2: AW2015FCR, require:AW2015FCR_QFN8L, F.Cu at (96.8, 56.1)
- SW1: value SW_Push -> SW_SKSC_4PIN; footprint require:HYP_1TS003A_SIDE_PUSH -> require:SW_ALPS_SKSC
- moved R92 37.5 mm to (96.5, 76.0), turned to 270 degrees
- moved SW1 23.0 mm to (96.2, 76.4)
Connections:
- net Net-(U1000-PadV3) renamed /test/CORE_DVS
- net Net-(U1000-PadY3) renamed /test/POWER_SLEEP
- SW1 pad 1: Net-(R987-Pad1) -> GND
- U1000 pad T10: /rk3308-lcdc-mac-i2s1-jtag/SPI2_CS -> /rk3308-lcdc-mac-i2s1-jtag/DIO10
- U1000 pad T9: /rk3308-lcdc-mac-i2s1-jtag/SPI2_TX_UART2_TX_M0 -> /rk3308-lcdc-mac-i2s1-jtag/DIO8
- U1000 pad U14: Net-(U1000-PadU14) -> /rk3308-lcdc-mac-i2s1-jtag/DIO3
- U1000 pad U2: Net-(U1000-PadU2) -> /test/PWM3
- U1000 pad V1: Net-(U1000-PadV1) -> /test/I2C1_SCL
- U1000 pad V10: /rk3308-lcdc-mac-i2s1-jtag/SPI2_CLK -> /rk3308-lcdc-mac-i2s1-jtag/DIO9
- U1000 pad V16: Net-(U1000-PadV16) -> /rk3308-lcdc-mac-i2s1-jtag/DIO4
- U1000 pad V2: Net-(U1000-PadV2) -> /test/I2C1_SDA
- U1000 pad W1: Net-(U1000-PadW1) -> /test/PWM2
- U1000 pad W16: Net-(U1000-PadW16) -> /rk3308-lcdc-mac-i2s1-jtag/DIO6
- U1000 pad W2: Net-(U1000-PadW2) -> /test/PWM1
- U1000 pad W9: /rk3308-lcdc-mac-i2s1-jtag/SPI2_RX_UART2_RX_M0 -> /rk3308-lcdc-mac-i2s1-jtag/DIO7
- U1000 pad Y16: Net-(U1000-PadY16) -> /rk3308-lcdc-mac-i2s1-jtag/DIO5
Routing:
- net Net-(P13-Pad1): track 0.00 -> 4.75 mm, vias 0 -> 1
- net /emmc/EMMC_RST: track 15.0 -> 11.4 mm
- net GND: track 213.4 -> 210.6 mm, vias 161 -> 160
- net /test/LED3: track 0.00 -> 0.90 mm
- net /rk3308-lcdc-mac-i2s1-jtag/DIO9: track 0.00 -> 0.46 mm, vias 0 -> 1
- net /rk3308-lcdc-mac-i2s1-jtag/DIO10: track 0.00 -> 0.46 mm, vias 0 -> 1
- net Net-(P14-Pad1): track 0.00 -> 0.46 mm, vias 0 -> 1

Commit message: wip
Parts:
- removed R90: 22R, Resistors_SMD:R_0402
- added C101: C, Capacitors_SMD:C_0402, F.Cu at (54.8, 58.2)
- moved D9 63.3 mm to (101.0, 47.0)
- moved R91 0.45 mm to (58.5, 68.2)
Connections:
- U1000 pad J18: Net-(R90-Pad2) -> /test/SDIO_CLK
- U4 pad C1: Net-(U4-PadC1) -> Net-(C101-Pad1)
- U4 pad C2: Net-(U4-PadC2) -> Net-(C101-Pad1)
Routing:
- net /test/UART4_RTS: track 25.1 -> 0.00 mm
- net /test/UART4_CTS: track 20.8 -> 0.00 mm
- net /test/UART4_RXD: track 25.2 -> 5.93 mm, vias 2 -> 1
- net /test/UART4_TXD: track 25.7 -> 6.58 mm, vias 2 -> 1
- net /emmc/EMMC_RST: track 11.4 -> 2.67 mm
- net /test/PCM_SYNC: track 0.46 -> 7.40 mm
- net /test/PCM_OUT: track 0.46 -> 7.38 mm
- net /test/BT_REG_ON: track 14.6 -> 8.17 mm, vias 2 -> 1
- net /test/HOST_WAKE_BT: track 0.46 -> 6.80 mm
- net /test/BT_WAKE_HOST: track 0.46 -> 6.44 mm
- net /test/SDIO_D1: track 16.3 -> 22.0 mm
- net /test/PCM_IN: track 0.46 -> 5.95 mm
- net /test/PCM_CLK: track 0.00 -> 5.01 mm, vias 0 -> 1
- net /test/SDIO_CLK: track 24.0 -> 22.0 mm, vias 1 -> 0
- net /rk3308-power/RESET: track 3.13 -> 1.34 mm
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
Commit message: wip
Parts:
- moved U4 3.00 mm to (54.0, 62.0)
- moved C101 2.57 mm to (52.5, 57.0)
Connections:
- U1 pad 25: Net-(U1-Pad25) -> /test/PCM_OUT
- U1 pad 26: Net-(U1-Pad26) -> /test/PCM_CLK
- U1 pad 27: Net-(U1-Pad27) -> /test/PCM_IN
- U1 pad 28: Net-(U1-Pad28) -> /test/PCM_SYNC
- U4 pad B1: Net-(U4-PadB1) -> /emmc/FLASH_D3
Routing:
- net /test/WIFI_REG_ON: track 0.00 -> 31.1 mm, vias 0 -> 2
- net /test/WIFI_WAKE_HOST: track 0.00 -> 30.5 mm, vias 0 -> 2
- net /test/UART4_RTS: track 0.00 -> 21.1 mm, vias 0 -> 2
- net Net-(P14-Pad1): track 0.46 -> 19.7 mm
- net /test/UART4_CTS: track 0.00 -> 17.9 mm, vias 0 -> 2
- net Net-(P13-Pad1): track 4.75 -> 22.0 mm
- net /test/UART4_RXD: track 5.93 -> 22.4 mm, vias 1 -> 2
- net /rk3308-power/A0: track 0.81 -> 17.2 mm, vias 0 -> 1
- net /test/UART4_TXD: track 6.58 -> 22.4 mm, vias 1 -> 2
- net /test/HOST_WAKE_BT: track 6.80 -> 21.2 mm
- net /rk3308-power/A1: track 1.60 -> 15.3 mm, vias 0 -> 1
- net /test/BT_WAKE_HOST: track 6.44 -> 19.9 mm
- net /emmc/EMMC_RST: track 2.67 -> 14.8 mm
- net /rk3308-power/A2: track 2.25 -> 14.2 mm, vias 0 -> 1
- net /test/PCM_IN: track 5.95 -> 16.9 mm, vias 1 -> 2
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