File: hardware/require.kicad_pcb (KiCad board)
At the start: 6 copper layers, 66 x 26 mm, 169 parts, among them J1 USB_B_Micro, Q1 BSS138, U1 ap6255, U1000 RK3308, U2 SIT1532, U30 SY8089AAC, U4 DDR3_FBGA96, U40 SY8089AAC, U45 LDO_1.8V_SOT_23_5, U6 SY8089AAC, U8 ATECC608A-MAHDA, U994 EMMC_BGA_153, Y1 Crystal_GND24, Y2 Crystal_GND24

Commit message: wip
Parts:
- removed C1912: 47uf,tant, Capacitors_Tantalum_SMD:CP_Tantalum_Case-B_EIA-3528-21_Reflow
- removed C30: 0.1u,10V, require:C_0402
- removed C45, C46: 1u, require:C_0402
- removed the LP12 at (73.3, 76.4)
- removed the LP17 at (86.0, 76.4)
- removed R31, R4, R40, R45: 10k, require:R_0402
- removed R66, R67: 22R, require:R_0402
- removed RP20: G, require:OVAL_PIN
- removed TP1, TP2: TestPoint, require:TPTH0503
- removed U45: LDO_1.8V_SOT_23_5, TO_SOT_Packages_SMD:SOT-23-5
- added C188: 22p, require:C_0402, F.Cu at (90.5, 69.5)
- added C189: 22p, require:C_0402, F.Cu at (89.5, 71.7)
- added C190: 22p, require:C_0402, F.Cu at (89.5, 70.9)
- added C191: 22p, require:C_0402, F.Cu at (91.9, 71.7)
- added C200: 0.1u,10V, require:C_0402, B.Cu at (95.0, 62.8)
- added C267: 10u,10V, require:C_0603, B.Cu at (94.5, 63.8)
- added C268: 10u,10V, require:C_0603, F.Cu at (90.5, 66.0)
- added C500: 1u, require:C_0402, B.Cu at (62.9, 65.1)
- added C501: 1u, require:C_0402, B.Cu at (61.6, 63.7)
- added D201: LED, LEDs:LED_0402, F.Cu at (95.5, 58.2)
- added D400: D_Schottky, Diodes_SMD:D_SOD-523, B.Cu at (65.2, 56.0)
- added L191: 2.2u, Inductors_SMD:L_0603, F.Cu at (91.5, 70.1)
- added LP18: 5V, require:OVAL_PIN, F.Cu at (86.0, 76.4)
- added LP8: RST, require:OVAL_PIN, F.Cu at (60.6, 76.4)
- added Q200: NPND_SOT_363, TO_SOT_Packages_SMD:SOT-363_SC-70-6, F.Cu at (95.1, 60.0)
- added R200: R, require:R_0402, B.Cu at (92.0, 59.2)
- added R202: R, require:R_0402, F.Cu at (95.0, 62.0)
- added RP18: G, require:OVAL_PIN, F.Cu at (86.0, 53.6)
- added RP19: BYP, require:OVAL_PIN, F.Cu at (88.5, 53.6)
- added SW1: SW_SKSC_4PIN, require:SW_ALPS_SKSCLCE010, F.Cu at (90.5, 76.4)
- added U187: TPS62088_FIXED, require:TPS62088_DSBGA6, F.Cu at (89.4, 69.5)
- added U500: NCP707_XDFN4, require:XDFN4, B.Cu at (61.6, 65.0)
- C15, C32, C332, C42, C50, C51: footprint require:C_0805 -> require:C_0603
- C18: footprint require:C_0805 -> require:C_0603; moved to B.Cu
- C3, C4, R1, R2: moved to B.Cu
- J1: footprint Connectors_USB:USB_Micro-B_Molex_47346-0001 -> require:USB_Micro-B_Molex_47346-0001
- LP14: value RST -> NC
- Q1: value BSS138 -> Q_NMOS_GSD; footprint require:SOT-323_SC-70 -> require:SOT-883
- moved R1 28.7 mm to (71.2, 61.6), turned to 180 degrees
- moved R8 25.3 mm to (89.5, 68.0)
- moved R7 25.3 mm to (89.5, 67.1)
- moved D2 24.9 mm to (91.5, 67.6), turned to 180 degrees
- moved R37 24.1 mm to (90.0, 59.2), turned to 180 degrees
- moved R36 23.4 mm to (90.0, 60.2), turned to 180 degrees
- moved R35 22.7 mm to (90.0, 61.2), turned to 180 degrees
- moved U8 22.5 mm to (71.2, 57.5), turned to 270 degrees
- moved R2 22.4 mm to (71.2, 60.6), turned to 180 degrees
- moved C34 22.1 mm to (90.0, 62.2), turned to 180 degrees
- moved C25 21.6 mm to (69.5, 57.5), turned to 90 degrees
- moved R34 21.6 mm to (90.0, 63.2), turned to 0 degrees
- moved R47 21.3 mm to (61.8, 72.2), turned to 0 degrees
- moved R46 21.1 mm to (60.9, 73.8)
- moved Q1 19.6 mm to (61.8, 73.8), turned to 270 degrees
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- renumbered LP9 to LP10, LP10 to LP11, LP11 to LP12, LP18 to LP15, LP15 to LP16, LP16 to LP17, LP8 to LP9
Connections:
- net /emmc/EMMC_D0 renamed /EMMC_D0
- D6 pad 1: Net-(D6-Pad1) -> /rk3308-io/D20
- D6 pad 2: Net-(D6-Pad2) -> /rk3308-io/D19
- J1 pad 2: Net-(D2-Pad1) -> Net-(D2-Pad2)
- J1 pad 3: Net-(D2-Pad2) -> Net-(D2-Pad1)
- LP11 pad 1: Net-(D6-Pad2) -> /rk3308-io/D19
- LP12 pad 1: Net-(D6-Pad1) -> /rk3308-io/D20
- LP14 pad 1: /RESET -> GND
- R7 pad 1: Net-(D2-Pad2) -> Net-(D2-Pad1)
- R8 pad 1: Net-(D2-Pad1) -> Net-(D2-Pad2)
- U40 pad 1: Net-(R40-Pad1) -> +3V3
- U6 pad 1: Net-(R4-Pad1) -> +3V3
Routing:
- net +3V3: track 50.4 -> 74.7 mm, vias 18 -> 26
- net Net-(D400-Pad1): track 0.00 -> 24.1 mm, vias 0 -> 2
- net /rk3308-io/I2C1_SCL: track 25.4 -> 2.18 mm
- net /rk3308-io/I2C1_SDA: track 25.3 -> 5.54 mm
- net /rk3308-io/D20: track 3.62 -> 19.6 mm, vias 1 -> 2
- net /rk3308-io/D19: track 3.00 -> 16.8 mm, vias 1 -> 2
- net Net-(D6-Pad1): track 13.6 -> 0.00 mm, vias 1 -> 0
- net GND: track 231.5 -> 244.6 mm, vias 139 -> 160
- net VCC_DDR: track 42.3 -> 53.7 mm, vias 23 -> 26
- net +1V8: track 10.8 -> 19.9 mm, vias 2 -> 4
- net Net-(D6-Pad2): track 8.89 -> 0.00 mm, vias 1 -> 0
- net +5V: track 0.00 -> 8.87 mm, vias 0 -> 1
- net +1V0C: track 41.1 -> 50.0 mm, vias 6 -> 8
- net /USB_OTG_D_P: track 27.0 -> 34.1 mm, vias 1 -> 2
- net Net-(C33-Pad2): track 3.45 -> 10.2 mm
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Other:
- board size 66 x 26 mm -> 68 x 26 mm

Commit message: wip
Parts:
- removed C4, C57, C74, C76, C82, C88: 0.1u, require:C_0402
- removed C50: 10u, require:C_0603
- removed the C500 at (62.9, 65.1)
- removed the C501 at (61.6, 63.7)
- removed R41: 110k,1%, require:R_0402
- removed R42: 150k,1%, require:R_0402
- removed U2: SIT1532, require:SITIME_1508
- removed Y1: Crystal_GND24, require:EPSON_FA_128
- added C110: 0.1u, require:C_0402, B.Cu at (62.6, 73.8)
- added C255: 0.1u, require:C_0402, B.Cu at (70.2, 63.7)
- added C257: 0.1u, require:C_0402, B.Cu at (63.0, 65.1)
- added C259: 1u, require:C_0402, B.Cu at (62.4, 63.0)
- added C260: 1u, require:C_0402, B.Cu at (61.6, 66.3)
- added C261: 1u, require:C_0402, B.Cu at (61.6, 63.9)
- added C300: 10u, require:C_0603, B.Cu at (86.0, 57.0)
- added C302: 10u, require:C_0603, B.Cu at (76.0, 57.0)
- added C315: 0.1u, require:C_0402, B.Cu at (86.0, 69.0)
- added C352: 0.1u, require:C_0402, B.Cu at (67.7, 65.1)
- added C405: 1u, require:C_0402, F.Cu at (56.0, 59.4)
- added C511: 10u, require:C_0603, F.Cu at (40.1, 66.8)
- added C550: 4.7u, require:C_0402, B.Cu at (45.4, 69.9)
- added D850: ESD5302F, require:ESD_DFN1006_3L, B.Cu at (90.0, 76.4)
- added H1: MountingHole, require:MTG_1.8mm_2.4mm_NPL, F.Cu at (31.4, 53.9)
- added H2: MountingHole, require:MTG_1.8mm_2.4mm_NPL, F.Cu at (31.4, 76.1)
- added H3: MountingHole_Pad, require:MTG_1.8mm_2.4mm_PL, F.Cu at (95.6, 53.9)
- added H4: MountingHole_Pad, require:MTG_1.8mm_2.4mm_PL, F.Cu at (95.6, 76.1)
- added R222: 110k,1%, require:R_0402, B.Cu at (95.2, 69.5)
- added R223: 150k,1%, require:R_0402, B.Cu at (95.2, 68.5)
- added R850: 4.7k, require:R_0402, B.Cu at (91.0, 76.4)
- added Y520: Crystal_GND24, require:EPSON_FA_128, F.Cu at (39.5, 69.7)
- added Y550: SG-3030CM, Oscillators:Oscillator_SMD_SeikoEpson_SG3030CM, B.Cu at (45.4, 72.3)
- C201: renamed from C267; value 10u,10V -> 10u
- C220: renamed from C40; value 0.1u,10V -> 0.1u
- C221: renamed from C18; value 10u,10V -> 10u
- C230: renamed from C17; value 0.1u,10V -> 0.1u
- C231: renamed from C268; value 10u,10V -> 10u
- C256: renamed from C75; value 0.1u -> 1u
- C258: renamed from C87; value 0.1u -> 1u
- C400: renamed from C10; value C -> 10u
- C401: renamed from C12; value C -> 0.1u
- C402: renamed from C11; value C -> 0.1u
- C406: renamed from C8; value C -> 0.1u
- C410: renamed from C6; value C -> 10u
- C411: renamed from C7; value C -> 0.1u
- C510: renamed from C3; moved to F.Cu
- C520: renamed from C905; moved to F.Cu
- C521: renamed from C906; moved to F.Cu
- L540: renamed from L2; value 3.3u -> 2.2u
- R830: renamed from R2; value 22R -> 4.7k
- R831: renamed from R1; value 22R -> 4.7k
- R840: renamed from R202; value R -> 470R
- moved C520 7.64 mm to (38.0, 69.5)
- moved C510 4.69 mm to (38.9, 66.8)
- moved C521 4.58 mm to (39.5, 71.5), turned to 180 degrees
- moved C320 2.00 mm to (76.0, 63.4)
- moved C321 1.20 mm to (76.0, 65.4)
- moved C322 0.80 mm to (76.0, 68.2)
- moved C420 0.75 mm to (56.0, 58.5)
- moved R340 0.71 mm to (83.3, 66.5)
- moved C314 0.50 mm to (86.0, 66.3)
- moved R410 0.49 mm to (71.2, 62.6)
- moved C340 0.40 mm to (86.0, 65.4)
- moved R341 0.14 mm to (83.3, 65.1)
- moved R330 0.10 mm to (80.9, 63.9)
- moved C351 0.08 mm to (66.9, 65.1)
- moved C225 0.08 mm to (64.8, 65.3)
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- renumbered C91 to C100, C90 to C101, C33 to C202, C32 to C203, C332 to C204, C70 to C205, C71 to C206, C72 to C207, C73 to C208, C34 to C210, C43 to C222, C42 to C223, C78 to C225, C77 to C226, C86 to C229, C16 to C232, C15 to C233, C188 to C250, C190 to C251, C189 to C252, C191 to C253, C84 to C265, C85 to C269, C51 to C301, C52 to C310, C53 to C311, C54 to C312, C55 to C313, C56 to C314, C58 to C316, C59 to C317, C60 to C318, C61 to C319, C62 to C320, C63 to C321, C64 to C322, C65 to C323, C66 to C330, C69 to C331, C67 to C332, C68 to C340, C80 to C350, C81 to C351, C5 to C420, C1 to C500, C2 to C501, C907 to C530, C908 to C540, C25 to C830, D2 to D800, D5 to D810, D6 to D820, D201 to D840, FB1 to F229, FB2 to F269, J1 to J800, L30 to L200, L40 to L220, L10 to L230, L191 to L250, L1 to L500, Q1 to Q110, Q200 to Q840, R91 to R100, R47 to R110, R46 to R111, R30 to R201, R32 to R202, R33 to R203, R34 to R210, R35 to R211, R36 to R212, R37 to R213, R5 to R232, R6 to R233, R51 to R330, R52 to R331, R53 to R340, R54 to R341, R60 to R400, R62 to R410, R63 to R700, R64 to R701, R7 to R800, R8 to R801, R72 to R805, R68 to R810, R69 to R811, SW1 to SW850, U30 to U200, U40 to U220, U6 to U230, U187 to U250, U500 to U260, U4 to U300, U994 to U400, U1 to U500, U8 to U830, Y2 to Y100
Connections:
- net /wireless/PCM_CLK renamed Net-(U500-Pad26)
- net /wireless/PCM_IN renamed Net-(U500-Pad27)
- net /wireless/PCM_OUT renamed Net-(U500-Pad25)
- net /wireless/PCM_SYNC renamed Net-(U500-Pad28)
- net Net-(D400-Pad1) renamed /EMMC_D0_SHORT
- R410 pad 1: GND -> /emmc/EMMC_VSEL
- R410 pad 2: Net-(R62-Pad2) -> GND
- R805 pad 1: GND -> /rk3308-io/USB_EXTR
- R805 pad 2: Net-(R72-Pad2) -> GND
- R830 pad 1: /rk3308-io/I2C1_SCL -> +3V3
- R830 pad 2: +3V3 -> /rk3308-io/I2C1_SCL
- R831 pad 1: /rk3308-io/I2C1_SDA -> +3V3
- R831 pad 2: +3V3 -> /rk3308-io/I2C1_SDA
- SW850 pad 1: Net-(SW1-Pad1) -> GND
- SW850 pad 2: Net-(SW1-Pad2) -> GND
- SW850 pad 3: Net-(SW1-Pad3) -> /KEY
- U1000 pad C15: Net-(R72-Pad2) -> /rk3308-io/USB_EXTR
- U1000 pad R3: Net-(R62-Pad2) -> /emmc/EMMC_VSEL
- U1000 pad T1: Net-(U1000-PadT1) -> /KEY
- U1000 pad W3: Net-(U1000-PadW3) -> /LED
- U300 pad A2: /ddr/DDR_D6 -> /ddr/DDR_D1
- U300 pad C2: /ddr/DDR_D5 -> /ddr/DDR_D0
- U300 pad C3: /ddr/DDR_D1 -> /ddr/DDR_D2
- U300 pad C8: /ddr/DDR_D0 -> /ddr/DDR_D5
- U300 pad D7: /ddr/DDR_D2 -> /ddr/DDR_D6
- U300 pad F8: /ddr/DDR_D15 -> /ddr/DDR_D14
- U300 pad G2: /ddr/DDR_D14 -> /ddr/DDR_D12
- U300 pad H3: /ddr/DDR_D12 -> /ddr/DDR_D15
Routing:
- net /KEY: track 0.00 -> 51.5 mm, vias 0 -> 3
- net /LED: track 4.50 -> 36.0 mm, vias 1 -> 2
- net +5V: track 8.87 -> 17.6 mm
- net +3V3: track 74.7 -> 82.7 mm, vias 26 -> 28
- net /wireless/LPO: track 3.85 -> 11.5 mm, vias 0 -> 2
- net +1V0C: track 50.0 -> 57.5 mm
- net /ddr/DDR_D7: track 24.0 -> 19.4 mm, vias 0 -> 2
- net /ddr/DDR_D5: track 24.1 -> 19.4 mm, vias 0 -> 2
- net /ddr/DDR_D2: track 24.0 -> 19.5 mm, vias 0 -> 2
- net /ddr/DDR_D3: track 24.1 -> 19.9 mm
- net /ddr/DDR_D4: track 24.0 -> 19.9 mm
- net /ddr/DDR_DQS0N: track 24.0 -> 19.9 mm
- net /ddr/DDR_DM0: track 24.0 -> 19.9 mm
- net /ddr/DDR_DQS0P: track 24.0 -> 19.9 mm
- net /ddr/DDR_D6: track 23.6 -> 19.5 mm
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
Commit message: wip
Parts:
- added C2551: 2.2u,10V, require:C_0402, F.Cu at (102.2, 74.0)
- added C2552: 2.2u, require:C_0402, F.Cu at (99.8, 74.0)
- added L255: 0.47u,3A, require:L_0806, F.Cu at (101.0, 72.0)
- added U255: LM3281, require:LM3281_DSBGA6, F.Cu at (101.0, 74.0)
- A500: renamed from ANT1; value ANT12 -> AH104N2450D1-T
- C100, C101: value 15p -> 22p
- C200: value 0.1u,10V -> 0.1u
- C540: value 4.7u -> 10u
- D400: footprint Diodes_SMD:D_SOD-523 -> require:D_SOD-523
- D800, D810, D820, D850: value ESD5302F -> PESDUC3FD5VU; footprint require:ESD_DFN1006_3L -> require:SOT-883
- D840: footprint LEDs:LED_0402 -> require:LED_0402
- J800: value USB_B_Micro -> Molex 47346-0001
- L250: value 2.2u -> 0.24u,3A
- L500: footprint Inductors_SMD:L_0402 -> require:L_0402
- Q110: value Q_NMOS_GSD -> LN235N3T5G
- Q840: value NPND_SOT_363 -> LMBT3904DW1T1G
- Y100: value Crystal_GND24 -> 24MHz,12pF,10ppm
- Y520: value Crystal_GND24 -> 37.4MHz,12pF,10ppm
- moved D400 0.18 mm to (65.3, 55.9)
- moved R111 0.16 mm to (60.8, 73.8)
- moved C110 0.08 mm to (62.6, 73.8)
- turned R410 to 0 degrees
- turned R805 to 0 degrees
- turned R830 to 0 degrees
- turned R831 to 0 degrees
- renumbered U1000 to U100
Connections:
- D820 pad 1: /rk3308-io/D20 -> /rk3308-io/D19
- D820 pad 2: /rk3308-io/D19 -> /rk3308-io/D20
- J800 pad 2: Net-(D800-Pad2) -> Net-(D800-Pad1)
- J800 pad 3: Net-(D800-Pad1) -> Net-(D800-Pad2)
- LP10 pad 1: Net-(D810-Pad2) -> Net-(D810-Pad1)
- LP9 pad 1: Net-(D810-Pad1) -> Net-(D810-Pad2)
- R800 pad 1: Net-(D800-Pad1) -> Net-(D800-Pad2)
- R801 pad 1: Net-(D800-Pad2) -> Net-(D800-Pad1)
- R810 pad 1: Net-(D810-Pad1) -> Net-(D810-Pad2)
- R811 pad 1: Net-(D810-Pad2) -> Net-(D810-Pad1)
Routing:
- net /rk3308-io/D9: track 9.12 -> 7.62 mm
- net Net-(R72-Pad2): track 1.42 -> 0.00 mm, vias 1 -> 0
- net /rk3308-io/USB_EXTR: track 0.00 -> 1.42 mm, vias 0 -> 1
- net /rk3308-io/D10: track 10.1 -> 9.32 mm
- net /EMMC_D0_SHORT: track 24.1 -> 23.5 mm
- net GND: track 242.1 -> 242.5 mm, vias 166 -> 167

Commit message: wip
Parts:
- removed C250, C251, C252, C253: 22p, require:C_0402
- removed C259: 1u, require:C_0402
- removed C550: 4.7u, require:C_0402
- removed L250: 0.24u,3A, Inductors_SMD:L_0603
- removed the L255 at (101.0, 72.0)
- removed U250: TPS62088_FIXED, require:TPS62088_DSBGA6
- removed the U255 at (101.0, 74.0)
- removed Y550: SG-3030CM, Oscillators:Oscillator_SMD_SeikoEpson_SG3030CM
- added L255: 0.47u,3A, require:L_0806, F.Cu at (89.5, 70.5)
- added L255: 0.47u,3A, require:L_0806, B.Cu at (100.0, 72.5)
- added REF**: C_0402, require:C_0402, B.Cu at (101.0, 68.8)
- added REF**: R_0402, require:R_0402, B.Cu at (101.0, 67.8)
- added REF**: R_0402, require:R_0402, B.Cu at (101.0, 66.8)
- added REF**: C_0603, require:C_0603, B.Cu at (102.8, 70.2)
- added REF**: C_0603, require:C_0603, B.Cu at (99.2, 70.2)
- added REF**: R_0402, require:R_0402, B.Cu at (89.0, 71.2)
- added REF**: R_0402, require:R_0402, B.Cu at (89.0, 72.2)
- added REF**: C_0402, require:C_0402, B.Cu at (89.0, 73.2)
- added U255: PAM2305CGFADJ, require:U-DFN2020-6, F.Cu at (90.5, 72.8)
- added U255: PAM2305CGFADJ, require:U-DFN2020-6, B.Cu at (101.0, 70.3)
- C2551, C2552: footprint require:C_0402 -> require:C_0603
- moved C2552 11.1 mm to (88.8, 72.8)
- moved C2551 10.0 mm to (92.2, 72.8)
Connections:
- U100 pad M17: +1V8 -> Net-(U100-PadM17)
- U100 pad N17: +1V8 -> Net-(U100-PadN17)
- U100 pad P16: +3V3 -> Net-(U100-PadP16)
- U100 pad Y2: Net-(U100-PadY2) -> /wireless/LPO
Routing:
- net /wireless/LPO: track 11.5 -> 40.9 mm
- net +3V3: track 82.7 -> 70.7 mm, vias 28 -> 21
- net +5V: track 17.6 -> 8.78 mm, vias 1 -> 0
- net GND: track 242.5 -> 236.8 mm, vias 167 -> 164
- net (no net): track 0.00 -> 3.08 mm, vias 0 -> 3
- net Net-(L250-Pad1): track 1.96 -> 0.00 mm
- net +1V8: track 19.7 -> 18.1 mm, vias 4 -> 3
- net /LED: track 36.0 -> 36.6 mm

Commit message: wip
Parts:
- removed C220, C230: 0.1u, require:C_0402
- removed L255: 0.47u,3A, require:L_0806
- removed R200: R, require:R_0402
- removed REF** (x2): C_0402, require:C_0402
- removed REF** (x4): R_0402, require:R_0402
- removed REF** (x2): C_0603, require:C_0603
- removed U255: PAM2305CGFADJ, require:U-DFN2020-6
- added C252: 22p, require:C_0402, F.Cu at (90.5, 65.2)
- added R252: 110k,1%, require:R_0402, F.Cu at (90.5, 66.2)
- added R253: 150k,1%, require:R_0402, F.Cu at (90.5, 67.2)
- C222, R222, R223: moved to F.Cu
- C251: renamed from C2551; moved to B.Cu
- C253: renamed from C2552; value 2.2u -> 22u; moved to B.Cu
- J800: footprint require:USB_Micro-B_Molex_47346-0001 -> require:USB_Micro-B_Molex-105164-0001
- L220, L230: value 2.2u -> 0.47u,3A; footprint require:L_murata_2520 -> require:L_0806
- L250: renamed from L255; moved to B.Cu
- U220, U230: value SY8089AAC -> PAM2305CGFADJ; footprint TO_SOT_Packages_SMD:SOT-23-5 -> require:U-DFN2020-6
- U250: renamed from U255; moved to B.Cu
- moved C251 6.86 mm to (93.5, 66.0), turned to 90 degrees
- moved C253 6.86 mm to (90.0, 66.0), turned to 90 degrees
- moved U250 6.86 mm to (91.8, 66.0)
- moved R223 6.21 mm to (90.5, 72.5)
- moved C223 5.40 mm to (90.0, 71.2), turned to 90 degrees
- moved R232 5.30 mm to (89.0, 63.8), turned to 90 degrees
- moved R233 5.30 mm to (91.0, 63.8), turned to 270 degrees
- moved R222 5.15 mm to (90.5, 71.5), turned to 0 degrees
- moved C221 5.06 mm to (93.5, 71.2), turned to 90 degrees
- moved C231 4.92 mm to (92.5, 61.5), turned to 270 degrees
- moved C222 4.75 mm to (90.5, 70.5), turned to 0 degrees
- moved C233 4.47 mm to (89.0, 61.5), turned to 270 degrees
- moved C232 3.47 mm to (90.0, 63.8), turned to 90 degrees
- moved L250 2.36 mm to (90.8, 68.5)
- moved L220 2.35 mm to (90.8, 73.8), turned to 180 degrees
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Connections:
- C200 pad 1: +3V3 -> +5V
- C201 pad 1: +3V3 -> +5V
- C221 pad 1: +3V3 -> +5V
- C231 pad 1: +3V3 -> +5V
- J800 pad 2: Net-(D800-Pad1) -> Net-(D800-Pad2)
- J800 pad 3: Net-(D800-Pad2) -> Net-(D800-Pad1)
- R800 pad 1: Net-(D800-Pad2) -> Net-(D800-Pad1)
- R801 pad 1: Net-(D800-Pad1) -> Net-(D800-Pad2)
- U200 pad 1: Net-(R200-Pad1) -> +5V
- U200 pad 4: +3V3 -> +5V
- U220 pad 1: +3V3 -> Net-(U220-Pad1)
- U220 pad 2: GND -> +5V
- U220 pad 3: Net-(L220-Pad1) -> +5V
- U220 pad 4: +3V3 -> Net-(L220-Pad1)
- U220 pad 5: Net-(C222-Pad2) -> GND
- U230 pad 1: +3V3 -> Net-(U230-Pad1)
- U230 pad 2: GND -> +5V
- U230 pad 3: Net-(L230-Pad1) -> +5V
- U230 pad 4: +3V3 -> Net-(L230-Pad1)
- U230 pad 5: Net-(C232-Pad2) -> GND
Routing:
- net +3V3: track 70.7 -> 49.2 mm, vias 21 -> 20
- net GND: track 236.8 -> 246.7 mm, vias 164 -> 272
- net /wireless/LPO: track 40.9 -> 31.8 mm
- net +1V0C: track 57.5 -> 50.1 mm
- net +5V: track 8.78 -> 15.1 mm, vias 0 -> 5
- net /KEY: track 51.8 -> 45.7 mm
- net Net-(C202-Pad2): track 10.2 -> 5.16 mm
- net Net-(C252-Pad2): track 0.00 -> 3.71 mm, vias 0 -> 1
- net (no net): track 3.08 -> 0.00 mm, vias 3 -> 0
- net VCC_DDR: track 56.5 -> 53.7 mm, vias 26 -> 27
- net Net-(C232-Pad2): track 5.58 -> 3.16 mm
- net /USB_OTG_D_N: track 35.7 -> 33.5 mm
- net Net-(L250-Pad1): track 0.00 -> 2.11 mm
- net /USB_OTG_D_P: track 35.8 -> 33.8 mm
- net +1V0L: track 10.4 -> 8.47 mm
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- added copper zone on In3.Cu, net +5V
Other:
- outline, holes or cut-outs redrawn

Commit message: wip
Parts:
- added L255: 0.47u,3A, require:L_0806, B.Cu at (90.8, 76.0)
- D850, R850: moved to F.Cu
- moved D850 3.05 mm to (87.7, 74.4), turned to 90 degrees
- moved R850 3.05 mm to (88.7, 74.4), turned to 270 degrees
Routing:
- net /KEY: track 45.7 -> 31.1 mm, vias 3 -> 1
- net +3V3: track 49.2 -> 48.6 mm, vias 20 -> 19
- net GND: vias 272 -> 271

Commit message: wip
Parts:
- removed L255: 0.47u,3A, require:L_0806
- added C324: 0.1u, require:C_0402, B.Cu at (86.0, 61.0)
- added C325: 0.1u, require:C_0402, B.Cu at (76.0, 61.2)
- added C326: 0.1u, require:C_0402, B.Cu at (81.1, 63.7)
- added L251: 2.2u,0806, require:L_0806, B.Cu at (90.8, 76.2)
- C201, C221, C231: value 10u -> 10u,10V; footprint require:C_0603 -> require:C_0805
- C202, C222, C232, C252: value 22p -> 100p
- C210: value 0.1u -> 10n
- C223, C233: value 22u -> 10u
- C251: value 2.2u,10V -> 10u,10V; footprint require:C_0603 -> require:C_0805
- C253: value 22u -> 10u,10V; footprint require:C_0603 -> require:C_0805
- D850, R850: moved to B.Cu
- L230: value 0.47u,3A -> 2.2u
- L250: value 0.47u,3A -> 2.2u,0806
- R201: value 100R,1% -> 100R
- R210: value 10k -> 169k,1%
- R232: value 110k,1% -> 150k,1%
- R233: value 150k,1% -> 100k,1%
- R252: value 110k,1% -> 540k,1%
- R253: value 150k,1% -> 120k,1%
- moved L250 5.50 mm to (90.8, 74.0)
- moved C221 5.26 mm to (93.8, 66.0)
- moved C251 5.26 mm to (93.8, 71.2)
- moved C253 5.26 mm to (89.8, 71.2)
- moved C222 5.25 mm to (90.5, 65.2)
- moved C223 5.25 mm to (90.0, 66.0)
- moved C252 5.25 mm to (90.5, 70.5)
- moved L220 5.25 mm to (90.8, 68.5)
- moved R222 5.25 mm to (90.5, 66.2)
- moved R223 5.25 mm to (90.5, 67.2)
- moved R252 5.25 mm to (90.5, 71.5)
- moved R253 5.25 mm to (90.5, 72.5)
- moved U220 5.25 mm to (91.8, 66.0)
- moved U250 5.25 mm to (91.8, 71.2)
- moved D840 3.58 mm to (96.0, 62.2), turned to 270 degrees
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Connections:
- SW850 pad 4: Net-(SW850-Pad4) -> /KEY
Routing:
- net GND: track 246.7 -> 274.3 mm, vias 271 -> 301
- net /KEY: track 31.1 -> 48.7 mm, vias 1 -> 3
- net +5V: track 15.1 -> 21.7 mm, vias 5 -> 10
- net +3V3: track 48.6 -> 54.5 mm, vias 19 -> 18
- net +1V8: track 18.1 -> 13.3 mm, vias 3 -> 2
- net /LED: track 37.7 -> 33.2 mm
- net VCC_DDR: track 53.7 -> 56.9 mm, vias 27 -> 28
- net Net-(L250-Pad1): track 2.11 -> 4.61 mm
- net Net-(C330-Pad1): track 17.2 -> 19.1 mm
- net +1V0L: track 8.47 -> 9.82 mm, vias 7 -> 8
- net Net-(C202-Pad2): track 5.16 -> 6.16 mm
- net Net-(D840-Pad1): track 2.03 -> 1.06 mm
- net +1V0C: track 50.1 -> 49.2 mm, vias 8 -> 9

Commit message: wip
Parts:
- moved C830 1.17 mm to (70.2, 58.5)
- moved U830 0.49 mm to (71.7, 57.5)
Routing:
- net GND: track 274.3 -> 277.9 mm, vias 301 -> 303
- net /wireless/LPO: track 31.8 -> 29.0 mm
- net /rk3308-io/D14: track 17.5 -> 14.7 mm
- net /LED: track 33.2 -> 35.2 mm
- net /KEY: track 48.7 -> 50.5 mm
- net /rk3308-io/D16: track 21.1 -> 22.1 mm
- net /rk3308-io/D13: track 11.1 -> 10.5 mm
- net +3V3: track 54.5 -> 53.8 mm
- net +1V0C: track 49.2 -> 48.6 mm
