File: hardware/require.kicad_pcb (KiCad board)
At the start: 6 copper layers, 68 x 26 mm, 184 parts, among them J800 Molex 47346-0001, Q110 LN235N3T5G, Q840 LMBT3904DW1T1G, SW850 SW_SKSC_4PIN, U100 RK3308, U200 SY8089AAC, U220 PAM2305CGFADJ, U230 PAM2305CGFADJ, U250 PAM2305CGFADJ, U260 NCP707_XDFN4, U300 DDR3_FBGA96, U400 EMMC_BGA_153, U500 ap6255, U830 ATECC608A-MAHDA, Y100 24MHz,12pF,10ppm, Y520 37.4MHz,12pF,10ppm

Commit message: wip
Parts:
- moved C255 0.49 mm to (70.2, 63.2)
- moved R410 0.16 mm to (71.2, 62.4)
- moved R831 0.16 mm to (71.2, 61.4)
- moved R830 0.16 mm to (71.2, 60.5)
- moved U830 0.10 mm to (71.8, 57.5)
Routing:
- net +3V3: track 53.8 -> 53.0 mm
- net GND: track 277.9 -> 278.5 mm, vias 303 -> 310
- net /rk3308-io/D12: track 7.41 -> 6.79 mm
- net /rk3308-io/D13: vias 1 -> 0

Commit message: wip
Parts:
- added R802: 0R, require:R_0603, B.Cu at (96.0, 69.2)
- A500: footprint require:YAIYO_YUDEN_AH104N -> require:ANT_AH104N
- C256, C258: value 1u -> 0.47u
- C405: value 1u -> 2.2u
- C420: value C -> 1u
- C520, C521: value 22p -> 15p
- D400: value D_Schottky -> RB521S
- J800: value Molex 47346-0001 -> Molex 105164-0001
- L200, L540: footprint require:L_murata_2520 -> require:L_1008
- L220: value 0.47u,3A -> 2.2u
- L250, L251: value 2.2u,0806 -> 2.2u
- LP14: value NC -> G
- Q840: footprint TO_SOT_Packages_SMD:SOT-363_SC-70-6 -> require:SOT-363_SC-70-6
- R330, R331: value R -> 1k,1%
- R700, R701: value R -> 51k,1%
- R800, R801: value 2.2R -> 22R
- R850: value 4.7k -> 10k
- RP19: value BYP -> U
- U100: footprint require:RK3308_BGA355 -> require:RK3308_TFBGA-355
- U200: footprint TO_SOT_Packages_SMD:SOT-23-5 -> require:SOT-23-5
- U260: value NCP707_XDFN4 -> NCP707CMX180TCG
- U300: footprint require:DDR3_BGA_96 -> require:DDR3_BGA-96
- Y520: value 37.4MHz,12pF,10ppm -> 37.4MHz,9pF,10ppm; footprint require:EPSON_FA_128 -> Crystals:Crystal_SMD_2016-4pin_2.0x1.6mm
- moved U260 0.17 mm to (61.8, 65.0)
Connections:
- net /EMMC_D0_SHORT renamed Net-(D400-Pad1)
- net /emmc/EMMC_VSEL renamed /rk3308-io/EMMC_VSEL
- J800 pad 6: GND -> /SHIELD
Routing:
- net GND: track 278.5 -> 282.2 mm, vias 310 -> 309
- net /SHIELD: track 0.00 -> 1.79 mm, vias 0 -> 2
- net +3V3: track 53.0 -> 52.3 mm
- added copper zone on F.Cu, net /SHIELD
Other:
- rule pad_to_mask_clearance: 0.05 -> 0.025

Commit message: wip
Parts:
- removed D400: RB521S, require:D_SOD-523
- removed D850: PESDUC3FD5VU, require:SOT-883
- removed R850: 10k, require:R_0402
- removed RP19: U, require:OVAL_PIN
- removed SW850: SW_SKSC_4PIN, require:SW_ALPS_SKSCLCE010
- moved R400 5.96 mm to (60.9, 55.5), turned to 0 degrees
Routing:
- net /KEY: track 50.4 -> 0.00 mm, vias 3 -> 0
- net Net-(D400-Pad1): track 23.5 -> 0.00 mm, vias 2 -> 0
- net /ddr/DDR_CS0N: track 21.7 -> 12.4 mm
- net /ddr/DDR_A11: track 22.1 -> 18.9 mm, vias 0 -> 2
- net /emmc/EMMC_D1: track 15.5 -> 12.7 mm
- net /emmc/EMMC_D5: track 15.4 -> 12.8 mm
- net /emmc/EMMC_CLK1: track 12.4 -> 9.77 mm
- net /emmc/EMMC_D7: track 15.5 -> 13.1 mm, vias 1 -> 2
- net /emmc/EMMC_D3: track 15.6 -> 13.2 mm
- net /EMMC_D0: track 16.4 -> 14.3 mm, vias 2 -> 1
- net /emmc/EMMC_D6: track 15.9 -> 14.0 mm
- net /emmc/EMMC_D2: track 15.5 -> 13.7 mm
- net /emmc/EMMC_D4: track 15.3 -> 13.7 mm
- net /emmc/EMMC_CMD: track 15.5 -> 14.2 mm
- net /emmc/EMMC_CLK: track 2.09 -> 3.14 mm
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
Commit message: wip
Parts:
- removed A500: AH104N2450D1-T, require:ANT_AH104N
- removed H1, H2: MountingHole, require:MTG_1.8mm_2.4mm_NPL
- removed L251: 2.2u, require:L_0806
- added C254: 10u,10V, require:C_0805, B.Cu at (42.5, 72.0)
- C202, C210, C540, L540, R201, R202, R203, R210, R211, R212, R213: moved to F.Cu
- C222, C231, C233, C510, C511, C520, C521, D800, J800, L230, R222, R223, R800, R801, U230, Y520: moved to B.Cu
- L250: footprint require:L_0806 -> require:L_1008
- U250: value PAM2305CGFADJ -> SY8089AAC; footprint require:U-DFN2020-6 -> require:SOT-23-5
- Y100: footprint Crystals:Crystal_SMD_3225-4pin_3.2x2.5mm -> Crystals:Crystal_SMD_2016-4pin_2.0x1.6mm
- moved C200 65.1 mm to (31.5, 58.0)
- moved R800 65.0 mm to (24.9, 66.1), turned to 0 degrees
- moved R801 65.0 mm to (24.9, 65.3), turned to 0 degrees
- moved R802 64.3 mm to (32.0, 63.2)
- moved J800 60.6 mm to (37.0, 65.0)
- moved H3 56.9 mm to (38.8, 53.8)
- moved H4 56.9 mm to (38.8, 76.2)
- moved C201 56.6 mm to (38.8, 59.2), turned to 0 degrees
- moved U200 55.8 mm to (38.8, 57.0), turned to 180 degrees
- moved C251 54.8 mm to (39.0, 73.8), turned to 0 degrees
- moved R203 54.8 mm to (37.8, 54.5), turned to 90 degrees
- moved C202 53.6 mm to (38.8, 54.5), turned to 270 degrees
- moved R252 53.0 mm to (37.5, 72.8)
- moved R253 53.0 mm to (37.5, 71.8)
- moved C252 53.0 mm to (37.5, 70.5)
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Connections:
- U250 pad 1: Net-(U250-Pad1) -> +5V
- U250 pad 2: +5V -> GND
- U250 pad 3: +5V -> Net-(L250-Pad1)
- U250 pad 4: Net-(L250-Pad1) -> +5V
- U250 pad 5: GND -> Net-(C252-Pad2)
- U300 pad A3: /ddr/DDR_D4 -> /ddr/DDR_D5
- U300 pad C8: /ddr/DDR_D5 -> /ddr/DDR_D4
Routing:
- net GND: track 281.7 -> 228.1 mm, vias 293 -> 115
- net +1V0C: track 48.6 -> 18.1 mm, vias 9 -> 6
- net /rk3308-io/USB_HOST_DP: track 3.41 -> 28.0 mm
- net /rk3308-io/USB_HOST_DM: track 2.62 -> 26.4 mm
- net +5V: track 21.7 -> 0.00 mm, vias 10 -> 0
- net /power/CORE_DVS: track 21.3 -> 0.46 mm, vias 2 -> 1
- net /rk3308-io/BT_WAKE_HOST: track 20.4 -> 0.00 mm, vias 3 -> 0
- net +3V3: track 51.3 -> 32.2 mm, vias 18 -> 12
- net /ddr/DDR_CLKN: track 20.9 -> 5.42 mm
- net /ddr/DDR_CLKP: track 20.7 -> 5.32 mm
- net /LED: track 35.2 -> 22.1 mm, vias 2 -> 1
- net /ddr/DDR_RESET: track 22.6 -> 9.53 mm, vias 3 -> 2
- net /rk3308-io/SDIO_D2: track 21.2 -> 9.48 mm
- net /rk3308-io/SDIO_D0: track 21.1 -> 9.50 mm
- net /rk3308-io/SDIO_CMD: track 21.4 -> 9.80 mm
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- removed copper zone on F.Cu, net /SHIELD
Other:
- board size 68 x 26 mm -> 50 x 26 mm

Commit message: wip
Parts:
- removed D840: LED, require:LED_0402
- removed H3, H4: MountingHole_Pad, require:MTG_1.8mm_2.4mm_PL
- removed the J800 at (37.0, 65.0)
- removed LP13: NC, require:OVAL_PIN
- removed LP6: A5, require:OVAL_PIN
- removed LP8: RST, require:OVAL_PIN
- removed Q110: LN235N3T5G, require:SOT-883
- removed Q840: LMBT3904DW1T1G, require:SOT-363_SC-70-6
- removed R111: 10k, require:R_0402
- removed R840: 470R, require:R_0402
- removed RP15: 14, require:OVAL_PIN
- removed RP16: 15, require:OVAL_PIN
- removed RP17: 16, require:OVAL_PIN
- added J800: Molex 105164-0001, require:USB_Micro-B_Molex-105164-0001, F.Cu at (44.5, 51.0)
- added J800: Molex 105164-0001, require:USB_Micro-B_Molex-105164-0001, F.Cu at (80.5, 79.0)
- C100, C101, C222, C530, D810, D820, R100, R222, R223, R810, R811, Y100: moved to F.Cu
- C252, R252, R253: moved to B.Cu
- LP2: value A1 -> A0
- LP3: value A2 -> A1
- LP4: value A3 -> A2
- LP5: value A4 -> A3
- moved LP15 43.5 mm to (44.0, 48.0)
- moved LP17 41.1 mm to (40.9, 77.7)
- moved LP16 38.5 mm to (40.9, 75.2)
- moved C200 37.5 mm to (69.0, 56.7), turned to 270 degrees
- moved LP14 30.9 mm to (43.5, 77.7)
- moved R203 30.2 mm to (67.8, 57.2)
- moved C202 30.0 mm to (68.6, 57.2), turned to 90 degrees
- moved R202 29.8 mm to (69.4, 57.2), turned to 90 degrees
- moved R210 29.4 mm to (69.4, 55.2), turned to 90 degrees
- moved C210 29.2 mm to (70.2, 55.2)
- moved R211 29.0 mm to (71.0, 55.2), turned to 90 degrees
- moved C201 28.2 mm to (66.6, 54.6), turned to 180 degrees
- moved U200 27.9 mm to (66.6, 56.8), turned to 0 degrees
- moved R212 27.2 mm to (70.2, 57.2), turned to 270 degrees
- moved R213 27.0 mm to (71.0, 57.2)
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Connections:
- net /EMMC_D0 renamed /emmc/EMMC_D0
- net /KEY renamed Net-(U100-PadT1)
- net /rk3308-io/PCM_CLK renamed Net-(U100-PadF18)
- net /rk3308-io/PCM_IN renamed Net-(U100-PadH14)
- net /rk3308-io/PCM_OUT renamed Net-(U100-PadH15)
- net /rk3308-io/PCM_SYNC renamed Net-(U100-PadJ15)
- net /rk3308-power/RESET_1V8 renamed Net-(C110-Pad1)
- LP2 pad 1: /rk3308-io/A1 -> /rk3308-io/A0
- LP3 pad 1: /rk3308-io/A2 -> /rk3308-io/A1
- LP4 pad 1: /rk3308-io/A3 -> /rk3308-io/A2
- LP5 pad 1: /rk3308-io/A4 -> /rk3308-io/A3
- R400 pad 1: /emmc/EMMC_CLK1 -> Net-(R400-Pad1)
- R400 pad 2: /emmc/EMMC_CLK -> Net-(R400-Pad2)
- R700 pad 2: /rk3308-io/A0 -> /rk3308-io/A4
- R701 pad 1: /rk3308-io/A0 -> /rk3308-io/A4
- R800 pad 1: Net-(D800-Pad1) -> Net-(D800-Pad2)
- R801 pad 1: Net-(D800-Pad2) -> Net-(D800-Pad1)
- U100 pad R4: /rk3308-io/D14 -> Net-(U100-PadR4)
- U100 pad T4: /rk3308-io/D16 -> Net-(U100-PadT4)
- U100 pad T5: /rk3308-io/D15 -> Net-(U100-PadT5)
- U100 pad W3: /LED -> Net-(U100-PadW3)
- U400 pad A8: /emmc/EMMC_D7 -> Net-(U400-PadA8)
- U400 pad B7: /emmc/EMMC_D7 -> Net-(U400-PadB7)
- U400 pad C7: Net-(U400-PadC7) -> /emmc/EMMC_D7
- U400 pad K1: /emmc/EMMC_CLK1 -> /emmc/EMMC_CLK
- U400 pad K2: /emmc/EMMC_CLK1 -> /emmc/EMMC_CLK
- U400 pad K3: /emmc/EMMC_CLK1 -> /emmc/EMMC_CLK
- U400 pad M6: /emmc/EMMC_CLK1 -> /emmc/EMMC_CLK
Routing:
- net +3V3: track 32.2 -> 56.2 mm, vias 12 -> 14
- net /rk3308-io/USB_HOST_DP: track 28.0 -> 5.15 mm, vias 1 -> 0
- net /LED: track 22.1 -> 0.00 mm, vias 1 -> 0
- net /rk3308-io/BT_REG_ON: track 8.77 -> 30.8 mm, vias 1 -> 2
- net /rk3308-io/D16: track 22.0 -> 0.00 mm, vias 1 -> 0
- net /rk3308-io/USB_HOST_DM: track 26.4 -> 5.06 mm, vias 1 -> 0
- net /rk3308-io/D15: track 19.9 -> 0.00 mm, vias 1 -> 0
- net /rk3308-io/BT_WAKE_HOST: track 0.00 -> 17.4 mm, vias 0 -> 2
- net /rk3308-io/D14: track 15.5 -> 0.00 mm, vias 2 -> 0
- net /rk3308-io/D20: track 19.6 -> 8.01 mm, vias 2 -> 0
- net /rk3308-io/A1: track 17.6 -> 6.01 mm, vias 1 -> 0
- net /emmc/EMMC_CLK: track 3.14 -> 13.7 mm
- net +5V: track 0.00 -> 10.3 mm, vias 0 -> 3
- net /rk3308-io/A5: track 10.0 -> 0.00 mm, vias 1 -> 0
- net /emmc/EMMC_CLK1: track 9.77 -> 0.00 mm
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- added copper zone on In4.Cu, net +5V
- removed copper zone on In3.Cu, net +5V
Other:
- board size 50 x 26 mm -> 48 x 28 mm

Commit message: wip
Parts:
- removed C530: 1u, require:C_0402
- removed LP15, RP1: G, require:OVAL_PIN
- removed R201: 100R, require:R_0402
- removed R802: 0R, require:R_0603
- added R812: 22R, require:R_0402, B.Cu at (73.1, 75.5)
- added R813: 22R, require:R_0402, B.Cu at (72.3, 75.5)
- D800, R800, R801: moved to F.Cu
- moved C300 19.5 mm to (84.5, 72.0)
- moved LP1 3.59 mm to (40.9, 72.6)
- moved R801 3.25 mm to (45.8, 57.7), turned to 0 degrees
- moved C540 3.01 mm to (50.2, 56.8)
- moved R810 2.53 mm to (69.1, 75.0)
- moved R811 2.53 mm to (69.1, 74.2)
- moved R100 2.02 mm to (54.8, 69.0), turned to 90 degrees
- moved C510 1.81 mm to (50.2, 68.8), turned to 0 degrees
- moved R800 1.75 mm to (46.2, 56.9), turned to 0 degrees
- moved C511 1.72 mm to (50.2, 69.8), turned to 0 degrees
- moved D800 1.64 mm to (44.7, 56.8), turned to 135 degrees
- moved L540 1.52 mm to (52.5, 56.8), turned to 180 degrees
- moved C400 1.50 mm to (57.0, 62.8)
- moved C401 1.50 mm to (56.0, 63.0)
- moved C402 1.50 mm to (55.2, 63.0)
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- renumbered J800 to J801
Connections:
- J800 pad 6: /SHIELD -> GND
- J801 pad 1: (no net) -> +5V
- J801 pad 2: (no net) -> Net-(J801-Pad2)
- J801 pad 3: (no net) -> Net-(J801-Pad3)
- J801 pad 4: (no net) -> Net-(J801-Pad4)
- J801 pad 5: (no net) -> GND
- J801 pad 6: (no net) -> GND
Routing:
- net GND: track 229.2 -> 251.4 mm, vias 117 -> 137
- net +5V: track 10.3 -> 23.9 mm, vias 3 -> 10
- net Net-(J801-Pad2): track 0.00 -> 11.6 mm, vias 0 -> 1
- net Net-(D810-Pad1): track 0.00 -> 10.3 mm
- net +3V3: track 56.2 -> 66.1 mm, vias 14 -> 18
- net /rk3308-io/D12: track 1.58 -> 11.5 mm
- net Net-(J801-Pad3): track 0.00 -> 9.88 mm, vias 0 -> 1
- net Net-(D810-Pad2): track 0.00 -> 9.61 mm
- net /ddr/DDR_CLKN: track 5.42 -> 14.7 mm
- net VCC_DDR: track 46.5 -> 55.2 mm, vias 24 -> 27
- net Net-(C520-Pad1): track 0.00 -> 8.56 mm, vias 0 -> 1
- net /rk3308-io/D11: track 1.60 -> 9.64 mm
- net +1V0C: track 11.0 -> 18.7 mm, vias 7 -> 8
- net Net-(C521-Pad1): track 0.00 -> 7.14 mm, vias 0 -> 1
- net Net-(C202-Pad2): track 0.00 -> 5.70 mm, vias 0 -> 1
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Other:
- board size 48 x 28 mm -> 48 x 28.6 mm
- net class mmc: trace_width 0.125 -> 0.1

Commit message: wip
Parts:
- added C530: 1u, require:C_0402, F.Cu at (49.2, 56.8)
- added TP100: TestPoint, require:TP08, B.Cu at (61.3, 62.7)
- added TP101: TestPoint, require:TP08, B.Cu at (63.4, 63.0)
- moved R400 17.7 mm to (61.8, 61.8)
- moved LP1 3.59 mm to (43.5, 75.2)
- moved C100 1.80 mm to (53.8, 69.2)
- moved R100 1.58 mm to (55.2, 67.5), turned to 0 degrees
- moved C340 1.39 mm to (79.6, 64.5), turned to 180 degrees
- moved C101 1.35 mm to (55.2, 71.0)
- moved Y100 1.35 mm to (55.2, 69.2)
- moved D810 0.50 mm to (70.5, 75.1)
- moved R810 0.50 mm to (69.1, 75.5)
- moved R811 0.50 mm to (69.1, 74.7)
- moved R341 0.30 mm to (79.6, 65.4)
- moved R340 0.30 mm to (79.6, 66.2)
Connections:
- R400 pad 2: Net-(R400-Pad2) -> /emmc/EMMC_CLK
- U400 pad K1: /emmc/EMMC_CLK -> Net-(R400-Pad1)
- U400 pad K2: /emmc/EMMC_CLK -> Net-(R400-Pad1)
- U400 pad K3: /emmc/EMMC_CLK -> Net-(R400-Pad1)
- U400 pad M6: /emmc/EMMC_CLK -> Net-(R400-Pad1)
Routing:
- net /emmc/EMMC_CLK: track 14.2 -> 1.31 mm
- net Net-(R400-Pad1): track 0.00 -> 10.6 mm
- net /ddr/DDR_CLKP: track 10.7 -> 18.1 mm
- net /ddr/DDR_A7: track 11.4 -> 16.8 mm
- net /ddr/DDR_A2: track 11.6 -> 16.7 mm
- net /ddr/DDR_CLKN: track 14.7 -> 18.9 mm
- net +3V3: track 66.1 -> 69.7 mm, vias 18 -> 19
- net GND: track 251.4 -> 247.9 mm, vias 137 -> 144
- net /ddr/DDR_A9: track 13.4 -> 16.7 mm
- net /ddr/DDR_A6: track 16.0 -> 19.2 mm
- net /ddr/DDR_A1: track 14.4 -> 17.3 mm
- net /ddr/DDR_A4: track 16.4 -> 19.1 mm
- net /emmc/EMMC_CMD: track 9.21 -> 11.8 mm
- net /ddr/DDR_DM0: track 19.8 -> 17.2 mm
- net /ddr/DDR_BA1: track 16.7 -> 19.2 mm
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
Commit message: prepare gerber and drill
Parts:
- removed the LP1 at (43.5, 75.2)
- removed LP16: 3V3, require:OVAL_PIN
- removed LP18: 5V, require:OVAL_PIN
- added ANT1: ANT_LA52H2450_5500_A28, require:LA52H2450_5500_A28, F.Cu at (49.3, 77.6)
- added LP8: 5V, require:OVAL_PIN, F.Cu at (68.8, 77.7)
- added R820: 22R, require:R_0402, F.Cu at (60.4, 73.6)
- added R821: 22R, require:R_0402, F.Cu at (63.6, 73.6)
- added R840: 10k, require:R_0402, F.Cu at (56.0, 54.2)
- added R841: 10k, require:R_0402, F.Cu at (56.0, 55.2)
- F229, F269: footprint Inductors_SMD:L_0402 -> require:L_0402
- Y100, Y520: footprint Crystals:Crystal_SMD_2016-4pin_2.0x1.6mm -> require:Crystal_SMD_2016-4pin_2.0x1.6mm
- moved R701 3.23 mm to (57.4, 69.8), turned to 90 degrees
- moved D820 2.83 mm to (62.8, 75.6)
- moved C500 1.86 mm to (45.2, 74.8), turned to 270 degrees
- moved C501 1.86 mm to (43.0, 74.8), turned to 270 degrees
- moved R700 1.68 mm to (58.2, 69.8)
- moved R222 1.60 mm to (61.2, 73.6)
- moved L500 1.50 mm to (44.1, 74.2)
- moved C110 1.44 mm to (59.0, 69.8), turned to 90 degrees
- moved R110 1.30 mm to (59.8, 70.1)
- moved R232 1.01 mm to (84.5, 56.6)
- moved C232 0.81 mm to (83.7, 56.6)
- moved R213 0.81 mm to (70.7, 56.6)
- moved R223 0.81 mm to (62.8, 73.6)
- moved R211 0.80 mm to (70.7, 54.8)
- moved R212 0.62 mm to (69.9, 56.6)
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- renumbered LP17 to LP1, LP14 to LP2, LP2 to LP3, LP3 to LP31, LP5 to LP41, LP11 to LP5, LP12 to LP6, RP2 to RP1, RP11 to RP10, RP12 to RP11, RP13 to RP12, RP14 to RP13, RP18 to RP14, RP3 to RP2, RP4 to RP3, RP5 to RP4, RP6 to RP5, RP7 to RP6, RP8 to RP7, RP9 to RP8, RP10 to RP9
Connections:
- net /rk3308-io/USB_HOST_DM renamed /USB_HOST_D1_N
- net /rk3308-io/USB_HOST_DP renamed /USB_HOST_D1_P
- net Net-(C501-Pad1) renamed /wireless/RFOUT
- net Net-(D810-Pad1) renamed /USB_HOST_D2_P
- net Net-(D810-Pad2) renamed /USB_HOST_D2_N
- net Net-(J801-Pad2) renamed /USB_HOST_D3_P
- net Net-(J801-Pad3) renamed /USB_HOST_D3_N
- C500 pad 1: Net-(C500-Pad1) -> GND
- D820 pad 1: /rk3308-io/D19 -> Net-(D820-Pad1)
- D820 pad 2: /rk3308-io/D20 -> Net-(D820-Pad2)
- L500 pad 2: Net-(C500-Pad1) -> GND
- LP5 pad 1: /rk3308-io/D19 -> Net-(D820-Pad1)
- LP6 pad 1: /rk3308-io/D20 -> Net-(D820-Pad2)
Routing:
- net +3V3: track 69.7 -> 76.1 mm, vias 19 -> 22
- net Net-(D820-Pad1): track 0.00 -> 5.47 mm
- net /rk3308-io/D20: track 8.01 -> 2.61 mm
- net /rk3308-io/D19: track 8.52 -> 3.32 mm
- net /rk3308-io/D2: track 23.0 -> 27.5 mm, vias 2 -> 3
- net Net-(D820-Pad2): track 0.00 -> 4.36 mm
- net /rk3308-io/A4: track 2.00 -> 5.18 mm
- net /rk3308-io/BT_WAKE_HOST: track 19.8 -> 18.0 mm
- net /rk3308-io/HOST_WAKE_BT: track 19.4 -> 17.6 mm
- net /USB_HOST_D3_N: track 9.88 -> 11.6 mm
- net +1V0L: track 9.15 -> 7.98 mm
- net +1V8: track 9.54 -> 10.6 mm
- net /rk3308-io/D1: track 16.8 -> 17.7 mm, vias 1 -> 2
- net Net-(C520-Pad1): track 8.56 -> 7.66 mm
- net /USB_OTG_D_N: track 28.3 -> 29.0 mm
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- added copper zone on F.Cu, net /wireless/RFOUT
Other:
- outline, holes or cut-outs redrawn
- net class Default: trace_width 0.2 -> 0.15
- board text added: "2.4G/5G 802.11ac Wifi + Bluetooth 4.1"
- board text added: "3V3"
- board text added: "512MB DDR3"
- board text added: "5V"
- board text added: "A0"
- board text added: "A1"
- board text added: "A2"
- board text added: "A3"
- board text added: "CK0"
- board text added: "CK2"
- board text added: "CS0"
- board text added: "CS2"
- board text added: "CTS0"
- board text added: "CTS1"
- board text added: "D+"
- board text added: "D-"
- board text added: "D1"
- board text added: "D10"
- board text added: "D11"
- board text added: "D12"
- board text added: "D13"
- board text added: "D2"
- board text added: "D3"
- board text added: "D4"
- board text added: "D5"
- board text added: "D6"
- board text added: "D7"
- board text added: "D8"
- board text added: "D9"
- board text added: "GND"
- board text added: "GPIO0_B6"
- board text added: "GPIO0_B7"
- board text added: "GPIO0_C0"
- board text added: "GPIO1_C6"
- board text added: "GPIO1_C7"
- board text added: "GPIO1_D0"
- board text added: "GPIO1_D1"
- board text added: "GPIO2_A0"
- board text added: "GPIO2_A1"
- board text added: "GPIO2_A2"
- board text added: "GPIO2_A3"
- board text added: "GPIO3_B4"
- board text added: "GPIO3_B5"
- board text added: "GPIO4_D2"
- board text added: "GPIO4_D3"
- board text added: "MI0"
- board text added: "MI2"
- board text added: "MO0"
- board text added: "MO2"
- board text added: "On-board 8G/16G eMMC (bottom side)"
- board text added: "On-board Microchip CryptoAuth chip for secure authentication (bottom side)"
- board text added: "PWM1"
- board text added: "PWM2"
- board text added: "PWM3"
- board text added: "RTS0"
- board text added: "RTS1"
- board text added: "RX0"
- board text added: "RX1"
- board text added: "RX2"
- board text added: "RX2/TCK"
- board text added: "RX3"
- board text added: "Rockchip RK3308, Quad-Core A35"
- board text added: "SCL0"
- board text added: "SCL2"
- board text added: "SCL3"
- board text added: "SDA0"
- board text added: "SDA2"
- board text added: "SDA3"
- board text added: "TX0"
- board text added: "TX1"
- board text added: "TX2"
- board text added: "TX2/TMS"
- board text added: "TX3"
- board text added: "USB Device & Power"
- board text added: "USB Host"
- board text added: "chip antenna"
