File: hardware/test.sch (KiCad schematic (older format))
At the start: 8 parts, among them J1 Conn_01x02, J9100 microSD-13p, U1000 RK3308, U6000 ap6255

Commit message: wip
Parts:
- removed J9100: microSD-13p, require:xunpu_microSD_tf_115, symbol require-rescue:microSD-13p
- removed R1712: 22R, Resistors_SMD:R_0402, symbol Device:R
- added C122, C123: C, Capacitors_SMD:C_0402, symbol Device:C
- added C6008: 4.7u, Capacitors_SMD:C_0603, symbol Device:C
- added L123: L, Inductors_SMD:L_0402, symbol Device:L
- added L6002: 3.3u, require:L_murata_2520, symbol Device:L
Connections:
- net labels removed: SDMMC_CLK, SDMMC_CMD, SDMMC_D0, SDMMC_D1, SDMMC_D2, SDMMC_D3, SDMMC_PWREN
- wire segments 73 -> 71
- no-connect marks 4 -> 11

Commit message: wip
Connections:
- net labels added: VCC_IO
- net labels removed: VCCIO_SDMMC
- wire segments 71 -> 72
Changed lines of the file:
@@
 	4300 4300 4300 4400
 Connection ~ 4300 4400
-$Comp
-L require:VCCIO_SDMMC #PWR0137
-U 1 1 5D24957E
-P 4350 7250
-F 0 "#PWR0137" H 4350 7100 50  0001 C CNN
-F 1 "VCCIO_SDMMC" H 4367 7423 50  0000 C CNN
-F 2 "" H 4350 7250 50  0001 C CNN
-F 3 "" H 4350 7250 50  0001 C CNN
-	1    4350 7250
-	1    0    0    -1
-$EndComp
 Wire Wire Line
 	4350 7250 4350 7350
@@
 	1    0    0    -1
 $EndComp
+$Comp
+L require:VCC_IO #PWR0137
+U 1 1 5CA02A89
+P 4350 7250
+F 0 "#PWR0137" H 4350 7100 50  0001 C CNN
+F 1 "VCC_IO" H 4367 7423 50  0000 C CNN
+F 2 "" H 4350 7250 50  0001 C CNN
+F 3 "" H 4350 7250 50  0001 C CNN
+	1    4350 7250
+	1    0    0    -1
+$EndComp
+Wire Wire Line
+	13750 4750 14000 4750
+$Comp
+L power:GND #PWR?
+U 1 1 5CB230DF
+P 14000 4750
+F 0 "#PWR?" H 14000 4500 50  0001 C CNN
+F 1 "GND" V 14005 4622 50  0000 R CNN
+F 2 "" H 14000 4750 50  0001 C CNN
+F 3 "" H 14000 4750 50  0001 C CNN
+	1    14000 4750
+	0    -1   -1   0
+$EndComp
 $EndSCHEMATC

Commit message: wip
Parts:
- added C901: 10u, Capacitors_SMD:C_0603, symbol Device:C
- added C902: 0.1u, Capacitors_SMD:C_0402, symbol Device:C
- added C910, C911: 22p, Capacitors_SMD:C_0402, symbol Device:C
- added Y123: Crystal_GND24, require:EPSON_FA_128, symbol Device:Crystal_GND24
Connections:
- wire segments 72 -> 98
Other:
- note added: "epson fa-128"
Changed lines of the file:
@@
 $EndComp
 Wire Wire Line
-	12850 3250 12850 3050
-Wire Wire Line
-	12850 3050 12650 3050
+	12850 3250 12850 1950
 Wire Wire Line
 	13050 3250 13050 3050
@@
 L power:GND #PWR0143
 U 1 1 5D284FAE
-P 12650 3050
-F 0 "#PWR0143" H 12650 2800 50  0001 C CNN
-F 1 "GND" V 12655 2922 50  0000 R CNN
-F 2 "" H 12650 3050 50  0001 C CNN
-F 3 "" H 12650 3050 50  0001 C CNN
-	1    12650 3050
-	0    1    1    0
+P 12850 1950
+F 0 "#PWR0143" H 12850 1700 50  0001 C CNN
+F 1 "GND" V 12855 1822 50  0000 R CNN
+F 2 "" H 12850 1950 50  0001 C CNN
+F 3 "" H 12850 1950 50  0001 C CNN
+	1    12850 1950
+	-1   0    0    1
 $EndComp
 $Comp
@@
 	13750 4750 14000 4750
 $Comp
-L power:GND #PWR?
+L power:GND #PWR0208
 U 1 1 5CB230DF
 P 14000 4750
-F 0 "#PWR?" H 14000 4500 50  0001 C CNN
+F 0 "#PWR0208" H 14000 4500 50  0001 C CNN
 F 1 "GND" V 14005 4622 50  0000 R CNN
 F 2 "" H 14000 4750 50  0001 C CNN
@@
 	0    -1   -1   0
 $EndComp
+Wire Wire Line
+	12050 3250 12050 3100
+Wire Wire Line
+	12150 3250 12150 2800
+Wire Wire Line
+	12250 2150 12250 3250
+Wire Wire Line
+	12450 3250 12450 2050
+Wire Wire Line
+	12450 2050 11200 2050
+Wire Wire Line
+	12550 3250 12550 1950
+Wire Wire Line
+	12550 1950 11200 1950
+Text Label 11200 1950 0    50   ~ 0
+HOST_WAKE_BT
+Text Label 11200 2050 0    50   ~ 0
+BT_WAKE_HOST
+Text HLabel 11200 2050 0    50   Input ~ 0
+BT_WAKE_HOST
+Text HLabel 11200 1950 0    50   Input ~ 0
+HOST_WAKE_BT
+Wire Wire Line
+	9400 2150 9400 2050
+$Comp
+L require:VCC_IO #PWR0209
+U 1 1 5CB3B3D2
+P 9400 2050
+F 0 "#PWR0209" H 9400 1900 50  0001 C CNN
+F 1 "VCC_IO" H 9417 2223 50  0000 C CNN
+F 2 "" H 9400 2050 50  0001 C CNN
+F 3 "" H 9400 2050 50  0001 C CNN
+	1    9400 2050
+	1    0    0    -1
+$EndComp
+$Comp
+L Device:C C901
+U 1 1 5CB3CB45
+P 9400 2500
+F 0 "C901" H 9515 2546 50  0000 L CNN
+F 1 "10u" H 9515 2455 50  0000 L CNN
+F 2 "Capacitors_SMD:C_0603" H 9438 2350 50  0001 C CNN
+F 3 "~" H 9400 2500 50  0001 C CNN
+	1    9400 2500
+	1    0    0    -1
+$EndComp
+$Comp
+L Device:C C902
+U 1 1 5CB3CBB9
+P 10100 2500
+F 0 "C902" H 10215 2546 50  0000 L CNN
+F 1 "0.1u" H 10215 2455 50  0000 L CNN
+F 2 "Capacitors_SMD:C_0402" H 10138 2350 50  0001 C CNN
+F 3 "~" H 10100 2500 50  0001 C CNN
+	1    10100 2500
+	1    0    0    -1
+$EndComp
+Wire Wire Line
+	10100 2750 9400 2750
+Wire Wire Line
+	9400 2750 9400 2650
+Wire Wire Line
+	9400 2750 9400 2850
+Connection ~ 9400 2750
+$Comp
+L power:GND #PWR0210
+U 1 1 5CB4048A
+P 9400 2850
+F 0 "#PWR0210" H 9400 2600 50  0001 C CNN
+F 1 "GND" H 9405 2677 50  0000 C CNN
+F 2 "" H 9400 2850 50  0001 C CNN
+F 3 "" H 9400 2850 50  0001 C CNN
+	1    9400 2850
+	1    0    0    -1
+$EndComp
+Wire Wire Line
+	9400 2350 9400 2150
+Connection ~ 9400 2150
+$Comp
+L Device:Crystal_GND24 Y123
+U 1 1 5CB46F9E
+P 10700 3100
+F 0 "Y123" H 10891 3146 50  0000 L CNN
+F 1 "Crystal_GND24" H 10891 3055 50  0000 L CNN
+F 2 "require:EPSON_FA_128" H 10700 3100 50  0001 C CNN
+F 3 "~" H 10700 3100 50  0001 C CNN
+	1    10700 3100
+	1    0    0    -1
+$EndComp
+Wire Wire Line
+	9400 2150 10100 2150
+Wire Wire Line
+	10100 2350 10100 2150
+Connection ~ 10100 2150
+Wire Wire Line
+	10100 2150 12250 2150
+Wire Wire Line
+	10100 2650 10100 2750
+Wire Wire Line
+	10700 2900 10700 2700
+$Comp
+L power:GND #PWR0211
+U 1 1 5CB54632
+P 10700 2700
+F 0 "#PWR0211" H 10700 2450 50  0001 C CNN
+F 1 "GND" H 10705 2527 50  0000 C CNN
+F 2 "" H 10700 2700 50  0001 C CNN
+F 3 "" H 10700 2700 50  0001 C CNN
+	1    10700 2700
+	-1   0    0    1
+$EndComp
+Wire Wire Line
+	10700 3300 10700 3500
+$Comp
+L power:GND #PWR0212
+U 1 1 5CB5A5A2
+P 10700 3500
+F 0 "#PWR0212" H 10700 3250 50  0001 C CNN
+F 1 "GND" H 10705 3327 50  0000 C CNN
+F 2 "" H 10700 3500 50  0001 C CNN
+F 3 "" H 10700 3500 50  0001 C CNN
+	1    10700 3500
+	1    0    0    -1
+$EndComp
+Wire Wire Line
+	10100 2800 10100 3100
+Wire Wire Line
+	10100 3100 10550 3100
+Wire Wire Line
+	10100 2800 12150 2800
+Wire Wire Line
+	10850 3100 11100 3100
+Text Notes 10900 2950 0    50   ~ 0
+epson fa-128
+$Comp
+L Device:C C911
+U 1 1 5CB62E04
+P 11100 3350
+F 0 "C911" H 11215 3396 50  0000 L CNN
+F 1 "22p" H 11215 3305 50  0000 L CNN
+F 2 "Capacitors_SMD:C_0402" H 11138 3200 50  0001 C CNN
+F 3 "~" H 11100 3350 50  0001 C CNN
+	1    11100 3350
+	1    0    0    -1
+$EndComp
+Wire Wire Line
+	11100 3200 11100 3100
+Connection ~ 11100 3100
+Wire Wire Line
+	11100 3100 12050 3100
+Wire Wire Line
+	11100 3500 11100 3600
+$Comp
+L power:GND #PWR0213
+U 1 1 5CB674FF
+P 11100 3600
+F 0 "#PWR0213" H 11100 3350 50  0001 C CNN
+F 1 "GND" H 11105 3427 50  0000 C CNN
+F 2 "" H 11100 3600 50  0001 C CNN
+F 3 "" H 11100 3600 50  0001 C CNN
+	1    11100 3600
+	1    0    0    -1
+$EndComp
+$Comp
+L Device:C C910
+U 1 1 5CB67581
+P 10100 3350
+F 0 "C910" H 10215 3396 50  0000 L CNN
+F 1 "22p" H 10215 3305 50  0000 L CNN
+F 2 "Capacitors_SMD:C_0402" H 10138 3200 50  0001 C CNN
+F 3 "~" H 10100 3350 50  0001 C CNN
+	1    10100 3350
+	1    0    0    -1
+$EndComp
+Wire Wire Line
+	10100 3200 10100 3100
+Connection ~ 10100 3100
+Wire Wire Line
+	10100 3500 10100 3600
+$Comp
+L power:GND #PWR0214
+U 1 1 5CB6C013
+P 10100 3600
+F 0 "#PWR0214" H 10100 3350 50  0001 C CNN
+F 1 "GND" H 10105 3427 50  0000 C CNN
+F 2 "" H 10100 3600 50  0001 C CNN
+F 3 "" H 10100 3600 50  0001 C CNN
+	1    10100 3600
+	1    0    0    -1
+$EndComp
 $EndSCHEMATC

Commit message: wip
Parts:
- removed C1701: 0.1u, Capacitors_SMD:C_0402, symbol Device:C
- removed J1: Conn_01x02, Connectors_JST:JST_EH_B02B-EH-A_02x2.50mm_Straight, symbol require-rescue:Conn_01x02
- added ANT1: ANT12, require:YAIYO_YUDEN_AH104N, symbol require:ANT12
- added C7: 1u, Capacitors_SMD:C_0402, symbol Device:C
- added C74, C9: 0.1u, Capacitors_SMD:C_0402, symbol Device:C
- added unit 2 of U1000
- added Y4: SG-3030CM, Oscillators:Oscillator_SMD_SeikoEpson_SG3030CM, symbol Oscillator:SG-3030CM
- renumbered C123 to C1, C122 to C2, C901 to C3, C902 to C4, C910 to C5, C911 to C6, C1700 to C76, C6008 to C8, L123 to L1, L6002 to L2, R1700 to R90, U6000 to U1, Y123 to Y1
Connections:
- net labels added: LPO, WIFI_REG_ON, WIFI_WAKE_HOST
- net labels removed: VCC5V0_SYS, VCCIO_SDIO
- wire segments 98 -> 118
- no-connect marks 11 -> 16
Other:
- note added: "SDIO 3.0, 1.8V\nVDDIO 1.8V"
- note added: "Share cap with E14, D14, D13, C14"
- note added: "Use SDIO 2.0 (3V3)"

Commit message: wip
Parts:
- added C14: 1u, Capacitors_SMD:C_0402, symbol Device:C
- added D9: LED_GBAR_0603X2, require:LED_RGB_0603X2, symbol require:LED_GBAR_0603X2
- added LP10: TX2, require:OVAL_PIN, symbol require:OP
- added LP9: RX2, require:OVAL_PIN, symbol require:OP
- added P10: 16, require:OVAL_PIN, symbol require:OP
- added P11: 17, require:OVAL_PIN, symbol require:OP
- added P12: 18, require:OVAL_PIN, symbol require:OP
- added P23: 11, require:OVAL_PIN, symbol require:OP
- added P24: 12, require:OVAL_PIN, symbol require:OP
- added P25: 13, require:OVAL_PIN, symbol require:OP
- added P26: 14, require:OVAL_PIN, symbol require:OP
- added P7: 15, require:OVAL_PIN, symbol require:OP
- added R3: 30k, Resistors_SMD:R_0402, symbol Device:R
- added R4, R5: 22R, Resistors_SMD:R_0402, symbol Device:R
- added U2: AW2015FCR, require:AW2015FCR_QFN8L, symbol require:AW2015FCR
Connections:
- net labels added: CORE_DVS, I2C1_SCL, I2C1_SDA, LED1, LED2, LED3, POWER_SLEEP, PWM1, PWM2, PWM3
- wire segments 118 -> 168
- no-connect marks 16 -> 15

Commit message: wip
Parts:
- removed R90: 22R, Resistors_SMD:R_0402, symbol Device:R
Connections:
- wire segments 168 -> 167
Changed lines of the file:
@@
 Wire Wire Line
 	4150 7350 4350 7350
-$Comp
-L Device:R R90
-U 1 1 5D22225C
-P 5100 2700
-F 0 "R90" V 4893 2700 50  0000 C CNN
-F 1 "22R" V 4984 2700 50  0000 C CNN
-F 2 "Resistors_SMD:R_0402" V 5030 2700 50  0001 C CNN
-F 3 "~" H 5100 2700 50  0001 C CNN
-	1    5100 2700
-	0    1    1    0
-$EndComp
-Wire Wire Line
-	4100 2700 4950 2700
-Text Label 5450 2700 0    50   ~ 0
+Text Label 4250 2700 0    50   ~ 0
 SDIO_CLK
-Wire Wire Line
-	5250 2700 5850 2700
 Connection ~ 4300 4400
 Wire Wire Line
@@
 	8300 9200 8300 9100
 $Comp
-L require:VCC_IO #PWR?
+L require:VCC_IO #PWR0229
 U 1 1 5CA12DDB
 P 8300 9100
-F 0 "#PWR?" H 8300 8950 50  0001 C CNN
+F 0 "#PWR0229" H 8300 8950 50  0001 C CNN
 F 1 "VCC_IO" H 8317 9273 50  0000 C CNN
 F 2 "" H 8300 9100 50  0001 C CNN
@@
 	1    0    0    -1
 $EndComp
+Wire Wire Line
+	4100 2700 5850 2700
 $EndSCHEMATC

Commit message: wip
Connections:
- wire segments 167 -> 175
- no-connect marks 15 -> 11
Changed lines of the file:
@@
 	1    0    0    -1
 $EndComp
-Text Notes 12000 6200 0    50   ~ 10
+Text Notes 13300 5850 0    50   ~ 10
 Use SDIO 2.0 (3V3)
 $Comp
@@
 Text Label 11200 6050 0    50   ~ 0
 LPO
-NoConn ~ 12250 5650
-NoConn ~ 12350 5650
-NoConn ~ 12450 5650
-NoConn ~ 12550 5650
 $Comp
 L Device:C C9
@@
 Wire Wire Line
 	4100 2700 5850 2700
+Wire Wire Line
+	12550 5650 12550 6400
+Wire Wire Line
+	12550 6400 13200 6400
+Wire Wire Line
+	12450 5650 12450 6550
+Wire Wire Line
+	12450 6550 13200 6550
+Wire Wire Line
+	12350 5650 12350 6700
+Wire Wire Line
+	12350 6700 13200 6700
+Wire Wire Line
+	12250 5650 12250 6850
+Wire Wire Line
+	12250 6850 13200 6850
+Text Label 12650 6400 0    50   ~ 0
+PCM_SYNC
+Text Label 12650 6550 0    50   ~ 0
+PCM_IN
+Text Label 12650 6700 0    50   ~ 0
+PCM_CLK
+Text Label 12650 6850 0    50   ~ 0
+PCM_OUT
 $EndSCHEMATC
