File: hardware/test.sch (KiCad schematic (older format))
At the start: 34 parts, among them P10 16, P11 17, P12 18, P23 11, P24 12, P25 13, P26 14, P7 15, U1 ap6255, U1000 RK3308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

Commit message: wip
Parts:
- removed C74, C76: 0.1u, Capacitors_SMD:C_0402, symbol Device:C
- removed LP10: TX2, require:OVAL_PIN, symbol require:OP
- removed LP9: RX2, require:OVAL_PIN, symbol require:OP
- removed P10: 16, require:OVAL_PIN, symbol require:OP
- removed P11: 17, require:OVAL_PIN, symbol require:OP
- removed P12: 18, require:OVAL_PIN, symbol require:OP
- removed P23: 11, require:OVAL_PIN, symbol require:OP
- removed P24: 12, require:OVAL_PIN, symbol require:OP
- removed P25: 13, require:OVAL_PIN, symbol require:OP
- removed P26: 14, require:OVAL_PIN, symbol require:OP
- removed P7: 15, require:OVAL_PIN, symbol require:OP
- removed U1000: RK3308, symbol require:RK3308
Connections:
- net labels removed: CORE_DVS, POWER_SLEEP, PWM1, PWM2, PWM3
- wire segments 175 -> 133
- no-connect marks 11 -> 4
Other:
- note removed: "SDIO 3.0, 1.8V\nVDDIO 1.8V"
- note removed: "Share cap with E14, D14, D13, C14"
