File: hardware/rk3308-acodec.sch (KiCad schematic (older format))
At the start: 1 part, among them U1000 RK3308

Commit message: wip
Parts:
- removed U1000: RK3308, require:RK3308_BGA355, symbol require:RK3308
Connections:
- net labels removed: GND
- wire segments 16 -> 0
- no-connect marks 24 -> 0
Changed lines of the file:
@@
 Comment4 ""
 $EndDescr
-$Comp
-L require:RK3308 U1000
-U 8 1 5C46A4FA
-P 2700 6600
-F 0 "U1000" H 3306 11787 60  0000 C CNN
-F 1 "RK3308" H 3306 11681 60  0000 C CNN
-F 2 "require:RK3308_BGA355" H 2700 6600 60  0001 C CNN
-F 3 "" H 2700 6600 60  0001 C CNN
-	8    2700 6600
-	1    0    0    -1
-$EndComp
-NoConn ~ 3900 2100
-NoConn ~ 3900 2200
-NoConn ~ 3900 2300
-NoConn ~ 3900 2400
-NoConn ~ 3900 2500
-NoConn ~ 3900 2600
-NoConn ~ 3900 2700
-NoConn ~ 3900 2800
-NoConn ~ 3900 2900
-NoConn ~ 3900 3000
-NoConn ~ 3900 3100
-NoConn ~ 3900 3200
-NoConn ~ 3900 3300
-NoConn ~ 3900 3400
-NoConn ~ 3900 3500
-NoConn ~ 3900 3600
-NoConn ~ 3900 3800
-NoConn ~ 3900 3900
-NoConn ~ 3900 4100
-NoConn ~ 3900 4200
-NoConn ~ 3900 4400
-NoConn ~ 3900 4500
-NoConn ~ 3900 4900
-NoConn ~ 3950 5000
-Wire Wire Line
-	3900 5700 4100 5700
-Wire Wire Line
-	4100 5700 4100 5800
-$Comp
-L power:GND #PWR0105
-U 1 1 5C46A5ED
-P 4100 6600
-F 0 "#PWR0105" H 4100 6350 50  0001 C CNN
-F 1 "GND" H 4105 6427 50  0000 C CNN
-F 2 "" H 4100 6600 50  0001 C CNN
-F 3 "" H 4100 6600 50  0001 C CNN
-	1    4100 6600
-	1    0    0    -1
-$EndComp
-Wire Wire Line
-	3900 5800 4100 5800
-Connection ~ 4100 5800
-Wire Wire Line
-	4100 5800 4100 5900
-Wire Wire Line
-	3900 5900 4100 5900
-Connection ~ 4100 5900
-Wire Wire Line
-	4100 5900 4100 6000
-Wire Wire Line
-	3900 6000 4100 6000
-Connection ~ 4100 6000
-Wire Wire Line
-	4100 6000 4100 6100
-Wire Wire Line
-	3900 6100 4100 6100
-Connection ~ 4100 6100
-Wire Wire Line
-	4100 6100 4100 6200
-Wire Wire Line
-	3900 6200 4100 6200
-Connection ~ 4100 6200
-Wire Wire Line
-	4100 6200 4100 6300
-Wire Wire Line
-	3900 6300 4100 6300
-Connection ~ 4100 6300
-Wire Wire Line
-	4100 6300 4100 6400
-Wire Wire Line
-	3900 6400 4100 6400
-Connection ~ 4100 6400
-Wire Wire Line
-	4100 6400 4100 6600
 $EndSCHEMATC
