File: hardware/emmc.sch (KiCad schematic (older format))
At the start: 3 parts, among them U1000 RK3308, U3 EMMC_BGA_153

Commit message: wip
Connections:
- net labels added: VCC_1V8
- net labels removed: VCCIO_FLASH
- wire segments 88 -> 96
- no-connect marks 4 -> 85

Commit message: wip
Parts:
- removed C1984: 0.1u, Capacitors_SMD:C_0402, symbol Device:C
- renumbered U3 to U4
Connections:
- net labels removed: VCC_1V8
- wire segments 96 -> 92
Other:
- note added: "EMMC\nInterface power → VDD(VCCQ) (1.70V - 1.95V or 2.7V - 3.6V) \nMemory power → VDDF(VCC) (2.7V - 3.6V)"
- note added: "Share cap with R11, T11"
- note added: "Use 3V3 for emmc io"
- moved on the sheet: U1000E
Changed lines of the file:
@@
 $Descr A4 11693 8268
 encoding utf-8
-Sheet 7 8
+Sheet 7 9
 Title ""
 Date ""
@@
 L require:RK3308 U1000
 U 5 1 5CDB90C0
-P 1050 3000
-F 0 "U1000" H 1836 5287 60  0000 C CNN
-F 1 "RK3308" H 1836 5181 60  0000 C CNN
-F 2 "" H 1050 3000 60  0001 C CNN
-F 3 "" H 1050 3000 60  0001 C CNN
-	5    1050 3000
-	1    0    0    -1
-$EndComp
-Wire Wire Line
-	3250 1200 4000 1200
-Wire Wire Line
-	3250 1300 4000 1300
-Wire Wire Line
-	3250 1400 4000 1400
-Wire Wire Line
-	3250 1500 4000 1500
-Wire Wire Line
-	3250 1600 4000 1600
-Wire Wire Line
-	3250 1700 4000 1700
-Wire Wire Line
-	3250 1800 4000 1800
-Wire Wire Line
-	3250 1900 4000 1900
-Wire Wire Line
-	3250 2000 4000 2000
-Text Label 3450 1200 0    50   ~ 0
+P 1450 4350
+F 0 "U1000" H 2236 6637 60  0000 C CNN
+F 1 "RK3308" H 2236 6531 60  0000 C CNN
+F 2 "" H 1450 4350 60  0001 C CNN
+F 3 "" H 1450 4350 60  0001 C CNN
+	5    1450 4350
+	1    0    0    -1
+$EndComp
+Wire Wire Line
+	3650 2550 4400 2550
+Wire Wire Line
+	3650 2650 4400 2650
+Wire Wire Line
+	3650 2750 4400 2750
+Wire Wire Line
+	3650 2850 4400 2850
+Wire Wire Line
+	3650 2950 4400 2950
+Wire Wire Line
+	3650 3050 4400 3050
+Wire Wire Line
+	3650 3150 4400 3150
+Wire Wire Line
+	3650 3250 4400 3250
+Wire Wire Line
+	3650 3350 4400 3350
+Text Label 3850 2550 0    50   ~ 0
 FLASH_D1
-Text Label 3450 1300 0    50   ~ 0
+Text Label 3850 2650 0    50   ~ 0
 FLASH_D2
-Text Label 3450 1400 0    50   ~ 0
+Text Label 3850 2750 0    50   ~ 0
 FLASH_D3
-Text Label 3450 1500 0    50   ~ 0
+Text Label 3850 2850 0    50   ~ 0
 FLASH_D4
-Text Label 3450 1600 0    50   ~ 0
+Text Label 3850 2950 0    50   ~ 0
 FLASH_D5
-Text Label 3450 1700 0    50   ~ 0
+Text Label 3850 3050 0    50   ~ 0
 FLASH_D6
-Text Label 3450 1800 0    50   ~ 0
+Text Label 3850 3150 0    50   ~ 0
 FLASH_D7
-Text Label 3450 1900 0    50   ~ 0
+Text Label 3850 3250 0    50   ~ 0
 FLASH_CMD
-Text Label 3450 2000 0    50   ~ 0
+Text Label 3850 3350 0    50   ~ 0
 FLASH_CLK
-Text Label 3450 1100 0    50   ~ 0
+Text Label 3850 2450 0    50   ~ 0
 FLASH_D0
 Wire Wire Line
-	3250 1100 4000 1100
+	3650 2450 4400 2450
 Text Label 6200 1650 0    50   ~ 0
 FLASH_D3
@@
 	8000 3250 8200 3250
 Wire Wire Line
-	8100 1250 8700 1250
-Text Label 8100 1250 0    50   ~ 0
+	8200 1250 8800 1250
+Text Label 8200 1250 0    50   ~ 0
 FLASH_D7
 Text Label 5950 3250 0    50   ~ 0
 FLASH_D6
 Wire Wire Line
-	3250 2200 4000 2200
-Text Label 3450 2200 0    50   ~ 0
+	3650 3550 4400 3550
+Text Label 3850 3550 0    50   ~ 0
 EMMC_RST
 $Comp
@@
 Connection ~ 7000 2050
 $Comp
-L require:EMMC_BGA_153 U3
+L require:EMMC_BGA_153 U4
 U 1 1 5CF1B07B
 P 8100 4850
-F 0 "U3" H 9628 6396 50  0000 L CNN
+F 0 "U4" H 9628 6396 50  0000 L CNN
 F 1 "EMMC_BGA_153" H 9628 6305 50  0000 L CNN
 F 2 "require:BGA-153_14x14_11.5x13.0mm" H 8100 4850 50  0001 C CNN
@@
 	5550 4050 5550 4150
 NoConn ~ 7600 3450
-NoConn ~ 3250 2100
-NoConn ~ 3250 2300
-NoConn ~ 3250 2400
-Wire Wire Line
-	3250 2800 3450 2800
-Wire Wire Line
-	3450 2800 3450 2650
-$Comp
-L Device:C C1984
-U 1 1 5D203A8A
-P 3450 3150
-F 0 "C1984" H 3565 3196 50  0000 L CNN
-F 1 "0.1u" H 3565 3105 50  0000 L CNN
-F 2 "Capacitors_SMD:C_0402" H 3488 3000 50  0001 C CNN
-F 3 "~" H 3450 3150 50  0001 C CNN
-	1    3450 3150
-	1    0    0    -1
-$EndComp
-Wire Wire Line
-	3450 3000 3450 2800
-Connection ~ 3450 2800
-Wire Wire Line
-	3450 3300 3450 3500
-$Comp
-L power:GND #PWR0125
-U 1 1 5D206B15
-P 3450 3500
-F 0 "#PWR0125" H 3450 3250 50  0001 C CNN
-F 1 "GND" H 3455 3327 50  0000 C CNN
-F 2 "" H 3450 3500 50  0001 C CNN
-F 3 "" H 3450 3500 50  0001 C CNN
-	1    3450 3500
-	1    0    0    -1
-$EndComp
+NoConn ~ 3650 3450
+NoConn ~ 3650 3650
+NoConn ~ 3650 3750
+Wire Wire Line
+	3650 4150 3850 4150
+Wire Wire Line
+	3850 4150 3850 4000
 Wire Wire Line
 	7000 2650 6800 2850
 Connection ~ 6800 2850
-$Comp
-L require:VCC_1V8 #PWR0124
-U 1 1 5CA04985
-P 3450 2650
-F 0 "#PWR0124" H 3450 2500 50  0001 C CNN
-F 1 "VCC_1V8" H 3467 2823 50  0000 C CNN
-F 2 "" H 3450 2650 50  0001 C CNN
-F 3 "" H 3450 2650 50  0001 C CNN
-	1    3450 2650
-	1    0    0    -1
-$EndComp
-$Comp
-L require:VCC_1V8 #PWR0136
-U 1 1 5CA0607E
-P 5550 4050
-F 0 "#PWR0136" H 5550 3900 50  0001 C CNN
-F 1 "VCC_1V8" H 5567 4223 50  0000 C CNN
-F 2 "" H 5550 4050 50  0001 C CNN
-F 3 "" H 5550 4050 50  0001 C CNN
-	1    5550 4050
-	1    0    0    -1
-$EndComp
 Wire Wire Line
 	7400 2450 7200 2650
@@
 	8000 2250 8200 2050
 Connection ~ 8000 2250
-Wire Wire Line
-	8200 2050 8200 1800
-Wire Wire Line
-	8200 1800 8100 1800
 Connection ~ 8200 2050
-Wire Wire Line
-	8100 1800 8100 1250
 NoConn ~ 8400 4650
 NoConn ~ 8200 4650
@@
 	7600 4450 7800 4650
 Connection ~ 7800 4650
-$Comp
-L require:VCC_1V8 #PWR0135
-U 1 1 5CB0E558
+Wire Wire Line
+	6400 3050 6800 3050
+Wire Wire Line
+	5950 2850 6800 2850
+Wire Wire Line
+	6800 3250 5950 3250
+Connection ~ 6800 3250
+Connection ~ 8400 3750
+Wire Wire Line
+	8400 3750 8400 3850
+Wire Wire Line
+	8400 3750 10300 3750
+Text Notes 5650 5800 0    50   ~ 10
+EMMC\nInterface power → VDD(VCCQ) (1.70V - 1.95V or 2.7V - 3.6V) \nMemory power → VDDF(VCC) (2.7V - 3.6V)
+Text Notes 4050 4000 0    50   ~ 0
+Use 3V3 for emmc io
+Wire Wire Line
+	8200 1250 8200 2050
+$Comp
+L require:VCC_IO #PWR0124
+U 1 1 5CF36E42
+P 3850 4000
+F 0 "#PWR0124" H 3850 3850 50  0001 C CNN
+F 1 "VCC_IO" H 3867 4173 50  0000 C CNN
+F 2 "" H 3850 4000 50  0001 C CNN
+F 3 "" H 3850 4000 50  0001 C CNN
+	1    3850 4000
+	1    0    0    -1
+$EndComp
+$Comp
+L require:VCC_IO #PWR0135
+U 1 1 5CF36E83
 P 9900 2450
 F 0 "#PWR0135" H 9900 2300 50  0001 C CNN
-F 1 "VCC_1V8" H 9917 2623 50  0000 C CNN
+F 1 "VCC_IO" H 9917 2623 50  0000 C CNN
 F 2 "" H 9900 2450 50  0001 C CNN
 F 3 "" H 9900 2450 50  0001 C CNN
@@
 	1    0    0    -1
 $EndComp
-Wire Wire Line
-	6400 3050 6800 3050
-Wire Wire Line
-	5950 2850 6800 2850
-Wire Wire Line
-	6800 3250 5950 3250
-Connection ~ 6800 3250
-Connection ~ 8400 3750
-Wire Wire Line
-	8400 3750 8400 3850
-Wire Wire Line
-	8400 3750 10300 3750
+$Comp
+L require:VCC_IO #PWR0136
+U 1 1 5CF36EC4
+P 5550 4050
+F 0 "#PWR0136" H 5550 3900 50  0001 C CNN
+F 1 "VCC_IO" H 5567 4223 50  0000 C CNN
+F 2 "" H 5550 4050 50  0001 C CNN
+F 3 "" H 5550 4050 50  0001 C CNN
+	1    5550 4050
+	1    0    0    -1
+$EndComp
+Text Notes 3750 4350 0    50   ~ 10
+Share cap with R11, T11
 $EndSCHEMATC

Commit message: wip
Parts:
- added P13: 1, require:OVAL_PIN, symbol require:OP
- added P14: 2, require:OVAL_PIN, symbol require:OP
Connections:
- wire segments 92 -> 94
- no-connect marks 85 -> 83
Changed lines of the file:
@@
 $Descr A4 11693 8268
 encoding utf-8
-Sheet 7 9
+Sheet 7 10
 Title ""
 Date ""
@@
 	5550 4050 5550 4150
 NoConn ~ 7600 3450
-NoConn ~ 3650 3450
-NoConn ~ 3650 3650
-NoConn ~ 3650 3750
 Wire Wire Line
 	3650 4150 3850 4150
@@
 Text Notes 3750 4350 0    50   ~ 10
 Share cap with R11, T11
+Wire Wire Line
+	3650 3650 4400 3650
+Wire Wire Line
+	3650 3750 4400 3750
+$Comp
+L require:OP P13
+U 1 1 5C5EA528
+P 4600 3650
+F 0 "P13" H 4800 3650 50  0000 C CNN
+F 1 "1" H 4600 3650 50  0000 C CNN
+F 2 "require:OVAL_PIN" H 4600 3600 50  0001 C CNN
+F 3 "" H 4600 3600 50  0001 C CNN
+	1    4600 3650
+	1    0    0    -1
+$EndComp
+$Comp
+L require:OP P14
+U 1 1 5C5EA552
+P 4600 3750
+F 0 "P14" H 4800 3750 50  0000 C CNN
+F 1 "2" H 4600 3750 50  0000 C CNN
+F 2 "require:OVAL_PIN" H 4600 3700 50  0001 C CNN
+F 3 "" H 4600 3700 50  0001 C CNN
+	1    4600 3750
+	1    0    0    -1
+$EndComp
+NoConn ~ 3650 3450
 $EndSCHEMATC

Commit message: wip
Parts:
- added C101: C, Capacitors_SMD:C_0402, symbol Device:C
Connections:
- wire segments 94 -> 100
- no-connect marks 83 -> 81
Changed lines of the file:
@@
 	6200 1650 6800 1650
 Connection ~ 6800 2050
-NoConn ~ 6800 2450
-NoConn ~ 7000 2450
 NoConn ~ 6800 2650
 Wire Wire Line
@@
 $EndComp
 NoConn ~ 3650 3450
+Wire Wire Line
+	7000 2450 6800 2450
+Wire Wire Line
+	6800 2450 6250 2450
+Wire Wire Line
+	6250 2450 6250 1900
+Wire Wire Line
+	6250 1900 5550 1900
+Wire Wire Line
+	5550 1900 5550 2100
+Connection ~ 6800 2450
+$Comp
+L Device:C C101
+U 1 1 5C4D63A0
+P 5550 2250
+F 0 "C101" H 5665 2296 50  0000 L CNN
+F 1 "C" H 5665 2205 50  0000 L CNN
+F 2 "Capacitors_SMD:C_0402" H 5588 2100 50  0001 C CNN
+F 3 "~" H 5550 2250 50  0001 C CNN
+	1    5550 2250
+	1    0    0    -1
+$EndComp
+Wire Wire Line
+	5550 2400 5550 2500
+$Comp
+L power:GND #PWR0230
+U 1 1 5C4D81E0
+P 5550 2500
+F 0 "#PWR0230" H 5550 2250 50  0001 C CNN
+F 1 "GND" H 5555 2327 50  0000 C CNN
+F 2 "" H 5550 2500 50  0001 C CNN
+F 3 "" H 5550 2500 50  0001 C CNN
+	1    5550 2500
+	1    0    0    -1
+$EndComp
 $EndSCHEMATC

Commit message: wip
Connections:
- wire segments 100 -> 101
- no-connect marks 81 -> 80
Changed lines of the file:
@@
 Wire Wire Line
 	6200 1550 7000 1550
-NoConn ~ 6800 2250
 Wire Wire Line
 	7000 2250 6800 2050
@@
 	1    0    0    -1
 $EndComp
+Wire Wire Line
+	7000 2250 6800 2250
+Connection ~ 7000 2250
 $EndSCHEMATC

Commit message: wip
Parts:
- removed P13: 1, require:OVAL_PIN, symbol require:OP
- removed P14: 2, require:OVAL_PIN, symbol require:OP
- removed U1000: RK3308, symbol require:RK3308
Connections:
- net labels added: EMMC_CLK, EMMC_CMD, EMMC_D0, EMMC_D1, EMMC_D2, EMMC_D3, EMMC_D4, EMMC_D5, EMMC_D6, EMMC_D7, VDDi
- wire segments 101 -> 85
- no-connect marks 80 -> 79
Other:
- note removed: "Share cap with R11, T11"
- note removed: "Use 3V3 for emmc io"
- moved on the sheet: C101, U4
