File: hardware/emmc.sch (KiCad schematic (older format))
At the start: 2 parts, among them U4 EMMC_BGA_153

Commit message: wip
Connections:
- net labels removed: FLASH_CLK, FLASH_CMD, FLASH_D0, FLASH_D1, FLASH_D2, FLASH_D3, FLASH_D4, FLASH_D5, FLASH_D6, FLASH_D7
Changed lines of the file:
@@
 Comment4 ""
 $EndDescr
-Text Label 1900 1800 0    50   ~ 0
-FLASH_D3
-Text Label 2200 3000 0    50   ~ 0
-FLASH_D5
 Wire Wire Line
 	3450 2400 3250 2200
-Text Label 1900 1700 0    50   ~ 0
-FLASH_D4
 Wire Wire Line
 	3450 2200 3450 1600
-Text Label 1900 1600 0    50   ~ 0
-FLASH_D0
 Wire Wire Line
 	3650 2200 3650 1500
-Text Label 1900 1500 0    50   ~ 0
-FLASH_D1
 Wire Wire Line
 	3850 2200 3850 1400
-Text Label 1900 1400 0    50   ~ 0
-FLASH_D2
 Wire Wire Line
 	4050 2200 4050 1800
@@
 Wire Wire Line
 	4250 3400 4450 3400
-Text Label 1900 1300 0    50   ~ 0
-FLASH_D7
-Text Label 2200 3400 0    50   ~ 0
-FLASH_D6
 $Comp
 L require:VCC_IO #PWR0133
@@
 Wire Wire Line
 	3450 3800 3250 3800
-Text Label 2200 3800 0    50   ~ 0
-EMMC_RST
 Wire Wire Line
 	4050 4400 3650 4000
@@
 Wire Wire Line
 	3450 4200 3250 4200
-Text Label 2200 4000 0    50   ~ 0
-FLASH_CLK
-Text Label 2200 4200 0    50   ~ 0
-FLASH_CMD
 Wire Wire Line
 	3250 1700 3250 2200

Commit message: wip
Parts:
- added C505, C600, C700, C800: C, require:C_0603, symbol Device:C
- added C506, C507, C601, C701, C801, C802: C, require:C_0402, symbol Device:C
- C101: footprint Capacitors_SMD:C_0402 -> require:C_0402
Connections:
- wire segments 85 -> 125

Commit message: wip
Parts:
- added R9675: 22R, require:R_0402, symbol Device:R
- added TP1, TP2: TestPoint, require:TPTH0603, symbol Connector:TestPoint
Connections:
- net labels added: EMMC_CLK1
- wire segments 125 -> 128
Changed lines of the file:
@@
 Wire Wire Line
 	3650 4000 3450 4000
-Connection ~ 3050 4000
 Connection ~ 3250 4000
 Wire Wire Line
@@
 Wire Wire Line
 	1800 5000 1800 5100
-Wire Wire Line
-	1800 4000 3050 4000
 Text HLabel 1800 4000 0    50   Input ~ 0
 EMMC_CLK
@@
 	1    0    0    -1
 $EndComp
+$Comp
+L Connector:TestPoint TP1
+U 1 1 5C5BDCB5
+P 3450 900
+F 0 "TP1" H 3508 1020 50  0000 L CNN
+F 1 "TestPoint" H 3508 929 50  0000 L CNN
+F 2 "require:TPTH0603" H 3650 900 50  0001 C CNN
+F 3 "~" H 3650 900 50  0001 C CNN
+	1    3450 900
+	1    0    0    -1
+$EndComp
+Wire Wire Line
+	3450 1600 3450 900
+Connection ~ 3450 1600
+$Comp
+L Connector:TestPoint TP2
+U 1 1 5C5C292E
+P 3950 900
+F 0 "TP2" H 4008 1020 50  0000 L CNN
+F 1 "TestPoint" H 4008 929 50  0000 L CNN
+F 2 "require:TPTH0603" H 4150 900 50  0001 C CNN
+F 3 "~" H 4150 900 50  0001 C CNN
+	1    3950 900
+	1    0    0    -1
+$EndComp
+$Comp
+L power:GND #PWR0242
+U 1 1 5C5C29C3
+P 3950 1000
+F 0 "#PWR0242" H 3950 750 50  0001 C CNN
+F 1 "GND" H 3955 827 50  0000 C CNN
+F 2 "" H 3950 1000 50  0001 C CNN
+F 3 "" H 3950 1000 50  0001 C CNN
+	1    3950 1000
+	1    0    0    -1
+$EndComp
+Wire Wire Line
+	3950 1000 3950 900
+$Comp
+L Device:R R9675
+U 1 1 5C5CEDA4
+P 2150 4000
+F 0 "R9675" V 2050 4000 50  0000 C CNN
+F 1 "22R" V 2250 4000 50  0000 C CNN
+F 2 "require:R_0402" V 2080 4000 50  0001 C CNN
+F 3 "~" H 2150 4000 50  0001 C CNN
+	1    2150 4000
+	0    1    1    0
+$EndComp
+Wire Wire Line
+	1800 4000 2000 4000
+Wire Wire Line
+	2300 4000 3050 4000
+Connection ~ 3050 4000
+Text Label 2350 4000 0    50   ~ 0
+EMMC_CLK1
 $EndSCHEMATC

Commit message: wip
Parts:
- removed C600, C700: C, require:C_0603, symbol Device:C
- removed C601, C701: C, require:C_0402, symbol Device:C
Connections:
- wire segments 128 -> 112
Changed lines of the file:
@@
 	5150 5400 5150 5500
-$Comp
-L Device:C C600
-U 1 1 5C5FDEC0
-P 6350 5750
-F 0 "C600" H 6465 5796 50  0000 L CNN
-F 1 "C" H 6465 5705 50  0000 L CNN
-F 2 "require:C_0603" H 6388 5600 50  0001 C CNN
-F 3 "~" H 6350 5750 50  0001 C CNN
-	1    6350 5750
-	1    0    0    -1
-$EndComp
-$Comp
-L Device:C C601
-U 1 1 5C5FDF2A
-P 6750 5750
-F 0 "C601" H 6865 5796 50  0000 L CNN
-F 1 "C" H 6865 5705 50  0000 L CNN
-F 2 "require:C_0402" H 6788 5600 50  0001 C CNN
-F 3 "~" H 6750 5750 50  0001 C CNN
-	1    6750 5750
-	1    0    0    -1
-$EndComp
-$Comp
-L Device:C C700
-U 1 1 5C5FDF80
-P 7350 5750
-F 0 "C700" H 7465 5796 50  0000 L CNN
-F 1 "C" H 7465 5705 50  0000 L CNN
-F 2 "require:C_0603" H 7388 5600 50  0001 C CNN
-F 3 "~" H 7350 5750 50  0001 C CNN
-	1    7350 5750
-	1    0    0    -1
-$EndComp
-$Comp
-L Device:C C701
-U 1 1 5C5FDFE0
-P 7750 5750
-F 0 "C701" H 7865 5796 50  0000 L CNN
-F 1 "C" H 7865 5705 50  0000 L CNN
-F 2 "require:C_0402" H 7788 5600 50  0001 C CNN
-F 3 "~" H 7750 5750 50  0001 C CNN
-	1    7750 5750
-	1    0    0    -1
-$EndComp
-Wire Wire Line
-	7750 5600 7750 5500
-Wire Wire Line
-	7750 5500 7350 5500
-Wire Wire Line
-	7350 5500 7350 5600
-Wire Wire Line
-	7350 5900 7350 6000
-Wire Wire Line
-	7350 6000 7750 6000
-Wire Wire Line
-	7750 6000 7750 5900
-Wire Wire Line
-	6350 5600 6350 5500
-Wire Wire Line
-	6350 5500 6750 5500
-Wire Wire Line
-	6750 5500 6750 5600
-Wire Wire Line
-	6350 5900 6350 6000
-Wire Wire Line
-	6350 6000 6750 6000
-Wire Wire Line
-	6750 6000 6750 5900
-$Comp
-L require:VCC_IO #PWR0236
-U 1 1 5C60DA61
-P 6350 5400
-F 0 "#PWR0236" H 6350 5250 50  0001 C CNN
-F 1 "VCC_IO" H 6367 5573 50  0000 C CNN
-F 2 "" H 6350 5400 50  0001 C CNN
-F 3 "" H 6350 5400 50  0001 C CNN
-	1    6350 5400
-	1    0    0    -1
-$EndComp
-$Comp
-L require:VCC_IO #PWR0237
-U 1 1 5C60DA9E
-P 7350 5400
-F 0 "#PWR0237" H 7350 5250 50  0001 C CNN
-F 1 "VCC_IO" H 7367 5573 50  0000 C CNN
-F 2 "" H 7350 5400 50  0001 C CNN
-F 3 "" H 7350 5400 50  0001 C CNN
-	1    7350 5400
-	1    0    0    -1
-$EndComp
-$Comp
-L power:GND #PWR0238
-U 1 1 5C60DB21
-P 6350 6100
-F 0 "#PWR0238" H 6350 5850 50  0001 C CNN
-F 1 "GND" H 6355 5927 50  0000 C CNN
-F 2 "" H 6350 6100 50  0001 C CNN
-F 3 "" H 6350 6100 50  0001 C CNN
-	1    6350 6100
-	1    0    0    -1
-$EndComp
-$Comp
-L power:GND #PWR0239
-U 1 1 5C60DB5E
-P 7350 6100
-F 0 "#PWR0239" H 7350 5850 50  0001 C CNN
-F 1 "GND" H 7355 5927 50  0000 C CNN
-F 2 "" H 7350 6100 50  0001 C CNN
-F 3 "" H 7350 6100 50  0001 C CNN
-	1    7350 6100
-	1    0    0    -1
-$EndComp
-Wire Wire Line
-	7350 5400 7350 5500
-Connection ~ 7350 5500
-Wire Wire Line
-	6350 5400 6350 5500
-Connection ~ 6350 5500
-Wire Wire Line
-	6350 6100 6350 6000
-Connection ~ 6350 6000
-Wire Wire Line
-	7350 6100 7350 6000
-Connection ~ 7350 6000
 $Comp
 L Device:C C800

Commit message: wip
Parts:
- TP1, TP2: footprint require:TPTH0603 -> require:TPTH0503
- renumbered C505 to C10, C506 to C11, C507 to C12, C101 to C5, C800 to C6, C801 to C7, C802 to C8, R9675 to R60, U4 to U994
Connections:
- net labels added: +3V3
- net labels removed: VCC_IO
Changed lines of the file:
@@
 Wire Wire Line
 	4250 3400 4450 3400
-$Comp
-L require:VCC_IO #PWR0133
-U 1 1 5D136F94
-P 6050 3800
-F 0 "#PWR0133" H 6050 3650 50  0001 C CNN
-F 1 "VCC_IO" H 6067 3973 50  0000 C CNN
-F 2 "" H 6050 3800 50  0001 C CNN
-F 3 "" H 6050 3800 50  0001 C CNN
-	1    6050 3800
-	1    0    0    -1
-$EndComp
 Connection ~ 3250 2800
 Wire Wire Line
@@
 Connection ~ 3250 2200
 $Comp
-L require:EMMC_BGA_153 U4
+L require:EMMC_BGA_153 U994
 U 1 1 5CF1B07B
 P 4350 5000
-F 0 "U4" H 5700 8400 50  0000 L CNN
+F 0 "U994" H 5700 8400 50  0000 L CNN
 F 1 "EMMC_BGA_153" H 5700 8300 50  0000 L CNN
 F 2 "require:BGA-153_14x14_11.5x13.0mm" H 4350 5000 50  0001 C CNN
@@
 Text Notes 1900 5950 0    50   ~ 10
 EMMC\nInterface power → VDD(VCCQ) (1.70V - 1.95V or 2.7V - 3.6V) \nMemory power → VDDF(VCC) (2.7V - 3.6V)
-$Comp
-L require:VCC_IO #PWR0135
-U 1 1 5CF36E83
-P 6050 2600
-F 0 "#PWR0135" H 6050 2450 50  0001 C CNN
-F 1 "VCC_IO" H 6067 2773 50  0000 C CNN
-F 2 "" H 6050 2600 50  0001 C CNN
-F 3 "" H 6050 2600 50  0001 C CNN
-	1    6050 2600
-	1    0    0    -1
-$EndComp
-$Comp
-L require:VCC_IO #PWR0136
-U 1 1 5CF36EC4
-P 1800 5000
-F 0 "#PWR0136" H 1800 4850 50  0001 C CNN
-F 1 "VCC_IO" H 1817 5173 50  0000 C CNN
-F 2 "" H 1800 5000 50  0001 C CNN
-F 3 "" H 1800 5000 50  0001 C CNN
-	1    1800 5000
-	1    0    0    -1
-$EndComp
 Wire Wire Line
 	3250 2600 3050 2600
@@
 Connection ~ 3050 2600
 $Comp
-L Device:C C101
+L Device:C C5
 U 1 1 5C4D63A0
 P 1800 2400
-F 0 "C101" H 1915 2446 50  0000 L CNN
+F 0 "C5" H 1915 2446 50  0000 L CNN
 F 1 "C" H 1915 2355 50  0000 L CNN
 F 2 "require:C_0402" H 1838 2250 50  0001 C CNN
@@
 	4450 1300 4450 2200
 Wire Wire Line
-	4050 3000 4050 2700
-Connection ~ 4050 3000
-Connection ~ 4050 2700
-Wire Wire Line
 	1800 3000 3050 3000
 Wire Wire Line
@@
 Connection ~ 3050 2400
 $Comp
-L Device:C C505
+L Device:C C10
 U 1 1 5C5EFDE2
 P 4750 5750
-F 0 "C505" H 4865 5796 50  0000 L CNN
+F 0 "C10" H 4865 5796 50  0000 L CNN
 F 1 "C" H 4865 5705 50  0000 L CNN
-F 2 "require:C_0603" H 4788 5600 50  0001 C CNN
+F 2 "require:C_0603" H 4788 5600 50  0000 C CNN
 F 3 "~" H 4750 5750 50  0001 C CNN
 	1    4750 5750
@@
 $EndComp
 $Comp
-L Device:C C506
+L Device:C C11
 U 1 1 5C5EFE7D
 P 5150 5750
-F 0 "C506" H 5265 5796 50  0000 L CNN
+F 0 "C11" H 5265 5796 50  0000 L CNN
 F 1 "C" H 5265 5705 50  0000 L CNN
 F 2 "require:C_0402" H 5188 5600 50  0001 C CNN
@@
 $EndComp
 $Comp
-L Device:C C507
+L Device:C C12
 U 1 1 5C5EFEA5
 P 5550 5750
-F 0 "C507" H 5665 5796 50  0000 L CNN
+F 0 "C12" H 5665 5796 50  0000 L CNN
 F 1 "C" H 5665 5705 50  0000 L CNN
 F 2 "require:C_0402" H 5588 5600 50  0001 C CNN
@@
 Wire Wire Line
 	5150 6000 5150 6100
-$Comp
-L require:VCC_IO #PWR0229
-U 1 1 5C5F8213
-P 5150 5400
-F 0 "#PWR0229" H 5150 5250 50  0001 C CNN
-F 1 "VCC_IO" H 5167 5573 50  0000 C CNN
-F 2 "" H 5150 5400 50  0001 C CNN
-F 3 "" H 5150 5400 50  0001 C CNN
-	1    5150 5400
-	1    0    0    -1
-$EndComp
 Wire Wire Line
 	5150 5400 5150 5500
 $Comp
-L Device:C C800
+L Device:C C6
 U 1 1 5C618955
 P 7950 4850
-F 0 "C800" H 8065 4896 50  0000 L CNN
+F 0 "C6" H 8065 4896 50  0000 L CNN
 F 1 "C" H 8065 4805 50  0000 L CNN
-F 2 "require:C_0603" H 7988 4700 50  0001 C CNN
+F 2 "require:C_0603" H 7988 4700 50  0000 C CNN
 F 3 "~" H 7950 4850 50  0001 C CNN
 	1    7950 4850
@@
 $EndComp
 $Comp
-L Device:C C801
+L Device:C C7
 U 1 1 5C6189A1
 P 8350 4850
-F 0 "C801" H 8465 4896 50  0000 L CNN
+F 0 "C7" H 8465 4896 50  0000 L CNN
 F 1 "C" H 8465 4805 50  0000 L CNN
 F 2 "require:C_0402" H 8388 4700 50  0001 C CNN
@@
 	1    0    0    -1
 $EndComp
-$Comp
-L require:VCC_IO #PWR0241
-U 1 1 5C62D6F0
-P 8350 4500
-F 0 "#PWR0241" H 8350 4350 50  0001 C CNN
-F 1 "VCC_IO" H 8367 4673 50  0000 C CNN
-F 2 "" H 8350 4500 50  0001 C CNN
-F 3 "" H 8350 4500 50  0001 C CNN
-	1    8350 4500
-	1    0    0    -1
-$EndComp
 Wire Wire Line
 	8350 4500 8350 4600
 $Comp
-L Device:C C802
+L Device:C C8
 U 1 1 5C6189D7
 P 8750 4850
-F 0 "C802" H 8865 4896 50  0000 L CNN
+F 0 "C8" H 8865 4896 50  0000 L CNN
 F 1 "C" H 8865 4805 50  0000 L CNN
 F 2 "require:C_0402" H 8788 4700 50  0001 C CNN
@@
 F 0 "TP1" H 3508 1020 50  0000 L CNN
 F 1 "TestPoint" H 3508 929 50  0000 L CNN
-F 2 "require:TPTH0603" H 3650 900 50  0001 C CNN
+F 2 "require:TPTH0503" H 3650 900 50  0001 C CNN
 F 3 "~" H 3650 900 50  0001 C CNN
 	1    3450 900
@@
 F 0 "TP2" H 4008 1020 50  0000 L CNN
 F 1 "TestPoint" H 4008 929 50  0000 L CNN
-F 2 "require:TPTH0603" H 4150 900 50  0001 C CNN
+F 2 "require:TPTH0503" H 4150 900 50  0001 C CNN
 F 3 "~" H 4150 900 50  0001 C CNN
 	1    3950 900
@@
 	3950 1000 3950 900
 $Comp
-L Device:R R9675
+L Device:R R60
 U 1 1 5C5CEDA4
 P 2150 4000
-F 0 "R9675" V 2050 4000 50  0000 C CNN
+F 0 "R60" V 2050 4000 50  0000 C CNN
 F 1 "22R" V 2250 4000 50  0000 C CNN
 F 2 "require:R_0402" V 2080 4000 50  0001 C CNN
@@
 Text Label 2350 4000 0    50   ~ 0
 EMMC_CLK1
+Connection ~ 4050 2700
+Connection ~ 4050 3000
+Wire Wire Line
+	4050 3000 4050 2700
+$Comp
+L power:+3V3 #PWR0224
+U 1 1 5C7E8A09
+P 6050 2600
+F 0 "#PWR0224" H 6050 2450 50  0001 C CNN
+F 1 "+3V3" H 6065 2773 50  0000 C CNN
+F 2 "" H 6050 2600 50  0001 C CNN
+F 3 "" H 6050 2600 50  0001 C CNN
+	1    6050 2600
+	1    0    0    -1
+$EndComp
+$Comp
+L power:+3V3 #PWR0226
+U 1 1 5C7E8A3D
+P 6050 3800
+F 0 "#PWR0226" H 6050 3650 50  0001 C CNN
+F 1 "+3V3" H 6065 3973 50  0000 C CNN
+F 2 "" H 6050 3800 50  0001 C CNN
+F 3 "" H 6050 3800 50  0001 C CNN
+	1    6050 3800
+	1    0    0    -1
+$EndComp
+$Comp
+L power:+3V3 #PWR0229
+U 1 1 5C7E8AA1
+P 8350 4500
+F 0 "#PWR0229" H 8350 4350 50  0001 C CNN
+F 1 "+3V3" H 8365 4673 50  0000 C CNN
+F 2 "" H 8350 4500 50  0001 C CNN
+F 3 "" H 8350 4500 50  0001 C CNN
+	1    8350 4500
+	1    0    0    -1
+$EndComp
+$Comp
+L power:+3V3 #PWR0239
+U 1 1 5C7E8B05
+P 5150 5400
+F 0 "#PWR0239" H 5150 5250 50  0001 C CNN
+F 1 "+3V3" H 5165 5573 50  0000 C CNN
+F 2 "" H 5150 5400 50  0001 C CNN
+F 3 "" H 5150 5400 50  0001 C CNN
+	1    5150 5400
+	1    0    0    -1
+$EndComp
+$Comp
+L power:+3V3 #PWR0241
+U 1 1 5C7E8BA0
+P 1800 5000
+F 0 "#PWR0241" H 1800 4850 50  0001 C CNN
+F 1 "+3V3" H 1815 5173 50  0000 C CNN
+F 2 "" H 1800 5000 50  0001 C CNN
+F 3 "" H 1800 5000 50  0001 C CNN
+	1    1800 5000
+	1    0    0    -1
+$EndComp
 $EndSCHEMATC

Commit message: wip
Parts:
- removed TP1, TP2: TestPoint, require:TPTH0503, symbol Connector:TestPoint
Changed lines of the file:
@@
 $EndComp
-$Comp
-L Connector:TestPoint TP1
-U 1 1 5C5BDCB5
-P 3450 900
-F 0 "TP1" H 3508 1020 50  0000 L CNN
-F 1 "TestPoint" H 3508 929 50  0000 L CNN
-F 2 "require:TPTH0503" H 3650 900 50  0001 C CNN
-F 3 "~" H 3650 900 50  0001 C CNN
-	1    3450 900
-	1    0    0    -1
-$EndComp
-Wire Wire Line
-	3450 1600 3450 900
-Connection ~ 3450 1600
-$Comp
-L Connector:TestPoint TP2
-U 1 1 5C5C292E
-P 3950 900
-F 0 "TP2" H 4008 1020 50  0000 L CNN
-F 1 "TestPoint" H 4008 929 50  0000 L CNN
-F 2 "require:TPTH0503" H 4150 900 50  0001 C CNN
-F 3 "~" H 4150 900 50  0001 C CNN
-	1    3950 900
-	1    0    0    -1
-$EndComp
-$Comp
-L power:GND #PWR0242
-U 1 1 5C5C29C3
-P 3950 1000
-F 0 "#PWR0242" H 3950 750 50  0001 C CNN
-F 1 "GND" H 3955 827 50  0000 C CNN
-F 2 "" H 3950 1000 50  0001 C CNN
-F 3 "" H 3950 1000 50  0001 C CNN
-	1    3950 1000
-	1    0    0    -1
-$EndComp
-Wire Wire Line
-	3950 1000 3950 900
 $Comp
 L Device:R R60

Commit message: wip
Parts:
- added C405: 1u, require:C_0402, symbol Device:C
- added D400: D_Schottky, Diodes_SMD:D_SOD-523, symbol Device:D_Schottky
- added R410: 2.2k, require:R_0402, symbol Device:R
- C400: renamed from C10; value C -> 10u
- C401: renamed from C11; value C -> 0.1u
- C402: renamed from C12; value C -> 0.1u
- C406: renamed from C8; value C -> 0.1u
- C410: renamed from C6; value C -> 10u
- C411: renamed from C7; value C -> 0.1u
- renumbered C5 to C420, R60 to R400, U994 to U400
Connections:
- net +3V3: now also C405.1
- net EMMC_D0: now also D400.2 (A)
- net GND: now also C405.2, R410.2
- new net EMMC_D0_SHORT: D400.1 (K)
- new net EMMC_VSEL: R410.1
Other:
- moved on the sheet: C400, C401, C402, C406, C410, C411

Commit message: wip
Parts:
- D400: footprint Diodes_SMD:D_SOD-523 -> require:D_SOD-523
Changed lines of the file:
@@
 F 0 "D400" H 7250 5584 50  0000 C CNN
 F 1 "D_Schottky" H 7250 5675 50  0000 C CNN
-F 2 "Diodes_SMD:D_SOD-523" H 7250 5800 50  0001 C CNN
+F 2 "require:D_SOD-523" H 7250 5800 50  0001 C CNN
 F 3 "~" H 7250 5800 50  0001 C CNN
 	1    7250 5800
