File: hardware/emmc.sch (KiCad schematic (older format))
At the start: 12 parts, among them U400 EMMC_BGA_153

Commit message: wip
Parts:
- C405: value 1u -> 2.2u
- C420: value C -> 1u
Other:
- moved on the sheet: C400, C401, C402, C405, C406, C410, C411, C420, D400, R400, R410, U400

Commit message: wip
Parts:
- removed D400: D_Schottky, require:D_SOD-523, symbol Device:D_Schottky
- removed R410: 2.2k, require:R_0402, symbol Device:R
Changed lines of the file:
@@
 Wire Wire Line
 	7600 3700 7600 3800
-Text HLabel 8450 4650 2    50   Input ~ 0
-EMMC_VSEL
-$Comp
-L Device:D_Schottky D?
-U 1 1 5C89A16B
-P 8100 5200
-AR Path="/5C89A16B" Ref="D?"  Part="1"
-AR Path="/5CDAE2B6/5C89A16B" Ref="D400"  Part="1"
-F 0 "D400" H 8100 4984 50  0000 C CNN
-F 1 "D_Schottky" H 8100 5075 50  0000 C CNN
-F 2 "require:D_SOD-523" H 8100 5200 50  0001 C CNN
-F 3 "~" H 8100 5200 50  0001 C CNN
-	1    8100 5200
-	-1   0    0    1
-$EndComp
-Wire Wire Line
-	7950 5200 7600 5200
-Text Label 7600 5200 0    50   ~ 0
-EMMC_D0
-Text HLabel 8450 5200 2    50   Input ~ 0
-EMMC_D0_SHORT
-Wire Wire Line
-	8250 5200 8450 5200
-$Comp
-L Device:R R410
-U 1 1 5C8A763A
-P 8100 4650
-F 0 "R410" V 8000 4650 50  0000 C CNN
-F 1 "2.2k" V 8200 4650 50  0000 C CNN
-F 2 "require:R_0402" V 8030 4650 50  0001 C CNN
-F 3 "~" H 8100 4650 50  0001 C CNN
-	1    8100 4650
-	0    1    1    0
-$EndComp
-$Comp
-L power:GND #PWR0180
-U 1 1 5C8A77BF
-P 7850 4650
-F 0 "#PWR0180" H 7850 4400 50  0001 C CNN
-F 1 "GND" V 7855 4522 50  0000 R CNN
-F 2 "" H 7850 4650 50  0001 C CNN
-F 3 "" H 7850 4650 50  0001 C CNN
-	1    7850 4650
-	0    1    1    0
-$EndComp
-Wire Wire Line
-	7850 4650 7950 4650
-Wire Wire Line
-	8450 4650 8250 4650
 Wire Wire Line
 	4900 2400 4900 2250
@@
 	7150 2500 7150 2600
 $Comp
-L power:GND #PWR?
+L power:GND #PWR0169
 U 1 1 5C852246
 P 7600 2600
-F 0 "#PWR?" H 7600 2350 50  0001 C CNN
+F 0 "#PWR0169" H 7600 2350 50  0001 C CNN
 F 1 "GND" H 7605 2427 50  0000 C CNN
 F 2 "" H 7600 2600 50  0001 C CNN
@@
 $EndComp
 $Comp
-L power:GND #PWR?
+L power:GND #PWR0171
 U 1 1 5C854B2B
 P 7600 3800
-F 0 "#PWR?" H 7600 3550 50  0001 C CNN
+F 0 "#PWR0171" H 7600 3550 50  0001 C CNN
 F 1 "GND" H 7605 3627 50  0000 C CNN
 F 2 "" H 7600 3800 50  0001 C CNN
@@
 	3900 5400 3900 5500
 $Comp
-L power:GND #PWR?
+L power:GND #PWR0177
 U 1 1 5C85BC25
 P 3200 5500
-F 0 "#PWR?" H 3200 5250 50  0001 C CNN
+F 0 "#PWR0177" H 3200 5250 50  0001 C CNN
 F 1 "GND" H 3205 5327 50  0000 C CNN
 F 2 "" H 3200 5500 50  0001 C CNN
@@
 $EndComp
 $Comp
-L power:GND #PWR?
+L power:GND #PWR0220
 U 1 1 5C85BC48
 P 4300 5500
-F 0 "#PWR?" H 4300 5250 50  0001 C CNN
+F 0 "#PWR0220" H 4300 5250 50  0001 C CNN
 F 1 "GND" H 4305 5327 50  0000 C CNN
 F 2 "" H 4300 5500 50  0001 C CNN

Commit message: wip
Connections:
- net EMMC_CLK: now also U400.K1, U400.K2, U400.K3, U400.M6 (CLK); no longer R400.2
- net EMMC_D7: now also U400.C7; no longer U400.A8, U400.B7
- removed net EMMC_CLK1: R400.1, U400.K1, U400.K2, U400.K3, U400.M6 (CLK)
- no-connect marks 79 -> 80
Other:
- moved on the sheet: R400
Changed lines of the file:
@@
 	4100 2600 3900 2800
 Connection ~ 4100 2600
-Wire Wire Line
-	4900 1800 5100 1800
-Wire Wire Line
-	5100 1800 5300 1600
-Connection ~ 5100 1800
-Connection ~ 5300 1600
 NoConn ~ 5500 4200
 NoConn ~ 5300 4200
@@
 NoConn ~ 5900 2000
 NoConn ~ 5500 2000
-NoConn ~ 5300 2000
-NoConn ~ 5100 2000
 NoConn ~ 5700 2000
 NoConn ~ 6100 2200
@@
 L Device:R R400
 U 1 1 5C5CEDA4
-P 2700 3400
-F 0 "R400" V 2600 3400 50  0000 C CNN
-F 1 "22R" V 2800 3400 50  0000 C CNN
-F 2 "require:R_0402" V 2630 3400 50  0001 C CNN
-F 3 "~" H 2700 3400 50  0001 C CNN
-	1    2700 3400
+P 2700 4000
+F 0 "R400" V 2600 4000 50  0000 C CNN
+F 1 "22R" V 2800 4000 50  0000 C CNN
+F 2 "require:R_0402" V 2630 4000 50  0001 C CNN
+F 3 "~" H 2700 4000 50  0001 C CNN
+	1    2700 4000
 	0    1    1    0
 $EndComp
-Wire Wire Line
-	2850 3400 3900 3400
 Connection ~ 3900 3400
-Text Label 3000 3400 0    50   ~ 0
-EMMC_CLK1
 $Comp
 L power:+3V3 #PWR0229
@@
 	3200 1300 3200 900
 Wire Wire Line
-	3200 900  5300 900
-Wire Wire Line
-	5300 900  5300 1600
-Wire Wire Line
 	2650 1900 2650 2400
 Wire Wire Line
@@
 	2350 3400 2350 2200
 Wire Wire Line
-	2350 3400 2550 3400
-Wire Wire Line
 	2250 3600 2250 2300
 Wire Wire Line
@@
 Wire Wire Line
 	2150 2000 2550 2000
+NoConn ~ 5300 1600
+Wire Wire Line
+	3200 900  5200 900
+NoConn ~ 5100 1800
+NoConn ~ 5300 2000
+Wire Wire Line
+	4900 1800 5100 2000
+Wire Wire Line
+	5100 2000 5200 2000
+Wire Wire Line
+	5200 2000 5200 900
+Connection ~ 5100 2000
+Wire Wire Line
+	2350 3400 3900 3400
 $EndSCHEMATC

Commit message: wip
Parts:
- added TP100, TP101: TestPoint, require:TP08, symbol Connector:TestPoint
Connections:
- net EMMC_CLK: now also R400.2; no longer U400.K1, U400.K2, U400.K3, U400.M6 (CLK)
- net GND: now also TP101.1
- net at R400.1: now also U400.K1, U400.K2, U400.K3, U400.M6 (CLK), TP100.1
Other:
- moved on the sheet: R400
Changed lines of the file:
@@
 Wire Wire Line
 	4500 3600 4300 3600
-Connection ~ 3900 3600
 Connection ~ 4100 3600
 Wire Wire Line
@@
 L Device:R R400
 U 1 1 5C5CEDA4
-P 2700 4000
-F 0 "R400" V 2600 4000 50  0000 C CNN
-F 1 "22R" V 2800 4000 50  0000 C CNN
-F 2 "require:R_0402" V 2630 4000 50  0001 C CNN
-F 3 "~" H 2700 4000 50  0001 C CNN
-	1    2700 4000
+P 2950 3400
+F 0 "R400" V 2850 3400 50  0000 C CNN
+F 1 "22R" V 3050 3400 50  0000 C CNN
+F 2 "require:R_0402" V 2880 3400 50  0001 C CNN
+F 3 "~" H 2950 3400 50  0001 C CNN
+	1    2950 3400
 	0    1    1    0
 $EndComp
-Connection ~ 3900 3400
 $Comp
 L power:+3V3 #PWR0229
@@
 	2250 3600 2250 2300
 Wire Wire Line
-	2250 3600 3900 3600
-Wire Wire Line
 	2150 2100 2450 2100
 Wire Wire Line
@@
 	5200 2000 5200 900
 Connection ~ 5100 2000
-Wire Wire Line
-	2350 3400 3900 3400
+Connection ~ 3900 3600
+Wire Wire Line
+	2250 3600 3900 3600
+Wire Wire Line
+	3100 3400 3300 3400
+Connection ~ 3900 3400
+Wire Wire Line
+	2800 3400 2350 3400
+$Comp
+L Connector:TestPoint TP100
+U 1 1 5CD619C9
+P 2550 4000
+F 0 "TP100" H 2608 4120 50  0000 L CNN
+F 1 "TestPoint" H 2608 4029 50  0000 L CNN
+F 2 "require:TP08" H 2750 4000 50  0001 C CNN
+F 3 "~" H 2750 4000 50  0001 C CNN
+	1    2550 4000
+	1    0    0    -1
+$EndComp
+Wire Wire Line
+	2550 4000 2550 4150
+Wire Wire Line
+	2550 4150 3300 4150
+Wire Wire Line
+	3300 4150 3300 3400
+Connection ~ 3300 3400
+Wire Wire Line
+	3300 3400 3900 3400
+$Comp
+L Connector:TestPoint TP101
+U 1 1 5CD6708D
+P 2100 4000
+F 0 "TP101" H 2158 4120 50  0000 L CNN
+F 1 "TestPoint" H 2158 4029 50  0000 L CNN
+F 2 "require:TP08" H 2300 4000 50  0001 C CNN
+F 3 "~" H 2300 4000 50  0001 C CNN
+	1    2100 4000
+	1    0    0    -1
+$EndComp
+$Comp
+L power:GND #PWR0181
+U 1 1 5CD67129
+P 2100 4100
+F 0 "#PWR0181" H 2100 3850 50  0001 C CNN
+F 1 "GND" H 2105 3927 50  0000 C CNN
+F 2 "" H 2100 4100 50  0001 C CNN
+F 3 "" H 2100 4100 50  0001 C CNN
+	1    2100 4100
+	1    0    0    -1
+$EndComp
+Wire Wire Line
+	2100 4000 2100 4100
 $EndSCHEMATC
