File: hardware/rk3308-lcdc-mac-i2s1-jtag.sch (KiCad schematic (older format))
At the start: 3 parts, among them U1000 RK3308

Commit message: wip
Parts:
- removed C5124: 0.1u, Capacitors_SMD:C_0402, symbol Device:C
- removed unit 2 of U1000
- added unit 4 of U1000
- renumbered C5123 to C75
Connections:
- net labels removed: WIFI_REG_ON, WIFI_WAKE_HOST
- wire segments 14 -> 10
- no-connect marks 26 -> 22
Other:
- note added: "Share cap with R12,R11\n"
Changed lines of the file:
@@
 $Descr A3 16535 11693
 encoding utf-8
-Sheet 8 8
+Sheet 8 9
 Title ""
 Date ""
@@
 $EndComp
 $Comp
-L Device:C C5123
+L Device:C C75
 U 1 1 5C70D031
 P 4600 5250
-F 0 "C5123" H 4715 5296 50  0000 L CNN
+F 0 "C75" H 4715 5296 50  0000 L CNN
 F 1 "0.1u" H 4715 5205 50  0000 L CNN
 F 2 "Capacitors_SMD:C_0402" H 4638 5100 50  0001 C CNN
@@
 $Comp
 L require:RK3308 U1000
-U 2 1 5C70F9F9
-P 6500 5200
-F 0 "U1000" H 7306 9287 60  0000 C CNN
-F 1 "RK3308" H 7306 9181 60  0000 C CNN
-F 2 "" H 6500 5200 60  0001 C CNN
-F 3 "" H 6500 5200 60  0001 C CNN
-	2    6500 5200
-	1    0    0    -1
-$EndComp
-Text Label 8300 1500 0    50   ~ 0
-WIFI_WAKE_HOST
-NoConn ~ 8100 1600
-Wire Wire Line
-	8100 1700 8900 1700
-Wire Wire Line
-	8100 1500 8900 1500
-Text Label 8300 1700 0    50   ~ 0
-WIFI_REG_ON
-NoConn ~ 8100 1800
-NoConn ~ 8100 4500
-NoConn ~ 8100 4600
-$Comp
-L Device:C C5124
-U 1 1 5C70FD6C
-P 8300 5350
-F 0 "C5124" H 8415 5396 50  0000 L CNN
-F 1 "0.1u" H 8415 5305 50  0000 L CNN
-F 2 "Capacitors_SMD:C_0402" H 8338 5200 50  0001 C CNN
-F 3 "~" H 8300 5350 50  0001 C CNN
-	1    8300 5350
+U 4 1 5D04A3D0
+P 7200 4700
+F 0 "U1000" H 8186 8287 60  0000 C CNN
+F 1 "RK3308" H 8186 8181 60  0000 C CNN
+F 2 "" H 7200 4700 60  0001 C CNN
+F 3 "" H 7200 4700 60  0001 C CNN
+	4    7200 4700
 	1    0    0    -1
 $EndComp
 Wire Wire Line
-	8100 5000 8300 5000
+	9400 4500 9900 4500
 Wire Wire Line
-	8300 5000 8300 5200
-Wire Wire Line
-	8300 5500 8300 5700
+	9900 4500 9900 4300
 $Comp
-L power:GND #PWR0173
-U 1 1 5C70FF11
-P 8300 5700
-F 0 "#PWR0173" H 8300 5450 50  0001 C CNN
-F 1 "GND" H 8305 5527 50  0000 C CNN
-F 2 "" H 8300 5700 50  0001 C CNN
-F 3 "" H 8300 5700 50  0001 C CNN
-	1    8300 5700
+L require:VCC_IO #PWR0221
+U 1 1 5D04A5C2
+P 9900 4300
+F 0 "#PWR0221" H 9900 4150 50  0001 C CNN
+F 1 "VCC_IO" H 9917 4473 50  0000 C CNN
+F 2 "" H 9900 4300 50  0001 C CNN
+F 3 "" H 9900 4300 50  0001 C CNN
+	1    9900 4300
 	1    0    0    -1
 $EndComp
-Wire Wire Line
-	8300 5000 8300 4900
-Connection ~ 8300 5000
-$Comp
-L require:VCC_IO #PWR0175
-U 1 1 5C70FFEA
-P 8300 4900
-F 0 "#PWR0175" H 8300 4750 50  0001 C CNN
-F 1 "VCC_IO" H 8317 5073 50  0000 C CNN
-F 2 "" H 8300 4900 50  0001 C CNN
-F 3 "" H 8300 4900 50  0001 C CNN
-	1    8300 4900
-	1    0    0    -1
-$EndComp
+Text Notes 9900 4650 0    50   ~ 10
+Share cap with R12,R11\n
 $EndSCHEMATC

Commit message: wip
Parts:
- added LP1, LP18, LP8, RP1, RP20: GND, require:OVAL_PIN, symbol require:OP
- added LP13: DNC, require:OVAL_PIN, symbol require:OP
- added LP15, LP16: 3V3, require:OVAL_PIN, symbol require:OP
- added LP17: 5V, require:OVAL_PIN, symbol require:OP
- added P15: 7, require:OVAL_PIN, symbol require:OP
- added P16: 8, require:OVAL_PIN, symbol require:OP
- added P17: 9, require:OVAL_PIN, symbol require:OP
- added P18: 10, require:OVAL_PIN, symbol require:OP
- added P19: 3, require:OVAL_PIN, symbol require:OP
- added P20: 4, require:OVAL_PIN, symbol require:OP
- added P21: 5, require:OVAL_PIN, symbol require:OP
- added P22: 6, require:OVAL_PIN, symbol require:OP
Connections:
- net labels added: DIO10, DIO3, DIO4, DIO5, DIO6, DIO7, DIO8, DIO9, VCC5V0_SYS
- net labels removed: SPI2_CLK, SPI2_CS, SPI2_RX_UART2_RX_M0, SPI2_TX_UART2_TX_M0
- wire segments 10 -> 30
- no-connect marks 22 -> 23

Commit message: wip
Parts:
- removed C75: 0.1u, Capacitors_SMD:C_0402, symbol Device:C
- removed P15: 7, require:OVAL_PIN, symbol require:OP
- removed P16: 8, require:OVAL_PIN, symbol require:OP
- removed P17: 9, require:OVAL_PIN, symbol require:OP
- removed P18: 10, require:OVAL_PIN, symbol require:OP
- removed P19: 3, require:OVAL_PIN, symbol require:OP
- removed P20: 4, require:OVAL_PIN, symbol require:OP
- removed P21: 5, require:OVAL_PIN, symbol require:OP
- removed P22: 6, require:OVAL_PIN, symbol require:OP
- removed U1000: RK3308, symbol require:RK3308
Connections:
- net labels removed: DIO10, DIO3, DIO4, DIO5, DIO6, DIO7, DIO8, DIO9
- wire segments 30 -> 16
- no-connect marks 23 -> 1
Other:
- note removed: "Share cap with R12,R11\n"
Changed lines of the file:
@@
 $Descr A3 16535 11693
 encoding utf-8
-Sheet 8 10
+Sheet 7 9
 Title ""
 Date ""
@@
 Comment4 ""
 $EndDescr
-$Comp
-L require:RK3308 U1000
-U 3 1 5C70CE31
-P 1200 5100
-F 0 "U1000" H 2636 9087 60  0000 C CNN
-F 1 "RK3308" H 2636 8981 60  0000 C CNN
-F 2 "" H 1200 5100 60  0001 C CNN
-F 3 "" H 1200 5100 60  0001 C CNN
-	3    1200 5100
-	1    0    0    -1
-$EndComp
-NoConn ~ 4400 1400
-NoConn ~ 4400 1500
-NoConn ~ 4400 1600
-NoConn ~ 4400 1700
-NoConn ~ 4400 1800
-NoConn ~ 4400 1900
-NoConn ~ 4400 2000
-NoConn ~ 4400 2100
-NoConn ~ 4400 2200
-NoConn ~ 4400 2300
-NoConn ~ 4400 2400
-NoConn ~ 4400 2500
-NoConn ~ 4400 2700
-NoConn ~ 4400 2900
-NoConn ~ 4400 3000
-NoConn ~ 4400 3100
-NoConn ~ 4400 3200
-NoConn ~ 4400 3300
-NoConn ~ 4400 3400
-NoConn ~ 4400 3500
-NoConn ~ 4400 3600
-NoConn ~ 4400 3700
-Wire Wire Line
-	4400 4100 5400 4100
-Text Label 4600 4100 0    50   ~ 0
-DIO7
-Wire Wire Line
-	4400 4200 5400 4200
-Text Label 4600 4200 0    50   ~ 0
-DIO8
-Wire Wire Line
-	4400 4400 5400 4400
-Wire Wire Line
-	4400 4500 5400 4500
-Text Label 4600 4400 0    50   ~ 0
-DIO9
-Text Label 4600 4500 0    50   ~ 0
-DIO10
-Wire Wire Line
-	4400 4900 4600 4900
-Wire Wire Line
-	4600 4900 4600 4800
-$Comp
-L require:VCC_IO #PWR0170
-U 1 1 5C70CFF6
-P 4600 4800
-F 0 "#PWR0170" H 4600 4650 50  0001 C CNN
-F 1 "VCC_IO" H 4617 4973 50  0000 C CNN
-F 2 "" H 4600 4800 50  0001 C CNN
-F 3 "" H 4600 4800 50  0001 C CNN
-	1    4600 4800
-	1    0    0    -1
-$EndComp
-$Comp
-L Device:C C75
-U 1 1 5C70D031
-P 4600 5250
-F 0 "C75" H 4715 5296 50  0000 L CNN
-F 1 "0.1u" H 4715 5205 50  0000 L CNN
-F 2 "Capacitors_SMD:C_0402" H 4638 5100 50  0001 C CNN
-F 3 "~" H 4600 5250 50  0001 C CNN
-	1    4600 5250
-	1    0    0    -1
-$EndComp
-Wire Wire Line
-	4600 5100 4600 4900
-Connection ~ 4600 4900
-Wire Wire Line
-	4600 5400 4600 5600
-$Comp
-L power:GND #PWR0171
-U 1 1 5C70D0C1
-P 4600 5600
-F 0 "#PWR0171" H 4600 5350 50  0001 C CNN
-F 1 "GND" H 4605 5427 50  0000 C CNN
-F 2 "" H 4600 5600 50  0001 C CNN
-F 3 "" H 4600 5600 50  0001 C CNN
-	1    4600 5600
-	1    0    0    -1
-$EndComp
-$Comp
-L require:RK3308 U1000
-U 4 1 5D04A3D0
-P 7200 4700
-F 0 "U1000" H 8186 8287 60  0000 C CNN
-F 1 "RK3308" H 8186 8181 60  0000 C CNN
-F 2 "" H 7200 4700 60  0001 C CNN
-F 3 "" H 7200 4700 60  0001 C CNN
-	4    7200 4700
-	1    0    0    -1
-$EndComp
-Wire Wire Line
-	9400 4500 9900 4500
-Wire Wire Line
-	9900 4500 9900 4300
-$Comp
-L require:VCC_IO #PWR0221
-U 1 1 5D04A5C2
-P 9900 4300
-F 0 "#PWR0221" H 9900 4150 50  0001 C CNN
-F 1 "VCC_IO" H 9917 4473 50  0000 C CNN
-F 2 "" H 9900 4300 50  0001 C CNN
-F 3 "" H 9900 4300 50  0001 C CNN
-	1    9900 4300
-	1    0    0    -1
-$EndComp
-Text Notes 9900 4650 0    50   ~ 10
-Share cap with R12,R11\n
-Wire Wire Line
-	9400 1500 10050 1500
-Wire Wire Line
-	9400 1600 10050 1600
-Wire Wire Line
-	9400 1800 10050 1800
-Wire Wire Line
-	9400 2000 10050 2000
-$Comp
-L require:OP P15
-U 1 1 5C5EFD91
-P 5600 4100
-F 0 "P15" H 5850 4100 50  0000 C CNN
-F 1 "7" H 5600 4100 50  0000 C CNN
-F 2 "require:OVAL_PIN" H 5600 4050 50  0001 C CNN
-F 3 "" H 5600 4050 50  0001 C CNN
-	1    5600 4100
-	1    0    0    -1
-$EndComp
-$Comp
-L require:OP P16
-U 1 1 5C5EFE28
-P 5600 4200
-F 0 "P16" H 5850 4200 50  0000 C CNN
-F 1 "8" H 5600 4200 50  0000 C CNN
-F 2 "require:OVAL_PIN" H 5600 4150 50  0001 C CNN
-F 3 "" H 5600 4150 50  0001 C CNN
-	1    5600 4200
-	1    0    0    -1
-$EndComp
-$Comp
-L require:OP P17
-U 1 1 5C5EFE42
-P 5600 4400
-F 0 "P17" H 5850 4400 50  0000 C CNN
-F 1 "9" H 5600 4400 50  0000 C CNN
-F 2 "require:OVAL_PIN" H 5600 4350 50  0001 C CNN
-F 3 "" H 5600 4350 50  0001 C CNN
-	1    5600 4400
-	1    0    0    -1
-$EndComp
-$Comp
-L require:OP P18
-U 1 1 5C5EFE66
-P 5600 4500
-F 0 "P18" H 5850 4500 50  0000 C CNN
-F 1 "10" H 5600 4500 50  0000 C CNN
-F 2 "require:OVAL_PIN" H 5600 4450 50  0001 C CNN
-F 3 "" H 5600 4450 50  0001 C CNN
-	1    5600 4500
-	1    0    0    -1
-$EndComp
-$Comp
-L require:OP P19
-U 1 1 5C5F0013
-P 10250 1500
-F 0 "P19" H 10450 1500 50  0000 C CNN
-F 1 "3" H 10250 1500 50  0000 C CNN
-F 2 "require:OVAL_PIN" H 10250 1450 50  0001 C CNN
-F 3 "" H 10250 1450 50  0001 C CNN
-	1    10250 1500
-	1    0    0    -1
-$EndComp
-$Comp
-L require:OP P20
-U 1 1 5C5F00C8
-P 10250 1600
-F 0 "P20" H 10450 1600 50  0000 C CNN
-F 1 "4" H 10250 1600 50  0000 C CNN
-F 2 "require:OVAL_PIN" H 10250 1550 50  0001 C CNN
-F 3 "" H 10250 1550 50  0001 C CNN
-	1    10250 1600
-	1    0    0    -1
-$EndComp
-$Comp
-L require:OP P21
-U 1 1 5C5F00EA
-P 10250 1800
-F 0 "P21" H 10450 1800 50  0000 C CNN
-F 1 "5" H 10250 1800 50  0000 C CNN
-F 2 "require:OVAL_PIN" H 10250 1750 50  0001 C CNN
-F 3 "" H 10250 1750 50  0001 C CNN
-	1    10250 1800
-	1    0    0    -1
-$EndComp
-$Comp
-L require:OP P22
-U 1 1 5C5F0112
-P 10250 2000
-F 0 "P22" H 10450 2000 50  0000 C CNN
-F 1 "6" H 10250 2000 50  0000 C CNN
-F 2 "require:OVAL_PIN" H 10250 1950 50  0001 C CNN
-F 3 "" H 10250 1950 50  0001 C CNN
-	1    10250 2000
-	1    0    0    -1
-$EndComp
 $Comp
 L require:OP RP1
@@
 Wire Wire Line
 	8250 6350 8250 6550
-Text Label 9550 1500 0    50   ~ 0
-DIO3
-Text Label 9550 1600 0    50   ~ 0
-DIO4
-Text Label 9550 1800 0    50   ~ 0
-DIO5
-Text Label 9550 2000 0    50   ~ 0
-DIO6
 $Comp
 L require:OP LP13

Commit message: wip
Parts:
- removed LP1, LP18, LP8, RP1, RP20: GND, require:OVAL_PIN, symbol require:OP
- removed LP13: DNC, require:OVAL_PIN, symbol require:OP
- removed LP15, LP16: 3V3, require:OVAL_PIN, symbol require:OP
- removed LP17: 5V, require:OVAL_PIN, symbol require:OP
Connections:
- no-connect marks 1 -> 0
Changed lines of the file:
@@
 Comment4 ""
 $EndDescr
-$Comp
-L require:OP RP1
-U 1 1 5C6074E9
-P 10750 6150
-F 0 "RP1" H 11000 6150 50  0000 C CNN
-F 1 "GND" H 10750 6150 50  0000 C CNN
-F 2 "require:OVAL_PIN" H 10750 6100 50  0001 C CNN
-F 3 "" H 10750 6100 50  0001 C CNN
-	1    10750 6150
-	1    0    0    -1
-$EndComp
-$Comp
-L require:OP RP20
-U 1 1 5C6075BF
-P 10750 6350
-F 0 "RP20" H 11000 6350 50  0000 C CNN
-F 1 "GND" H 10750 6350 50  0000 C CNN
-F 2 "require:OVAL_PIN" H 10750 6300 50  0001 C CNN
-F 3 "" H 10750 6300 50  0001 C CNN
-	1    10750 6350
-	1    0    0    -1
-$EndComp
-$Comp
-L require:OP LP1
-U 1 1 5C6075EB
-P 8650 6150
-F 0 "LP1" H 8900 6150 50  0000 C CNN
-F 1 "GND" H 8650 6150 50  0000 C CNN
-F 2 "require:OVAL_PIN" H 8650 6100 50  0001 C CNN
-F 3 "" H 8650 6100 50  0001 C CNN
-	1    8650 6150
-	1    0    0    -1
-$EndComp
-$Comp
-L require:OP LP8
-U 1 1 5C607619
-P 8650 6350
-F 0 "LP8" H 8900 6350 50  0000 C CNN
-F 1 "GND" H 8650 6350 50  0000 C CNN
-F 2 "require:OVAL_PIN" H 8650 6300 50  0001 C CNN
-F 3 "" H 8650 6300 50  0001 C CNN
-	1    8650 6350
-	1    0    0    -1
-$EndComp
-Wire Wire Line
-	10550 6150 10350 6150
-Wire Wire Line
-	10350 6150 10350 6350
-$Comp
-L power:GND #PWR01
-U 1 1 5C607840
-P 8250 6750
-F 0 "#PWR01" H 8250 6500 50  0001 C CNN
-F 1 "GND" H 8255 6577 50  0000 C CNN
-F 2 "" H 8250 6750 50  0001 C CNN
-F 3 "" H 8250 6750 50  0001 C CNN
-	1    8250 6750
-	1    0    0    -1
-$EndComp
-Wire Wire Line
-	10550 6350 10350 6350
-Wire Wire Line
-	8450 6150 8250 6150
-Wire Wire Line
-	8250 6150 8250 6350
-Wire Wire Line
-	8450 6350 8250 6350
-Connection ~ 8250 6350
-Wire Wire Line
-	8250 6350 8250 6550
-$Comp
-L require:OP LP13
-U 1 1 5C6CA58D
-P 8450 7300
-F 0 "LP13" H 8700 7300 50  0000 C CNN
-F 1 "DNC" H 8450 7300 50  0000 C CNN
-F 2 "require:OVAL_PIN" H 8450 7250 50  0001 C CNN
-F 3 "" H 8450 7250 50  0001 C CNN
-	1    8450 7300
-	1    0    0    1
-$EndComp
-$Comp
-L require:OP LP15
-U 1 1 5C6CC801
-P 11700 7250
-F 0 "LP15" H 11950 7250 50  0000 C CNN
-F 1 "3V3" H 11700 7250 50  0000 C CNN
-F 2 "require:OVAL_PIN" H 11700 7200 50  0001 C CNN
-F 3 "" H 11700 7200 50  0001 C CNN
-	1    11700 7250
-	1    0    0    -1
-$EndComp
-$Comp
-L require:OP LP16
-U 1 1 5C6CC8C7
-P 11700 7450
-F 0 "LP16" H 11950 7450 50  0000 C CNN
-F 1 "3V3" H 11700 7450 50  0000 C CNN
-F 2 "require:OVAL_PIN" H 11700 7400 50  0001 C CNN
-F 3 "" H 11700 7400 50  0001 C CNN
-	1    11700 7450
-	1    0    0    -1
-$EndComp
-$Comp
-L require:OP LP17
-U 1 1 5C6CC93F
-P 8650 8300
-F 0 "LP17" H 8900 8300 50  0000 C CNN
-F 1 "5V" H 8650 8300 50  0000 C CNN
-F 2 "require:OVAL_PIN" H 8650 8250 50  0001 C CNN
-F 3 "" H 8650 8250 50  0001 C CNN
-	1    8650 8300
-	1    0    0    -1
-$EndComp
-$Comp
-L require:OP LP18
-U 1 1 5C6CCA42
-P 8650 6550
-F 0 "LP18" H 8900 6550 50  0000 C CNN
-F 1 "GND" H 8650 6550 50  0000 C CNN
-F 2 "require:OVAL_PIN" H 8650 6500 50  0001 C CNN
-F 3 "" H 8650 6500 50  0001 C CNN
-	1    8650 6550
-	1    0    0    -1
-$EndComp
-Wire Wire Line
-	11500 7250 11100 7250
-Wire Wire Line
-	8250 6550 8450 6550
-Wire Wire Line
-	8250 8300 8450 8300
-Connection ~ 8250 6550
-Wire Wire Line
-	8250 6550 8250 6750
-$Comp
-L power:GND #PWR0225
-U 1 1 5C6D5A58
-P 10350 6550
-F 0 "#PWR0225" H 10350 6300 50  0001 C CNN
-F 1 "GND" H 10355 6377 50  0000 C CNN
-F 2 "" H 10350 6550 50  0001 C CNN
-F 3 "" H 10350 6550 50  0001 C CNN
-	1    10350 6550
-	1    0    0    -1
-$EndComp
-Wire Wire Line
-	10350 6350 10350 6550
-Connection ~ 10350 6350
-Wire Wire Line
-	11100 6900 11100 7250
-Wire Wire Line
-	8250 8200 8250 8300
-Wire Wire Line
-	11500 7450 11100 7450
-Wire Wire Line
-	11100 7450 11100 7250
-Connection ~ 11100 7250
-$Comp
-L require:VCC5V0_SYS #PWR0227
-U 1 1 5C6DB54B
-P 8250 8200
-F 0 "#PWR0227" H 8250 8050 50  0001 C CNN
-F 1 "VCC5V0_SYS" H 8267 8373 50  0000 C CNN
-F 2 "" H 8250 8200 50  0001 C CNN
-F 3 "" H 8250 8200 50  0001 C CNN
-	1    8250 8200
-	1    0    0    -1
-$EndComp
-$Comp
-L require:VCC_IO #PWR0228
-U 1 1 5C6DB5B3
-P 11100 6900
-F 0 "#PWR0228" H 11100 6750 50  0001 C CNN
-F 1 "VCC_IO" H 11117 7073 50  0000 C CNN
-F 2 "" H 11100 6900 50  0001 C CNN
-F 3 "" H 11100 6900 50  0001 C CNN
-	1    11100 6900
-	1    0    0    -1
-$EndComp
-NoConn ~ 8250 7300
 $EndSCHEMATC
