File: hardware/usb.sch (KiCad schematic (older format))
At the start: 12 parts, among them J10 USB_B_Micro, U1000 RK3308

Commit message: wip
Parts:
- added LP11: DM, require:OVAL_PIN, symbol require:OP
- added LP12: DP, require:OVAL_PIN, symbol require:OP
Changed lines of the file:
@@
 $Descr A4 11693 8268
 encoding utf-8
-Sheet 9 9
+Sheet 9 10
 Title ""
 Date ""
@@
 Wire Wire Line
 	2200 1800 3050 1800
-Wire Wire Line
-	2200 1900 3050 1900
 $Comp
 L Device:R R93
@@
 	6900 3450 6900 3050
 Connection ~ 6900 3050
+$Comp
+L require:OP LP11
+U 1 1 5C4F0BF5
+P 3250 1800
+F 0 "LP11" H 3500 1800 50  0000 C CNN
+F 1 "DM" H 3250 1800 50  0000 C CNN
+F 2 "require:OVAL_PIN" H 3250 1800 50  0001 C CNN
+F 3 "" H 3250 1800 50  0001 C CNN
+	1    3250 1800
+	1    0    0    -1
+$EndComp
+$Comp
+L require:OP LP12
+U 1 1 5C4F0C66
+P 3250 1900
+F 0 "LP12" H 3500 1900 50  0000 C CNN
+F 1 "DP" H 3250 1900 50  0000 C CNN
+F 2 "require:OVAL_PIN" H 3250 1900 50  0001 C CNN
+F 3 "" H 3250 1900 50  0001 C CNN
+	1    3250 1900
+	1    0    0    -1
+$EndComp
+Wire Wire Line
+	2200 1900 3050 1900
 $EndSCHEMATC

Commit message: wip
Parts:
- removed C85, C87: 0.1u, Capacitors_SMD:C_0402, symbol Device:C
Connections:
- net labels removed: AVDD_1V8, VDD_1V0
- wire segments 45 -> 32
Other:
- note removed: "Share cap with pll"
Changed lines of the file:
@@
 $Descr A4 11693 8268
 encoding utf-8
-Sheet 9 10
+Sheet 8 9
 Title ""
 Date ""
@@
 	0    -1   -1   0
 $EndComp
-Wire Wire Line
-	2200 2300 3650 2300
-Wire Wire Line
-	3650 2300 3650 2200
-Wire Wire Line
-	2200 2400 3650 2400
-Wire Wire Line
-	3650 2400 3650 2300
-Connection ~ 3650 2300
-$Comp
-L Device:C C87
-U 1 1 5CED3FFD
-P 3650 2650
-F 0 "C87" H 3765 2696 50  0000 L CNN
-F 1 "0.1u" H 3765 2605 50  0000 L CNN
-F 2 "Capacitors_SMD:C_0402" H 3688 2500 50  0001 C CNN
-F 3 "~" H 3650 2650 50  0001 C CNN
-	1    3650 2650
-	1    0    0    -1
-$EndComp
-$Comp
-L power:GND #PWR0192
-U 1 1 5CED414D
-P 3650 2900
-F 0 "#PWR0192" H 3650 2650 50  0001 C CNN
-F 1 "GND" H 3655 2727 50  0000 C CNN
-F 2 "" H 3650 2900 50  0001 C CNN
-F 3 "" H 3650 2900 50  0001 C CNN
-	1    3650 2900
-	1    0    0    -1
-$EndComp
-Wire Wire Line
-	3650 2900 3650 2800
-Wire Wire Line
-	3650 2500 3650 2400
-Connection ~ 3650 2400
 $Comp
 L require:VCC_IO #PWR0195
 U 1 1 5CED42C8
-P 3650 2200
-F 0 "#PWR0195" H 3650 2050 50  0001 C CNN
-F 1 "VCC_IO" H 3667 2373 50  0000 C CNN
-F 2 "" H 3650 2200 50  0001 C CNN
-F 3 "" H 3650 2200 50  0001 C CNN
-	1    3650 2200
-	1    0    0    -1
-$EndComp
-$Comp
-L Device:C C85
-U 1 1 5CED42E0
-P 3200 3050
-F 0 "C85" H 3315 3096 50  0000 L CNN
-F 1 "0.1u" H 3315 3005 50  0000 L CNN
-F 2 "Capacitors_SMD:C_0402" H 3238 2900 50  0001 C CNN
-F 3 "~" H 3200 3050 50  0001 C CNN
-	1    3200 3050
-	1    0    0    -1
-$EndComp
-Wire Wire Line
-	2200 2800 3200 2800
-Wire Wire Line
-	3200 2800 3200 2900
-$Comp
-L require:AVDD_1V8 #PWR0196
-U 1 1 5CED44A9
-P 3200 2700
-F 0 "#PWR0196" H 3200 2550 50  0001 C CNN
-F 1 "AVDD_1V8" H 3217 2873 50  0000 C CNN
-F 2 "" H 3200 2700 50  0001 C CNN
-F 3 "" H 3200 2700 50  0001 C CNN
-	1    3200 2700
-	1    0    0    -1
-$EndComp
-Wire Wire Line
-	3200 2700 3200 2800
-Connection ~ 3200 2800
-Wire Wire Line
-	3200 3200 3200 3300
-$Comp
-L power:GND #PWR0197
-U 1 1 5CED46F9
-P 3200 3300
-F 0 "#PWR0197" H 3200 3050 50  0001 C CNN
-F 1 "GND" H 3205 3127 50  0000 C CNN
-F 2 "" H 3200 3300 50  0001 C CNN
-F 3 "" H 3200 3300 50  0001 C CNN
-	1    3200 3300
-	1    0    0    -1
-$EndComp
-Wire Wire Line
-	2200 3200 2400 3200
-Wire Wire Line
-	2400 3100 2400 3200
+P 4050 1100
+F 0 "#PWR0195" H 4050 950 50  0001 C CNN
+F 1 "VCC_IO" H 4067 1273 50  0000 C CNN
+F 2 "" H 4050 1100 50  0001 C CNN
+F 3 "" H 4050 1100 50  0001 C CNN
+	1    4050 1100
+	1    0    0    -1
+$EndComp
 Text Label 2350 1000 0    50   ~ 0
 USB_OTG_DM
@@
 	5500 4750 5500 4650
 Wire Wire Line
-	3850 1300 3850 2300
-Wire Wire Line
-	3850 2300 3650 2300
-Wire Wire Line
-	2200 1300 3850 1300
-$Comp
-L require:VDD_1V0 #PWR0173
-U 1 1 5CF02EB6
-P 2400 3100
-F 0 "#PWR0173" H 2400 2950 50  0001 C CNN
-F 1 "VDD_1V0" H 2417 3273 50  0000 C CNN
-F 2 "" H 2400 3100 50  0001 C CNN
-F 3 "" H 2400 3100 50  0001 C CNN
-	1    2400 3100
-	1    0    0    -1
-$EndComp
-Text Notes 2100 3350 0    50   ~ 10
-Share cap with pll
-Wire Wire Line
 	1800 5350 1800 5450
 $Comp
@@
 Wire Wire Line
 	2200 1900 3050 1900
+Wire Wire Line
+	4050 1100 4050 1300
+Wire Wire Line
+	2200 1300 4050 1300
 $EndSCHEMATC

Commit message: wip
Parts:
- removed D2: D_TVS, symbol Device:D_TVS
- removed H1, H2, H3, H4: MountingHole_Pad, require:PTH_MTG320_380, symbol Mechanical:MountingHole_Pad
- removed J10: USB_B_Micro, Connectors_USB:USB_Micro-B_Molex_47346-0001, symbol Connector:USB_B_Micro
- removed R1, R2: 2.2R, Resistors_SMD:R_0402, symbol Device:R
- removed R93: 133R,1%, Resistors_SMD:R_0402, symbol Device:R
- removed U1000: RK3308, symbol require:RK3308
Connections:
- net labels removed: GND, USB_OTG_DM, USB_OTG_DP, VCC5V0_SYS
- wire segments 32 -> 4
- no-connect marks 2 -> 1
Other:
- note removed: "USB_OTG_ID floating, dedicated device/peripheral mode. no OTG."
Changed lines of the file:
@@
 $Descr A4 11693 8268
 encoding utf-8
-Sheet 8 9
+Sheet 7 8
 Title ""
 Date ""
@@
 Comment4 ""
 $EndDescr
-$Comp
-L require:RK3308 U1000
-U 9 1 5CED3BF3
-P 1000 3400
-F 0 "U1000" H 1606 6187 60  0000 C CNN
-F 1 "RK3308" H 1606 6081 60  0000 C CNN
-F 2 "" H 1000 3400 60  0001 C CNN
-F 3 "" H 1000 3400 60  0001 C CNN
-	9    1000 3400
-	1    0    0    -1
-$EndComp
-Wire Wire Line
-	2200 1000 3050 1000
-Wire Wire Line
-	2200 1100 3050 1100
 Wire Wire Line
 	2200 1800 3050 1800
-$Comp
-L Device:R R93
-U 1 1 5CED3D45
-P 2550 2100
-F 0 "R93" V 2450 2100 50  0000 C CNN
-F 1 "133R,1%" V 2650 2100 50  0000 C CNN
-F 2 "Resistors_SMD:R_0402" V 2480 2100 50  0001 C CNN
-F 3 "~" H 2550 2100 50  0001 C CNN
-	1    2550 2100
-	0    1    1    0
-$EndComp
-Wire Wire Line
-	2200 2100 2400 2100
-Wire Wire Line
-	2700 2100 3050 2100
-$Comp
-L power:GND #PWR0191
-U 1 1 5CED3E64
-P 3050 2100
-F 0 "#PWR0191" H 3050 1850 50  0001 C CNN
-F 1 "GND" V 3055 1972 50  0000 R CNN
-F 2 "" H 3050 2100 50  0001 C CNN
-F 3 "" H 3050 2100 50  0001 C CNN
-	1    3050 2100
-	0    -1   -1   0
-$EndComp
 $Comp
 L require:VCC_IO #PWR0195
@@
 	1    0    0    -1
 $EndComp
-Text Label 2350 1000 0    50   ~ 0
-USB_OTG_DM
-Text Label 2350 1100 0    50   ~ 0
-USB_OTG_DP
 Text Label 2350 1800 0    50   ~ 0
 USB_HOST_DM
 Text Label 2350 1900 0    50   ~ 0
 USB_HOST_DP
-$Comp
-L Connector:USB_B_Micro J10
-U 1 1 5CED7FA5
-P 1800 4950
-F 0 "J10" H 1855 5417 50  0000 C CNN
-F 1 "USB_B_Micro" H 1855 5326 50  0000 C CNN
-F 2 "Connectors_USB:USB_Micro-B_Molex_47346-0001" H 1950 4900 50  0001 C CNN
-F 3 "~" H 1950 4900 50  0001 C CNN
-	1    1800 4950
-	1    0    0    -1
-$EndComp
-Wire Wire Line
-	2100 4750 5500 4750
-$Comp
-L require:VCC5V0_SYS #PWR0218
-U 1 1 5CED863A
-P 5500 4650
-F 0 "#PWR0218" H 5500 4500 50  0001 C CNN
-F 1 "VCC5V0_SYS" H 5517 4823 50  0000 C CNN
-F 2 "" H 5500 4650 50  0001 C CNN
-F 3 "" H 5500 4650 50  0001 C CNN
-	1    5500 4650
-	1    0    0    -1
-$EndComp
-$Comp
-L Device:D_TVS D2
-U 1 1 5CEDAEDE
-P 5500 5100
-F 0 "D2" V 5454 5179 50  0000 L CNN
-F 1 "D_TVS" V 5545 5179 50  0000 L CNN
-F 2 "" H 5500 5100 50  0001 C CNN
-F 3 "~" H 5500 5100 50  0001 C CNN
-	1    5500 5100
-	0    1    1    0
-$EndComp
-Wire Wire Line
-	5500 4950 5500 4750
-Connection ~ 5500 4750
-Wire Wire Line
-	5500 5250 5500 5450
-$Comp
-L power:GND #PWR0222
-U 1 1 5CEDB8B6
-P 5500 5450
-F 0 "#PWR0222" H 5500 5200 50  0001 C CNN
-F 1 "GND" H 5505 5277 50  0000 C CNN
-F 2 "" H 5500 5450 50  0001 C CNN
-F 3 "" H 5500 5450 50  0001 C CNN
-	1    5500 5450
-	1    0    0    -1
-$EndComp
-$Comp
-L Device:R R1
-U 1 1 5CEDEDE4
-P 3300 4950
-F 0 "R1" V 3400 5000 50  0000 C CNN
-F 1 "2.2R" V 3400 4850 50  0000 C CNN
-F 2 "Resistors_SMD:R_0402" V 3230 4950 50  0001 C CNN
-F 3 "~" H 3300 4950 50  0001 C CNN
-	1    3300 4950
-	0    -1   -1   0
-$EndComp
-$Comp
-L Device:R R2
-U 1 1 5CEDEE6B
-P 3300 5050
-F 0 "R2" V 3200 5100 50  0000 C CNN
-F 1 "2.2R" V 3200 4950 50  0000 C CNN
-F 2 "Resistors_SMD:R_0402" V 3230 5050 50  0001 C CNN
-F 3 "~" H 3300 5050 50  0001 C CNN
-	1    3300 5050
-	0    -1   -1   0
-$EndComp
-Wire Wire Line
-	2100 4950 3150 4950
-Wire Wire Line
-	2100 5050 3150 5050
-Wire Wire Line
-	3450 4950 4200 4950
-Wire Wire Line
-	3450 5050 4200 5050
-Text Label 3600 4950 0    50   ~ 0
-USB_OTG_DP
-Text Label 3600 5050 0    50   ~ 0
-USB_OTG_DM
-NoConn ~ 2100 5150
 NoConn ~ 2200 1400
-Text Notes 5100 800  0    100  ~ 20
-USB_OTG_ID floating, dedicated device/peripheral mode. no OTG.
-Wire Wire Line
-	5500 4750 5500 4650
-Wire Wire Line
-	1800 5350 1800 5450
-$Comp
-L power:GND #PWR0215
-U 1 1 5CF5439A
-P 1800 5550
-F 0 "#PWR0215" H 1800 5300 50  0001 C CNN
-F 1 "GND" H 1805 5377 50  0000 C CNN
-F 2 "" H 1800 5550 50  0001 C CNN
-F 3 "" H 1800 5550 50  0001 C CNN
-	1    1800 5550
-	1    0    0    -1
-$EndComp
-Wire Wire Line
-	1700 5350 1700 5450
-Wire Wire Line
-	1700 5450 1800 5450
-Connection ~ 1800 5450
-Wire Wire Line
-	1800 5450 1800 5550
-$Comp
-L Mechanical:MountingHole_Pad H1
-U 1 1 5CF638CE
-P 7200 1550
-F 0 "H1" H 7300 1601 50  0000 L CNN
-F 1 "MountingHole_Pad" H 7300 1510 50  0000 L CNN
-F 2 "require:PTH_MTG320_380" H 7200 1550 50  0001 C CNN
-F 3 "~" H 7200 1550 50  0001 C CNN
-	1    7200 1550
-	1    0    0    -1
-$EndComp
-$Comp
-L power:GND #PWR0216
-U 1 1 5CF6394E
-P 7200 1850
-F 0 "#PWR0216" H 7200 1600 50  0001 C CNN
-F 1 "GND" H 7205 1677 50  0000 C CNN
-F 2 "" H 7200 1850 50  0001 C CNN
-F 3 "" H 7200 1850 50  0001 C CNN
-	1    7200 1850
-	1    0    0    -1
-$EndComp
-Wire Wire Line
-	7200 1650 7200 1750
-$Comp
-L Mechanical:MountingHole_Pad H2
-U 1 1 5CF63EC1
-P 7200 2300
-F 0 "H2" H 7300 2351 50  0000 L CNN
-F 1 "MountingHole_Pad" H 7300 2260 50  0000 L CNN
-F 2 "require:PTH_MTG320_380" H 7200 2300 50  0001 C CNN
-F 3 "~" H 7200 2300 50  0001 C CNN
-	1    7200 2300
-	1    0    0    -1
-$EndComp
-$Comp
-L Mechanical:MountingHole_Pad H3
-U 1 1 5CF63FAF
-P 7200 2850
-F 0 "H3" H 7300 2901 50  0000 L CNN
-F 1 "MountingHole_Pad" H 7300 2810 50  0000 L CNN
-F 2 "require:PTH_MTG320_380" H 7200 2850 50  0001 C CNN
-F 3 "~" H 7200 2850 50  0001 C CNN
-	1    7200 2850
-	1    0    0    -1
-$EndComp
-$Comp
-L Mechanical:MountingHole_Pad H4
-U 1 1 5CF63FE5
-P 7200 3250
-F 0 "H4" H 7300 3301 50  0000 L CNN
-F 1 "MountingHole_Pad" H 7300 3210 50  0000 L CNN
-F 2 "require:PTH_MTG320_380" H 7200 3250 50  0001 C CNN
-F 3 "~" H 7200 3250 50  0001 C CNN
-	1    7200 3250
-	1    0    0    -1
-$EndComp
-Wire Wire Line
-	7200 2400 7200 2500
-Wire Wire Line
-	7200 2500 6900 2500
-Wire Wire Line
-	7200 1750 6900 1750
-Wire Wire Line
-	6900 1750 6900 2500
-Connection ~ 7200 1750
-Wire Wire Line
-	7200 1750 7200 1850
-Wire Wire Line
-	7200 2950 7200 3050
-Wire Wire Line
-	7200 3050 6900 3050
-Wire Wire Line
-	6900 3050 6900 2500
-Connection ~ 6900 2500
-Wire Wire Line
-	7200 3350 7200 3450
-Wire Wire Line
-	7200 3450 6900 3450
-Wire Wire Line
-	6900 3450 6900 3050
-Connection ~ 6900 3050
 $Comp
 L require:OP LP11
