File: hardware/wifi.sch (KiCad schematic (older format))
At the start: 21 parts, among them U1 ap6255, U2 AW2015FCR, Y1 Crystal_GND24, Y4 SG-3030CM

Commit message: wip
Connections:
- net labels added: UART_CTS, UART_RTS, UART_RXD, UART_TXD
Other:
- moved on the sheet: C3, C4, C9, Y4
