File: hardware/power.sch (KiCad schematic (older format))
At the start: 9 parts, among them U1 SY8088AAC

Commit message: wip
Parts:
- removed C1: 1u, Resistors_SMD:R_0402_NoSilk, symbol require-rescue:C
- removed C2200: 10uF,10V,X5R, Capacitors_SMD:C_0805, symbol require-rescue:C
- removed C2201: 22u, Resistors_SMD:R_0603, symbol require-rescue:C
- removed C2202: 0.1u, Resistors_SMD:R_0402_NoSilk, symbol require-rescue:C
- removed L1: 22uH, Inductors_SMD:L_Taiyo-Yuden_MD-4040, symbol require-rescue:L
- removed R111: 100,5%, Resistors_SMD:R_0402_NoSilk, symbol require-rescue:R
- removed R112: 10, Resistors_SMD:R_0402_NoSilk, symbol require-rescue:R
- removed R2200: 10k, Resistors_SMD:R_0402_NoSilk, symbol require-rescue:R
- removed U1: SY8088AAC, TO_SOT_Packages_SMD:SOT-23-5, symbol require-rescue:SY8088AAC
- added C16: 10uF,10V,X5R, Capacitors_SMD:C_0805, symbol require-rescue:C
- added C18: 1u, Resistors_SMD:R_0402_NoSilk, symbol require-rescue:C
- added C20: 22p, Resistors_SMD:R_0402_NoSilk, symbol require-rescue:C
- added C22: 22u, Resistors_SMD:R_0603, symbol require-rescue:C
- added C24: 0.1u, Resistors_SMD:R_0402_NoSilk, symbol require-rescue:C
- added L3: 3.3u, require:L_murata_2520, symbol Device:L
- added R10: 10, Resistors_SMD:R_0402_NoSilk, symbol require-rescue:R
- added R7: 10k, Resistors_SMD:R_0402_NoSilk, symbol require-rescue:R
- added R9: 100,5%, Resistors_SMD:R_0402_NoSilk, symbol require-rescue:R
- added U15: SY8088AAC, TO_SOT_Packages_SMD:SOT-23-5, symbol require:SY8088AAC
Connections:
- net labels added: VCC_IO
- net labels removed: VDD_CORE
- wire segments 20 -> 31

Commit message: wip
Parts:
- removed C16: 10uF,10V,X5R, Capacitors_SMD:C_0805, symbol require-rescue:C
- removed C18: 1u, Resistors_SMD:R_0402_NoSilk, symbol require-rescue:C
- removed C20: 22p, Resistors_SMD:R_0402_NoSilk, symbol require-rescue:C
- removed C22: 22u, Resistors_SMD:R_0603, symbol require-rescue:C
- removed C24: 0.1u, Resistors_SMD:R_0402_NoSilk, symbol require-rescue:C
- removed L3: 3.3u, require:L_murata_2520, symbol Device:L
- removed R10: 10, Resistors_SMD:R_0402_NoSilk, symbol require-rescue:R
- removed R7: 10k, Resistors_SMD:R_0402_NoSilk, symbol require-rescue:R
- removed R9: 100,5%, Resistors_SMD:R_0402_NoSilk, symbol require-rescue:R
- removed U15: SY8088AAC, TO_SOT_Packages_SMD:SOT-23-5, symbol require:SY8088AAC
- added C400: 0.1u,10V, Capacitors_SMD:C_0402, symbol require-rescue:C
- added C401: 10u,10V, Capacitors_SMD:C_0805, symbol require-rescue:C
- added C403: 22p, Capacitors_SMD:C_0402, symbol require-rescue:C
- added C404: 22u, Capacitors_SMD:C_0603, symbol require-rescue:C
- added L400: 2.2u, require:L_murata_2520, symbol require-rescue:L
- added R400: 10k, Resistors_SMD:R_0402, symbol require-rescue:R
- added R402: 110k,1%, Resistors_SMD:R_0402, symbol require-rescue:R
- added R403: 150k,1%, Resistors_SMD:R_0402, symbol require-rescue:R
- added U400: SY8089AAC, TO_SOT_Packages_SMD:SOT-23-5, symbol require:SY8089AAC
Connections:
- wire segments 31 -> 29
Other:
- note added: "Murata DFE252012R-H-2R2M#\n"

Commit message: wip
Parts:
- added C410, C413: 1u, Capacitors_SMD:C_0402, symbol require-rescue:C
- added FB400: L, Inductors_SMD:L_0603, symbol Device:L
- added R410: 10k, Resistors_SMD:R_0402, symbol require-rescue:R
- added R420, R421, R422, R425, R426: 0R, Resistors_SMD:R_0402, symbol Device:R
- added R423, R429: 1R, Resistors_SMD:R_0402, symbol Device:R
- added U410: LDO_1.8V_SOT_23_5, TO_SOT_Packages_SMD:SOT-23-5, symbol require:LDO_1.8V_SOT_23_5
Connections:
- net labels added: USB_VDD_1V8, VCCIO_FLASH, VCCIO_SDIO, VCCIO_SDMMC, VCC_1V8, VCC_1V8_CODEC, VCC_3V3_CODEC, VDD_1V0, VDD_LOG, VDD_USB_PLL_1V0
- wire segments 29 -> 73
Other:
- note added: "PT5108E23E-18, 500mA 1.8V LDO"
- note added: "Power Supply of arm core, cpu logic and ddr are drawn in corresponding pages."
- moved on the sheet: C400, C401, C403, C404, L400, R400, R402, R403, U400

Commit message: wip
Parts:
- removed R420, R421, R422, R425, R426: 0R, Resistors_SMD:R_0402, symbol Device:R
- removed R423, R429: 1R, Resistors_SMD:R_0402, symbol Device:R
- added C10, C32, C42: 22u, Capacitors_SMD:C_0603, symbol require-rescue:C
- added C11, C33, C43: 22p, Capacitors_SMD:C_0402, symbol require-rescue:C
- added C12, C30, C40: 0.1u,10V, Capacitors_SMD:C_0402, symbol require-rescue:C
- added C13, C31, C41: 10u,10V, Capacitors_SMD:C_0805, symbol require-rescue:C
- added C34: 0.1u, Capacitors_SMD:C_0402, symbol require-rescue:C
- added FB2: 180R,1.5A, Inductors_SMD:L_0402, symbol Device:L
- added L10, L30, L40: 2.2u, require:L_murata_2520, symbol require-rescue:L
- added R10, R31, R34, R40: 10k, Resistors_SMD:R_0402, symbol require-rescue:R
- added R11, R41: 110k,1%, Resistors_SMD:R_0402, symbol require-rescue:R
- added R12, R33, R42: 150k,1%, Resistors_SMD:R_0402, symbol require-rescue:R
- added R30: 100R,1%, Resistors_SMD:R_0402, symbol require-rescue:R
- added R32: 100k,1%, Resistors_SMD:R_0402, symbol require-rescue:R
- added R35: 10k,1%, Resistors_SMD:R_0402, symbol require-rescue:R
- added R36: 27k,1%, Resistors_SMD:R_0402, symbol require-rescue:R
- added R37: 12k,1%, Resistors_SMD:R_0402, symbol require-rescue:R
- added U10, U30, U40: SY8089AAC, TO_SOT_Packages_SMD:SOT-23-5, symbol require:SY8089AAC
- FB1: renamed from FB400; value L -> 180R,1.5A; footprint Inductors_SMD:L_0603 -> Inductors_SMD:L_0402
- renumbered C404 to C20, C403 to C21, C400 to C22, C401 to C23, C410 to C45, C413 to C46, L400 to L20, R400 to R20, R402 to R21, R403 to R22, R410 to R45, U400 to U20, U410 to U45
Connections:
- net labels added: AVDD_1V8, CORE_DVS, VCC_DDR, VDD_CORE
- net labels removed: USB_VDD_1V8, VCCIO_FLASH, VCCIO_SDIO, VCCIO_SDMMC, VCC_1V8_CODEC, VCC_3V3_CODEC, VDD_USB_PLL_1V0
- wire segments 73 -> 154
- no-connect marks 0 -> 1
Other:
- note added: "180 ohm @ 100MHz, 1.5A\nBLM15PX181SN1D (Tape)\nBLM15PX181SN1B (Bulk)"
- note added: "CORE"
- note added: "DDR3"
- note added: "IO 1V8"
- note added: "IO 3V3"
- note added: "LOGIC"
- note removed: "Power Supply of arm core, cpu logic and ddr are drawn in corresponding pages."
- moved on the sheet: C20, C21, C22, C23, C45, C46, FB1, L20, R20, R21, R22, R45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

Commit message: wip
Other:
- moved on the sheet: C10, C11, C12, C13, C20, C21, C22, C23, C32, C42, C43, C45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

Commit message: wip
Parts:
- added Q2: DTC143ZE_SOT523, require:SOT-523, symbol Transistor_FET:BSS138
Connections:
- net GND: now also Q2.2 (S)
- net at R31.1, U30.1 (EN): now also Q2.3 (D)
- new net POWER_SLEEP: Q2.1 (G)
Other:
- moved on the sheet: C30, C31, R31
Changed lines of the file:
@@
 L require-rescue:R R31
 U 1 1 5CCCBB3A
-P 2700 1500
+P 2400 1500
 AR Path="/5C2CD8AE/5CCCBB3A" Ref="R31"  Part="1"
 AR Path="/5C325762/5CCCBB3A" Ref="R?"  Part="1"
-F 0 "R31" V 2600 1500 50  0000 C CNN
-F 1 "10k" V 2800 1500 50  0000 C CNN
-F 2 "Resistors_SMD:R_0402" V 2630 1500 50  0001 C CNN
-F 3 "" H 2700 1500 50  0001 C CNN
-	1    2700 1500
+F 0 "R31" V 2300 1500 50  0000 C CNN
+F 1 "10k" V 2500 1500 50  0000 C CNN
+F 2 "Resistors_SMD:R_0402" V 2330 1500 50  0001 C CNN
+F 3 "" H 2400 1500 50  0001 C CNN
+	1    2400 1500
 	0    1    1    0
 $EndComp
@@
 L require-rescue:C C31
 U 1 1 5CCCBB50
-P 2150 1850
+P 1500 1850
 AR Path="/5C2CD8AE/5CCCBB50" Ref="C31"  Part="1"
 AR Path="/5C325762/5CCCBB50" Ref="C?"  Part="1"
-F 0 "C31" H 2250 1900 50  0000 L CNN
-F 1 "10u,10V" H 2250 1800 50  0000 L CNN
-F 2 "Capacitors_SMD:C_0805" H 2250 1700 50  0000 C CNN
-F 3 "" H 2150 1850 50  0001 C CNN
-F 4 "10V" H 2150 1850 60  0001 C CNN "Voltage"
-F 5 "X5R" H 2150 1850 60  0001 C CNN "Type"
-	1    2150 1850
+F 0 "C31" H 1600 1900 50  0000 L CNN
+F 1 "10u,10V" H 1600 1800 50  0000 L CNN
+F 2 "Capacitors_SMD:C_0805" H 1600 1700 50  0000 C CNN
+F 3 "" H 1500 1850 50  0001 C CNN
+F 4 "10V" H 1500 1850 60  0001 C CNN "Voltage"
+F 5 "X5R" H 1500 1850 60  0001 C CNN "Type"
+	1    1500 1850
 	1    0    0    -1
 $EndComp
@@
 L require-rescue:GND #PWR0182
 U 1 1 5CCCBB57
-P 2150 2200
+P 1500 2200
 AR Path="/5C2CD8AE/5CCCBB57" Ref="#PWR0182"  Part="1"
 AR Path="/5C325762/5CCCBB57" Ref="#PWR?"  Part="1"
-F 0 "#PWR0182" H 2150 1950 50  0001 C CNN
-F 1 "GND" H 2150 2050 50  0000 C CNN
-F 2 "" H 2150 2200 50  0001 C CNN
-F 3 "" H 2150 2200 50  0001 C CNN
-	1    2150 2200
+F 0 "#PWR0182" H 1500 1950 50  0001 C CNN
+F 1 "GND" H 1500 2050 50  0000 C CNN
+F 2 "" H 1500 2200 50  0001 C CNN
+F 3 "" H 1500 2200 50  0001 C CNN
+	1    1500 2200
 	1    0    0    -1
 $EndComp
@@
 Wire Wire Line
 	6200 1800 6200 2000
-Connection ~ 2150 1500
-Wire Wire Line
-	2150 2000 2150 2200
+Wire Wire Line
+	1500 2000 1500 2200
 $Comp
 L require-rescue:L L30
@@
 	4700 1300 5000 1300
 Wire Wire Line
-	2550 1500 2150 1500
-Wire Wire Line
-	2150 1300 2150 1500
+	2250 1500 2150 1500
 Wire Wire Line
 	5000 1300 5000 1500
@@
 $EndComp
 Wire Wire Line
-	2150 1500 2150 1700
-Wire Wire Line
 	5000 1800 5000 1950
 Connection ~ 5000 2200
@@
 	4200 1500 4550 1500
 Connection ~ 4550 2900
-Text HLabel 2150 3250 0    50   Input ~ 0
+Text HLabel 1900 3250 0    50   Input ~ 0
 CORE_DVS
 Wire Wire Line
-	2150 3250 2750 3250
+	1900 3250 2750 3250
 Connection ~ 2750 3250
 $Comp
 L require-rescue:C C?
 U 1 1 5CCCBBF6
-P 1400 1850
+P 950 1850
 AR Path="/5CCCBBF6" Ref="C?"  Part="1"
 AR Path="/5C2CD8AE/5CCCBBF6" Ref="C30"  Part="1"
 AR Path="/5C325762/5CCCBBF6" Ref="C?"  Part="1"
-F 0 "C30" H 1500 1900 50  0000 L CNN
-F 1 "0.1u,10V" H 1500 1800 50  0000 L CNN
-F 2 "Capacitors_SMD:C_0402" H 1438 1700 50  0001 C CNN
-F 3 "" H 1400 1850 50  0001 C CNN
-	1    1400 1850
+F 0 "C30" H 1050 1900 50  0000 L CNN
+F 1 "0.1u,10V" H 1050 1800 50  0000 L CNN
+F 2 "Capacitors_SMD:C_0402" H 988 1700 50  0001 C CNN
+F 3 "" H 950 1850 50  0001 C CNN
+	1    950  1850
 	1    0    0    -1
 $EndComp
@@
 L power:GND #PWR?
 U 1 1 5CCCBBFD
-P 1400 2200
+P 950 2200
 AR Path="/5C325762/5CCCBBFD" Ref="#PWR?"  Part="1"
 AR Path="/5C2CD8AE/5CCCBBFD" Ref="#PWR0188"  Part="1"
-F 0 "#PWR0188" H 1400 1950 50  0001 C CNN
-F 1 "GND" H 1405 2027 50  0000 C CNN
-F 2 "" H 1400 2200 50  0001 C CNN
-F 3 "" H 1400 2200 50  0001 C CNN
-	1    1400 2200
-	1    0    0    -1
-$EndComp
-Wire Wire Line
-	1400 2200 1400 2000
-Wire Wire Line
-	1400 1700 1400 1300
-Wire Wire Line
-	1400 1300 2150 1300
+F 0 "#PWR0188" H 950 1950 50  0001 C CNN
+F 1 "GND" H 955 2027 50  0000 C CNN
+F 2 "" H 950 2200 50  0001 C CNN
+F 3 "" H 950 2200 50  0001 C CNN
+	1    950  2200
+	1    0    0    -1
+$EndComp
+Wire Wire Line
+	950  2200 950  2000
+Wire Wire Line
+	950  1700 950  1300
+Wire Wire Line
+	950  1300 1500 1300
 Wire Wire Line
 	4350 3250 4550 3250
@@
 	2750 2650 2750 2750
 Wire Wire Line
-	2850 1500 3450 1500
+	2550 1500 2850 1500
 $Comp
 L require-rescue:VDD_CORE #PWR0189
@@
 Wire Wire Line
 	5000 9500 5000 9700
+$Comp
+L Transistor_FET:BSS138 Q2
+U 1 1 5C57C0E0
+P 2750 1850
+F 0 "Q2" H 2956 1896 50  0000 L CNN
+F 1 "DTC143ZE_SOT523" H 2956 1805 50  0000 L CNN
+F 2 "require:SOT-523" H 2950 1775 50  0001 L CIN
+F 3 "https://www.fairchildsemi.com/datasheets/BS/BSS138.pdf" H 2750 1850 50  0001 L CNN
+	1    2750 1850
+	1    0    0    -1
+$EndComp
+Wire Wire Line
+	1500 1700 1500 1300
+Connection ~ 1500 1300
+Wire Wire Line
+	1500 1300 2150 1300
+Wire Wire Line
+	2850 1650 2850 1500
+Connection ~ 2850 1500
+Wire Wire Line
+	2850 2050 2850 2200
+Wire Wire Line
+	2150 1850 2150 3000
+Wire Wire Line
+	2150 3000 1900 3000
+Text HLabel 1900 3000 0    50   Input ~ 0
+POWER_SLEEP
+Wire Wire Line
+	2150 1500 2150 1300
+$Comp
+L power:GND #PWR0231
+U 1 1 5C5FDC8C
+P 2850 2200
+F 0 "#PWR0231" H 2850 1950 50  0001 C CNN
+F 1 "GND" H 2855 2027 50  0000 C CNN
+F 2 "" H 2850 2200 50  0001 C CNN
+F 3 "" H 2850 2200 50  0001 C CNN
+	1    2850 2200
+	1    0    0    -1
+$EndComp
+Wire Wire Line
+	2850 1500 3450 1500
+Wire Wire Line
+	2150 1850 2550 1850
 $EndSCHEMATC
