File: hardware/power.sch (KiCad schematic (older format))
At the start: 49 parts, among them Q2 DTC143ZE_SOT523, U10 SY8089AAC, U20 SY8089AAC, U30 SY8089AAC, U40 SY8089AAC, U45 LDO_1.8V_SOT_23_5

Commit message: wip
Parts:
- C10, C20, C32, C42: footprint Capacitors_SMD:C_0603 -> require:C_0603
- C11, C12, C21, C22, C30, C33, C34, C40, C43, C45, C46: footprint Capacitors_SMD:C_0402 -> require:C_0402
- R10, R11, R12, R20, R21, R22, R30, R31, R32, R33, R34, R35, R36, R37, R40, R41, R42, R45: footprint Resistors_SMD:R_0402 -> require:R_0402
Changed lines of the file:
@@
 F 0 "R20" V 2600 9000 50  0000 C CNN
 F 1 "10k" V 2800 9000 50  0000 C CNN
-F 2 "Resistors_SMD:R_0402" V 2630 9000 50  0001 C CNN
+F 2 "require:R_0402" V 2630 9000 50  0001 C CNN
 F 3 "" H 2700 9000 50  0001 C CNN
 	1    2700 9000
@@
 F 0 "C20" H 6300 9200 50  0000 L CNN
 F 1 "22u" H 6300 9100 50  0000 L CNN
-F 2 "Capacitors_SMD:C_0603" H 6300 9000 50  0000 C CNN
+F 2 "require:C_0603" H 6300 9000 50  0000 C CNN
 F 3 "" H 6200 9150 50  0001 C CNN
 	1    6200 9150
@@
 F 0 "R21" H 5100 9200 50  0000 L CNN
 F 1 "110k,1%" H 5100 9100 50  0000 L CNN
-F 2 "Resistors_SMD:R_0402" V 4930 9150 50  0001 C CNN
+F 2 "require:R_0402" V 4930 9150 50  0001 C CNN
 F 3 "" H 5000 9150 50  0001 C CNN
 	1    5000 9150
@@
 F 0 "R22" H 5100 9900 50  0000 L CNN
 F 1 "150k,1%" H 5100 9800 50  0000 L CNN
-F 2 "Resistors_SMD:R_0402" V 4930 9850 50  0001 C CNN
+F 2 "require:R_0402" V 4930 9850 50  0001 C CNN
 F 3 "" H 5000 9850 50  0001 C CNN
 	1    5000 9850
@@
 F 0 "C21" H 5700 9200 50  0000 L CNN
 F 1 "22p" H 5700 9100 50  0000 L CNN
-F 2 "Capacitors_SMD:C_0402" H 5638 9000 50  0001 C CNN
+F 2 "require:C_0402" H 5638 9000 50  0001 C CNN
 F 3 "" H 5600 9150 50  0001 C CNN
 	1    5600 9150
@@
 F 0 "C22" H 1500 9400 50  0000 L CNN
 F 1 "0.1u,10V" H 1500 9300 50  0000 L CNN
-F 2 "Capacitors_SMD:C_0402" H 1438 9200 50  0001 C CNN
+F 2 "require:C_0402" H 1438 9200 50  0001 C CNN
 F 3 "" H 1400 9350 50  0001 C CNN
 	1    1400 9350
@@
 F 0 "C45" H 8050 1800 50  0000 L CNN
 F 1 "1u" H 8050 1700 50  0000 L CNN
-F 2 "Capacitors_SMD:C_0402" H 7988 1600 50  0001 C CNN
+F 2 "require:C_0402" H 7988 1600 50  0001 C CNN
 F 3 "" H 7950 1750 50  0001 C CNN
 	1    7950 1750
@@
 F 0 "R45" V 8100 1500 50  0000 C CNN
 F 1 "10k" V 8300 1500 50  0000 C CNN
-F 2 "Resistors_SMD:R_0402" V 8130 1500 50  0001 C CNN
+F 2 "require:R_0402" V 8130 1500 50  0001 C CNN
 F 3 "" H 8200 1500 50  0001 C CNN
 	1    8200 1500
@@
 F 0 "C46" H 10200 1800 50  0000 L CNN
 F 1 "1u" H 10200 1700 50  0000 L CNN
-F 2 "Capacitors_SMD:C_0402" H 10138 1600 50  0001 C CNN
+F 2 "require:C_0402" H 10138 1600 50  0001 C CNN
 F 3 "" H 10100 1750 50  0001 C CNN
 	1    10100 1750
@@
 F 0 "R31" V 2300 1500 50  0000 C CNN
 F 1 "10k" V 2500 1500 50  0000 C CNN
-F 2 "Resistors_SMD:R_0402" V 2330 1500 50  0001 C CNN
+F 2 "require:R_0402" V 2330 1500 50  0001 C CNN
 F 3 "" H 2400 1500 50  0001 C CNN
 	1    2400 1500
@@
 F 0 "C32" H 6300 1700 50  0000 L CNN
 F 1 "22u" H 6300 1600 50  0000 L CNN
-F 2 "Capacitors_SMD:C_0603" H 6300 1500 50  0000 C CNN
+F 2 "require:C_0603" H 6300 1500 50  0000 C CNN
 F 3 "" H 6200 1650 50  0001 C CNN
 	1    6200 1650
@@
 F 0 "R30" H 5100 1700 50  0000 L CNN
 F 1 "100R,1%" H 5100 1600 50  0000 L CNN
-F 2 "Resistors_SMD:R_0402" V 4930 1650 50  0001 C CNN
+F 2 "require:R_0402" V 4930 1650 50  0001 C CNN
 F 3 "" H 5000 1650 50  0001 C CNN
 	1    5000 1650
@@
 F 0 "R32" H 5100 2600 50  0000 L CNN
 F 1 "100k,1%" H 5100 2500 50  0000 L CNN
-F 2 "Resistors_SMD:R_0402" V 4930 2550 50  0001 C CNN
+F 2 "require:R_0402" V 4930 2550 50  0001 C CNN
 F 3 "" H 5000 2550 50  0001 C CNN
 	1    5000 2550
@@
 F 0 "R33" H 5100 3300 50  0000 L CNN
 F 1 "150k,1%" H 5100 3200 50  0000 L CNN
-F 2 "Resistors_SMD:R_0402" V 4930 3250 50  0001 C CNN
+F 2 "require:R_0402" V 4930 3250 50  0001 C CNN
 F 3 "" H 5000 3250 50  0001 C CNN
 	1    5000 3250
@@
 F 0 "C33" H 5700 2600 50  0000 L CNN
 F 1 "22p" H 5700 2500 50  0000 L CNN
-F 2 "Capacitors_SMD:C_0402" H 5638 2400 50  0001 C CNN
+F 2 "require:C_0402" H 5638 2400 50  0001 C CNN
 F 3 "" H 5600 2550 50  0001 C CNN
 	1    5600 2550
@@
 F 0 "R37" H 2850 2950 50  0000 L CNN
 F 1 "12k,1%" H 2850 2850 50  0000 L CNN
-F 2 "Resistors_SMD:R_0402" V 2680 2900 50  0001 C CNN
+F 2 "require:R_0402" V 2680 2900 50  0001 C CNN
 F 3 "" H 2750 2900 50  0001 C CNN
 	1    2750 2900
@@
 F 0 "R36" V 3000 3250 50  0000 C CNN
 F 1 "27k,1%" V 3200 3250 50  0000 C CNN
-F 2 "Resistors_SMD:R_0402" V 3030 3250 50  0001 C CNN
+F 2 "require:R_0402" V 3030 3250 50  0001 C CNN
 F 3 "" H 3100 3250 50  0001 C CNN
 	1    3100 3250
@@
 F 0 "R35" H 3550 3650 50  0000 L CNN
 F 1 "10k,1%" H 3550 3550 50  0000 L CNN
-F 2 "Resistors_SMD:R_0402" V 3380 3600 50  0001 C CNN
+F 2 "require:R_0402" V 3380 3600 50  0001 C CNN
 F 3 "" H 3450 3600 50  0001 C CNN
 	1    3450 3600
@@
 F 0 "C34" H 3950 3650 50  0000 L CNN
 F 1 "0.1u" H 3950 3550 50  0000 L CNN
-F 2 "Capacitors_SMD:C_0402" H 3888 3450 50  0001 C CNN
+F 2 "require:C_0402" H 3888 3450 50  0001 C CNN
 F 3 "" H 3850 3600 50  0001 C CNN
 	1    3850 3600
@@
 F 0 "R34" V 4100 3250 50  0000 C CNN
 F 1 "10k" V 4300 3250 50  0000 C CNN
-F 2 "Resistors_SMD:R_0402" V 4130 3250 50  0001 C CNN
+F 2 "require:R_0402" V 4130 3250 50  0001 C CNN
 F 3 "" H 4200 3250 50  0001 C CNN
 	1    4200 3250
@@
 F 0 "C30" H 1050 1900 50  0000 L CNN
 F 1 "0.1u,10V" H 1050 1800 50  0000 L CNN
-F 2 "Capacitors_SMD:C_0402" H 988 1700 50  0001 C CNN
+F 2 "require:C_0402" H 988 1700 50  0001 C CNN
 F 3 "" H 950 1850 50  0001 C CNN
 	1    950  1850
@@
 F 0 "R40" V 2600 4800 50  0000 C CNN
 F 1 "10k" V 2800 4800 50  0000 C CNN
-F 2 "Resistors_SMD:R_0402" V 2630 4800 50  0001 C CNN
+F 2 "require:R_0402" V 2630 4800 50  0001 C CNN
 F 3 "" H 2700 4800 50  0001 C CNN
 	1    2700 4800
@@
 F 0 "C42" H 6300 5000 50  0000 L CNN
 F 1 "22u" H 6300 4900 50  0000 L CNN
-F 2 "Capacitors_SMD:C_0603" H 6300 4800 50  0000 C CNN
+F 2 "require:C_0603" H 6300 4800 50  0000 C CNN
 F 3 "" H 6200 4950 50  0001 C CNN
 	1    6200 4950
@@
 F 0 "R41" H 5100 5000 50  0000 L CNN
 F 1 "110k,1%" H 5100 4900 50  0000 L CNN
-F 2 "Resistors_SMD:R_0402" V 4930 4950 50  0001 C CNN
+F 2 "require:R_0402" V 4930 4950 50  0001 C CNN
 F 3 "" H 5000 4950 50  0001 C CNN
 	1    5000 4950
@@
 F 0 "R42" H 5100 5700 50  0000 L CNN
 F 1 "150k,1%" H 5100 5600 50  0000 L CNN
-F 2 "Resistors_SMD:R_0402" V 4930 5650 50  0001 C CNN
+F 2 "require:R_0402" V 4930 5650 50  0001 C CNN
 F 3 "" H 5000 5650 50  0001 C CNN
 	1    5000 5650
@@
 F 0 "C43" H 5700 5000 50  0000 L CNN
 F 1 "22p" H 5700 4900 50  0000 L CNN
-F 2 "Capacitors_SMD:C_0402" H 5638 4800 50  0001 C CNN
+F 2 "require:C_0402" H 5638 4800 50  0001 C CNN
 F 3 "" H 5600 4950 50  0001 C CNN
 	1    5600 4950
@@
 F 0 "C40" H 1500 5200 50  0000 L CNN
 F 1 "0.1u,10V" H 1500 5100 50  0000 L CNN
-F 2 "Capacitors_SMD:C_0402" H 1438 5000 50  0001 C CNN
+F 2 "require:C_0402" H 1438 5000 50  0001 C CNN
 F 3 "" H 1400 5150 50  0001 C CNN
 	1    1400 5150
@@
 F 0 "R10" V 2600 6900 50  0000 C CNN
 F 1 "10k" V 2800 6900 50  0000 C CNN
-F 2 "Resistors_SMD:R_0402" V 2630 6900 50  0001 C CNN
+F 2 "require:R_0402" V 2630 6900 50  0001 C CNN
 F 3 "" H 2700 6900 50  0001 C CNN
 	1    2700 6900
@@
 F 0 "C10" H 6300 7100 50  0000 L CNN
 F 1 "22u" H 6300 7000 50  0000 L CNN
-F 2 "Capacitors_SMD:C_0603" H 6300 6900 50  0000 C CNN
+F 2 "require:C_0603" H 6300 6900 50  0000 C CNN
 F 3 "" H 6200 7050 50  0001 C CNN
 	1    6200 7050
@@
 F 0 "R11" H 5100 7100 50  0000 L CNN
 F 1 "110k,1%" H 5100 7000 50  0000 L CNN
-F 2 "Resistors_SMD:R_0402" V 4930 7050 50  0001 C CNN
+F 2 "require:R_0402" V 4930 7050 50  0001 C CNN
 F 3 "" H 5000 7050 50  0001 C CNN
 	1    5000 7050
@@
 F 0 "R12" H 5100 7800 50  0000 L CNN
 F 1 "150k,1%" H 5100 7700 50  0000 L CNN
-F 2 "Resistors_SMD:R_0402" V 4930 7750 50  0001 C CNN
+F 2 "require:R_0402" V 4930 7750 50  0001 C CNN
 F 3 "" H 5000 7750 50  0001 C CNN
 	1    5000 7750
@@
 F 0 "C11" H 5700 7100 50  0000 L CNN
 F 1 "22p" H 5700 7000 50  0000 L CNN
-F 2 "Capacitors_SMD:C_0402" H 5638 6900 50  0001 C CNN
+F 2 "require:C_0402" H 5638 6900 50  0001 C CNN
 F 3 "" H 5600 7050 50  0001 C CNN
 	1    5600 7050
@@
 F 0 "C12" H 1500 7300 50  0000 L CNN
 F 1 "0.1u,10V" H 1500 7200 50  0000 L CNN
-F 2 "Capacitors_SMD:C_0402" H 1438 7100 50  0001 C CNN
+F 2 "require:C_0402" H 1438 7100 50  0001 C CNN
 F 3 "" H 1400 7250 50  0001 C CNN
 	1    1400 7250

Commit message: wip
Parts:
- removed FB1, FB2: 180R,1.5A, Inductors_SMD:L_0402, symbol Device:L
- removed Q2: DTC143ZE_SOT523, require:SOT-523, symbol Transistor_FET:BSS138
- C18: renamed from C13; footprint Capacitors_SMD:C_0805 -> require:C_0805
- C23, C31, C41: footprint Capacitors_SMD:C_0805 -> require:C_0805
- renumbered C10 to C15, C11 to C16, C12 to C17, R21 to R10, R22 to R11, R10 to R4, R11 to R5, R12 to R6, R20 to R9, U10 to U6, U20 to U7
Connections:
- net labels added: +1V0C, +1V0L, +1V8, +3V3, +5V
- net labels removed: AVDD_1V8, POWER_SLEEP, VCC5V0_SYS, VCC_1V8, VCC_IO, VDD_1V0, VDD_CORE, VDD_LOG
- wire segments 158 -> 144
Other:
- note removed: "180 ohm @ 100MHz, 1.5A\nBLM15PX181SN1D (Tape)\nBLM15PX181SN1B (Bulk)"

Commit message: wip
Parts:
- removed C20: 22u, require:C_0603, symbol require-rescue:C
- removed C21: 22p, require:C_0402, symbol require-rescue:C
- removed C22: 0.1u,10V, require:C_0402, symbol require-rescue:C
- removed C23, C31, C41: 10u,10V, require:C_0805, symbol require-rescue:C
- removed L20: 2.2u, require:L_murata_2520, symbol require-rescue:L
- removed R10: 110k,1%, require:R_0402, symbol require-rescue:R
- removed R11: 150k,1%, require:R_0402, symbol require-rescue:R
- removed R9: 10k, require:R_0402, symbol require-rescue:R
- removed U7: SY8089AAC, TO_SOT_Packages_SMD:SOT-23-5, symbol require:SY8089AAC
- added C1912: 47uf,tant, Capacitors_Tantalum_SMD:CP_Tantalum_Case-B_EIA-3528-21_Reflow, symbol Device:C
- added C332: 22u, require:C_0805, symbol require-rescue:C
- C15, C32, C42: footprint require:C_0603 -> require:C_0805
- C18: footprint require:C_0805 -> require:C_0603
Connections:
- net labels added: +3.3V
- net labels removed: +5V
- wire segments 144 -> 118
Other:
- note removed: "IO 3V3"
- moved on the sheet: C18

Commit message: wip
Parts:
- removed C1912: 47uf,tant, Capacitors_Tantalum_SMD:CP_Tantalum_Case-B_EIA-3528-21_Reflow, symbol Device:C
- removed C30: 0.1u,10V, require:C_0402, symbol require-rescue:C
- removed C45, C46: 1u, require:C_0402, symbol require-rescue:C
- removed R31, R4, R40, R45: 10k, require:R_0402, symbol require-rescue:R
- removed U45: LDO_1.8V_SOT_23_5, TO_SOT_Packages_SMD:SOT-23-5, symbol require:LDO_1.8V_SOT_23_5
- added C188, C189, C190, C191: 22p, require:C_0402, symbol require-rescue:C
- added C200: 0.1u,10V, require:C_0402, symbol require-rescue:C
- added C267, C268: 10u,10V, require:C_0603, symbol require-rescue:C
- added C500, C501: 1u, require:C_0402, symbol require-rescue:C
- added L191: 2.2u, Inductors_SMD:L_0603, symbol require-rescue:L
- added R200: R, require:R_0402, symbol Device:R
- added U187: TPS62088_FIXED, require:TPS62088_DSBGA6, symbol require:TPS62088_FIXED
- added U500: NCP707_XDFN4, require:XDFN4, symbol require:NCP707_XDFN4
- C15, C32, C332, C42: footprint require:C_0805 -> require:C_0603
Connections:
- net labels added: +5V
- wire segments 118 -> 154
Other:
- note added: "Use TI TLV713 DQN"
- note removed: "IO 1V8"
- note removed: "PT5108E23E-18, 500mA 1.8V LDO"

Commit message: wip
Parts:
- C201: renamed from C267; value 10u,10V -> 10u
- C220: renamed from C40; value 0.1u,10V -> 0.1u
- C221: renamed from C18; value 10u,10V -> 10u
- C230: renamed from C17; value 0.1u,10V -> 0.1u
- C231: renamed from C268; value 10u,10V -> 10u
- renumbered C33 to C202, C32 to C203, C332 to C204, C34 to C210, C43 to C222, C42 to C223, C16 to C232, C15 to C233, C188 to C250, C189 to C251, C190 to C252, C191 to C253, C500 to C260, C501 to C261, L30 to L200, L40 to L220, L10 to L230, L191 to L250, R30 to R201, R32 to R202, R33 to R203, R34 to R210, R35 to R211, R36 to R212, R37 to R213, R41 to R222, R42 to R223, R5 to R232, R6 to R233, U30 to U200, U40 to U220, U6 to U230, U187 to U250, U500 to U260
Other:
- moved on the sheet: C221, C231, C260, C261, U260

Commit message: wip
Parts:
- removed C203, C204: 22u, require:C_0603, symbol require-rescue:C
- removed L250: 2.2u, Inductors_SMD:L_0603, symbol require-rescue:L
- added C203, C204: 22u, require:C_0603, symbol Device:C
- added C2551: 2.2u,10V, require:C_0402, symbol require-rescue:C
- added C2552: 2.2u, require:C_0402, symbol require-rescue:C
- added L250: 0.24u,3A, Inductors_SMD:L_0603, symbol Device:L
- added L255: 0.47u,3A, require:L_0806, symbol Device:L
- added U255: LM3281, require:LM3281_DSBGA6, symbol require:LM3281
- C200: value 0.1u,10V -> 0.1u; symbol require-rescue:C -> Device:C
- C202, C210, C222, C223, C233, C251: symbol require-rescue:C -> Device:C
- L200, L220, L230: symbol require-rescue:L -> Device:L
- R201, R202, R210, R211, R212, R213, R232, R233: symbol require-rescue:R -> Device:R
Connections:
- net +1V0C: now also C203.1, C204.1
- net +3V3: now also C2552.1, L250.2, L255.2, U255.A1 (FB)
- net +5V: now also C2551.1, U255.A2 (VIN), U255.C1 (EN)
- net GND: now also C203.2, C204.2, C2551.2, C2552.2, U255.B1 (MODE), U255.C2 (GND)
- net at U250.B2 (SW): now also L250.1
- new net: L255.1, U255.B2 (SW)
Changed lines of the file:
@@
-$EndComp
-$Comp
-L require-rescue:C C203
-U 1 1 5CCCBB41
-P 6200 1650
-AR Path="/5C2CD8AE/5CCCBB41" Ref="C203"  Part="1"
-AR Path="/5C325762/5CCCBB41" Ref="C?"  Part="1"
-F 0 "C203" H 6300 1700 50  0000 L CNN
-F 1 "22u" H 6300 1600 50  0000 L CNN
-F 2 "require:C_0603" H 6300 1500 50  0000 C CNN
-F 3 "" H 6200 1650 50  0001 C CNN
-	1    6200 1650
-	1    0    0    -1
 $EndComp
 $Comp
@@
 	6200 1800 6200 2000
 $Comp
-L require-rescue:L L200
+L Device:L L200
 U 1 1 5CCCBB64
 P 4550 1300
@@
 	6200 1300 6200 1500
 $Comp
-L require-rescue:R R201
+L Device:R R201
 U 1 1 5CCCBB6C
 P 5000 1650
@@
 $EndComp
 $Comp
-L require-rescue:R R202
+L Device:R R202
 U 1 1 5CCCBB73
 P 5000 2550
@@
 $EndComp
 $Comp
-L require-rescue:C C202
+L Device:C C202
 U 1 1 5CCCBB96
 P 5600 2550
@@
 	5600 1950 5600 1300
 $Comp
-L require-rescue:R R213
+L Device:R R213
 U 1 1 5CCCBBA2
 P 2750 2900
@@
 $EndComp
 $Comp
-L require-rescue:R R212
+L Device:R R212
 U 1 1 5CCCBBA9
 P 3100 3250
@@
 $EndComp
 $Comp
-L require-rescue:R R211
+L Device:R R211
 U 1 1 5CCCBBB0
 P 3450 3600
@@
 $EndComp
 $Comp
-L require-rescue:C C210
+L Device:C C210
 U 1 1 5CCCBBB7
 P 3850 3600
@@
 $EndComp
 $Comp
-L require-rescue:R R210
+L Device:R R210
 U 1 1 5CCCBBBE
 P 4200 3250
@@
 $EndComp
 $Comp
-L require-rescue:C C223
+L Device:C C223
 U 1 1 5CD09078
 P 6200 4950
@@
 	6200 5100 6200 5300
 $Comp
-L require-rescue:L L220
+L Device:L L220
 U 1 1 5CD0909B
 P 4550 4600
@@
 $EndComp
 $Comp
-L require-rescue:C C222
+L Device:C C222
 U 1 1 5CD090C4
 P 5600 4950
@@
 $EndComp
 $Comp
-L require-rescue:C C233
+L Device:C C233
 U 1 1 5CD9D5E0
 P 6200 7050
@@
 	6200 7200 6200 7400
 $Comp
-L require-rescue:L L230
+L Device:L L230
 U 1 1 5CD9D603
 P 4550 6700
@@
 	6200 6700 6200 6900
 $Comp
-L require-rescue:R R232
+L Device:R R232
 U 1 1 5CD9D60B
 P 5000 7050
@@
 Murata DFE252012R-H-2R2M#\n
 $Comp
-L require-rescue:R R233
+L Device:R R233
 U 1 1 5CD9D61E
 P 5000 7750
@@
 F 3 "" H 2150 6600 50  0001 C CNN
 	1    2150 6600
-	1    0    0    -1
-$EndComp
-$Comp
-L require-rescue:C C204
-U 1 1 5C673666
-P 6800 1650
-AR Path="/5C2CD8AE/5C673666" Ref="C204"  Part="1"
-AR Path="/5C325762/5C673666" Ref="C?"  Part="1"
-F 0 "C204" H 6900 1700 50  0000 L CNN
-F 1 "22u" H 6900 1600 50  0000 L CNN
-F 2 "require:C_0603" H 6900 1500 50  0000 C CNN
-F 3 "" H 6800 1650 50  0001 C CNN
-	1    6800 1650
 	1    0    0    -1
 $EndComp
@@
 $EndComp
 NoConn ~ 9350 4650
-$Comp
-L require-rescue:L L250
-U 1 1 5C65F0BE
-P 10300 4450
-AR Path="/5C2CD8AE/5C65F0BE" Ref="L250"  Part="1"
-AR Path="/5C325762/5C65F0BE" Ref="L?"  Part="1"
-F 0 "L250" V 10400 4450 50  0000 C CNN
-F 1 "2.2u" V 10500 4450 50  0000 C CNN
-F 2 "Inductors_SMD:L_0603" H 10300 4450 50  0001 C CNN
-F 3 "" H 10300 4450 50  0001 C CNN
-	1    10300 4450
-	0    -1   -1   0
-$EndComp
 Wire Wire Line
 	9950 4450 10150 4450
@@
 	10650 4550 10650 4450
 $Comp
-L require-rescue:C C251
+L Device:C C251
 U 1 1 5C66BA37
 P 10650 4800
@@
 	2150 4800 3450 4800
 $Comp
-L require-rescue:C C?
+L Device:C C?
 U 1 1 5C6C99C8
 P 950 1850
@@
 AR Path="/5C325762/5C6C99C8" Ref="C?"  Part="1"
 F 0 "C200" H 1050 1900 50  0000 L CNN
-F 1 "0.1u,10V" H 1050 1800 50  0000 L CNN
+F 1 "0.1u" H 1050 1800 50  0000 L CNN
 F 2 "require:C_0402" H 988 1700 50  0001 C CNN
 F 3 "" H 950 1850 50  0001 C CNN
@@
 Wire Wire Line
 	2150 7400 2150 7600
+$Comp
+L Device:L L250
+U 1 1 5C7C4941
+P 10300 4450
+AR Path="/5C2CD8AE/5C7C4941" Ref="L250"  Part="1"
+AR Path="/5C325762/5C7C4941" Ref="L?"  Part="1"
+AR Path="/5C2F0873/5C7C4941" Ref="L?"  Part="1"
+F 0 "L250" V 10400 4450 50  0000 C CNN
+F 1 "0.24u,3A" V 10500 4450 50  0000 C CNN
+F 2 "Inductors_SMD:L_0603" H 10300 4450 50  0001 C CNN
+F 3 "" H 10300 4450 50  0001 C CNN
+	1    10300 4450
+	0    -1   -1   0
+$EndComp
+$Comp
+L Device:C C203
+U 1 1 5C833838
+P 6200 1650
+AR Path="/5C2CD8AE/5C833838" Ref="C203"  Part="1"
+AR Path="/5C325762/5C833838" Ref="C?"  Part="1"
+F 0 "C203" H 6300 1700 50  0000 L CNN
+F 1 "22u" H 6300 1600 50  0000 L CNN
+F 2 "require:C_0603" H 6238 1500 50  0001 C CNN
+F 3 "" H 6200 1650 50  0001 C CNN
+	1    6200 1650
+	1    0    0    -1
+$EndComp
+$Comp
+L Device:C C204
+U 1 1 5C8338C6
+P 6800 1650
+AR Path="/5C2CD8AE/5C8338C6" Ref="C204"  Part="1"
+AR Path="/5C325762/5C8338C6" Ref="C?"  Part="1"
+F 0 "C204" H 6900 1700 50  0000 L CNN
+F 1 "22u" H 6900 1600 50  0000 L CNN
+F 2 "require:C_0603" H 6838 1500 50  0001 C CNN
+F 3 "" H 6800 1650 50  0001 C CNN
+	1    6800 1650
+	1    0    0    -1
+$EndComp
+$Comp
+L require:LM3281 U255
+U 1 1 5CA6F613
+P 9650 3050
+F 0 "U255" H 9650 3515 50  0000 C CNN
+F 1 "LM3281" H 9650 3424 50  0000 C CNN
+F 2 "require:LM3281_DSBGA6" H 9650 3050 50  0001 C CNN
+F 3 "" H 9650 3050 50  0001 C CNN
+	1    9650 3050
+	1    0    0    -1
+$EndComp
+$Comp
+L require-rescue:C C2551
+U 1 1 5CA6F70F
+P 8450 3100
+AR Path="/5C2CD8AE/5CA6F70F" Ref="C2551"  Part="1"
+AR Path="/5C325762/5CA6F70F" Ref="C?"  Part="1"
+F 0 "C2551" H 8550 3150 50  0000 L CNN
+F 1 "2.2u,10V" H 8550 3050 50  0000 L CNN
+F 2 "require:C_0402" H 8488 2950 50  0001 C CNN
+F 3 "" H 8450 3100 50  0001 C CNN
+	1    8450 3100
+	1    0    0    -1
+$EndComp
+Wire Wire Line
+	9250 2850 9150 2850
+Wire Wire Line
+	8450 2850 8450 2950
+Wire Wire Line
+	9250 2950 9150 2950
+Wire Wire Line
+	9150 2950 9150 2850
+Connection ~ 9150 2850
+Wire Wire Line
+	9150 2850 8450 2850
+Wire Wire Line
+	9250 3150 9150 3150
+Wire Wire Line
+	9150 3150 9150 3250
+Wire Wire Line
+	9150 3250 9250 3250
+Wire Wire Line
+	9150 3250 9150 3350
+Connection ~ 9150 3250
+$Comp
+L power:GND #PWR0232
+U 1 1 5CA8588D
+P 9150 3350
+F 0 "#PWR0232" H 9150 3100 50  0001 C CNN
+F 1 "GND" H 9155 3177 50  0000 C CNN
+F 2 "" H 9150 3350 50  0001 C CNN
+F 3 "" H 9150 3350 50  0001 C CNN
+	1    9150 3350
+	1    0    0    -1
+$EndComp
+Wire Wire Line
+	8450 3250 8450 3350
+$Comp
+L power:GND #PWR0242
+U 1 1 5CA8B6C8
+P 8450 3350
+F 0 "#PWR0242" H 8450 3100 50  0001 C CNN
+F 1 "GND" H 8455 3177 50  0000 C CNN
+F 2 "" H 8450 3350 50  0001 C CNN
+F 3 "" H 8450 3350 50  0001 C CNN
+	1    8450 3350
+	1    0    0    -1
+$EndComp
+$Comp
+L Device:L L255
+U 1 1 5CA8B856
+P 10300 2850
+AR Path="/5C2CD8AE/5CA8B856" Ref="L255"  Part="1"
+AR Path="/5C325762/5CA8B856" Ref="L?"  Part="1"
+AR Path="/5C2F0873/5CA8B856" Ref="L?"  Part="1"
+F 0 "L255" V 10400 2850 50  0000 C CNN
+F 1 "0.47u,3A" V 10500 2850 50  0000 C CNN
+F 2 "require:L_0806" H 10300 2850 50  0001 C CNN
+F 3 "" H 10300 2850 50  0001 C CNN
+	1    10300 2850
+	0    -1   -1   0
+$EndComp
+Wire Wire Line
+	10150 2850 10050 2850
+$Comp
+L require-rescue:C C2552
+U 1 1 5CA9189F
+P 10750 3100
+AR Path="/5C2CD8AE/5CA9189F" Ref="C2552"  Part="1"
+AR Path="/5C325762/5CA9189F" Ref="C?"  Part="1"
+F 0 "C2552" H 10850 3150 50  0000 L CNN
+F 1 "2.2u" H 10850 3050 50  0000 L CNN
+F 2 "require:C_0402" H 10788 2950 50  0001 C CNN
+F 3 "" H 10750 3100 50  0001 C CNN
+	1    10750 3100
+	1    0    0    -1
+$EndComp
+Wire Wire Line
+	10750 2850 10750 2950
+Wire Wire Line
+	10750 3250 10750 3350
+$Comp
+L power:GND #PWR0243
+U 1 1 5CA9D83E
+P 10750 3350
+F 0 "#PWR0243" H 10750 3100 50  0001 C CNN
+F 1 "GND" H 10755 3177 50  0000 C CNN
+F 2 "" H 10750 3350 50  0001 C CNN
+F 3 "" H 10750 3350 50  0001 C CNN
+	1    10750 3350
+	1    0    0    -1
+$EndComp
+Wire Wire Line
+	10450 2850 10550 2850
+Wire Wire Line
+	10550 2850 10550 3100
+Wire Wire Line
+	10550 3100 10300 3100
+Wire Wire Line
+	10300 3100 10300 3250
+Wire Wire Line
+	10300 3250 10050 3250
+Connection ~ 10550 2850
+Wire Wire Line
+	10550 2850 10750 2850
+$Comp
+L power:+5V #PWR?
+U 1 1 5CABF137
+P 8450 2750
+F 0 "#PWR?" H 8450 2600 50  0001 C CNN
+F 1 "+5V" H 8465 2923 50  0000 C CNN
+F 2 "" H 8450 2750 50  0001 C CNN
+F 3 "" H 8450 2750 50  0001 C CNN
+	1    8450 2750
+	1    0    0    -1
+$EndComp
+Wire Wire Line
+	8450 2750 8450 2850
+Connection ~ 8450 2850
+$Comp
+L power:+3V3 #PWR?
+U 1 1 5CAC5ACB
+P 10750 2750
+F 0 "#PWR?" H 10750 2600 50  0001 C CNN
+F 1 "+3V3" H 10765 2923 50  0000 C CNN
+F 2 "" H 10750 2750 50  0001 C CNN
+F 3 "" H 10750 2750 50  0001 C CNN
+	1    10750 2750
+	1    0    0    -1
+$EndComp
+Wire Wire Line
+	10750 2750 10750 2850
+Connection ~ 10750 2850
 $EndSCHEMATC

Commit message: wip
Parts:
- removed C250, C252, C253: 22p, require:C_0402, symbol require-rescue:C
- removed C251: 22p, require:C_0402, symbol Device:C
- removed L250: 0.24u,3A, Inductors_SMD:L_0603, symbol Device:L
- removed U250: TPS62088_FIXED, require:TPS62088_DSBGA6, symbol require:TPS62088_FIXED
- removed U255: LM3281, require:LM3281_DSBGA6, symbol require:LM3281
- added U255: PAM2305CGFADJ, require:U-DFN2020-6, symbol Regulator_Switching:PAM2305CGFADJ
- C2551, C2552: footprint require:C_0402 -> require:C_0603
Connections:
- net +5V: now also U255.2 (EN), U255.3 (Vin)
- net GND: now also U255.5 (GND), U255.7 (PAD)
- net at L255.1: now also U255.4 (SW)
Other:
- moved on the sheet: C2551, C2552, L255
