File: hardware/power.sch (KiCad schematic (older format))
At the start: 39 parts, among them U200 SY8089AAC, U220 SY8089AAC, U230 SY8089AAC, U255 PAM2305CGFADJ, U260 NCP707_XDFN4

Commit message: wip
Parts:
- removed C220, C230: 0.1u, require:C_0402, symbol require-rescue:C
- removed C232: 22p, require:C_0402, symbol require-rescue:C
- removed C2552: 2.2u, require:C_0603, symbol require-rescue:C
- removed R200: R, require:R_0402, symbol Device:R
- removed R232: 110k,1%, require:R_0402, symbol Device:R
- removed R233: 150k,1%, require:R_0402, symbol Device:R
- removed U220, U230: SY8089AAC, TO_SOT_Packages_SMD:SOT-23-5, symbol require:SY8089AAC
- added C232, C252: 22p, require:C_0402, symbol Device:C
- added C253: 22u, require:C_0603, symbol Device:C
- added R232, R252: 110k,1%, require:R_0402, symbol require-rescue:R
- added R233, R253: 150k,1%, require:R_0402, symbol require-rescue:R
- added U220, U230: PAM2305CGFADJ, require:U-DFN2020-6, symbol Regulator_Switching:PAM2305CGFADJ
- L220, L230: value 2.2u -> 0.47u,3A; footprint require:L_murata_2520 -> require:L_0806
- renumbered C2551 to C251, L255 to L250, U255 to U250
Connections:
- net +3V3: now also C252.1, C253.1, R252.1; no longer C200.1, C201.1, C221.1, C231.1, U200.4 (VIN)
- net +5V: now also C200.1, C201.1, C221.1, C231.1, U200.1 (EN), U200.4 (VIN), U220.2 (EN), U220.3 (Vin), U230.2 (EN), U230.3 (Vin)
- net GND: now also C253.2, R233.2, R253.2, U220.5 (GND), U220.7 (PAD), U230.5 (GND), U230.7 (PAD)
- net VCC_DDR: now also C232.1, R232.1
- net at U250.6 (FB): now also C252.2, R252.2, R253.1
- net at L220.1: now also U220.4 (SW)
- net at C222.2, R222.2, R223.1: now also U220.6 (FB)
- net at L230.1: now also U230.4 (SW)
- new net: C232.2, R232.2, R233.1, U230.6 (FB)
- no-connect marks 1 -> 0
Other:
- note removed: "DDR3"
- note removed: "LOGIC"
- moved on the sheet: C221, C222, C223, C231, C260, C261, R222, R223
