File: hardware/rk3308-power.sch (KiCad schematic (older format))
At the start: 1 part, among them U1000 RK3308

Commit message: wip
Parts:
- added C100, C200: 0.1u,10V, Capacitors_SMD:C_0402, symbol require-rescue:C
- added C101, C201: 10u,10V, Capacitors_SMD:C_0805, symbol require-rescue:C
- added C102, C202: 1n, Capacitors_SMD:C_0402, symbol require-rescue:C
- added C103, C203: 22p, Capacitors_SMD:C_0402, symbol require-rescue:C
- added C104, C204: 22u, Capacitors_SMD:C_0603, symbol require-rescue:C
- added C105, C106, C107, C108, C110, C205, C207, C208: 0.1u, Capacitors_SMD:C_0402, symbol require-rescue:C
- added C1102: 0.1u, Capacitors_SMD:C_0402, symbol Device:C
- added C206: 10u, Capacitors_SMD:C_0603, symbol require-rescue:C
- added L100, L200: 2.2u, require:L_murata_2520, symbol require-rescue:L
- added R100, R110, R200: 10k, Resistors_SMD:R_0402, symbol require-rescue:R
- added R101: 100R,1%, Resistors_SMD:R_0402, symbol require-rescue:R
- added R102: 100k,1%, Resistors_SMD:R_0402, symbol require-rescue:R
- added R103, R203: 150k,1%, Resistors_SMD:R_0402, symbol require-rescue:R
- added R111: 10k,1%, Resistors_SMD:R_0402, symbol require-rescue:R
- added R112: 27k,1%, Resistors_SMD:R_0402, symbol require-rescue:R
- added R113: 12k,1%, Resistors_SMD:R_0402, symbol require-rescue:R
- added R202: 110k,1%, Resistors_SMD:R_0402, symbol require-rescue:R
- added U100, U200: SY8089AAC, TO_SOT_Packages_SMD:SOT-23-5, symbol require:SY8089AAC
- added unit 1 of U1000
- added Y1: Crystal_GND24, Crystals:Crystal_SMD_3225-4pin_3.2x2.5mm, symbol Device:Crystal_GND24
Connections:
- net labels added: CORE_DVS, RESET, VCC5V0_SYS, VCC_IO, VDD_CORE, VDD_LOG
- wire segments 212 -> 369
- no-connect marks 0 -> 1
Other:
- note added: "Close to chip"
- note added: "Murata DFE252012R-H-2R2M#\n"
- moved on the sheet: U1000L, U1000M, U1000N

Commit message: wip
Parts:
- removed C102, C202: 1n, Capacitors_SMD:C_0402, symbol require-rescue:C
- removed C205: 0.1u, Capacitors_SMD:C_0402, symbol require-rescue:C
- C107: value 0.1u -> 2.2u
- C108: value 0.1u -> 22u; footprint Capacitors_SMD:C_0402 -> Capacitors_SMD:C_0603
Connections:
- wire segments 369 -> 362
Other:
- moved on the sheet: C105, C106, C107, C108, C1102, C206, C207, C208, U1000A, U1000L, Y1

Commit message: wip
Parts:
- added C220, C221: 15p, Capacitors_SMD:C_0402, symbol Device:C
- added C230, C231: 0.1u, Capacitors_SMD:C_0402, symbol Device:C
- added R220: 22R, Resistors_SMD:R_0402, symbol require-rescue:R
- added R230: 1R, Resistors_SMD:R_0402, symbol require-rescue:R
- renumbered C1102 to C225, Y1 to Y220
Connections:
- net labels added: VCC_1V8, VDD_1V0
- wire segments 362 -> 383
Changed lines of the file:
@@
 $EndComp
 $Comp
-L Device:Crystal_GND24 Y1
+L Device:Crystal_GND24 Y220
 U 1 1 5D440CD1
 P 8700 5200
-F 0 "Y1" H 8891 5246 50  0000 L CNN
+F 0 "Y220" H 8891 5246 50  0000 L CNN
 F 1 "Crystal_GND24" H 8891 5155 50  0000 L CNN
 F 2 "Crystals:Crystal_SMD_3225-4pin_3.2x2.5mm" H 8700 5200 50  0001 C CNN
@@
 $EndComp
 Wire Wire Line
-	8050 5200 8550 5200
-Wire Wire Line
 	8050 5600 8250 5600
 Wire Wire Line
@@
 RESET
 $Comp
-L Device:C C1102
+L Device:C C225
 U 1 1 5C42AEFD
 P 9050 6350
-F 0 "C1102" H 9165 6396 50  0000 L CNN
+F 0 "C225" H 9165 6396 50  0000 L CNN
 F 1 "0.1u" H 9165 6305 50  0000 L CNN
 F 2 "Capacitors_SMD:C_0402" H 9088 6200 50  0001 C CNN
@@
 	8650 1750 8250 1750
 Connection ~ 8650 1750
+$Comp
+L require-rescue:R R?
+U 1 1 5C745F21
+P 8300 5200
+AR Path="/5C2CD8AE/5C745F21" Ref="R?"  Part="1"
+AR Path="/5C325762/5C745F21" Ref="R220"  Part="1"
+F 0 "R220" V 8200 5200 50  0000 C CNN
+F 1 "22R" V 8400 5200 50  0000 C CNN
+F 2 "Resistors_SMD:R_0402" V 8230 5200 50  0001 C CNN
+F 3 "" H 8300 5200 50  0001 C CNN
+	1    8300 5200
+	0    1    1    0
+$EndComp
+Wire Wire Line
+	8150 5200 8050 5200
+Wire Wire Line
+	8450 5200 8500 5200
+$Comp
+L Device:C C220
+U 1 1 5C7967A1
+P 8100 4450
+F 0 "C220" H 8215 4496 50  0000 L CNN
+F 1 "15p" H 8215 4405 50  0000 L CNN
+F 2 "Capacitors_SMD:C_0402" H 8138 4300 50  0001 C CNN
+F 3 "~" H 8100 4450 50  0001 C CNN
+	1    8100 4450
+	1    0    0    -1
+$EndComp
+Wire Wire Line
+	8100 4300 8100 4100
+Wire Wire Line
+	8100 4100 8500 4100
+Wire Wire Line
+	8500 4100 8500 5200
+Connection ~ 8500 5200
+Wire Wire Line
+	8500 5200 8550 5200
+$Comp
+L power:GND #PWR0200
+U 1 1 5C7BF779
+P 8100 4700
+F 0 "#PWR0200" H 8100 4450 50  0001 C CNN
+F 1 "GND" H 8105 4527 50  0000 C CNN
+F 2 "" H 8100 4700 50  0001 C CNN
+F 3 "" H 8100 4700 50  0001 C CNN
+	1    8100 4700
+	1    0    0    -1
+$EndComp
+Wire Wire Line
+	8100 4600 8100 4700
+$Comp
+L Device:C C221
+U 1 1 5C7EA32C
+P 9850 5550
+F 0 "C221" H 9965 5596 50  0000 L CNN
+F 1 "15p" H 9965 5505 50  0000 L CNN
+F 2 "Capacitors_SMD:C_0402" H 9888 5400 50  0001 C CNN
+F 3 "~" H 9850 5550 50  0001 C CNN
+	1    9850 5550
+	1    0    0    -1
+$EndComp
+Wire Wire Line
+	9650 5200 9850 5200
+Wire Wire Line
+	9850 5200 9850 5400
+Connection ~ 9650 5200
+$Comp
+L power:GND #PWR0201
+U 1 1 5C813FE0
+P 9850 5900
+F 0 "#PWR0201" H 9850 5650 50  0001 C CNN
+F 1 "GND" H 9855 5727 50  0000 C CNN
+F 2 "" H 9850 5900 50  0001 C CNN
+F 3 "" H 9850 5900 50  0001 C CNN
+	1    9850 5900
+	1    0    0    -1
+$EndComp
+Wire Wire Line
+	9850 5700 9850 5900
+$Comp
+L require-rescue:R R?
+U 1 1 5C84B849
+P 10150 7000
+AR Path="/5C2CD8AE/5C84B849" Ref="R?"  Part="1"
+AR Path="/5C325762/5C84B849" Ref="R230"  Part="1"
+F 0 "R230" V 10050 7000 50  0000 C CNN
+F 1 "1R" V 10250 7000 50  0000 C CNN
+F 2 "Resistors_SMD:R_0402" V 10080 7000 50  0001 C CNN
+F 3 "" H 10150 7000 50  0001 C CNN
+	1    10150 7000
+	0    1    1    0
+$EndComp
+$Comp
+L Device:C C230
+U 1 1 5C84BC04
+P 9900 7300
+F 0 "C230" H 10015 7346 50  0000 L CNN
+F 1 "0.1u" H 10015 7255 50  0000 L CNN
+F 2 "Capacitors_SMD:C_0402" H 9938 7150 50  0001 C CNN
+F 3 "~" H 9900 7300 50  0001 C CNN
+	1    9900 7300
+	1    0    0    -1
+$EndComp
+Wire Wire Line
+	9900 7150 9900 7000
+Connection ~ 9900 7000
+Wire Wire Line
+	9900 7000 10000 7000
+Wire Wire Line
+	10300 7000 10500 7000
+Wire Wire Line
+	10500 7000 10500 6900
+$Comp
+L require:VDD_1V0 #PWR0202
+U 1 1 5C8CB6DB
+P 10500 6900
+F 0 "#PWR0202" H 10500 6750 50  0001 C CNN
+F 1 "VDD_1V0" H 10517 7073 50  0000 C CNN
+F 2 "" H 10500 6900 50  0001 C CNN
+F 3 "" H 10500 6900 50  0001 C CNN
+	1    10500 6900
+	1    0    0    -1
+$EndComp
+Wire Wire Line
+	8050 7000 9900 7000
+Wire Wire Line
+	9900 7450 9900 7650
+$Comp
+L power:GND #PWR0203
+U 1 1 5C9782CF
+P 9900 7650
+F 0 "#PWR0203" H 9900 7400 50  0001 C CNN
+F 1 "GND" H 9905 7477 50  0000 C CNN
+F 2 "" H 9900 7650 50  0001 C CNN
+F 3 "" H 9900 7650 50  0001 C CNN
+	1    9900 7650
+	1    0    0    -1
+$EndComp
+Wire Wire Line
+	8050 7200 8650 7200
+Wire Wire Line
+	8650 7200 8650 7500
+Wire Wire Line
+	8650 7500 9100 7500
+Wire Wire Line
+	9100 7500 9100 7400
+$Comp
+L require:VCC_1V8 #PWR0204
+U 1 1 5C9A4743
+P 9100 7400
+F 0 "#PWR0204" H 9100 7250 50  0001 C CNN
+F 1 "VCC_1V8" H 9117 7573 50  0000 C CNN
+F 2 "" H 9100 7400 50  0001 C CNN
+F 3 "" H 9100 7400 50  0001 C CNN
+	1    9100 7400
+	1    0    0    -1
+$EndComp
+$Comp
+L Device:C C231
+U 1 1 5C9A47A9
+P 8650 7850
+F 0 "C231" H 8765 7896 50  0000 L CNN
+F 1 "0.1u" H 8765 7805 50  0000 L CNN
+F 2 "Capacitors_SMD:C_0402" H 8688 7700 50  0001 C CNN
+F 3 "~" H 8650 7850 50  0001 C CNN
+	1    8650 7850
+	1    0    0    -1
+$EndComp
+Wire Wire Line
+	8650 7500 8650 7700
+Connection ~ 8650 7500
+Wire Wire Line
+	8650 8000 8650 8200
+$Comp
+L power:GND #PWR0205
+U 1 1 5C9FD96A
+P 8650 8200
+F 0 "#PWR0205" H 8650 7950 50  0001 C CNN
+F 1 "GND" H 8655 8027 50  0000 C CNN
+F 2 "" H 8650 8200 50  0001 C CNN
+F 3 "" H 8650 8200 50  0001 C CNN
+	1    8650 8200
+	1    0    0    -1
+$EndComp
 $EndSCHEMATC

Commit message: wip
Parts:
- removed C100, C200: 0.1u,10V, Capacitors_SMD:C_0402, symbol require-rescue:C
- removed C101, C201: 10u,10V, Capacitors_SMD:C_0805, symbol require-rescue:C
- removed C103, C203: 22p, Capacitors_SMD:C_0402, symbol require-rescue:C
- removed C104, C204: 22u, Capacitors_SMD:C_0603, symbol require-rescue:C
- removed C110, C208: 0.1u, Capacitors_SMD:C_0402, symbol require-rescue:C
- removed L100, L200: 2.2u, require:L_murata_2520, symbol require-rescue:L
- removed R100, R110, R200: 10k, Resistors_SMD:R_0402, symbol require-rescue:R
- removed R101: 100R,1%, Resistors_SMD:R_0402, symbol require-rescue:R
- removed R102: 100k,1%, Resistors_SMD:R_0402, symbol require-rescue:R
- removed R103, R203: 150k,1%, Resistors_SMD:R_0402, symbol require-rescue:R
- removed R111: 10k,1%, Resistors_SMD:R_0402, symbol require-rescue:R
- removed R112: 27k,1%, Resistors_SMD:R_0402, symbol require-rescue:R
- removed R113: 12k,1%, Resistors_SMD:R_0402, symbol require-rescue:R
- removed R202: 110k,1%, Resistors_SMD:R_0402, symbol require-rescue:R
- removed R230: 1R, Resistors_SMD:R_0402, symbol require-rescue:R
- removed U100, U200: SY8089AAC, TO_SOT_Packages_SMD:SOT-23-5, symbol require:SY8089AAC
- added R92, R987: 10k, Resistors_SMD:R_0402, symbol Device:R
- added SW1: SW_Push, require:HYP_1TS003A_SIDE_PUSH, symbol Switch:SW_Push
- added unit 10 of U1000
- renumbered C108 to C70, C105 to C71, C106 to C72, C107 to C73, C207 to C77, C206 to C78, C231 to C84, C230 to C86, C225 to C88, C221 to C90, C220 to C91, R220 to R91, Y220 to Y2
Connections:
- net labels added: A0, A1, A2, A3, A4, A5
- net labels removed: CORE_DVS, VCC5V0_SYS, VCC_IO
- wire segments 383 -> 323
Other:
- note added: "Share capacitor with E17"
- note removed: "Murata DFE252012R-H-2R2M#\n"
- moved on the sheet: C84, C86, C88, C90, C91, R91, U1000A, Y2

Commit message: wip
Parts:
- removed R987: 10k, Resistors_SMD:R_0402, symbol Device:R
- removed SW1: SW_Push, require:HYP_1TS003A_SIDE_PUSH, symbol Switch:SW_Push
- added LP14: RST, require:OVAL_PIN, symbol require:OP
- added LP2: A0, require:OVAL_PIN, symbol require:OP
- added LP3: A1, require:OVAL_PIN, symbol require:OP
- added LP4: A2, require:OVAL_PIN, symbol require:OP
- added LP5: A3, require:OVAL_PIN, symbol require:OP
- added LP6: A4, require:OVAL_PIN, symbol require:OP
- added LP7: A5, require:OVAL_PIN, symbol require:OP
- added Q1: BSS138, TO_SOT_Packages_SMD:SOT-23, symbol Transistor_FET:BSS138
- added R435: 10k, Resistors_SMD:R_0402, symbol Device:R
- added SW1: SW_SKSC_4PIN, require:SW_ALPS_SKSC, symbol require:SW_SKSC_4PIN
Connections:
- net labels added: VCC_IO
- wire segments 323 -> 339
Changed lines of the file:
@@
 $Descr A3 16535 11693
 encoding utf-8
-Sheet 5 9
+Sheet 5 10
 Title ""
 Date ""
@@
 	5650 6850 5650 6600
 Wire Wire Line
-	5650 6300 5650 6050
+	5650 6300 5650 6150
 $Comp
 L require:VCC_1V8 #PWR0219
@@
 Wire Wire Line
 	3000 2000 3450 2000
-Wire Wire Line
-	3000 2100 3450 2100
 Wire Wire Line
 	3000 2200 3450 2200
@@
 Text Label 3050 2400 0    50   ~ 0
 A5
-$Comp
-L Switch:SW_Push SW1
-U 1 1 5D1A103C
-P 6700 6850
-F 0 "SW1" H 6700 7135 50  0000 C CNN
-F 1 "SW_Push" H 6700 7044 50  0000 C CNN
-F 2 "require:HYP_1TS003A_SIDE_PUSH" H 6700 7050 50  0001 C CNN
-F 3 "" H 6700 7050 50  0001 C CNN
-	1    6700 6850
-	1    0    0    -1
-$EndComp
-$Comp
-L Device:R R987
-U 1 1 5D1A1230
-P 6050 6850
-F 0 "R987" H 6120 6896 50  0000 L CNN
-F 1 "10k" H 6120 6805 50  0000 L CNN
-F 2 "Resistors_SMD:R_0402" V 5980 6850 50  0001 C CNN
-F 3 "~" H 6050 6850 50  0001 C CNN
-	1    6050 6850
-	0    1    1    0
-$EndComp
-Wire Wire Line
-	6200 6850 6500 6850
-Wire Wire Line
-	5900 6850 5650 6850
 Connection ~ 5650 6850
-Wire Wire Line
-	6900 6850 7150 6850
-Wire Wire Line
-	7150 6850 7150 7100
 $Comp
 L power:GND #PWR0223
 U 1 1 5D1FE16C
-P 7150 7100
-F 0 "#PWR0223" H 7150 6850 50  0001 C CNN
-F 1 "GND" H 7155 6927 50  0000 C CNN
-F 2 "" H 7150 7100 50  0001 C CNN
-F 3 "" H 7150 7100 50  0001 C CNN
-	1    7150 7100
-	1    0    0    -1
-$EndComp
+P 7750 7400
+F 0 "#PWR0223" H 7750 7150 50  0001 C CNN
+F 1 "GND" H 7755 7227 50  0000 C CNN
+F 2 "" H 7750 7400 50  0001 C CNN
+F 3 "" H 7750 7400 50  0001 C CNN
+	1    7750 7400
+	1    0    0    -1
+$EndComp
+$Comp
+L require:OP LP2
+U 1 1 5C4D0C91
+P 3650 1900
+F 0 "LP2" H 3850 1900 50  0000 C CNN
+F 1 "A0" H 3650 1900 50  0000 C CNN
+F 2 "require:OVAL_PIN" H 3650 1900 50  0001 C CNN
+F 3 "" H 3650 1900 50  0001 C CNN
+	1    3650 1900
+	1    0    0    -1
+$EndComp
+$Comp
+L require:OP LP3
+U 1 1 5C4AB65C
+P 3650 2000
+F 0 "LP3" H 3850 2000 50  0000 C CNN
+F 1 "A1" H 3650 2000 50  0000 C CNN
+F 2 "require:OVAL_PIN" H 3650 2000 50  0001 C CNN
+F 3 "" H 3650 2000 50  0001 C CNN
+	1    3650 2000
+	1    0    0    -1
+$EndComp
+Wire Wire Line
+	3000 2100 3450 2100
+$Comp
+L require:OP LP4
+U 1 1 5C4EC7BD
+P 3650 2100
+F 0 "LP4" H 3850 2100 50  0000 C CNN
+F 1 "A2" H 3650 2100 50  0000 C CNN
+F 2 "require:OVAL_PIN" H 3650 2100 50  0001 C CNN
+F 3 "" H 3650 2100 50  0001 C CNN
+	1    3650 2100
+	1    0    0    -1
+$EndComp
+$Comp
+L require:OP LP5
+U 1 1 5C4EE56F
+P 3650 2200
+F 0 "LP5" H 3850 2200 50  0000 C CNN
+F 1 "A3" H 3650 2200 50  0000 C CNN
+F 2 "require:OVAL_PIN" H 3650 2200 50  0001 C CNN
+F 3 "" H 3650 2200 50  0001 C CNN
+	1    3650 2200
+	1    0    0    -1
+$EndComp
+$Comp
+L require:OP LP6
+U 1 1 5C4EE5D7
+P 3650 2300
+F 0 "LP6" H 3850 2300 50  0000 C CNN
+F 1 "A4" H 3650 2300 50  0000 C CNN
+F 2 "require:OVAL_PIN" H 3650 2300 50  0001 C CNN
+F 3 "" H 3650 2300 50  0001 C CNN
+	1    3650 2300
+	1    0    0    -1
+$EndComp
+$Comp
+L require:OP LP7
+U 1 1 5C4EE61B
+P 3650 2400
+F 0 "LP7" H 3850 2400 50  0000 C CNN
+F 1 "A5" H 3650 2400 50  0000 C CNN
+F 2 "require:OVAL_PIN" H 3650 2400 50  0001 C CNN
+F 3 "" H 3650 2400 50  0001 C CNN
+	1    3650 2400
+	1    0    0    -1
+$EndComp
+$Comp
+L require:SW_SKSC_4PIN SW1
+U 1 1 5C4B7DD5
+P 8300 6900
+F 0 "SW1" H 8300 7215 50  0000 C CNN
+F 1 "SW_SKSC_4PIN" H 8300 7124 50  0000 C CNN
+F 2 "require:SW_ALPS_SKSC" H 8300 6900 50  0001 C CNN
+F 3 "" H 8300 6900 50  0001 C CNN
+	1    8300 6900
+	1    0    0    -1
+$EndComp
+Wire Wire Line
+	8700 6850 8850 6850
+Wire Wire Line
+	8850 6850 8850 6500
+Wire Wire Line
+	8850 6500 7750 6500
+Wire Wire Line
+	7750 6500 7750 6850
+Wire Wire Line
+	7750 6850 7900 6850
+$Comp
+L require:OP LP?
+U 1 1 5C6E076D
+P 9250 6850
+AR Path="/5C70CDE2/5C6E076D" Ref="LP?"  Part="1"
+AR Path="/5C325762/5C6E076D" Ref="LP14"  Part="1"
+F 0 "LP14" H 9500 6850 50  0000 C CNN
+F 1 "RST" H 9250 6850 50  0000 C CNN
+F 2 "require:OVAL_PIN" H 9250 6800 50  0001 C CNN
+F 3 "" H 9250 6800 50  0001 C CNN
+	1    9250 6850
+	1    0    0    -1
+$EndComp
+$Comp
+L Transistor_FET:BSS138 Q1
+U 1 1 5C704641
+P 6450 6750
+F 0 "Q1" V 6700 6750 50  0000 C CNN
+F 1 "BSS138" V 6791 6750 50  0000 C CNN
+F 2 "TO_SOT_Packages_SMD:SOT-23" H 6650 6675 50  0001 L CIN
+F 3 "https://www.fairchildsemi.com/datasheets/BS/BSS138.pdf" H 6450 6750 50  0001 L CNN
+	1    6450 6750
+	0    1    1    0
+$EndComp
+Wire Wire Line
+	5650 6150 6450 6150
+Wire Wire Line
+	6450 6150 6450 6550
+Connection ~ 5650 6150
+Wire Wire Line
+	5650 6150 5650 6050
+Wire Wire Line
+	5650 6850 6250 6850
+$Comp
+L Device:R R435
+U 1 1 5C7F3B7D
+P 7150 6450
+F 0 "R435" H 7220 6496 50  0000 L CNN
+F 1 "10k" H 7220 6405 50  0000 L CNN
+F 2 "Resistors_SMD:R_0402" V 7080 6450 50  0001 C CNN
+F 3 "~" H 7150 6450 50  0001 C CNN
+	1    7150 6450
+	1    0    0    -1
+$EndComp
+$Comp
+L require:VCC_IO #PWR0226
+U 1 1 5C8165FF
+P 7150 6050
+F 0 "#PWR0226" H 7150 5900 50  0001 C CNN
+F 1 "VCC_IO" H 7167 6223 50  0000 C CNN
+F 2 "" H 7150 6050 50  0001 C CNN
+F 3 "" H 7150 6050 50  0001 C CNN
+	1    7150 6050
+	1    0    0    -1
+$EndComp
+Wire Wire Line
+	7150 6050 7150 6300
+Wire Wire Line
+	6650 6850 7150 6850
+Wire Wire Line
+	7150 6850 7150 6600
+Wire Wire Line
+	7150 6850 7750 6850
+Connection ~ 7150 6850
+Connection ~ 7750 6850
+Wire Wire Line
+	8850 6850 9050 6850
+Connection ~ 8850 6850
+Wire Wire Line
+	7900 7000 7750 7000
+Wire Wire Line
+	7750 7000 7750 7200
+Wire Wire Line
+	8700 7000 8850 7000
+Wire Wire Line
+	8850 7000 8850 7200
+Wire Wire Line
+	7750 7200 8850 7200
+Wire Wire Line
+	7750 7200 7750 7400
+Connection ~ 7750 7200
 $EndSCHEMATC

Commit message: wip
Parts:
- removed LP2: A0, require:OVAL_PIN, symbol require:OP
- removed LP3: A1, require:OVAL_PIN, symbol require:OP
- removed LP4: A2, require:OVAL_PIN, symbol require:OP
- removed LP5: A3, require:OVAL_PIN, symbol require:OP
- removed LP6: A4, require:OVAL_PIN, symbol require:OP
- removed LP7: A5, require:OVAL_PIN, symbol require:OP
- removed unit 10 of U1000
- added C74, C75, C76, C85, C87: 0.1u, Capacitors_SMD:C_0402, symbol Device:C
Connections:
- net labels added: AVDD_1V8, RESET_1V8
- net labels removed: A0, A1, A2, A3, A4, A5, RESET
- wire segments 339 -> 379
Other:
- note removed: "Close to chip"
- note removed: "Share capacitor with E17"
- moved on the sheet: C70, C71, C72, C73, C77, C78, C84, C86, C88, C90, C91, LP14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

Commit message: wip
Parts:
- removed LP14: RST, require:OVAL_PIN, symbol require:OP
- removed SW1: SW_SKSC_4PIN, require:SW_ALPS_SKSC, symbol require:SW_SKSC_4PIN
- added C89: 0.1u, Capacitors_SMD:C_0402, symbol Device:C
Connections:
- net GND: now also C89.2
- net RESET: now reaches Q1.3 (D), R435.2
- net RESET: now also C89.1
Other:
- moved on the sheet: C70, C71, C72, C73, C74, C75, C76, C77, C78, C84, C85, C86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

Commit message: wip
Parts:
- added C88: 0.1u, Capacitors_SMD:C_0402, symbol Device:C
- renumbered C89 to C47, C88 to C48, R435 to R46, R92 to R47
Connections:
- net GND: now also C88.2
- net RESET_1V8: now also C88.1
Changed lines of the file:
@@
 RESET_1V8
 $Comp
-L Device:C C88
+L Device:C C48
 U 1 1 5C42AEFD
 P 9450 5450
-F 0 "C88" H 9565 5496 50  0000 L CNN
+F 0 "C48" H 9565 5496 50  0000 L CNN
 F 1 "0.1u" H 9565 5405 50  0000 L CNN
 F 2 "Capacitors_SMD:C_0402" H 9488 5300 50  0001 C CNN
@@
 $EndComp
 $Comp
-L Device:R R92
+L Device:R R47
 U 1 1 5CF98D58
 P 9450 4950
-F 0 "R92" H 9520 4996 50  0000 L CNN
+F 0 "R47" H 9520 4996 50  0000 L CNN
 F 1 "10k" H 9520 4905 50  0000 L CNN
 F 2 "Resistors_SMD:R_0402" V 9380 4950 50  0001 C CNN
@@
 	9450 5200 9750 5200
 $Comp
-L Device:R R435
+L Device:R R46
 U 1 1 5C7F3B7D
 P 10450 4950
-F 0 "R435" H 10520 4996 50  0000 L CNN
+F 0 "R46" H 10520 4996 50  0000 L CNN
 F 1 "10k" H 10520 4905 50  0000 L CNN
 F 2 "Resistors_SMD:R_0402" V 10380 4950 50  0001 C CNN
@@
 	8400 3400 8500 3400
 Wire Wire Line
-	8400 5200 9450 5200
+	8400 5200 8900 5200
 Wire Wire Line
 	8400 4200 9700 4200
@@
 Connection ~ 10450 5200
 $Comp
-L Device:C C89
+L Device:C C47
 U 1 1 5C560B44
 P 10450 5450
-F 0 "C89" H 10565 5496 50  0000 L CNN
+F 0 "C47" H 10565 5496 50  0000 L CNN
 F 1 "0.1u" H 10565 5405 50  0000 L CNN
 F 2 "Capacitors_SMD:C_0402" H 10488 5300 50  0001 C CNN
@@
 	1    0    0    -1
 $EndComp
+$Comp
+L Device:C C88
+U 1 1 5C6BCD28
+P 8900 5450
+F 0 "C88" H 9015 5496 50  0000 L CNN
+F 1 "0.1u" H 9015 5405 50  0000 L CNN
+F 2 "Capacitors_SMD:C_0402" H 8938 5300 50  0001 C CNN
+F 3 "~" H 8900 5450 50  0001 C CNN
+	1    8900 5450
+	1    0    0    -1
+$EndComp
+Wire Wire Line
+	8900 5300 8900 5200
+Connection ~ 8900 5200
+Wire Wire Line
+	8900 5200 9450 5200
+Wire Wire Line
+	8900 5600 8900 5700
+$Comp
+L power:GND #PWR0195
+U 1 1 5C70F893
+P 8900 5700
+F 0 "#PWR0195" H 8900 5450 50  0001 C CNN
+F 1 "GND" H 8905 5527 50  0000 C CNN
+F 2 "" H 8900 5700 50  0001 C CNN
+F 3 "" H 8900 5700 50  0001 C CNN
+	1    8900 5700
+	1    0    0    -1
+$EndComp
