File: hardware/rk3308-power.sch (KiCad schematic (older format))
At the start: 24 parts, among them Q1 BSS138, U1000 RK3308, Y2 Crystal_GND24

Commit message: wip
Parts:
- C47, C48, C71, C72, C73, C74, C75, C76, C77, C84, C85, C86, C87, C88, C90, C91: footprint Capacitors_SMD:C_0402 -> require:C_0402
- C70, C78: footprint Capacitors_SMD:C_0603 -> require:C_0603
- R46, R47, R91: footprint Resistors_SMD:R_0402 -> require:R_0402
Changed lines of the file:
@@
 F 0 "C48" H 9565 5496 50  0000 L CNN
 F 1 "0.1u" H 9565 5405 50  0000 L CNN
-F 2 "Capacitors_SMD:C_0402" H 9488 5300 50  0001 C CNN
+F 2 "require:C_0402" H 9488 5300 50  0001 C CNN
 F 3 "~" H 9450 5450 50  0001 C CNN
 	1    9450 5450
@@
 F 0 "C71" H 3800 3050 50  0000 L CNN
 F 1 "0.1u" H 3800 2950 50  0000 L CNN
-F 2 "Capacitors_SMD:C_0402" H 3738 2850 50  0001 C CNN
+F 2 "require:C_0402" H 3738 2850 50  0001 C CNN
 F 3 "" H 3700 3000 50  0001 C CNN
 	1    3700 3000
@@
 F 0 "C72" H 4200 3050 50  0000 L CNN
 F 1 "0.1u" H 4200 2950 50  0000 L CNN
-F 2 "Capacitors_SMD:C_0402" H 4138 2850 50  0001 C CNN
+F 2 "require:C_0402" H 4138 2850 50  0001 C CNN
 F 3 "" H 4100 3000 50  0001 C CNN
 	1    4100 3000
@@
 F 0 "C73" H 4600 3050 50  0000 L CNN
 F 1 "2.2u" H 4600 2950 50  0000 L CNN
-F 2 "Capacitors_SMD:C_0402" H 4538 2850 50  0001 C CNN
+F 2 "require:C_0402" H 4538 2850 50  0001 C CNN
 F 3 "" H 4500 3000 50  0001 C CNN
 	1    4500 3000
@@
 F 0 "C70" H 5000 3050 50  0000 L CNN
 F 1 "22u" H 5000 2950 50  0000 L CNN
-F 2 "Capacitors_SMD:C_0603" H 5000 2850 50  0000 C CNN
+F 2 "require:C_0603" H 5000 2850 50  0000 C CNN
 F 3 "" H 4900 3000 50  0001 C CNN
 	1    4900 3000
@@
 F 0 "C78" H 3800 4250 50  0000 L CNN
 F 1 "10u" H 3800 4150 50  0000 L CNN
-F 2 "Capacitors_SMD:C_0603" H 3800 4050 50  0000 C CNN
+F 2 "require:C_0603" H 3800 4050 50  0000 C CNN
 F 3 "" H 3700 4200 50  0001 C CNN
 	1    3700 4200
@@
 F 0 "C77" H 4400 4250 50  0000 L CNN
 F 1 "0.1u" H 4400 4150 50  0000 L CNN
-F 2 "Capacitors_SMD:C_0402" H 4338 4050 50  0001 C CNN
+F 2 "require:C_0402" H 4338 4050 50  0001 C CNN
 F 3 "" H 4300 4200 50  0001 C CNN
 	1    4300 4200
@@
 F 0 "R91" V 8550 3400 50  0000 C CNN
 F 1 "22R" V 8750 3400 50  0000 C CNN
-F 2 "Resistors_SMD:R_0402" V 8580 3400 50  0001 C CNN
+F 2 "require:R_0402" V 8580 3400 50  0001 C CNN
 F 3 "" H 8650 3400 50  0001 C CNN
 	1    8650 3400
@@
 F 0 "C91" H 9015 3696 50  0000 L CNN
 F 1 "15p" H 9015 3605 50  0000 L CNN
-F 2 "Capacitors_SMD:C_0402" H 8938 3500 50  0001 C CNN
+F 2 "require:C_0402" H 8938 3500 50  0001 C CNN
 F 3 "~" H 8900 3650 50  0001 C CNN
 	1    8900 3650
@@
 F 0 "C90" H 10015 3696 50  0000 L CNN
 F 1 "15p" H 10015 3605 50  0000 L CNN
-F 2 "Capacitors_SMD:C_0402" H 9938 3500 50  0001 C CNN
+F 2 "require:C_0402" H 9938 3500 50  0001 C CNN
 F 3 "~" H 9900 3650 50  0001 C CNN
 	1    9900 3650
@@
 F 0 "C86" H 4265 7696 50  0000 L CNN
 F 1 "0.1u" H 4265 7605 50  0000 L CNN
-F 2 "Capacitors_SMD:C_0402" H 4188 7500 50  0001 C CNN
+F 2 "require:C_0402" H 4188 7500 50  0001 C CNN
 F 3 "~" H 4150 7650 50  0001 C CNN
 	1    4150 7650
@@
 F 0 "C84" H 3615 6846 50  0000 L CNN
 F 1 "0.1u" H 3615 6755 50  0000 L CNN
-F 2 "Capacitors_SMD:C_0402" H 3538 6650 50  0001 C CNN
+F 2 "require:C_0402" H 3538 6650 50  0001 C CNN
 F 3 "~" H 3500 6800 50  0001 C CNN
 	1    3500 6800
@@
 F 0 "R47" H 9520 4996 50  0000 L CNN
 F 1 "10k" H 9520 4905 50  0000 L CNN
-F 2 "Resistors_SMD:R_0402" V 9380 4950 50  0001 C CNN
+F 2 "require:R_0402" V 9380 4950 50  0001 C CNN
 F 3 "~" H 9450 4950 50  0001 C CNN
 	1    9450 4950
@@
 F 0 "R46" H 10520 4996 50  0000 L CNN
 F 1 "10k" H 10520 4905 50  0000 L CNN
-F 2 "Resistors_SMD:R_0402" V 10380 4950 50  0001 C CNN
+F 2 "require:R_0402" V 10380 4950 50  0001 C CNN
 F 3 "~" H 10450 4950 50  0001 C CNN
 	1    10450 4950
@@
 F 0 "C74" H 3815 5146 50  0000 L CNN
 F 1 "0.1u" H 3815 5055 50  0000 L CNN
-F 2 "Capacitors_SMD:C_0402" H 3738 4950 50  0001 C CNN
+F 2 "require:C_0402" H 3738 4950 50  0001 C CNN
 F 3 "~" H 3700 5100 50  0001 C CNN
 	1    3700 5100
@@
 F 0 "C75" H 4415 5146 50  0000 L CNN
 F 1 "0.1u" H 4415 5055 50  0000 L CNN
-F 2 "Capacitors_SMD:C_0402" H 4338 4950 50  0001 C CNN
+F 2 "require:C_0402" H 4338 4950 50  0001 C CNN
 F 3 "~" H 4300 5100 50  0001 C CNN
 	1    4300 5100
@@
 F 0 "C76" H 4965 5146 50  0000 L CNN
 F 1 "0.1u" H 4965 5055 50  0000 L CNN
-F 2 "Capacitors_SMD:C_0402" H 4888 4950 50  0001 C CNN
+F 2 "require:C_0402" H 4888 4950 50  0001 C CNN
 F 3 "~" H 4850 5100 50  0001 C CNN
 	1    4850 5100
@@
 F 0 "C85" H 4965 6646 50  0000 L CNN
 F 1 "0.1u" H 4965 6555 50  0000 L CNN
-F 2 "Capacitors_SMD:C_0402" H 4888 6450 50  0001 C CNN
+F 2 "require:C_0402" H 4888 6450 50  0001 C CNN
 F 3 "~" H 4850 6600 50  0001 C CNN
 	1    4850 6600
@@
 F 0 "C87" H 5565 5146 50  0000 L CNN
 F 1 "0.1u" H 5565 5055 50  0000 L CNN
-F 2 "Capacitors_SMD:C_0402" H 5488 4950 50  0001 C CNN
+F 2 "require:C_0402" H 5488 4950 50  0001 C CNN
 F 3 "~" H 5450 5100 50  0001 C CNN
 	1    5450 5100
@@
 F 0 "C47" H 10565 5496 50  0000 L CNN
 F 1 "0.1u" H 10565 5405 50  0000 L CNN
-F 2 "Capacitors_SMD:C_0402" H 10488 5300 50  0001 C CNN
+F 2 "require:C_0402" H 10488 5300 50  0001 C CNN
 F 3 "~" H 10450 5450 50  0001 C CNN
 	1    10450 5450
@@
 F 0 "C88" H 9015 5496 50  0000 L CNN
 F 1 "0.1u" H 9015 5405 50  0000 L CNN
-F 2 "Capacitors_SMD:C_0402" H 8938 5300 50  0001 C CNN
+F 2 "require:C_0402" H 8938 5300 50  0001 C CNN
 F 3 "~" H 8900 5450 50  0001 C CNN
 	1    8900 5450

Commit message: wip
Parts:
- removed C47, C48: 0.1u, require:C_0402, symbol Device:C
- added FB1, FB2: 180R,1.5A, Inductors_SMD:L_0402, symbol Device:L
- Q1: footprint TO_SOT_Packages_SMD:SOT-23 -> require:SOT-323_SC-70
Connections:
- net labels added: +1V0, +1V0C, +1V0L, +1V8, +1V8A, +3V3
- net labels removed: AVDD_1V8, VCC_1V8, VCC_IO, VDD_1V0, VDD_CORE, VDD_LOG
- wire segments 372 -> 375
Other:
- note added: "180 ohm @ 100MHz, 1.5A\nBLM15PX181SN1D (Tape)\nBLM15PX181SN1B (Bulk)"
Changed lines of the file:
@@
 	3300 2750 3300 2650
 Connection ~ 3300 2750
-$Comp
-L require:VDD_CORE #PWR0147
-U 1 1 5D30F1B1
-P 3300 2650
-F 0 "#PWR0147" H 3300 2500 50  0001 C CNN
-F 1 "VDD_CORE" H 3317 2823 50  0000 C CNN
-F 2 "" H 3300 2650 50  0001 C CNN
-F 3 "" H 3300 2650 50  0001 C CNN
-	1    3300 2650
-	1    0    0    -1
-$EndComp
 Wire Wire Line
 	3100 3950 3300 3950
@@
 Wire Wire Line
 	3300 4050 3300 4150
-$Comp
-L require:VDD_LOG #PWR0148
-U 1 1 5D35275B
-P 3300 3850
-F 0 "#PWR0148" H 3300 3700 50  0001 C CNN
-F 1 "VDD_LOG" H 3317 4023 50  0000 C CNN
-F 2 "" H 3300 3850 50  0001 C CNN
-F 3 "" H 3300 3850 50  0001 C CNN
-	1    3300 3850
-	1    0    0    -1
-$EndComp
-Wire Wire Line
-	3300 3850 3300 3950
 Connection ~ 3300 3950
 $Comp
@@
 Text Label 8600 5200 0    50   ~ 0
 RESET_1V8
-$Comp
-L Device:C C48
-U 1 1 5C42AEFD
-P 9450 5450
-F 0 "C48" H 9565 5496 50  0000 L CNN
-F 1 "0.1u" H 9565 5405 50  0000 L CNN
-F 2 "require:C_0402" H 9488 5300 50  0001 C CNN
-F 3 "~" H 9450 5450 50  0001 C CNN
-	1    9450 5450
-	1    0    0    -1
-$EndComp
-Wire Wire Line
-	9450 5300 9450 5200
-Wire Wire Line
-	9450 5600 9450 5700
-$Comp
-L power:GND #PWR0155
-U 1 1 5C4535B5
-P 9450 5700
-F 0 "#PWR0155" H 9450 5450 50  0001 C CNN
-F 1 "GND" H 9455 5527 50  0000 C CNN
-F 2 "" H 9450 5700 50  0001 C CNN
-F 3 "" H 9450 5700 50  0001 C CNN
-	1    9450 5700
-	1    0    0    -1
-$EndComp
 $Comp
 L require-rescue:C C?
@@
 	1    0    0    -1
 $EndComp
-$Comp
-L require:VDD_1V0 #PWR0202
-U 1 1 5C8CB6DB
-P 4150 7250
-F 0 "#PWR0202" H 4150 7100 50  0001 C CNN
-F 1 "VDD_1V0" H 4167 7423 50  0000 C CNN
-F 2 "" H 4150 7250 50  0001 C CNN
-F 3 "" H 4150 7250 50  0001 C CNN
-	1    4150 7250
-	1    0    0    -1
-$EndComp
 Wire Wire Line
 	4150 7800 4150 8000
@@
 $EndComp
 $Comp
-L require:VCC_1V8 #PWR0204
-U 1 1 5C9A4743
-P 3500 5950
-F 0 "#PWR0204" H 3500 5800 50  0001 C CNN
-F 1 "VCC_1V8" H 3517 6123 50  0000 C CNN
-F 2 "" H 3500 5950 50  0001 C CNN
-F 3 "" H 3500 5950 50  0001 C CNN
-	1    3500 5950
-	1    0    0    -1
-$EndComp
-$Comp
 L Device:C C84
 U 1 1 5C9A47A9
@@
 	9450 5200 9450 5100
 $Comp
-L require:VCC_1V8 #PWR0219
-U 1 1 5CFD03F5
-P 9450 4600
-F 0 "#PWR0219" H 9450 4450 50  0001 C CNN
-F 1 "VCC_1V8" H 9467 4773 50  0000 C CNN
-F 2 "" H 9450 4600 50  0001 C CNN
-F 3 "" H 9450 4600 50  0001 C CNN
-	1    9450 4600
-	1    0    0    -1
-$EndComp
-$Comp
 L Transistor_FET:BSS138 Q1
 U 1 1 5C704641
@@
 F 0 "Q1" V 10200 5100 50  0000 C CNN
 F 1 "BSS138" V 10291 5100 50  0000 C CNN
-F 2 "TO_SOT_Packages_SMD:SOT-23" H 10150 5025 50  0001 L CIN
+F 2 "require:SOT-323_SC-70" V 10400 5100 50  0000 C CIN
 F 3 "https://www.fairchildsemi.com/datasheets/BS/BSS138.pdf" H 9950 5100 50  0001 L CNN
 	1    9950 5100
@@
 Wire Wire Line
 	3300 4950 3300 5050
-Wire Wire Line
-	3300 4850 3300 4750
 Connection ~ 3300 4850
-$Comp
-L require:VCC_IO #PWR0137
-U 1 1 5CA7CF6B
-P 3300 4750
-F 0 "#PWR0137" H 3300 4600 50  0001 C CNN
-F 1 "VCC_IO" H 3317 4923 50  0000 C CNN
-F 2 "" H 3300 4750 50  0001 C CNN
-F 3 "" H 3300 4750 50  0001 C CNN
-	1    3300 4750
-	1    0    0    -1
-$EndComp
 Wire Wire Line
 	3300 4850 3700 4850
@@
 	1    0    0    -1
 $EndComp
-$Comp
-L require:AVDD_1V8 #PWR?
-U 1 1 5CF5F381
-P 4850 6050
-AR Path="/5CED3BD3/5CF5F381" Ref="#PWR?"  Part="1"
-AR Path="/5C325762/5CF5F381" Ref="#PWR0141"  Part="1"
-F 0 "#PWR0141" H 4850 5900 50  0001 C CNN
-F 1 "AVDD_1V8" H 4867 6223 50  0000 C CNN
-F 2 "" H 4850 6050 50  0001 C CNN
-F 3 "" H 4850 6050 50  0001 C CNN
-	1    4850 6050
-	1    0    0    -1
-$EndComp
 Wire Wire Line
 	4850 6750 4850 6850
@@
 	3500 6250 3500 6350
 Wire Wire Line
-	4850 6050 4850 6150
+	4850 5950 4850 6050
 Wire Wire Line
 	3100 6150 4850 6150
@@
 Wire Wire Line
 	10450 4800 10450 4600
-$Comp
-L require:VCC_IO #PWR0153
-U 1 1 5DE4DB0E
-P 10450 4600
-F 0 "#PWR0153" H 10450 4450 50  0001 C CNN
-F 1 "VCC_IO" H 10467 4773 50  0000 C CNN
-F 2 "" H 10450 4600 50  0001 C CNN
-F 3 "" H 10450 4600 50  0001 C CNN
-	1    10450 4600
-	1    0    0    -1
-$EndComp
 Wire Wire Line
 	10450 5100 10450 5200
@@
 Connection ~ 10450 5200
 $Comp
-L Device:C C47
-U 1 1 5C560B44
-P 10450 5450
-F 0 "C47" H 10565 5496 50  0000 L CNN
-F 1 "0.1u" H 10565 5405 50  0000 L CNN
-F 2 "require:C_0402" H 10488 5300 50  0001 C CNN
-F 3 "~" H 10450 5450 50  0001 C CNN
-	1    10450 5450
-	1    0    0    -1
-$EndComp
-Wire Wire Line
-	10450 5300 10450 5200
-Wire Wire Line
-	10450 5600 10450 5700
-$Comp
-L power:GND #PWR0173
-U 1 1 5C5B8584
-P 10450 5700
-F 0 "#PWR0173" H 10450 5450 50  0001 C CNN
-F 1 "GND" H 10455 5527 50  0000 C CNN
-F 2 "" H 10450 5700 50  0001 C CNN
-F 3 "" H 10450 5700 50  0001 C CNN
-	1    10450 5700
-	1    0    0    -1
-$EndComp
-$Comp
 L Device:C C88
 U 1 1 5C6BCD28
@@
 	1    0    0    -1
 $EndComp
+$Comp
+L power:+3V3 #PWR0137
+U 1 1 5C821550
+P 10450 4600
+F 0 "#PWR0137" H 10450 4450 50  0001 C CNN
+F 1 "+3V3" H 10465 4773 50  0000 C CNN
+F 2 "" H 10450 4600 50  0001 C CNN
+F 3 "" H 10450 4600 50  0001 C CNN
+	1    10450 4600
+	1    0    0    -1
+$EndComp
+Wire Wire Line
+	5450 4850 5450 4750
+Connection ~ 5450 4850
+$Comp
+L power:+3V3 #PWR0153
+U 1 1 5C84A2A6
+P 5450 4750
+F 0 "#PWR0153" H 5450 4600 50  0001 C CNN
+F 1 "+3V3" H 5465 4923 50  0000 C CNN
+F 2 "" H 5450 4750 50  0001 C CNN
+F 3 "" H 5450 4750 50  0001 C CNN
+	1    5450 4750
+	1    0    0    -1
+$EndComp
+$Comp
+L power:+1V8 #PWR0204
+U 1 1 5C8583C0
+P 9450 4600
+F 0 "#PWR0204" H 9450 4450 50  0001 C CNN
+F 1 "+1V8" H 9465 4773 50  0000 C CNN
+F 2 "" H 9450 4600 50  0001 C CNN
+F 3 "" H 9450 4600 50  0001 C CNN
+	1    9450 4600
+	1    0    0    -1
+$EndComp
+$Comp
+L power:+1V8 #PWR0219
+U 1 1 5C85A555
+P 3500 5950
+F 0 "#PWR0219" H 3500 5800 50  0001 C CNN
+F 1 "+1V8" H 3515 6123 50  0000 C CNN
+F 2 "" H 3500 5950 50  0001 C CNN
+F 3 "" H 3500 5950 50  0001 C CNN
+	1    3500 5950
+	1    0    0    -1
+$EndComp
+$Comp
+L Device:L FB?
+U 1 1 5C86B836
+P 4100 6050
+AR Path="/5C2CD8AE/5C86B836" Ref="FB?"  Part="1"
+AR Path="/5C325762/5C86B836" Ref="FB2"  Part="1"
+F 0 "FB2" V 4290 6050 50  0000 C CNN
+F 1 "180R,1.5A" V 4199 6050 50  0000 C CNN
+F 2 "Inductors_SMD:L_0402" H 4100 6050 50  0001 C CNN
+F 3 "~" H 4100 6050 50  0001 C CNN
+	1    4100 6050
+	0    -1   -1   0
+$EndComp
+Wire Wire Line
+	4250 6050 4850 6050
+Connection ~ 4850 6050
+Wire Wire Line
+	4850 6050 4850 6150
+Wire Wire Line
+	3950 6050 3500 6050
+$Comp
+L require:+1V8A #PWR0141
+U 1 1 5C989EFE
+P 4850 5950
+F 0 "#PWR0141" H 4850 5800 50  0001 C CNN
+F 1 "+1V8A" H 4865 6123 50  0000 C CNN
+F 2 "" H 4850 5950 50  0001 C CNN
+F 3 "" H 4850 5950 50  0001 C CNN
+	1    4850 5950
+	1    0    0    -1
+$EndComp
+Wire Wire Line
+	4300 3850 4300 3950
+Connection ~ 4300 3950
+$Comp
+L require:+1V0L #PWR0176
+U 1 1 5C9E0D26
+P 4300 3850
+F 0 "#PWR0176" H 4300 3700 50  0001 C CNN
+F 1 "+1V0L" H 4315 4023 50  0000 C CNN
+F 2 "" H 4300 3850 50  0001 C CNN
+F 3 "" H 4300 3850 50  0001 C CNN
+	1    4300 3850
+	1    0    0    -1
+$EndComp
+$Comp
+L require:+1V0C #PWR0189
+U 1 1 5C9EBE59
+P 3300 2650
+F 0 "#PWR0189" H 3300 2500 50  0001 C CNN
+F 1 "+1V0C" H 3315 2823 50  0000 C CNN
+F 2 "" H 3300 2650 50  0001 C CNN
+F 3 "" H 3300 2650 50  0001 C CNN
+	1    3300 2650
+	1    0    0    -1
+$EndComp
+$Comp
+L power:+1V0 #PWR0190
+U 1 1 5C9F5772
+P 4150 7250
+F 0 "#PWR0190" H 4150 7100 50  0001 C CNN
+F 1 "+1V0" H 4165 7423 50  0000 C CNN
+F 2 "" H 4150 7250 50  0001 C CNN
+F 3 "" H 4150 7250 50  0001 C CNN
+	1    4150 7250
+	1    0    0    -1
+$EndComp
+Wire Wire Line
+	5200 7250 5200 7350
+Wire Wire Line
+	5200 7350 5400 7350
+Wire Wire Line
+	5700 7350 5900 7350
+Wire Wire Line
+	5900 7350 5900 7250
+$Comp
+L Device:L FB?
+U 1 1 5C9FE521
+P 5550 7350
+AR Path="/5C2CD8AE/5C9FE521" Ref="FB?"  Part="1"
+AR Path="/5C325762/5C9FE521" Ref="FB1"  Part="1"
+F 0 "FB1" V 5740 7350 50  0000 C CNN
+F 1 "180R,1.5A" V 5649 7350 50  0000 C CNN
+F 2 "Inductors_SMD:L_0402" H 5550 7350 50  0001 C CNN
+F 3 "~" H 5550 7350 50  0001 C CNN
+	1    5550 7350
+	0    -1   -1   0
+$EndComp
+Text Notes 5200 7700 0    50   ~ 10
+180 ohm @ 100MHz, 1.5A\nBLM15PX181SN1D (Tape)\nBLM15PX181SN1B (Bulk)
+$Comp
+L require:+1V0L #PWR?
+U 1 1 5C9FE529
+P 5200 7250
+AR Path="/5C2CD8AE/5C9FE529" Ref="#PWR?"  Part="1"
+AR Path="/5C325762/5C9FE529" Ref="#PWR0148"  Part="1"
+F 0 "#PWR0148" H 5200 7100 50  0001 C CNN
+F 1 "+1V0L" H 5215 7423 50  0000 C CNN
+F 2 "" H 5200 7250 50  0001 C CNN
+F 3 "" H 5200 7250 50  0001 C CNN
+	1    5200 7250
+	1    0    0    -1
+$EndComp
+$Comp
+L power:+1V0 #PWR?
+U 1 1 5C9FE52F
+P 5900 7250
+AR Path="/5C2CD8AE/5C9FE52F" Ref="#PWR?"  Part="1"
+AR Path="/5C325762/5C9FE52F" Ref="#PWR0177"  Part="1"
+F 0 "#PWR0177" H 5900 7100 50  0001 C CNN
+F 1 "+1V0" H 5915 7423 50  0000 C CNN
+F 2 "" H 5900 7250 50  0001 C CNN
+F 3 "" H 5900 7250 50  0001 C CNN
+	1    5900 7250
+	1    0    0    -1
+$EndComp

Commit message: wip
Parts:
- removed Q1: BSS138, require:SOT-323_SC-70, symbol Transistor_FET:BSS138
- added Q1: Q_NMOS_GSD, require:SOT-883, symbol Device:Q_NMOS_GSD
Changed lines of the file:
@@
 Wire Wire Line
 	9450 5200 9450 5100
-$Comp
-L Transistor_FET:BSS138 Q1
-U 1 1 5C704641
-P 9950 5100
-F 0 "Q1" V 10200 5100 50  0000 C CNN
-F 1 "BSS138" V 10291 5100 50  0000 C CNN
-F 2 "require:SOT-323_SC-70" V 10400 5100 50  0000 C CIN
-F 3 "https://www.fairchildsemi.com/datasheets/BS/BSS138.pdf" H 9950 5100 50  0001 L CNN
-	1    9950 5100
-	0    1    1    0
-$EndComp
 Wire Wire Line
 	9450 5200 9750 5200
@@
 	1    0    0    -1
 $EndComp
+$Comp
+L Device:Q_NMOS_GSD Q1
+U 1 1 5C85D5B8
+P 9950 5100
+F 0 "Q1" V 10201 5100 50  0000 C CNN
+F 1 "Q_NMOS_GSD" V 10292 5100 50  0000 C CNN
+F 2 "require:SOT-883" V 10383 5100 50  0000 C CNN
+F 3 "~" H 9950 5100 50  0001 C CNN
+	1    9950 5100
+	0    1    1    0
+$EndComp
 $EndSCHEMATC
