File: hardware/rk3308-power.sch (KiCad schematic (older format))
At the start: 24 parts, among them Q1 Q_NMOS_GSD, U1000 RK3308, Y2 Crystal_GND24

Commit message: wip
Parts:
- added C259: 1u, require:C_0402, symbol Device:C
- C256: renamed from C75; value 0.1u -> 1u
- C258: renamed from C87; value 0.1u -> 1u
- renumbered C91 to C100, C90 to C101, C88 to C110, C70 to C205, C71 to C206, C72 to C207, C73 to C208, C78 to C225, C77 to C226, C86 to C229, C74 to C255, C76 to C257, C84 to C265, C85 to C269, FB1 to F229, FB2 to F269, Q1 to Q110, R91 to R100, R47 to R110, R46 to R111, Y2 to Y100
Connections:
- net +3V3: now also C259.1
- net GND: now also C259.2
Other:
- note added: "D14/D13/E14"
- note added: "J14"
- note added: "N5"
- note added: "P16"
- note added: "R11/T11/R12"
Changed lines of the file:
@@
 $EndComp
 $Comp
-L Device:Crystal_GND24 Y2
+L Device:Crystal_GND24 Y100
 U 1 1 5D440CD1
 P 9350 3400
-F 0 "Y2" H 9500 3650 50  0000 L CNN
+F 0 "Y100" H 9500 3650 50  0000 L CNN
 F 1 "Crystal_GND24" H 9500 3750 50  0000 L CNN
 F 2 "Crystals:Crystal_SMD_3225-4pin_3.2x2.5mm" H 9350 3400 50  0001 C CNN
@@
 P 3700 3000
 AR Path="/5C2CD8AE/5C4672BA" Ref="C?"  Part="1"
-AR Path="/5C325762/5C4672BA" Ref="C71"  Part="1"
-F 0 "C71" H 3800 3050 50  0000 L CNN
+AR Path="/5C325762/5C4672BA" Ref="C206"  Part="1"
+F 0 "C206" H 3800 3050 50  0000 L CNN
 F 1 "0.1u" H 3800 2950 50  0000 L CNN
 F 2 "require:C_0402" H 3738 2850 50  0001 C CNN
@@
 P 4100 3000
 AR Path="/5C2CD8AE/5D13500C" Ref="C?"  Part="1"
-AR Path="/5C325762/5D13500C" Ref="C72"  Part="1"
-F 0 "C72" H 4200 3050 50  0000 L CNN
+AR Path="/5C325762/5D13500C" Ref="C207"  Part="1"
+F 0 "C207" H 4200 3050 50  0000 L CNN
 F 1 "0.1u" H 4200 2950 50  0000 L CNN
 F 2 "require:C_0402" H 4138 2850 50  0001 C CNN
@@
 P 4500 3000
 AR Path="/5C2CD8AE/5D135096" Ref="C?"  Part="1"
-AR Path="/5C325762/5D135096" Ref="C73"  Part="1"
-F 0 "C73" H 4600 3050 50  0000 L CNN
+AR Path="/5C325762/5D135096" Ref="C208"  Part="1"
+F 0 "C208" H 4600 3050 50  0000 L CNN
 F 1 "2.2u" H 4600 2950 50  0000 L CNN
 F 2 "require:C_0402" H 4538 2850 50  0001 C CNN
@@
 P 4900 3000
 AR Path="/5C2CD8AE/5D135164" Ref="C?"  Part="1"
-AR Path="/5C325762/5D135164" Ref="C70"  Part="1"
-F 0 "C70" H 5000 3050 50  0000 L CNN
+AR Path="/5C325762/5D135164" Ref="C205"  Part="1"
+F 0 "C205" H 5000 3050 50  0000 L CNN
 F 1 "22u" H 5000 2950 50  0000 L CNN
 F 2 "require:C_0603" H 5000 2850 50  0000 C CNN
@@
 P 3700 4200
 AR Path="/5C2CD8AE/5D240387" Ref="C?"  Part="1"
-AR Path="/5C325762/5D240387" Ref="C78"  Part="1"
-F 0 "C78" H 3800 4250 50  0000 L CNN
+AR Path="/5C325762/5D240387" Ref="C225"  Part="1"
+F 0 "C225" H 3800 4250 50  0000 L CNN
 F 1 "10u" H 3800 4150 50  0000 L CNN
 F 2 "require:C_0603" H 3800 4050 50  0000 C CNN
@@
 P 4300 4200
 AR Path="/5C2CD8AE/5D291CA2" Ref="C?"  Part="1"
-AR Path="/5C325762/5D291CA2" Ref="C77"  Part="1"
-F 0 "C77" H 4400 4250 50  0000 L CNN
+AR Path="/5C325762/5D291CA2" Ref="C226"  Part="1"
+F 0 "C226" H 4400 4250 50  0000 L CNN
 F 1 "0.1u" H 4400 4150 50  0000 L CNN
 F 2 "require:C_0402" H 4338 4050 50  0001 C CNN
@@
 P 8650 3400
 AR Path="/5C2CD8AE/5C745F21" Ref="R?"  Part="1"
-AR Path="/5C325762/5C745F21" Ref="R91"  Part="1"
-F 0 "R91" V 8550 3400 50  0000 C CNN
+AR Path="/5C325762/5C745F21" Ref="R100"  Part="1"
+F 0 "R100" V 8550 3400 50  0000 C CNN
 F 1 "22R" V 8750 3400 50  0000 C CNN
 F 2 "require:R_0402" V 8580 3400 50  0001 C CNN
@@
 	8800 3400 8900 3400
 $Comp
-L Device:C C91
+L Device:C C100
 U 1 1 5C7967A1
 P 8900 3650
-F 0 "C91" H 9015 3696 50  0000 L CNN
+F 0 "C100" H 9015 3696 50  0000 L CNN
 F 1 "15p" H 9015 3605 50  0000 L CNN
 F 2 "require:C_0402" H 8938 3500 50  0001 C CNN
@@
 	8900 3800 8900 3900
 $Comp
-L Device:C C90
+L Device:C C101
 U 1 1 5C7EA32C
 P 9900 3650
-F 0 "C90" H 10015 3696 50  0000 L CNN
+F 0 "C101" H 10015 3696 50  0000 L CNN
 F 1 "15p" H 10015 3605 50  0000 L CNN
 F 2 "require:C_0402" H 9938 3500 50  0001 C CNN
@@
 $EndComp
 $Comp
-L Device:C C86
+L Device:C C229
 U 1 1 5C84BC04
 P 4150 7650
-F 0 "C86" H 4265 7696 50  0000 L CNN
+F 0 "C229" H 4265 7696 50  0000 L CNN
 F 1 "0.1u" H 4265 7605 50  0000 L CNN
 F 2 "require:C_0402" H 4188 7500 50  0001 C CNN
@@
 $EndComp
 $Comp
-L Device:C C84
+L Device:C C265
 U 1 1 5C9A47A9
 P 3500 6800
-F 0 "C84" H 3615 6846 50  0000 L CNN
+F 0 "C265" H 3615 6846 50  0000 L CNN
 F 1 "0.1u" H 3615 6755 50  0000 L CNN
 F 2 "require:C_0402" H 3538 6650 50  0001 C CNN
@@
 $EndComp
 $Comp
-L Device:R R47
+L Device:R R110
 U 1 1 5CF98D58
 P 9450 4950
-F 0 "R47" H 9520 4996 50  0000 L CNN
+F 0 "R110" H 9520 4996 50  0000 L CNN
 F 1 "10k" H 9520 4905 50  0000 L CNN
 F 2 "require:R_0402" V 9380 4950 50  0001 C CNN
@@
 	9450 5200 9750 5200
 $Comp
-L Device:R R46
+L Device:R R111
 U 1 1 5C7F3B7D
 P 10450 4950
-F 0 "R46" H 10520 4996 50  0000 L CNN
+F 0 "R111" H 10520 4996 50  0000 L CNN
 F 1 "10k" H 10520 4905 50  0000 L CNN
 F 2 "require:R_0402" V 10380 4950 50  0001 C CNN
@@
 AR Path="/5C2D00B3/5C92C2F5" Ref="C?"  Part="1"
 AR Path="/5C87E279/5C92C2F5" Ref="C?"  Part="1"
-AR Path="/5C325762/5C92C2F5" Ref="C74"  Part="1"
-F 0 "C74" H 3815 5146 50  0000 L CNN
+AR Path="/5C325762/5C92C2F5" Ref="C255"  Part="1"
+F 0 "C255" H 3815 5146 50  0000 L CNN
 F 1 "0.1u" H 3815 5055 50  0000 L CNN
 F 2 "require:C_0402" H 3738 4950 50  0001 C CNN
@@
 AR Path="/5C70CDE2/5C9504D9" Ref="C?"  Part="1"
 AR Path="/5C87E279/5C9504D9" Ref="C?"  Part="1"
-AR Path="/5C325762/5C9504D9" Ref="C75"  Part="1"
-F 0 "C75" H 4415 5146 50  0000 L CNN
-F 1 "0.1u" H 4415 5055 50  0000 L CNN
+AR Path="/5C325762/5C9504D9" Ref="C256"  Part="1"
+F 0 "C256" H 4415 5146 50  0000 L CNN
+F 1 "1u" H 4415 5055 50  0000 L CNN
 F 2 "require:C_0402" H 4338 4950 50  0001 C CNN
 F 3 "~" H 4300 5100 50  0001 C CNN
@@
 AR Path="/5C2D00B3/5C9753AD" Ref="C?"  Part="1"
 AR Path="/5C87E279/5C9753AD" Ref="C?"  Part="1"
-AR Path="/5C325762/5C9753AD" Ref="C76"  Part="1"
-F 0 "C76" H 4965 5146 50  0000 L CNN
+AR Path="/5C325762/5C9753AD" Ref="C257"  Part="1"
+F 0 "C257" H 4965 5146 50  0000 L CNN
 F 1 "0.1u" H 4965 5055 50  0000 L CNN
 F 2 "require:C_0402" H 4888 4950 50  0001 C CNN
@@
 P 4850 6600
 AR Path="/5CED3BD3/5CF5F378" Ref="C?"  Part="1"
-AR Path="/5C325762/5CF5F378" Ref="C85"  Part="1"
-F 0 "C85" H 4965 6646 50  0000 L CNN
+AR Path="/5C325762/5CF5F378" Ref="C269"  Part="1"
+F 0 "C269" H 4965 6646 50  0000 L CNN
 F 1 "0.1u" H 4965 6555 50  0000 L CNN
 F 2 "require:C_0402" H 4888 6450 50  0001 C CNN
@@
 P 5450 5100
 AR Path="/5CED3BD3/5E151295" Ref="C?"  Part="1"
-AR Path="/5C325762/5E151295" Ref="C87"  Part="1"
-F 0 "C87" H 5565 5146 50  0000 L CNN
-F 1 "0.1u" H 5565 5055 50  0000 L CNN
+AR Path="/5C325762/5E151295" Ref="C258"  Part="1"
+F 0 "C258" H 5565 5146 50  0000 L CNN
+F 1 "1u" H 5565 5055 50  0000 L CNN
 F 2 "require:C_0402" H 5488 4950 50  0001 C CNN
 F 3 "~" H 5450 5100 50  0001 C CNN
@@
 Connection ~ 10450 5200
 $Comp
-L Device:C C88
+L Device:C C110
 U 1 1 5C6BCD28
 P 8900 5450
-F 0 "C88" H 9015 5496 50  0000 L CNN
+F 0 "C110" H 9015 5496 50  0000 L CNN
 F 1 "0.1u" H 9015 5405 50  0000 L CNN
 F 2 "require:C_0402" H 8938 5300 50  0001 C CNN
@@
 P 4100 6050
 AR Path="/5C2CD8AE/5C86B836" Ref="FB?"  Part="1"
-AR Path="/5C325762/5C86B836" Ref="FB2"  Part="1"
-F 0 "FB2" V 4290 6050 50  0000 C CNN
+AR Path="/5C325762/5C86B836" Ref="F269"  Part="1"
+F 0 "F269" V 4290 6050 50  0000 C CNN
 F 1 "180R,1.5A" V 4199 6050 50  0000 C CNN
 F 2 "Inductors_SMD:L_0402" H 4100 6050 50  0001 C CNN
@@
 P 5550 7350
 AR Path="/5C2CD8AE/5C9FE521" Ref="FB?"  Part="1"
-AR Path="/5C325762/5C9FE521" Ref="FB1"  Part="1"
-F 0 "FB1" V 5740 7350 50  0000 C CNN
+AR Path="/5C325762/5C9FE521" Ref="F229"  Part="1"
+F 0 "F229" V 5740 7350 50  0000 C CNN
 F 1 "180R,1.5A" V 5649 7350 50  0000 C CNN
 F 2 "Inductors_SMD:L_0402" H 5550 7350 50  0001 C CNN
@@
 $EndComp
 $Comp
-L Device:Q_NMOS_GSD Q1
+L Device:Q_NMOS_GSD Q110
 U 1 1 5C85D5B8
 P 9950 5100
-F 0 "Q1" V 10201 5100 50  0000 C CNN
+F 0 "Q110" V 10201 5100 50  0000 C CNN
 F 1 "Q_NMOS_GSD" V 10292 5100 50  0000 C CNN
 F 2 "require:SOT-883" V 10383 5100 50  0000 C CNN
@@
 	0    1    1    0
 $EndComp
+Text Notes 3750 5300 0    50   ~ 0
+N5
+Text Notes 4250 5300 0    50   ~ 0
+R11/T11/R12
+Text Notes 4900 5300 0    50   ~ 0
+J14
+Text Notes 5400 5300 0    50   ~ 0
+D14/D13/E14
+$Comp
+L Device:C C?
+U 1 1 5C781190
+P 6050 5100
+AR Path="/5CED3BD3/5C781190" Ref="C?"  Part="1"
+AR Path="/5C325762/5C781190" Ref="C259"  Part="1"
+F 0 "C259" H 6165 5146 50  0000 L CNN
+F 1 "1u" H 6165 5055 50  0000 L CNN
+F 2 "require:C_0402" H 6088 4950 50  0001 C CNN
+F 3 "~" H 6050 5100 50  0001 C CNN
+	1    6050 5100
+	1    0    0    -1
+$EndComp
+Wire Wire Line
+	5450 4850 6050 4850
+Wire Wire Line
+	6050 4850 6050 4950
+$Comp
+L power:GND #PWR?
+U 1 1 5C7ABB6E
+P 6050 5350
+AR Path="/5CED3BD3/5C7ABB6E" Ref="#PWR?"  Part="1"
+AR Path="/5C325762/5C7ABB6E" Ref="#PWR0110"  Part="1"
+F 0 "#PWR0110" H 6050 5100 50  0001 C CNN
+F 1 "GND" H 6055 5177 50  0000 C CNN
+F 2 "" H 6050 5350 50  0001 C CNN
+F 3 "" H 6050 5350 50  0001 C CNN
+	1    6050 5350
+	1    0    0    -1
+$EndComp
+Wire Wire Line
+	6050 5250 6050 5350
+Text Notes 6100 5300 0    50   ~ 0
+P16
 $EndSCHEMATC

Commit message: wip
Parts:
- C100, C101: value 15p -> 22p
- C205, C206, C207, C208: symbol require-rescue:C -> Device:C
- F229, F269: symbol Device:L -> Device:Ferrite_Bead
- Q110: value Q_NMOS_GSD -> LN235N3T5G
- Y100: value Crystal_GND24 -> 24MHz,12pF,10ppm
- renumbered U1000 to U100
Changed lines of the file:
@@
 $EndDescr
 $Comp
-L require:RK3308 U1000
+L require:RK3308 U100
 U 12 1 5C32630C
 P 1900 9400
-F 0 "U1000" H 1200 14650 60  0000 C CNN
+F 0 "U100" H 1200 14650 60  0000 C CNN
 F 1 "RK3308" H 1200 14750 60  0000 C CNN
 F 2 "require:RK3308_BGA355" H 1900 9400 60  0001 C CNN
@@
 $EndComp
 $Comp
-L require:RK3308 U1000
+L require:RK3308 U100
 U 13 1 5C3263AE
 P 14100 4150
-F 0 "U1000" H 14600 7137 60  0000 C CNN
+F 0 "U100" H 14600 7137 60  0000 C CNN
 F 1 "RK3308" H 14600 7031 60  0000 C CNN
 F 2 "require:RK3308_BGA355" H 14100 4150 60  0001 C CNN
@@
 $EndComp
 $Comp
-L require:RK3308 U1000
+L require:RK3308 U100
 U 14 1 5C32644B
 P 14100 7950
-F 0 "U1000" H 14600 11237 60  0000 C CNN
+F 0 "U100" H 14600 11237 60  0000 C CNN
 F 1 "RK3308" H 14600 11131 60  0000 C CNN
 F 2 "require:RK3308_BGA355" H 14100 7950 60  0001 C CNN
@@
 Connection ~ 3300 3950
 $Comp
-L require:RK3308 U1000
+L require:RK3308 U100
 U 1 1 5D42A919
 P 7200 5800
-F 0 "U1000" H 7806 8587 60  0000 C CNN
+F 0 "U100" H 7806 8587 60  0000 C CNN
 F 1 "RK3308" H 7806 8481 60  0000 C CNN
 F 2 "" H 7200 5800 60  0001 C CNN
@@
 P 9350 3400
 F 0 "Y100" H 9500 3650 50  0000 L CNN
-F 1 "Crystal_GND24" H 9500 3750 50  0000 L CNN
+F 1 "24MHz,12pF,10ppm" H 9500 3550 50  0000 L CNN
 F 2 "Crystals:Crystal_SMD_3225-4pin_3.2x2.5mm" H 9350 3400 50  0001 C CNN
 F 3 "~" H 9350 3400 50  0001 C CNN
@@
 RESET_1V8
 $Comp
-L require-rescue:C C?
+L Device:C C?
 U 1 1 5C4672BA
 P 3700 3000
@@
 	3700 2750 3700 2850
 $Comp
-L require-rescue:C C?
+L Device:C C?
 U 1 1 5D13500C
 P 4100 3000
@@
 $EndComp
 $Comp
-L require-rescue:C C?
+L Device:C C?
 U 1 1 5D135096
 P 4500 3000
@@
 $EndComp
 $Comp
-L require-rescue:C C?
+L Device:C C?
 U 1 1 5D135164
 P 4900 3000
@@
 P 8900 3650
 F 0 "C100" H 9015 3696 50  0000 L CNN
-F 1 "15p" H 9015 3605 50  0000 L CNN
+F 1 "22p" H 9015 3605 50  0000 L CNN
 F 2 "require:C_0402" H 8938 3500 50  0001 C CNN
 F 3 "~" H 8900 3650 50  0001 C CNN
@@
 P 9900 3650
 F 0 "C101" H 10015 3696 50  0000 L CNN
-F 1 "15p" H 10015 3605 50  0000 L CNN
+F 1 "22p" H 10015 3605 50  0000 L CNN
 F 2 "require:C_0402" H 9938 3500 50  0001 C CNN
 F 3 "~" H 9900 3650 50  0001 C CNN
@@
 $EndComp
 $Comp
-L Device:L FB?
+L Device:Ferrite_Bead FB?
 U 1 1 5C86B836
 P 4100 6050
@@
 	5900 7350 5900 7250
 $Comp
-L Device:L FB?
+L Device:Ferrite_Bead FB?
 U 1 1 5C9FE521
 P 5550 7350
@@
 P 9950 5100
 F 0 "Q110" V 10201 5100 50  0000 C CNN
-F 1 "Q_NMOS_GSD" V 10292 5100 50  0000 C CNN
+F 1 "LN235N3T5G " V 10292 5100 50  0000 C CNN
 F 2 "require:SOT-883" V 10383 5100 50  0000 C CNN
 F 3 "~" H 9950 5100 50  0001 C CNN

Commit message: wip
Parts:
- removed C259: 1u, require:C_0402, symbol Device:C
Connections:
- net +1V8: no longer U100.M17 (CODEC_AVDD_1V8_1), U100.N17 (CODEC_AVDD_1V8_2)
- net +3V3: no longer U100.P16 (CODEC_AVDD_3V3)
- no-connect marks 1 -> 4
Other:
- note removed: "P16"
Changed lines of the file:
@@
 	3300 5550 3300 5450
 Connection ~ 3300 5450
-Wire Wire Line
-	3100 5650 3300 5650
-Wire Wire Line
-	3300 5650 3300 5550
-Connection ~ 3300 5550
 $Comp
 L Device:C C?
@@
 Wire Wire Line
 	4850 6150 4850 6450
-Wire Wire Line
-	3500 6350 3500 6450
-Wire Wire Line
-	3100 6450 3500 6450
-Connection ~ 3500 6450
-Wire Wire Line
-	3500 6450 3500 6550
-Wire Wire Line
-	3100 6550 3500 6550
-Connection ~ 3500 6550
-Wire Wire Line
-	3500 6550 3500 6650
 Wire Wire Line
 	3100 8050 3300 8050
@@
 Text Notes 5400 5300 0    50   ~ 0
 D14/D13/E14
-$Comp
-L Device:C C?
-U 1 1 5C781190
-P 6050 5100
-AR Path="/5CED3BD3/5C781190" Ref="C?"  Part="1"
-AR Path="/5C325762/5C781190" Ref="C259"  Part="1"
-F 0 "C259" H 6165 5146 50  0000 L CNN
-F 1 "1u" H 6165 5055 50  0000 L CNN
-F 2 "require:C_0402" H 6088 4950 50  0001 C CNN
-F 3 "~" H 6050 5100 50  0001 C CNN
-	1    6050 5100
-	1    0    0    -1
-$EndComp
-Wire Wire Line
-	5450 4850 6050 4850
-Wire Wire Line
-	6050 4850 6050 4950
-$Comp
-L power:GND #PWR?
-U 1 1 5C7ABB6E
-P 6050 5350
-AR Path="/5CED3BD3/5C7ABB6E" Ref="#PWR?"  Part="1"
-AR Path="/5C325762/5C7ABB6E" Ref="#PWR0110"  Part="1"
-F 0 "#PWR0110" H 6050 5100 50  0001 C CNN
-F 1 "GND" H 6055 5177 50  0000 C CNN
-F 2 "" H 6050 5350 50  0001 C CNN
-F 3 "" H 6050 5350 50  0001 C CNN
-	1    6050 5350
-	1    0    0    -1
-$EndComp
-Wire Wire Line
-	6050 5250 6050 5350
-Text Notes 6100 5300 0    50   ~ 0
-P16
+NoConn ~ 3100 5650
+Wire Wire Line
+	3500 6350 3500 6650
+NoConn ~ 3100 6450
+NoConn ~ 3100 6550
 $EndSCHEMATC

Commit message: wip
Other:
- moved on the sheet: C229, C265
Changed lines of the file:
@@
 L Device:C C229
 U 1 1 5C84BC04
-P 4150 7650
-F 0 "C229" H 4265 7696 50  0000 L CNN
-F 1 "0.1u" H 4265 7605 50  0000 L CNN
-F 2 "require:C_0402" H 4188 7500 50  0001 C CNN
-F 3 "~" H 4150 7650 50  0001 C CNN
-	1    4150 7650
-	1    0    0    -1
-$EndComp
-Wire Wire Line
-	4150 7800 4150 8000
+P 4150 7600
+F 0 "C229" H 4265 7646 50  0000 L CNN
+F 1 "0.1u" H 4265 7555 50  0000 L CNN
+F 2 "require:C_0402" H 4188 7450 50  0001 C CNN
+F 3 "~" H 4150 7600 50  0001 C CNN
+	1    4150 7600
+	1    0    0    -1
+$EndComp
+Wire Wire Line
+	4150 7750 4150 7850
 $Comp
 L power:GND #PWR0203
 U 1 1 5C9782CF
-P 4150 8000
-F 0 "#PWR0203" H 4150 7750 50  0001 C CNN
-F 1 "GND" H 4155 7827 50  0000 C CNN
-F 2 "" H 4150 8000 50  0001 C CNN
-F 3 "" H 4150 8000 50  0001 C CNN
-	1    4150 8000
+P 4150 7850
+F 0 "#PWR0203" H 4150 7600 50  0001 C CNN
+F 1 "GND" H 4155 7677 50  0000 C CNN
+F 2 "" H 4150 7850 50  0001 C CNN
+F 3 "" H 4150 7850 50  0001 C CNN
+	1    4150 7850
 	1    0    0    -1
 $EndComp
@@
 L Device:C C265
 U 1 1 5C9A47A9
-P 3500 6800
-F 0 "C265" H 3615 6846 50  0000 L CNN
-F 1 "0.1u" H 3615 6755 50  0000 L CNN
-F 2 "require:C_0402" H 3538 6650 50  0001 C CNN
-F 3 "~" H 3500 6800 50  0001 C CNN
-	1    3500 6800
+P 3500 6600
+F 0 "C265" H 3615 6646 50  0000 L CNN
+F 1 "0.1u" H 3615 6555 50  0000 L CNN
+F 2 "require:C_0402" H 3538 6450 50  0001 C CNN
+F 3 "~" H 3500 6600 50  0001 C CNN
+	1    3500 6600
 	1    0    0    -1
 $EndComp
@@
 L power:GND #PWR0205
 U 1 1 5C9FD96A
-P 3500 7050
-F 0 "#PWR0205" H 3500 6800 50  0001 C CNN
-F 1 "GND" H 3505 6877 50  0000 C CNN
-F 2 "" H 3500 7050 50  0001 C CNN
-F 3 "" H 3500 7050 50  0001 C CNN
-	1    3500 7050
+P 3500 6850
+F 0 "#PWR0205" H 3500 6600 50  0001 C CNN
+F 1 "GND" H 3505 6677 50  0000 C CNN
+F 2 "" H 3500 6850 50  0001 C CNN
+F 3 "" H 3500 6850 50  0001 C CNN
+	1    3500 6850
 	1    0    0    -1
 $EndComp
@@
 Connection ~ 4850 6150
 Wire Wire Line
-	3500 6950 3500 7050
+	3500 6750 3500 6850
 Wire Wire Line
 	3100 6250 3500 6250
@@
 Connection ~ 4150 7350
 Wire Wire Line
-	4150 7350 4150 7500
+	4150 7350 4150 7450
 Wire Wire Line
 	3100 7450 3300 7450
@@
 NoConn ~ 3100 5650
 Wire Wire Line
-	3500 6350 3500 6650
+	3500 6350 3500 6450
 NoConn ~ 3100 6450
 NoConn ~ 3100 6550

Commit message: wip
Parts:
- C256, C258: value 1u -> 0.47u
Other:
- note added: "TSX-3225, X1E0000210129, 0.8@1k"
- moved on the sheet: C229, F229
Changed lines of the file:
@@
 L Device:C C229
 U 1 1 5C84BC04
-P 4150 7600
-F 0 "C229" H 4265 7646 50  0000 L CNN
-F 1 "0.1u" H 4265 7555 50  0000 L CNN
-F 2 "require:C_0402" H 4188 7450 50  0001 C CNN
-F 3 "~" H 4150 7600 50  0001 C CNN
-	1    4150 7600
-	1    0    0    -1
-$EndComp
-Wire Wire Line
-	4150 7750 4150 7850
+P 3600 7600
+F 0 "C229" H 3715 7646 50  0000 L CNN
+F 1 "0.1u" H 3715 7555 50  0000 L CNN
+F 2 "require:C_0402" H 3638 7450 50  0001 C CNN
+F 3 "~" H 3600 7600 50  0001 C CNN
+	1    3600 7600
+	1    0    0    -1
+$EndComp
+Wire Wire Line
+	3600 7750 3600 7850
 $Comp
 L power:GND #PWR0203
 U 1 1 5C9782CF
-P 4150 7850
-F 0 "#PWR0203" H 4150 7600 50  0001 C CNN
-F 1 "GND" H 4155 7677 50  0000 C CNN
-F 2 "" H 4150 7850 50  0001 C CNN
-F 3 "" H 4150 7850 50  0001 C CNN
-	1    4150 7850
+P 3600 7850
+F 0 "#PWR0203" H 3600 7600 50  0001 C CNN
+F 1 "GND" H 3605 7677 50  0000 C CNN
+F 2 "" H 3600 7850 50  0001 C CNN
+F 3 "" H 3600 7850 50  0001 C CNN
+	1    3600 7850
 	1    0    0    -1
 $EndComp
@@
 AR Path="/5C325762/5C9504D9" Ref="C256"  Part="1"
 F 0 "C256" H 4415 5146 50  0000 L CNN
-F 1 "1u" H 4415 5055 50  0000 L CNN
+F 1 "0.47u" H 4415 5055 50  0000 L CNN
 F 2 "require:C_0402" H 4338 4950 50  0001 C CNN
 F 3 "~" H 4300 5100 50  0001 C CNN
@@
 	3300 8950 3300 9050
 Wire Wire Line
-	4150 7250 4150 7350
+	3600 7250 3600 7350
 Wire Wire Line
 	3100 7350 3300 7350
-Connection ~ 4150 7350
-Wire Wire Line
-	4150 7350 4150 7450
+Connection ~ 3600 7350
+Wire Wire Line
+	3600 7350 3600 7450
 Wire Wire Line
 	3100 7450 3300 7450
 Wire Wire Line
 	3300 7450 3300 7350
-Connection ~ 3300 7350
-Wire Wire Line
-	3300 7350 4150 7350
+Wire Wire Line
+	3300 7350 3600 7350
 Wire Wire Line
 	8400 3400 8500 3400
@@
 AR Path="/5C325762/5E151295" Ref="C258"  Part="1"
 F 0 "C258" H 5565 5146 50  0000 L CNN
-F 1 "1u" H 5565 5055 50  0000 L CNN
+F 1 "0.47u" H 5565 5055 50  0000 L CNN
 F 2 "require:C_0402" H 5488 4950 50  0001 C CNN
 F 3 "~" H 5450 5100 50  0001 C CNN
@@
 L power:+1V0 #PWR0190
 U 1 1 5C9F5772
-P 4150 7250
-F 0 "#PWR0190" H 4150 7100 50  0001 C CNN
-F 1 "+1V0" H 4165 7423 50  0000 C CNN
-F 2 "" H 4150 7250 50  0001 C CNN
-F 3 "" H 4150 7250 50  0001 C CNN
-	1    4150 7250
-	1    0    0    -1
-$EndComp
-Wire Wire Line
-	5200 7250 5200 7350
-Wire Wire Line
-	5200 7350 5400 7350
-Wire Wire Line
-	5700 7350 5900 7350
-Wire Wire Line
-	5900 7350 5900 7250
+P 3600 7250
+F 0 "#PWR0190" H 3600 7100 50  0001 C CNN
+F 1 "+1V0" H 3615 7423 50  0000 C CNN
+F 2 "" H 3600 7250 50  0001 C CNN
+F 3 "" H 3600 7250 50  0001 C CNN
+	1    3600 7250
+	1    0    0    -1
+$EndComp
+Wire Wire Line
+	3600 7350 3800 7350
+Wire Wire Line
+	4100 7350 4300 7350
+Wire Wire Line
+	4300 7350 4300 7250
 $Comp
 L Device:Ferrite_Bead FB?
 U 1 1 5C9FE521
-P 5550 7350
+P 3950 7350
 AR Path="/5C2CD8AE/5C9FE521" Ref="FB?"  Part="1"
 AR Path="/5C325762/5C9FE521" Ref="F229"  Part="1"
-F 0 "F229" V 5740 7350 50  0000 C CNN
-F 1 "180R,1.5A" V 5649 7350 50  0000 C CNN
-F 2 "Inductors_SMD:L_0402" H 5550 7350 50  0001 C CNN
-F 3 "~" H 5550 7350 50  0001 C CNN
-	1    5550 7350
-	0    -1   -1   0
-$EndComp
-Text Notes 5200 7700 0    50   ~ 10
+F 0 "F229" V 3650 7350 50  0000 C CNN
+F 1 "180R,1.5A" V 3750 7350 50  0000 C CNN
+F 2 "Inductors_SMD:L_0402" H 3950 7350 50  0001 C CNN
+F 3 "~" H 3950 7350 50  0001 C CNN
+	1    3950 7350
+	0    1    1    0
+$EndComp
+Text Notes 5200 7900 0    50   ~ 10
 180 ohm @ 100MHz, 1.5A\nBLM15PX181SN1D (Tape)\nBLM15PX181SN1B (Bulk)
 $Comp
 L require:+1V0L #PWR?
 U 1 1 5C9FE529
-P 5200 7250
+P 4300 7250
 AR Path="/5C2CD8AE/5C9FE529" Ref="#PWR?"  Part="1"
 AR Path="/5C325762/5C9FE529" Ref="#PWR0148"  Part="1"
-F 0 "#PWR0148" H 5200 7100 50  0001 C CNN
-F 1 "+1V0L" H 5215 7423 50  0000 C CNN
-F 2 "" H 5200 7250 50  0001 C CNN
-F 3 "" H 5200 7250 50  0001 C CNN
-	1    5200 7250
-	1    0    0    -1
-$EndComp
-$Comp
-L power:+1V0 #PWR?
-U 1 1 5C9FE52F
-P 5900 7250
-AR Path="/5C2CD8AE/5C9FE52F" Ref="#PWR?"  Part="1"
-AR Path="/5C325762/5C9FE52F" Ref="#PWR0177"  Part="1"
-F 0 "#PWR0177" H 5900 7100 50  0001 C CNN
-F 1 "+1V0" H 5915 7423 50  0000 C CNN
-F 2 "" H 5900 7250 50  0001 C CNN
-F 3 "" H 5900 7250 50  0001 C CNN
-	1    5900 7250
+F 0 "#PWR0148" H 4300 7100 50  0001 C CNN
+F 1 "+1V0L" H 4315 7423 50  0000 C CNN
+F 2 "" H 4300 7250 50  0001 C CNN
+F 3 "" H 4300 7250 50  0001 C CNN
+	1    4300 7250
 	1    0    0    -1
 $EndComp
@@
 NoConn ~ 3100 6450
 NoConn ~ 3100 6550
+Connection ~ 3300 7350
+Text Notes 9500 3000 0    50   ~ 0
+TSX-3225, X1E0000210129, 0.8@1k
 $EndSCHEMATC
