File: hardware/rk3308-power.sch (KiCad schematic (older format))
At the start: 24 parts, among them Q110 LN235N3T5G, U100 RK3308, Y100 24MHz,12pF,10ppm

Commit message: wip
Parts:
- U100: footprint require:RK3308_BGA355 -> require:RK3308_TFBGA-355
- U100: footprint (none) -> require:RK3308_TFBGA-355
Changed lines of the file:
@@
 F 0 "U100" H 1200 14650 60  0000 C CNN
 F 1 "RK3308" H 1200 14750 60  0000 C CNN
-F 2 "require:RK3308_BGA355" H 1900 9400 60  0001 C CNN
+F 2 "require:RK3308_TFBGA-355" H 1900 9400 60  0001 C CNN
 F 3 "" H 1900 9400 60  0001 C CNN
 	12   1900 9400
@@
 F 0 "U100" H 14600 7137 60  0000 C CNN
 F 1 "RK3308" H 14600 7031 60  0000 C CNN
-F 2 "require:RK3308_BGA355" H 14100 4150 60  0001 C CNN
+F 2 "require:RK3308_TFBGA-355" H 14100 4150 60  0001 C CNN
 F 3 "" H 14100 4150 60  0001 C CNN
 	13   14100 4150
@@
 F 0 "U100" H 14600 11237 60  0000 C CNN
 F 1 "RK3308" H 14600 11131 60  0000 C CNN
-F 2 "require:RK3308_BGA355" H 14100 7950 60  0001 C CNN
+F 2 "require:RK3308_TFBGA-355" H 14100 7950 60  0001 C CNN
 F 3 "" H 14100 7950 60  0001 C CNN
 	14   14100 7950
@@
 F 0 "U100" H 7806 8587 60  0000 C CNN
 F 1 "RK3308" H 7806 8481 60  0000 C CNN
-F 2 "" H 7200 5800 60  0001 C CNN
+F 2 "require:RK3308_TFBGA-355" H 7200 5800 60  0001 C CNN
 F 3 "" H 7200 5800 60  0001 C CNN
 	1    7200 5800

Commit message: wip
Parts:
- Y100: footprint Crystals:Crystal_SMD_3225-4pin_3.2x2.5mm -> Crystals:Crystal_SMD_2016-4pin_2.0x1.6mm
Changed lines of the file:
@@
 F 0 "Y100" H 9500 3650 50  0000 L CNN
 F 1 "24MHz,12pF,10ppm" H 9500 3550 50  0000 L CNN
-F 2 "Crystals:Crystal_SMD_3225-4pin_3.2x2.5mm" H 9350 3400 50  0001 C CNN
+F 2 "Crystals:Crystal_SMD_2016-4pin_2.0x1.6mm" H 9350 3400 50  0001 C CNN
 F 3 "~" H 9350 3400 50  0001 C CNN
 	1    9350 3400

Commit message: wip
Parts:
- removed Q110: LN235N3T5G, require:SOT-883, symbol Device:Q_NMOS_GSD
- removed R111: 10k, require:R_0402, symbol Device:R
Connections:
- net RESET_1V8: no longer names the net of C110.1, R110.2, U100.B20 (NPOR_u)
Changed lines of the file:
@@
 	1    0    0    -1
 $EndComp
-Text Label 8600 5200 0    50   ~ 0
-RESET_1V8
 $Comp
 L Device:C C?
@@
 	9450 5200 9450 5100
 Wire Wire Line
-	9450 5200 9750 5200
-$Comp
-L Device:R R111
-U 1 1 5C7F3B7D
-P 10450 4950
-F 0 "R111" H 10520 4996 50  0000 L CNN
-F 1 "10k" H 10520 4905 50  0000 L CNN
-F 2 "require:R_0402" V 10380 4950 50  0001 C CNN
-F 3 "~" H 10450 4950 50  0001 C CNN
-	1    10450 4950
-	1    0    0    -1
-$EndComp
-Wire Wire Line
-	10150 5200 10450 5200
-Wire Wire Line
 	3700 4450 4300 4450
 Connection ~ 3700 4450
@@
 Wire Wire Line
 	8900 3500 8900 3400
-Wire Wire Line
-	9450 4800 9450 4700
-Wire Wire Line
-	9450 4700 9950 4700
-Wire Wire Line
-	9950 4700 9950 4900
-Wire Wire Line
-	9450 4600 9450 4700
-Connection ~ 9450 4700
 NoConn ~ 8400 5700
 Wire Wire Line
@@
 Wire Wire Line
 	9900 3800 9900 3900
-Connection ~ 9450 5200
-Wire Wire Line
-	10450 4800 10450 4600
-Wire Wire Line
-	10450 5100 10450 5200
 $Comp
 L Device:C C?
@@
 	4850 4850 5450 4850
 Connection ~ 4850 4850
-Text HLabel 10750 5200 2    50   Input ~ 0
-RESET
-Wire Wire Line
-	10750 5200 10450 5200
-Connection ~ 10450 5200
 $Comp
 L Device:C C110
@@
 F 3 "" H 8900 5700 50  0001 C CNN
 	1    8900 5700
-	1    0    0    -1
-$EndComp
-$Comp
-L power:+3V3 #PWR0137
-U 1 1 5C821550
-P 10450 4600
-F 0 "#PWR0137" H 10450 4450 50  0001 C CNN
-F 1 "+3V3" H 10465 4773 50  0000 C CNN
-F 2 "" H 10450 4600 50  0001 C CNN
-F 3 "" H 10450 4600 50  0001 C CNN
-	1    10450 4600
 	1    0    0    -1
 $EndComp
@@
 	1    0    0    -1
 $EndComp
-$Comp
-L Device:Q_NMOS_GSD Q110
-U 1 1 5C85D5B8
-P 9950 5100
-F 0 "Q110" V 10201 5100 50  0000 C CNN
-F 1 "LN235N3T5G " V 10292 5100 50  0000 C CNN
-F 2 "require:SOT-883" V 10383 5100 50  0000 C CNN
-F 3 "~" H 9950 5100 50  0001 C CNN
-	1    9950 5100
-	0    1    1    0
-$EndComp
 Text Notes 3750 5300 0    50   ~ 0
 N5
@@
 Text Notes 9500 3000 0    50   ~ 0
 TSX-3225, X1E0000210129, 0.8@1k
+Wire Wire Line
+	9450 4600 9450 4800
 $EndSCHEMATC

Commit message: prepare gerber and drill
Parts:
- F229, F269: footprint Inductors_SMD:L_0402 -> require:L_0402
- Y100: footprint Crystals:Crystal_SMD_2016-4pin_2.0x1.6mm -> require:Crystal_SMD_2016-4pin_2.0x1.6mm
Changed lines of the file:
@@
 F 0 "Y100" H 9500 3650 50  0000 L CNN
 F 1 "24MHz,12pF,10ppm" H 9500 3550 50  0000 L CNN
-F 2 "Crystals:Crystal_SMD_2016-4pin_2.0x1.6mm" H 9350 3400 50  0001 C CNN
+F 2 "require:Crystal_SMD_2016-4pin_2.0x1.6mm" H 9350 3400 50  0001 C CNN
 F 3 "~" H 9350 3400 50  0001 C CNN
 	1    9350 3400
@@
 F 0 "F269" V 4290 6050 50  0000 C CNN
 F 1 "180R,1.5A" V 4199 6050 50  0000 C CNN
-F 2 "Inductors_SMD:L_0402" H 4100 6050 50  0001 C CNN
+F 2 "require:L_0402" H 4100 6050 50  0001 C CNN
 F 3 "~" H 4100 6050 50  0001 C CNN
 	1    4100 6050
@@
 F 0 "F229" V 3650 7350 50  0000 C CNN
 F 1 "180R,1.5A" V 3750 7350 50  0000 C CNN
-F 2 "Inductors_SMD:L_0402" H 3950 7350 50  0001 C CNN
+F 2 "require:L_0402" H 3950 7350 50  0001 C CNN
 F 3 "~" H 3950 7350 50  0001 C CNN
 	1    3950 7350
