File: hardware/ddr.sch (KiCad schematic (older format))
At the start: 40 parts, among them U1000 RK3308, U13 SY8088AAC, U3000 DDR3_FBGA96

Commit message: wip
Parts:
- removed C2, C6: C, Capacitors_SMD:C_0603, symbol Device:C
- removed C3, C4, C5: C, Capacitors_SMD:C_0402, symbol Device:C
- removed L2: L, Inductors_SMD:L_Taiyo-Yuden_MD-4040, symbol Device:L
- removed R1, R2, R3: R, Resistors_SMD:R_0402, symbol Device:R
- removed U13: SY8088AAC, TO_SOT_Packages_SMD:SOT-23-5, symbol require:SY8088AAC
- added C300: 0.1u,10V, Capacitors_SMD:C_0402, symbol require-rescue:C
- added C301: 10u,10V, Capacitors_SMD:C_0805, symbol require-rescue:C
- added C302: 1n, Capacitors_SMD:C_0402, symbol require-rescue:C
- added C303: 22p, Capacitors_SMD:C_0402, symbol require-rescue:C
- added C304: 22u, Capacitors_SMD:C_0603, symbol require-rescue:C
- added C305: 0.1u, Capacitors_SMD:C_0402, symbol require-rescue:C
- added L300: 2.2u, require:L_murata_2520, symbol require-rescue:L
- added R300: 10k, Resistors_SMD:R_0402, symbol require-rescue:R
- added R302: 110k,1%, Resistors_SMD:R_0402, symbol require-rescue:R
- added R303: 150k,1%, Resistors_SMD:R_0402, symbol require-rescue:R
- added U300: SY8089AAC, TO_SOT_Packages_SMD:SOT-23-5, symbol require:SY8089AAC
Connections:
- net labels added: VDD_CORE
- wire segments 327 -> 331
Other:
- note added: "Murata DFE252012R-H-2R2M#\n"

Commit message: wip
Parts:
- removed C10: C, Capacitors_SMD:C_0402, symbol Device:C
- removed C302: 1n, Capacitors_SMD:C_0402, symbol require-rescue:C
- removed C305: 0.1u, Capacitors_SMD:C_0402, symbol require-rescue:C
- C310: renamed from C7; value C -> 10u
- C311: renamed from C8; value C -> 0.1u
- C312: renamed from C9; value C -> 0.1u
Connections:
- net labels removed: VDD_CORE
- wire segments 331 -> 321
Changed lines of the file:
@@
 $Descr A3 16535 11693
 encoding utf-8
-Sheet 4 7
+Sheet 4 8
 Title ""
 Date ""
@@
 Connection ~ 3750 4900
 $Comp
-L Device:C C10
-U 1 1 5C59BB3D
-P 3350 5250
-F 0 "C10" H 3465 5296 50  0000 L CNN
-F 1 "C" H 3465 5205 50  0000 L CNN
-F 2 "Capacitors_SMD:C_0402" H 3388 5100 50  0001 C CNN
-F 3 "~" H 3350 5250 50  0001 C CNN
-	1    3350 5250
-	1    0    0    -1
-$EndComp
-$Comp
-L Device:C C9
+L Device:C C312
 U 1 1 5C59BC64
 P 2950 5250
-F 0 "C9" H 3065 5296 50  0000 L CNN
-F 1 "C" H 3065 5205 50  0000 L CNN
+F 0 "C312" H 3065 5296 50  0000 L CNN
+F 1 "0.1u" H 3065 5205 50  0000 L CNN
 F 2 "Capacitors_SMD:C_0402" H 2988 5100 50  0001 C CNN
 F 3 "~" H 2950 5250 50  0001 C CNN
@@
 $EndComp
 $Comp
-L Device:C C8
+L Device:C C311
 U 1 1 5C59BCE6
 P 2550 5250
-F 0 "C8" H 2665 5296 50  0000 L CNN
-F 1 "C" H 2665 5205 50  0000 L CNN
+F 0 "C311" H 2665 5296 50  0000 L CNN
+F 1 "0.1u" H 2665 5205 50  0000 L CNN
 F 2 "Capacitors_SMD:C_0402" H 2588 5100 50  0001 C CNN
 F 3 "~" H 2550 5250 50  0001 C CNN
@@
 $EndComp
 $Comp
-L Device:C C7
+L Device:C C310
 U 1 1 5C59BD5B
 P 2150 5250
-F 0 "C7" H 2265 5296 50  0000 L CNN
-F 1 "C" H 2265 5205 50  0000 L CNN
+F 0 "C310" H 2265 5296 50  0000 L CNN
+F 1 "10u" H 2265 5205 50  0000 L CNN
 F 2 "Capacitors_SMD:C_0603" H 2188 5100 50  0001 C CNN
 F 3 "~" H 2150 5250 50  0001 C CNN
@@
 Connection ~ 2950 4900
 Wire Wire Line
-	2950 4900 3350 4900
-Wire Wire Line
-	3350 5100 3350 4900
-Connection ~ 3350 4900
-Wire Wire Line
-	3350 4900 3750 4900
-Wire Wire Line
-	3350 5400 3350 5600
-Wire Wire Line
-	3350 5600 2950 5600
-Wire Wire Line
 	2150 5600 2150 5400
 Wire Wire Line
@@
 Wire Wire Line
 	2950 5400 2950 5600
-Connection ~ 2950 5600
 Wire Wire Line
 	2950 5600 2550 5600
@@
 	1    2950 7800
 	0    1    1    0
-$EndComp
-$Comp
-L require-rescue:C C?
-U 1 1 5D112053
-P 3500 8150
-AR Path="/5D112053" Ref="C?"  Part="1"
-AR Path="/5C2CD8AE/5D112053" Ref="C?"  Part="1"
-AR Path="/5C325762/5D112053" Ref="C?"  Part="1"
-AR Path="/5C2F0873/5D112053" Ref="C302"  Part="1"
-F 0 "C302" H 3600 8200 50  0000 L CNN
-F 1 "1n" H 3600 8100 50  0000 L CNN
-F 2 "Capacitors_SMD:C_0402" H 3538 8000 50  0001 C CNN
-F 3 "" H 3500 8150 50  0001 C CNN
-	1    3500 8150
-	1    0    0    -1
-$EndComp
-$Comp
-L require-rescue:GND #PWR?
-U 1 1 5D11205A
-P 3500 8500
-AR Path="/5C2CD8AE/5D11205A" Ref="#PWR?"  Part="1"
-AR Path="/5C325762/5D11205A" Ref="#PWR?"  Part="1"
-AR Path="/5C2F0873/5D11205A" Ref="#PWR0156"  Part="1"
-F 0 "#PWR0156" H 3500 8250 50  0001 C CNN
-F 1 "GND" H 3500 8350 50  0000 C CNN
-F 2 "" H 3500 8500 50  0001 C CNN
-F 3 "" H 3500 8500 50  0001 C CNN
-	1    3500 8500
-	1    0    0    -1
-$EndComp
-$Comp
-L require-rescue:VDD_CORE #PWR?
-U 1 1 5D112060
-P 7050 7500
-AR Path="/5C2CD8AE/5D112060" Ref="#PWR?"  Part="1"
-AR Path="/5C325762/5D112060" Ref="#PWR?"  Part="1"
-AR Path="/5C2F0873/5D112060" Ref="#PWR0157"  Part="1"
-F 0 "#PWR0157" H 7050 7350 50  0001 C CNN
-F 1 "VDD_CORE" H 7050 7650 50  0000 C CNN
-F 2 "" H 7050 7500 50  0001 C CNN
-F 3 "" H 7050 7500 50  0001 C CNN
-	1    7050 7500
-	1    0    0    -1
 $EndComp
 $Comp
@@
 Wire Wire Line
 	3700 7700 3500 7700
-Wire Wire Line
-	3100 7800 3500 7800
 Connection ~ 2400 7600
-Wire Wire Line
-	3500 8300 3500 8500
 Wire Wire Line
 	6050 8100 6050 8300
@@
 	0    -1   -1   0
 $EndComp
-$Comp
-L require-rescue:C C?
-U 1 1 5D112092
-P 7050 7950
-AR Path="/5C2CD8AE/5D112092" Ref="C?"  Part="1"
-AR Path="/5C325762/5D112092" Ref="C?"  Part="1"
-AR Path="/5C2F0873/5D112092" Ref="C305"  Part="1"
-F 0 "C305" H 7150 8000 50  0000 L CNN
-F 1 "0.1u" H 7150 7900 50  0000 L CNN
-F 2 "Capacitors_SMD:C_0402" H 7088 7800 50  0001 C CNN
-F 3 "" H 7050 7950 50  0001 C CNN
-	1    7050 7950
-	1    0    0    -1
-$EndComp
 Wire Wire Line
 	6050 7600 6050 7800
-$Comp
-L require-rescue:GND #PWR?
-U 1 1 5D11209A
-P 7050 8300
-AR Path="/5C2CD8AE/5D11209A" Ref="#PWR?"  Part="1"
-AR Path="/5C325762/5D11209A" Ref="#PWR?"  Part="1"
-AR Path="/5C2F0873/5D11209A" Ref="#PWR0160"  Part="1"
-F 0 "#PWR0160" H 7050 8050 50  0001 C CNN
-F 1 "GND" H 7050 8150 50  0000 C CNN
-F 2 "" H 7050 8300 50  0001 C CNN
-F 3 "" H 7050 8300 50  0001 C CNN
-	1    7050 8300
-	1    0    0    -1
-$EndComp
-Wire Wire Line
-	7050 8100 7050 8300
 $Comp
 L require-rescue:R R?
@@
 Wire Wire Line
 	2400 7600 2400 7800
-Wire Wire Line
-	7050 7600 7050 7800
 $Comp
 L require:SY8089AAC U?
@@
 	4450 7600 4650 7600
 Wire Wire Line
-	3500 7800 3500 8000
-Wire Wire Line
 	2400 7800 2400 8000
-Connection ~ 3500 7800
-Wire Wire Line
-	3500 7800 3700 7800
 Connection ~ 5250 8500
 Wire Wire Line
@@
 Wire Wire Line
 	4450 7800 4800 7800
+Wire Wire Line
+	5250 7600 6050 7600
+Wire Wire Line
+	5250 7600 5250 8500
+$Comp
+L require:VCC_DDR #PWR0157
+U 1 1 5C4182E4
+P 6050 7500
+F 0 "#PWR0157" H 6050 7350 50  0001 C CNN
+F 1 "VCC_DDR" H 6067 7673 50  0000 C CNN
+F 2 "" H 6050 7500 50  0001 C CNN
+F 3 "" H 6050 7500 50  0001 C CNN
+	1    6050 7500
+	1    0    0    -1
+$EndComp
+Wire Wire Line
+	3100 7800 3700 7800
 $Comp
 L require-rescue:C C?
-U 1 1 5D1120DB
-P 1650 8150
-AR Path="/5D1120DB" Ref="C?"  Part="1"
-AR Path="/5C2CD8AE/5D1120DB" Ref="C?"  Part="1"
-AR Path="/5C325762/5D1120DB" Ref="C?"  Part="1"
-AR Path="/5C2F0873/5D1120DB" Ref="C300"  Part="1"
-F 0 "C300" H 1750 8200 50  0000 L CNN
-F 1 "0.1u,10V" H 1750 8100 50  0000 L CNN
-F 2 "Capacitors_SMD:C_0402" H 1688 8000 50  0001 C CNN
-F 3 "" H 1650 8150 50  0001 C CNN
-	1    1650 8150
-	1    0    0    -1
-$EndComp
-$Comp
-L power:GND #PWR?
-U 1 1 5D1120E2
-P 1650 8500
-AR Path="/5C325762/5D1120E2" Ref="#PWR?"  Part="1"
-AR Path="/5C2F0873/5D1120E2" Ref="#PWR0173"  Part="1"
-F 0 "#PWR0173" H 1650 8250 50  0001 C CNN
-F 1 "GND" H 1655 8327 50  0000 C CNN
-F 2 "" H 1650 8500 50  0001 C CNN
-F 3 "" H 1650 8500 50  0001 C CNN
-	1    1650 8500
-	1    0    0    -1
-$EndComp
-Wire Wire Line
-	1650 8500 1650 8300
-Wire Wire Line
-	1650 8000 1650 7600
-Connection ~ 7050 7600
-Wire Wire Line
-	7050 7500 7050 7600
-Wire Wire Line
-	6050 7600 7050 7600
+U 1 1 5C488E4A
+P 1800 8150
+AR Path="/5C2CD8AE/5C488E4A" Ref="C?"  Part="1"
+AR Path="/5C325762/5C488E4A" Ref="C?"  Part="1"
+AR Path="/5C2F0873/5C488E4A" Ref="C300"  Part="1"
+F 0 "C300" H 1900 8200 50  0000 L CNN
+F 1 "0.1u,10V" H 1900 8100 50  0000 L CNN
+F 2 "Capacitors_SMD:C_0402" H 1838 8000 50  0001 C CNN
+F 3 "" H 1800 8150 50  0001 C CNN
+	1    1800 8150
+	1    0    0    -1
+$EndComp
+Wire Wire Line
+	1800 8300 1800 8500
+$Comp
+L power:GND #PWR0156
+U 1 1 5C4A78F6
+P 1800 8500
+F 0 "#PWR0156" H 1800 8250 50  0001 C CNN
+F 1 "GND" H 1805 8327 50  0000 C CNN
+F 2 "" H 1800 8500 50  0001 C CNN
+F 3 "" H 1800 8500 50  0001 C CNN
+	1    1800 8500
+	1    0    0    -1
+$EndComp
+Wire Wire Line
+	1800 8000 1800 7600
+Wire Wire Line
+	1800 7600 2400 7600
+Wire Wire Line
+	6050 7600 6050 7500
 Connection ~ 6050 7600
 Wire Wire Line
-	1650 7600 2400 7600
-Wire Wire Line
-	5250 7600 6050 7600
-Wire Wire Line
-	5250 7600 5250 8500
+	2950 4900 3750 4900
 $EndSCHEMATC

Commit message: wip
Parts:
- removed C300: 0.1u,10V, Capacitors_SMD:C_0402, symbol require-rescue:C
- removed C301: 10u,10V, Capacitors_SMD:C_0805, symbol require-rescue:C
- removed C303: 22p, Capacitors_SMD:C_0402, symbol require-rescue:C
- removed C304: 22u, Capacitors_SMD:C_0603, symbol require-rescue:C
- removed L300: 2.2u, require:L_murata_2520, symbol require-rescue:L
- removed R300: 10k, Resistors_SMD:R_0402, symbol require-rescue:R
- removed R302: 110k,1%, Resistors_SMD:R_0402, symbol require-rescue:R
- removed R303: 150k,1%, Resistors_SMD:R_0402, symbol require-rescue:R
- removed U300: SY8089AAC, TO_SOT_Packages_SMD:SOT-23-5, symbol require:SY8089AAC
- renumbered C150 to C50, C151 to C51, C160 to C52, C161 to C53, C162 to C54, C163 to C55, C164 to C56, C165 to C57, C166 to C58, C167 to C59, C168 to C60, C169 to C61, C170 to C62, C171 to C63, C172 to C64, C173 to C65, C181 to C66, C180 to C67, C190 to C68, C310 to C80, C311 to C81, C312 to C82, R150 to R50, R180 to R51, R181 to R52, R190 to R53, R191 to R54, U3000 to U3
Connections:
- net labels removed: VCC5V0_SYS
- wire segments 321 -> 292
Other:
- note removed: "Murata DFE252012R-H-2R2M#\n"

Commit message: wip
Changed lines of the file:
@@
 DDR_D8
 Text Label 3500 3400 0    60   ~ 0
-DDR_D9
+DDR_D13
 Text Label 3500 3500 0    60   ~ 0
 DDR_D10
@@
 DDR_D12
 Text Label 3500 3800 0    60   ~ 0
-DDR_D13
+DDR_D9
 Text Label 3500 3900 0    60   ~ 0
 DDR_D14
@@
 DDR_D2
 Text Label 10600 2550 0    60   ~ 0
-DDR_D5
+DDR_D1
 Text Label 10600 2650 0    60   ~ 0
 DDR_D0
 Text Label 10600 2750 0    60   ~ 0
-DDR_D1
+DDR_D5
 Text Label 10600 2850 0    60   ~ 0
 DDR_D3

Commit message: wip
Parts:
- added C143: 1n, require:C_0402, symbol Device:C
- C52, C53, C54, C55, C56, C57, C58, C59, C60, C61, C62, C63, C64, C65, C66, C67, C68, C81, C82: footprint Capacitors_SMD:C_0402 -> require:C_0402
- C80: footprint Capacitors_SMD:C_0603 -> require:C_0603
- R50, R51, R52, R53, R54: footprint Resistors_SMD:R_0402 -> require:R_0402
Connections:
- wire segments 292 -> 296
Changed lines of the file:
@@
 F 0 "C82" H 3065 5296 50  0000 L CNN
 F 1 "0.1u" H 3065 5205 50  0000 L CNN
-F 2 "Capacitors_SMD:C_0402" H 2988 5100 50  0001 C CNN
+F 2 "require:C_0402" H 2988 5100 50  0001 C CNN
 F 3 "~" H 2950 5250 50  0001 C CNN
 	1    2950 5250
@@
 F 0 "C81" H 2665 5296 50  0000 L CNN
 F 1 "0.1u" H 2665 5205 50  0000 L CNN
-F 2 "Capacitors_SMD:C_0402" H 2588 5100 50  0001 C CNN
+F 2 "require:C_0402" H 2588 5100 50  0001 C CNN
 F 3 "~" H 2550 5250 50  0001 C CNN
 	1    2550 5250
@@
 F 0 "C80" H 2265 5296 50  0000 L CNN
 F 1 "10u" H 2265 5205 50  0000 L CNN
-F 2 "Capacitors_SMD:C_0603" H 2188 5100 50  0001 C CNN
+F 2 "require:C_0603" H 2188 5100 50  0001 C CNN
 F 3 "~" H 2150 5250 50  0001 C CNN
 	1    2150 5250
@@
 F 0 "R50" V 10043 4650 50  0000 C CNN
 F 1 "240R, 1%" V 10134 4650 50  0000 C CNN
-F 2 "Resistors_SMD:R_0402" V 10180 4650 50  0001 C CNN
+F 2 "require:R_0402" V 10180 4650 50  0001 C CNN
 F 3 "~" H 10250 4650 50  0001 C CNN
 	1    10250 4650
@@
 F 0 "C66" H 10715 7546 50  0000 L CNN
 F 1 "0.1u" H 10715 7455 50  0000 L CNN
-F 2 "Capacitors_SMD:C_0402" H 10638 7350 50  0001 C CNN
+F 2 "require:C_0402" H 10638 7350 50  0001 C CNN
 F 3 "~" H 10600 7500 50  0001 C CNN
 	1    10600 7500
@@
 F 0 "C67" H 10315 7546 50  0000 L CNN
 F 1 "1n" H 10315 7455 50  0000 L CNN
-F 2 "Capacitors_SMD:C_0402" H 10238 7350 50  0001 C CNN
+F 2 "require:C_0402" H 10238 7350 50  0001 C CNN
 F 3 "~" H 10200 7500 50  0001 C CNN
 	1    10200 7500
@@
 F 0 "R52" H 9870 7546 50  0000 L CNN
 F 1 "R" H 9870 7455 50  0000 L CNN
-F 2 "Resistors_SMD:R_0402" V 9730 7500 50  0001 C CNN
+F 2 "require:R_0402" V 9730 7500 50  0001 C CNN
 F 3 "~" H 9800 7500 50  0001 C CNN
 	1    9800 7500
@@
 F 0 "R51" H 9870 6846 50  0000 L CNN
 F 1 "R" H 9870 6755 50  0000 L CNN
-F 2 "Resistors_SMD:R_0402" V 9730 6800 50  0001 C CNN
+F 2 "require:R_0402" V 9730 6800 50  0001 C CNN
 F 3 "~" H 9800 6800 50  0001 C CNN
 	1    9800 6800
@@
 F 0 "C52" H 9915 8996 50  0000 L CNN
 F 1 "0.1u" H 9915 8905 50  0000 L CNN
-F 2 "Capacitors_SMD:C_0402" H 9838 8800 50  0001 C CNN
+F 2 "require:C_0402" H 9838 8800 50  0001 C CNN
 F 3 "~" H 9800 8950 50  0001 C CNN
 	1    9800 8950
@@
 F 0 "C53" H 10315 8996 50  0000 L CNN
 F 1 "0.1u" H 10315 8905 50  0000 L CNN
-F 2 "Capacitors_SMD:C_0402" H 10238 8800 50  0001 C CNN
+F 2 "require:C_0402" H 10238 8800 50  0001 C CNN
 F 3 "~" H 10200 8950 50  0001 C CNN
 	1    10200 8950
@@
 F 0 "C54" H 10715 8996 50  0000 L CNN
 F 1 "0.1u" H 10715 8905 50  0000 L CNN
-F 2 "Capacitors_SMD:C_0402" H 10638 8800 50  0001 C CNN
+F 2 "require:C_0402" H 10638 8800 50  0001 C CNN
 F 3 "~" H 10600 8950 50  0001 C CNN
 	1    10600 8950
@@
 F 0 "C55" H 11115 8996 50  0000 L CNN
 F 1 "0.1u" H 11115 8905 50  0000 L CNN
-F 2 "Capacitors_SMD:C_0402" H 11038 8800 50  0001 C CNN
+F 2 "require:C_0402" H 11038 8800 50  0001 C CNN
 F 3 "~" H 11000 8950 50  0001 C CNN
 	1    11000 8950
@@
 F 0 "C56" H 11515 8996 50  0000 L CNN
 F 1 "0.1u" H 11515 8905 50  0000 L CNN
-F 2 "Capacitors_SMD:C_0402" H 11438 8800 50  0001 C CNN
+F 2 "require:C_0402" H 11438 8800 50  0001 C CNN
 F 3 "~" H 11400 8950 50  0001 C CNN
 	1    11400 8950
@@
 F 0 "C57" H 11915 8996 50  0000 L CNN
 F 1 "0.1u" H 11915 8905 50  0000 L CNN
-F 2 "Capacitors_SMD:C_0402" H 11838 8800 50  0001 C CNN
+F 2 "require:C_0402" H 11838 8800 50  0001 C CNN
 F 3 "~" H 11800 8950 50  0001 C CNN
 	1    11800 8950
@@
 F 0 "C58" H 12315 8996 50  0000 L CNN
 F 1 "0.1u" H 12315 8905 50  0000 L CNN
-F 2 "Capacitors_SMD:C_0402" H 12238 8800 50  0001 C CNN
+F 2 "require:C_0402" H 12238 8800 50  0001 C CNN
 F 3 "~" H 12200 8950 50  0001 C CNN
 	1    12200 8950
@@
 F 0 "C59" H 12715 8996 50  0000 L CNN
 F 1 "0.1u" H 12715 8905 50  0000 L CNN
-F 2 "Capacitors_SMD:C_0402" H 12638 8800 50  0001 C CNN
+F 2 "require:C_0402" H 12638 8800 50  0001 C CNN
 F 3 "~" H 12600 8950 50  0001 C CNN
 	1    12600 8950
@@
 F 0 "C60" H 13115 8996 50  0000 L CNN
 F 1 "0.1u" H 13115 8905 50  0000 L CNN
-F 2 "Capacitors_SMD:C_0402" H 13038 8800 50  0001 C CNN
+F 2 "require:C_0402" H 13038 8800 50  0001 C CNN
 F 3 "~" H 13000 8950 50  0001 C CNN
 	1    13000 8950
@@
 F 0 "C61" H 13515 8996 50  0000 L CNN
 F 1 "0.1u" H 13515 8905 50  0000 L CNN
-F 2 "Capacitors_SMD:C_0402" H 13438 8800 50  0001 C CNN
+F 2 "require:C_0402" H 13438 8800 50  0001 C CNN
 F 3 "~" H 13400 8950 50  0001 C CNN
 	1    13400 8950
@@
 F 0 "C62" H 13915 8996 50  0000 L CNN
 F 1 "0.1u" H 13915 8905 50  0000 L CNN
-F 2 "Capacitors_SMD:C_0402" H 13838 8800 50  0001 C CNN
+F 2 "require:C_0402" H 13838 8800 50  0001 C CNN
 F 3 "~" H 13800 8950 50  0001 C CNN
 	1    13800 8950
@@
 F 0 "C63" H 14315 8996 50  0000 L CNN
 F 1 "0.1u" H 14315 8905 50  0000 L CNN
-F 2 "Capacitors_SMD:C_0402" H 14238 8800 50  0001 C CNN
+F 2 "require:C_0402" H 14238 8800 50  0001 C CNN
 F 3 "~" H 14200 8950 50  0001 C CNN
 	1    14200 8950
@@
 F 0 "C64" H 14715 8996 50  0000 L CNN
 F 1 "0.1u" H 14715 8905 50  0000 L CNN
-F 2 "Capacitors_SMD:C_0402" H 14638 8800 50  0001 C CNN
+F 2 "require:C_0402" H 14638 8800 50  0001 C CNN
 F 3 "~" H 14600 8950 50  0001 C CNN
 	1    14600 8950
@@
 F 0 "C65" H 15115 8996 50  0000 L CNN
 F 1 "0.1u" H 15115 8905 50  0000 L CNN
-F 2 "Capacitors_SMD:C_0402" H 15038 8800 50  0001 C CNN
+F 2 "require:C_0402" H 15038 8800 50  0001 C CNN
 F 3 "~" H 15000 8950 50  0001 C CNN
 	1    15000 8950
@@
 F 0 "R53" H 13930 4454 50  0000 R CNN
 F 1 "49.9R,1%" H 13930 4545 50  0000 R CNN
-F 2 "Resistors_SMD:R_0402" V 13930 4500 50  0001 C CNN
+F 2 "require:R_0402" V 13930 4500 50  0001 C CNN
 F 3 "~" H 14000 4500 50  0001 C CNN
 	1    14000 4500
@@
 F 0 "R54" H 14430 4454 50  0000 R CNN
 F 1 "49.9R,1%" H 14430 4545 50  0000 R CNN
-F 2 "Resistors_SMD:R_0402" V 14430 4500 50  0001 C CNN
+F 2 "require:R_0402" V 14430 4500 50  0001 C CNN
 F 3 "~" H 14500 4500 50  0001 C CNN
 	1    14500 4500
@@
 F 0 "C68" H 14115 5246 50  0000 L CNN
 F 1 "100p" H 14115 5155 50  0000 L CNN
-F 2 "Capacitors_SMD:C_0402" H 14038 5050 50  0001 C CNN
+F 2 "require:C_0402" H 14038 5050 50  0001 C CNN
 F 3 "~" H 14000 5200 50  0001 C CNN
 	1    14000 5200
@@
 Wire Wire Line
 	2950 4900 3750 4900
+$Comp
+L Device:C C143
+U 1 1 5C573356
+P 9400 7500
+F 0 "C143" H 9515 7546 50  0000 L CNN
+F 1 "1n" H 9515 7455 50  0000 L CNN
+F 2 "require:C_0402" H 9438 7350 50  0001 C CNN
+F 3 "~" H 9400 7500 50  0001 C CNN
+	1    9400 7500
+	1    0    0    -1
+$EndComp
+Wire Wire Line
+	9800 7150 9400 7150
+Wire Wire Line
+	9400 7150 9400 7350
+Wire Wire Line
+	9800 7850 9400 7850
+Wire Wire Line
+	9400 7850 9400 7650
 $EndSCHEMATC
