File: hardware/ddr.sch (KiCad schematic (older format))
At the start: 30 parts, among them U1000 RK3308, U3 DDR3_FBGA96

Commit message: wip
Parts:
- C50, C51: footprint Capacitors_SMD:C_0805 -> require:C_0805
- renumbered C143 to C69, U3 to U4
Changed lines of the file:
@@
 $EndDescr
 $Comp
-L require-rescue:DDR3_FBGA96 U3
+L require-rescue:DDR3_FBGA96 U4
 U 1 1 5C2F087E
 P 11800 1550
-F 0 "U3" H 11800 1700 60  0000 C CNN
+F 0 "U4" H 11800 1700 60  0000 C CNN
 F 1 "DDR3_FBGA96" H 11850 1600 60  0000 C CNN
 F 2 "require:DDR3_BGA_96" H 11800 1550 60  0001 C CNN
@@
 F 0 "C51" H 9115 5546 50  0000 L CNN
 F 1 "10u" H 9115 5455 50  0000 L CNN
-F 2 "Capacitors_SMD:C_0805" H 9038 5350 50  0001 C CNN
+F 2 "require:C_0805" H 9038 5350 50  0001 C CNN
 F 3 "~" H 9000 5500 50  0001 C CNN
 	1    9000 5500
@@
 F 0 "C50" H 8715 5546 50  0000 L CNN
 F 1 "10u" H 8715 5455 50  0000 L CNN
-F 2 "Capacitors_SMD:C_0805" H 8638 5350 50  0000 C CNN
+F 2 "require:C_0805" H 8638 5350 50  0000 C CNN
 F 3 "~" H 8600 5500 50  0001 C CNN
 	1    8600 5500
@@
 	2950 4900 3750 4900
 $Comp
-L Device:C C143
+L Device:C C69
 U 1 1 5C573356
 P 9400 7500
-F 0 "C143" H 9515 7546 50  0000 L CNN
+F 0 "C69" H 9515 7546 50  0000 L CNN
 F 1 "1n" H 9515 7455 50  0000 L CNN
 F 2 "require:C_0402" H 9438 7350 50  0001 C CNN

Commit message: wip
Parts:
- C50, C51: footprint require:C_0805 -> require:C_0603
Changed lines of the file:
@@
 F 0 "C51" H 9115 5546 50  0000 L CNN
 F 1 "10u" H 9115 5455 50  0000 L CNN
-F 2 "require:C_0805" H 9038 5350 50  0001 C CNN
+F 2 "require:C_0603" H 9038 5350 50  0001 C CNN
 F 3 "~" H 9000 5500 50  0001 C CNN
 	1    9000 5500
@@
 F 0 "C50" H 8715 5546 50  0000 L CNN
 F 1 "10u" H 8715 5455 50  0000 L CNN
-F 2 "require:C_0805" H 8638 5350 50  0000 C CNN
+F 2 "require:C_0603" H 8638 5350 50  0000 C CNN
 F 3 "~" H 8600 5500 50  0001 C CNN
 	1    8600 5500

Commit message: wip
Parts:
- added C302: 10u, require:C_0603, symbol Device:C
- renumbered C50 to C300, C51 to C301, C52 to C310, C53 to C311, C54 to C312, C55 to C313, C56 to C314, C57 to C315, C58 to C316, C59 to C317, C60 to C318, C61 to C319, C62 to C320, C63 to C321, C64 to C322, C65 to C323, C66 to C330, C69 to C331, C67 to C332, C68 to C340, C80 to C350, C81 to C351, C82 to C352, R51 to R330, R52 to R331, R53 to R340, R54 to R341, U4 to U300
Connections:
- wire segments 296 -> 300
Changed lines of the file:
@@
 $EndDescr
 $Comp
-L require-rescue:DDR3_FBGA96 U4
+L require-rescue:DDR3_FBGA96 U300
 U 1 1 5C2F087E
 P 11800 1550
-F 0 "U4" H 11800 1700 60  0000 C CNN
+F 0 "U300" H 11800 1700 60  0000 C CNN
 F 1 "DDR3_FBGA96" H 11850 1600 60  0000 C CNN
 F 2 "require:DDR3_BGA_96" H 11800 1550 60  0001 C CNN
@@
 DDR_D9
 Text Label 10600 1950 0    60   ~ 0
+DDR_D14
+Text Label 10600 2050 0    60   ~ 0
 DDR_D15
-Text Label 10600 2050 0    60   ~ 0
-DDR_D12
 Text Label 10600 2150 0    60   ~ 0
 DDR_D11
 Text Label 10600 2250 0    60   ~ 0
-DDR_D14
+DDR_D12
 Text Label 10600 2350 0    60   ~ 0
 DDR_D8
 Text Label 10600 2450 0    60   ~ 0
+DDR_D6
+Text Label 10600 2550 0    60   ~ 0
 DDR_D2
-Text Label 10600 2550 0    60   ~ 0
-DDR_D1
 Text Label 10600 2650 0    60   ~ 0
+DDR_D5
+Text Label 10600 2750 0    60   ~ 0
 DDR_D0
-Text Label 10600 2750 0    60   ~ 0
-DDR_D5
 Text Label 10600 2850 0    60   ~ 0
 DDR_D3
 Text Label 10600 2950 0    60   ~ 0
-DDR_D6
+DDR_D1
 Text Label 10600 3050 0    60   ~ 0
 DDR_D7
@@
 Connection ~ 3750 4900
 $Comp
-L Device:C C82
+L Device:C C352
 U 1 1 5C59BC64
 P 2950 5250
-F 0 "C82" H 3065 5296 50  0000 L CNN
+F 0 "C352" H 3065 5296 50  0000 L CNN
 F 1 "0.1u" H 3065 5205 50  0000 L CNN
 F 2 "require:C_0402" H 2988 5100 50  0001 C CNN
@@
 $EndComp
 $Comp
-L Device:C C81
+L Device:C C351
 U 1 1 5C59BCE6
 P 2550 5250
-F 0 "C81" H 2665 5296 50  0000 L CNN
+F 0 "C351" H 2665 5296 50  0000 L CNN
 F 1 "0.1u" H 2665 5205 50  0000 L CNN
 F 2 "require:C_0402" H 2588 5100 50  0001 C CNN
@@
 $EndComp
 $Comp
-L Device:C C80
+L Device:C C350
 U 1 1 5C59BD5B
 P 2150 5250
-F 0 "C80" H 2265 5296 50  0000 L CNN
+F 0 "C350" H 2265 5296 50  0000 L CNN
 F 1 "10u" H 2265 5205 50  0000 L CNN
-F 2 "require:C_0603" H 2188 5100 50  0001 C CNN
+F 2 "require:C_0603" H 2188 5100 50  0000 C CNN
 F 3 "~" H 2150 5250 50  0001 C CNN
 	1    2150 5250
@@
 Connection ~ 11000 6150
 $Comp
-L Device:C C51
+L Device:C C301
 U 1 1 5C738430
 P 9000 5500
-F 0 "C51" H 9115 5546 50  0000 L CNN
+F 0 "C301" H 9115 5546 50  0000 L CNN
 F 1 "10u" H 9115 5455 50  0000 L CNN
-F 2 "require:C_0603" H 9038 5350 50  0001 C CNN
+F 2 "require:C_0603" H 9038 5350 50  0000 C CNN
 F 3 "~" H 9000 5500 50  0001 C CNN
 	1    9000 5500
@@
 $EndComp
 $Comp
-L Device:C C50
+L Device:C C300
 U 1 1 5C7384A7
 P 8600 5500
-F 0 "C50" H 8715 5546 50  0000 L CNN
+F 0 "C300" H 8715 5546 50  0000 L CNN
 F 1 "10u" H 8715 5455 50  0000 L CNN
 F 2 "require:C_0603" H 8638 5350 50  0000 C CNN
@@
 	11000 7250 11200 7250
 $Comp
-L Device:C C66
+L Device:C C330
 U 1 1 5C8A1A28
 P 10600 7500
-F 0 "C66" H 10715 7546 50  0000 L CNN
+F 0 "C330" H 10715 7546 50  0000 L CNN
 F 1 "0.1u" H 10715 7455 50  0000 L CNN
 F 2 "require:C_0402" H 10638 7350 50  0001 C CNN
@@
 Connection ~ 11000 7150
 $Comp
-L Device:C C67
+L Device:C C332
 U 1 1 5C8B7D29
 P 10200 7500
-F 0 "C67" H 10315 7546 50  0000 L CNN
+F 0 "C332" H 10315 7546 50  0000 L CNN
 F 1 "1n" H 10315 7455 50  0000 L CNN
 F 2 "require:C_0402" H 10238 7350 50  0001 C CNN
@@
 Connection ~ 10600 7150
 $Comp
-L Device:R R52
+L Device:R R331
 U 1 1 5C8CE3CA
 P 9800 7500
-F 0 "R52" H 9870 7546 50  0000 L CNN
+F 0 "R331" H 9870 7546 50  0000 L CNN
 F 1 "R" H 9870 7455 50  0000 L CNN
 F 2 "require:R_0402" V 9730 7500 50  0001 C CNN
@@
 $EndComp
 $Comp
-L Device:R R51
+L Device:R R330
 U 1 1 5C8CE4D2
 P 9800 6800
-F 0 "R51" H 9870 6846 50  0000 L CNN
+F 0 "R330" H 9870 6846 50  0000 L CNN
 F 1 "R" H 9870 6755 50  0000 L CNN
 F 2 "require:R_0402" V 9730 6800 50  0001 C CNN
@@
 $EndComp
 $Comp
-L Device:C C52
+L Device:C C310
 U 1 1 5C979E19
 P 9800 8950
-F 0 "C52" H 9915 8996 50  0000 L CNN
+F 0 "C310" H 9915 8996 50  0000 L CNN
 F 1 "0.1u" H 9915 8905 50  0000 L CNN
 F 2 "require:C_0402" H 9838 8800 50  0001 C CNN
@@
 $EndComp
 $Comp
-L Device:C C53
+L Device:C C311
 U 1 1 5C97A08B
 P 10200 8950
-F 0 "C53" H 10315 8996 50  0000 L CNN
+F 0 "C311" H 10315 8996 50  0000 L CNN
 F 1 "0.1u" H 10315 8905 50  0000 L CNN
 F 2 "require:C_0402" H 10238 8800 50  0001 C CNN
@@
 $EndComp
 $Comp
-L Device:C C54
+L Device:C C312
 U 1 1 5C97A26C
 P 10600 8950
-F 0 "C54" H 10715 8996 50  0000 L CNN
+F 0 "C312" H 10715 8996 50  0000 L CNN
 F 1 "0.1u" H 10715 8905 50  0000 L CNN
 F 2 "require:C_0402" H 10638 8800 50  0001 C CNN
@@
 $EndComp
 $Comp
-L Device:C C55
+L Device:C C313
 U 1 1 5C97A3E8
 P 11000 8950
-F 0 "C55" H 11115 8996 50  0000 L CNN
+F 0 "C313" H 11115 8996 50  0000 L CNN
 F 1 "0.1u" H 11115 8905 50  0000 L CNN
 F 2 "require:C_0402" H 11038 8800 50  0001 C CNN
@@
 $EndComp
 $Comp
-L Device:C C56
+L Device:C C314
 U 1 1 5C97A44E
 P 11400 8950
-F 0 "C56" H 11515 8996 50  0000 L CNN
+F 0 "C314" H 11515 8996 50  0000 L CNN
 F 1 "0.1u" H 11515 8905 50  0000 L CNN
 F 2 "require:C_0402" H 11438 8800 50  0001 C CNN
@@
 $EndComp
 $Comp
-L Device:C C57
+L Device:C C315
 U 1 1 5C97A4AA
 P 11800 8950
-F 0 "C57" H 11915 8996 50  0000 L CNN
+F 0 "C315" H 11915 8996 50  0000 L CNN
 F 1 "0.1u" H 11915 8905 50  0000 L CNN
 F 2 "require:C_0402" H 11838 8800 50  0001 C CNN
@@
 $EndComp
 $Comp
-L Device:C C58
+L Device:C C316
 U 1 1 5C97A508
 P 12200 8950
-F 0 "C58" H 12315 8996 50  0000 L CNN
+F 0 "C316" H 12315 8996 50  0000 L CNN
 F 1 "0.1u" H 12315 8905 50  0000 L CNN
 F 2 "require:C_0402" H 12238 8800 50  0001 C CNN
@@
 $EndComp
 $Comp
-L Device:C C59
+L Device:C C317
 U 1 1 5C97A56A
 P 12600 8950
-F 0 "C59" H 12715 8996 50  0000 L CNN
+F 0 "C317" H 12715 8996 50  0000 L CNN
 F 1 "0.1u" H 12715 8905 50  0000 L CNN
 F 2 "require:C_0402" H 12638 8800 50  0001 C CNN
@@
 $EndComp
 $Comp
-L Device:C C60
+L Device:C C318
 U 1 1 5C97A966
 P 13000 8950
-F 0 "C60" H 13115 8996 50  0000 L CNN
+F 0 "C318" H 13115 8996 50  0000 L CNN
 F 1 "0.1u" H 13115 8905 50  0000 L CNN
 F 2 "require:C_0402" H 13038 8800 50  0001 C CNN
@@
 $EndComp
 $Comp
-L Device:C C61
+L Device:C C319
 U 1 1 5C97A9CC
 P 13400 8950
-F 0 "C61" H 13515 8996 50  0000 L CNN
+F 0 "C319" H 13515 8996 50  0000 L CNN
 F 1 "0.1u" H 13515 8905 50  0000 L CNN
 F 2 "require:C_0402" H 13438 8800 50  0001 C CNN
@@
 $EndComp
 $Comp
-L Device:C C62
+L Device:C C320
 U 1 1 5C97AA36
 P 13800 8950
-F 0 "C62" H 13915 8996 50  0000 L CNN
+F 0 "C320" H 13915 8996 50  0000 L CNN
 F 1 "0.1u" H 13915 8905 50  0000 L CNN
 F 2 "require:C_0402" H 13838 8800 50  0001 C CNN
@@
 $EndComp
 $Comp
-L Device:C C63
+L Device:C C321
 U 1 1 5C97AAC4
 P 14200 8950
-F 0 "C63" H 14315 8996 50  0000 L CNN
+F 0 "C321" H 14315 8996 50  0000 L CNN
 F 1 "0.1u" H 14315 8905 50  0000 L CNN
 F 2 "require:C_0402" H 14238 8800 50  0001 C CNN
@@
 $EndComp
 $Comp
-L Device:C C64
+L Device:C C322
 U 1 1 5C97AB2E
 P 14600 8950
-F 0 "C64" H 14715 8996 50  0000 L CNN
+F 0 "C322" H 14715 8996 50  0000 L CNN
 F 1 "0.1u" H 14715 8905 50  0000 L CNN
 F 2 "require:C_0402" H 14638 8800 50  0001 C CNN
@@
 $EndComp
 $Comp
-L Device:C C65
+L Device:C C323
 U 1 1 5C97AB9A
 P 15000 8950
-F 0 "C65" H 15115 8996 50  0000 L CNN
+F 0 "C323" H 15115 8996 50  0000 L CNN
 F 1 "0.1u" H 15115 8905 50  0000 L CNN
 F 2 "require:C_0402" H 15038 8800 50  0001 C CNN
@@
 0402, 0.1u x 14
 Wire Wire Line
-	9000 5150 11000 5150
-$Comp
-L Device:R R53
+	9000 5150 9600 5150
+$Comp
+L Device:R R340
 U 1 1 5CC9FD8E
 P 14000 4500
-F 0 "R53" H 13930 4454 50  0000 R CNN
+F 0 "R340" H 13930 4454 50  0000 R CNN
 F 1 "49.9R,1%" H 13930 4545 50  0000 R CNN
 F 2 "require:R_0402" V 13930 4500 50  0001 C CNN
@@
 $EndComp
 $Comp
-L Device:R R54
+L Device:R R341
 U 1 1 5CC9FF46
 P 14500 4500
-F 0 "R54" H 14430 4454 50  0000 R CNN
+F 0 "R341" H 14430 4454 50  0000 R CNN
 F 1 "49.9R,1%" H 14430 4545 50  0000 R CNN
 F 2 "require:R_0402" V 14430 4500 50  0001 C CNN
@@
 	14000 4650 14000 4850
 $Comp
-L Device:C C68
+L Device:C C340
 U 1 1 5CCF6D8A
 P 14000 5200
-F 0 "C68" H 14115 5246 50  0000 L CNN
+F 0 "C340" H 14115 5246 50  0000 L CNN
 F 1 "100p" H 14115 5155 50  0000 L CNN
 F 2 "require:C_0402" H 14038 5050 50  0001 C CNN
@@
 	2950 4900 3750 4900
 $Comp
-L Device:C C69
+L Device:C C331
 U 1 1 5C573356
 P 9400 7500
-F 0 "C69" H 9515 7546 50  0000 L CNN
+F 0 "C331" H 9515 7546 50  0000 L CNN
 F 1 "1n" H 9515 7455 50  0000 L CNN
 F 2 "require:C_0402" H 9438 7350 50  0001 C CNN
@@
 Wire Wire Line
 	9400 7850 9400 7650
+$Comp
+L Device:C C302
+U 1 1 5C74EB52
+P 9600 5500
+F 0 "C302" H 9715 5546 50  0000 L CNN
+F 1 "10u" H 9715 5455 50  0000 L CNN
+F 2 "require:C_0603" H 9638 5350 50  0000 C CNN
+F 3 "~" H 9600 5500 50  0001 C CNN
+	1    9600 5500
+	1    0    0    -1
+$EndComp
+Wire Wire Line
+	9600 5350 9600 5150
+Connection ~ 9600 5150
+Wire Wire Line
+	9600 5150 11000 5150
+Wire Wire Line
+	9600 5650 9600 5850
+Wire Wire Line
+	9600 5850 9000 5850
+Connection ~ 9000 5850
 $EndSCHEMATC

Commit message: wip
Parts:
- U100: renamed from U1000; symbol require-rescue:RK3308 -> require:RK3308
- U300: symbol require-rescue:DDR3_FBGA96 -> require:DDR3_FBGA96
Other:
- moved on the sheet: C301, C340, R340, R341
Changed lines of the file:
@@
 $EndDescr
 $Comp
-L require-rescue:DDR3_FBGA96 U300
+L require:DDR3_FBGA96 U300
 U 1 1 5C2F087E
 P 11800 1550
@@
 $EndComp
 $Comp
-L require-rescue:RK3308 U1000
+L require:RK3308 U100
 U 11 1 5C2F758B
 P 4150 5700
-F 0 "U1000" H 4150 5650 60  0000 L CNN
+F 0 "U100" H 4150 5650 60  0000 L CNN
 F 1 "RK3308" H 4150 5550 60  0000 L CNN
 F 2 "require:RK3308_BGA355" H 4150 5700 60  0001 C CNN
@@
 F 0 "C350" H 2265 5296 50  0000 L CNN
 F 1 "10u" H 2265 5205 50  0000 L CNN
-F 2 "require:C_0603" H 2188 5100 50  0000 C CNN
+F 2 "require:C_0603" H 2188 5100 50  0001 C CNN
 F 3 "~" H 2150 5250 50  0001 C CNN
 	1    2150 5250
@@
 L Device:C C301
 U 1 1 5C738430
-P 9000 5500
-F 0 "C301" H 9115 5546 50  0000 L CNN
-F 1 "10u" H 9115 5455 50  0000 L CNN
-F 2 "require:C_0603" H 9038 5350 50  0000 C CNN
-F 3 "~" H 9000 5500 50  0001 C CNN
-	1    9000 5500
+P 9100 5500
+F 0 "C301" H 9215 5546 50  0000 L CNN
+F 1 "10u" H 9215 5455 50  0000 L CNN
+F 2 "require:C_0603" H 9138 5350 50  0001 C CNN
+F 3 "~" H 9100 5500 50  0001 C CNN
+	1    9100 5500
 	1    0    0    -1
 $EndComp
@@
 F 0 "C300" H 8715 5546 50  0000 L CNN
 F 1 "10u" H 8715 5455 50  0000 L CNN
-F 2 "require:C_0603" H 8638 5350 50  0000 C CNN
+F 2 "require:C_0603" H 8638 5350 50  0001 C CNN
 F 3 "~" H 8600 5500 50  0001 C CNN
 	1    8600 5500
@@
 Connection ~ 11000 5150
 Wire Wire Line
-	9000 5350 9000 5150
-Connection ~ 9000 5150
-Wire Wire Line
-	9000 5150 8600 5150
+	9100 5350 9100 5150
+Connection ~ 9100 5150
+Wire Wire Line
+	9100 5150 8600 5150
 Wire Wire Line
 	8600 5850 8600 5650
 Wire Wire Line
-	9000 5650 9000 5850
-Wire Wire Line
-	9000 5850 8600 5850
+	9100 5650 9100 5850
+Wire Wire Line
+	9100 5850 8600 5850
 $Comp
 L require:VCC_DDR #PWR0116
@@
 0402, 0.1u x 14
 Wire Wire Line
-	9000 5150 9600 5150
+	9100 5150 9600 5150
 $Comp
 L Device:R R340
 U 1 1 5CC9FD8E
-P 14000 4500
-F 0 "R340" H 13930 4454 50  0000 R CNN
-F 1 "49.9R,1%" H 13930 4545 50  0000 R CNN
-F 2 "require:R_0402" V 13930 4500 50  0001 C CNN
-F 3 "~" H 14000 4500 50  0001 C CNN
-	1    14000 4500
+P 14000 4100
+F 0 "R340" H 13930 4054 50  0000 R CNN
+F 1 "49.9R,1%" H 13930 4145 50  0000 R CNN
+F 2 "require:R_0402" V 13930 4100 50  0001 C CNN
+F 3 "~" H 14000 4100 50  0001 C CNN
+	1    14000 4100
 	-1   0    0    1
 $EndComp
@@
 L Device:R R341
 U 1 1 5CC9FF46
-P 14500 4500
-F 0 "R341" H 14430 4454 50  0000 R CNN
-F 1 "49.9R,1%" H 14430 4545 50  0000 R CNN
-F 2 "require:R_0402" V 14430 4500 50  0001 C CNN
-F 3 "~" H 14500 4500 50  0001 C CNN
-	1    14500 4500
+P 14500 4100
+F 0 "R341" H 14430 4054 50  0000 R CNN
+F 1 "49.9R,1%" H 14430 4145 50  0000 R CNN
+F 2 "require:R_0402" V 14430 4100 50  0001 C CNN
+F 3 "~" H 14500 4100 50  0001 C CNN
+	1    14500 4100
 	-1   0    0    1
 $EndComp
 Wire Wire Line
-	14000 3850 14000 4350
+	14000 3850 14000 3950
 Wire Wire Line
 	12400 3850 14000 3850
 Wire Wire Line
-	14000 4650 14000 4850
+	14000 4250 14000 4350
 $Comp
 L Device:C C340
 U 1 1 5CCF6D8A
-P 14000 5200
-F 0 "C340" H 14115 5246 50  0000 L CNN
-F 1 "100p" H 14115 5155 50  0000 L CNN
-F 2 "require:C_0402" H 14038 5050 50  0001 C CNN
-F 3 "~" H 14000 5200 50  0001 C CNN
-	1    14000 5200
-	1    0    0    -1
-$EndComp
-Wire Wire Line
-	14000 4850 14000 5050
-Connection ~ 14000 4850
-Wire Wire Line
-	14000 5350 14000 5550
+P 14000 4600
+F 0 "C340" H 14115 4646 50  0000 L CNN
+F 1 "100p" H 14115 4555 50  0000 L CNN
+F 2 "require:C_0402" H 14038 4450 50  0001 C CNN
+F 3 "~" H 14000 4600 50  0001 C CNN
+	1    14000 4600
+	1    0    0    -1
+$EndComp
+Wire Wire Line
+	14000 4750 14000 4850
 $Comp
 L power:GND #PWR0123
 U 1 1 5CD314AE
-P 14000 5550
-F 0 "#PWR0123" H 14000 5300 50  0001 C CNN
-F 1 "GND" H 14005 5377 50  0000 C CNN
-F 2 "" H 14000 5550 50  0001 C CNN
-F 3 "" H 14000 5550 50  0001 C CNN
-	1    14000 5550
-	1    0    0    -1
-$EndComp
-Wire Wire Line
-	14500 4350 14500 3750
+P 14000 4850
+F 0 "#PWR0123" H 14000 4600 50  0001 C CNN
+F 1 "GND" H 14005 4677 50  0000 C CNN
+F 2 "" H 14000 4850 50  0001 C CNN
+F 3 "" H 14000 4850 50  0001 C CNN
+	1    14000 4850
+	1    0    0    -1
+$EndComp
+Wire Wire Line
+	14500 3950 14500 3750
 Wire Wire Line
 	12400 3750 14500 3750
 Wire Wire Line
-	14500 4650 14500 4850
-Wire Wire Line
-	14000 4850 14500 4850
+	14500 4250 14500 4350
 Wire Wire Line
 	2950 4900 3750 4900
@@
 F 0 "C302" H 9715 5546 50  0000 L CNN
 F 1 "10u" H 9715 5455 50  0000 L CNN
-F 2 "require:C_0603" H 9638 5350 50  0000 C CNN
+F 2 "require:C_0603" H 9638 5350 50  0001 C CNN
 F 3 "~" H 9600 5500 50  0001 C CNN
 	1    9600 5500
@@
 	9600 5650 9600 5850
 Wire Wire Line
-	9600 5850 9000 5850
-Connection ~ 9000 5850
+	9600 5850 9100 5850
+Connection ~ 9100 5850
+Wire Wire Line
+	14000 4350 14500 4350
+Connection ~ 14000 4350
+Wire Wire Line
+	14000 4350 14000 4450
 $EndSCHEMATC

Commit message: wip
Parts:
- added C324, C325, C326: 0.1u, require:C_0402, symbol Device:C
Connections:
- wire segments 300 -> 312
Changed lines of the file:
@@
 Wire Wire Line
 	14000 4350 14000 4450
+$Comp
+L Device:C C324
+U 1 1 5C869FEB
+P 15400 8950
+F 0 "C324" H 15515 8996 50  0000 L CNN
+F 1 "0.1u" H 15515 8905 50  0000 L CNN
+F 2 "require:C_0402" H 15438 8800 50  0001 C CNN
+F 3 "~" H 15400 8950 50  0001 C CNN
+	1    15400 8950
+	1    0    0    -1
+$EndComp
+Wire Wire Line
+	15400 8800 15400 8600
+Wire Wire Line
+	15400 8600 15000 8600
+Connection ~ 15000 8600
+Wire Wire Line
+	15400 9100 15400 9300
+Wire Wire Line
+	15400 9300 15000 9300
+Connection ~ 15000 9300
+$Comp
+L Device:C C325
+U 1 1 5C8A335A
+P 15800 8950
+F 0 "C325" H 15915 8996 50  0000 L CNN
+F 1 "0.1u" H 15915 8905 50  0000 L CNN
+F 2 "require:C_0402" H 15838 8800 50  0001 C CNN
+F 3 "~" H 15800 8950 50  0001 C CNN
+	1    15800 8950
+	1    0    0    -1
+$EndComp
+Wire Wire Line
+	15800 8800 15800 8600
+Wire Wire Line
+	15800 8600 15400 8600
+Connection ~ 15400 8600
+Wire Wire Line
+	15800 9100 15800 9300
+Wire Wire Line
+	15800 9300 15400 9300
+Connection ~ 15400 9300
+$Comp
+L Device:C C326
+U 1 1 5C990D30
+P 16200 8950
+F 0 "C326" H 16315 8996 50  0000 L CNN
+F 1 "0.1u" H 16315 8905 50  0000 L CNN
+F 2 "require:C_0402" H 16238 8800 50  0001 C CNN
+F 3 "~" H 16200 8950 50  0001 C CNN
+	1    16200 8950
+	1    0    0    -1
+$EndComp
+Wire Wire Line
+	15800 8600 16200 8600
+Wire Wire Line
+	16200 8600 16200 8800
+Connection ~ 15800 8600
+Wire Wire Line
+	16200 9100 16200 9300
+Wire Wire Line
+	16200 9300 15800 9300
+Connection ~ 15800 9300
 $EndSCHEMATC

Commit message: wip
Parts:
- R330, R331: value R -> 1k,1%
Other:
- note added: "0402, 0.1u x 17"
- note removed: "0402, 0.1u x 14"
- moved on the sheet: C310, C311, C312, C313, C314, C315, C316, C317, C318, C319, C320, C321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

Commit message: wip
Parts:
- U100: footprint require:RK3308_BGA355 -> require:RK3308_TFBGA-355
- U300: footprint require:DDR3_BGA_96 -> require:DDR3_BGA-96
Changed lines of the file:
@@
 F 0 "U300" H 11800 1700 60  0000 C CNN
 F 1 "DDR3_FBGA96" H 11850 1600 60  0000 C CNN
-F 2 "require:DDR3_BGA_96" H 11800 1550 60  0001 C CNN
+F 2 "require:DDR3_BGA-96" H 11800 1550 60  0001 C CNN
 F 3 "" H 11800 1550 60  0001 C CNN
 	1    11800 1550
@@
 F 0 "U100" H 4150 5650 60  0000 L CNN
 F 1 "RK3308" H 4150 5550 60  0000 L CNN
-F 2 "require:RK3308_BGA355" H 4150 5700 60  0001 C CNN
+F 2 "require:RK3308_TFBGA-355" H 4150 5700 60  0001 C CNN
 F 3 "" H 4150 5700 60  0001 C CNN
 	11   4150 5700

Commit message: wip
Changed lines of the file:
@@
 DDR_D2
 Text Label 10600 2650 0    60   ~ 0
-DDR_D5
+DDR_D4
 Text Label 10600 2750 0    60   ~ 0
 DDR_D0
@@
 DDR_D7
 Text Label 10600 3150 0    60   ~ 0
-DDR_D4
+DDR_D5
 Wire Wire Line
 	12600 5250 12600 5350
