File: hardware/require.sch (KiCad schematic (older format))
At the start: 0 parts

Commit message: wip
Changed lines of the file:
@@
 EELAYER 26 0
 EELAYER END
-$Descr A3 16535 11693
+$Descr A4 11693 8268
 encoding utf-8
-Sheet 1 7
+Sheet 1 8
 Title ""
 Date ""
@@
 $EndSheet
 $Sheet
-S 7300 4000 900  1650
+S 2700 950  900  1650
 U 5C2F0873
 F0 "ddr" 60
@@
 $EndSheet
 $Sheet
-S 2650 5450 1600 800
+S 850  1150 1400 1250
 U 5C325762
 F0 "rk3308-power" 50
@@
 $EndSheet
 $Sheet
-S 8400 4000 900  1650
+S 5700 4400 900  1650
 U 5CDAE2B6
 F0 "emmc" 50
 F1 "emmc.sch" 50
 $EndSheet
+$Sheet
+S 4600 6500 900  550
+U 5C70CDE2
+F0 "rk3308-lcdc-mac-i2s1-jtag" 50
+F1 "rk3308-lcdc-mac-i2s1-jtag.sch" 50
+$EndSheet
 $EndSCHEMATC

Commit message: wip
Changed lines of the file:
@@
 $Descr A4 11693 8268
 encoding utf-8
-Sheet 1 8
+Sheet 1 9
 Title ""
 Date ""
@@
 $EndSheet
 $Sheet
-S 850  1150 1400 1250
+S 7400 2400 1400 1250
 U 5C325762
 F0 "rk3308-power" 50
@@
 $EndSheet
 $Sheet
-S 5700 4400 900  1650
+S 4050 950  900  1650
 U 5CDAE2B6
 F0 "emmc" 50
@@
 F1 "rk3308-lcdc-mac-i2s1-jtag.sch" 50
 $EndSheet
+$Sheet
+S 5500 4100 1550 1200
+U 5CED3BD3
+F0 "usb" 50
+F1 "usb.sch" 50
+$EndSheet
 $EndSCHEMATC

Commit message: wip
Changed lines of the file:
@@
 $Descr A4 11693 8268
 encoding utf-8
-Sheet 1 9
+Sheet 1 10
 Title ""
 Date ""
@@
 $EndSheet
 $Sheet
-S 2700 950  900  1650
+S 1250 950  900  1650
 U 5C2F0873
 F0 "ddr" 60
@@
 F1 "usb.sch" 50
 $EndSheet
+$Sheet
+S 5350 950  1000 700
+U 5C48B775
+F0 "pin-header" 50
+F1 "pin-header.sch" 50
+$EndSheet
 $EndSCHEMATC

Commit message: wip
Changed lines of the file:
@@
 EELAYER 26 0
 EELAYER END
-$Descr A4 11693 8268
+$Descr A3 16535 11693
 encoding utf-8
-Sheet 1 10
+Sheet 1 9
 Title ""
 Date ""
@@
 $EndDescr
 $Sheet
-S 2650 3150 1600 750
+S 1900 1650 1250 1050
 U 5C2CD8AE
 F0 "power" 60
 F1 "power.sch" 60
+F2 "CORE_DVS" I L 1900 2500 50
 $EndSheet
 $Sheet
-S 2650 4400 1600 650
+S 7550 3200 1700 2100
 U 5C2D00B3
-F0 "test" 60
-F1 "test.sch" 60
+F0 "wifi" 60
+F1 "wifi.sch" 60
+F2 "HOST_WAKE_BT" I L 7550 4300 50
+F3 "BT_WAKE_HOST" I L 7550 4400 50
+F4 "WIFI_REG_ON" I L 7550 3300 50
+F5 "WIFI_WAKE_HOST" I L 7550 3400 50
+F6 "SDIO_D0" I L 7550 3500 50
+F7 "SDIO_D1" I L 7550 3600 50
+F8 "SDIO_D2" I L 7550 3700 50
+F9 "SDIO_D3" I L 7550 3800 50
+F10 "SDIO_CMD" I L 7550 3900 50
+F11 "SDIO_CLK" I L 7550 4000 50
+F12 "BT_REG_ON" I L 7550 4200 50
+F13 "UART_RTS" I L 7550 4500 50
+F14 "UART_CTS" I L 7550 4600 50
+F15 "UART_TXD" I L 7550 4700 50
+F16 "UART_RXD" I L 7550 4800 50
+F17 "PCM_SYNC" I L 7550 4900 50
+F18 "PCM_CLK" I L 7550 5000 50
+F19 "PCM_OUT" I L 7550 5100 50
+F20 "PCM_IN" I L 7550 5200 50
 $EndSheet
 $Sheet
-S 1250 950  900  1650
+S 7550 1650 1700 1050
 U 5C2F0873
 F0 "ddr" 60
@@
 $EndSheet
 $Sheet
-S 7400 2400 1400 1250
+S 3750 1650 1450 1050
 U 5C325762
 F0 "rk3308-power" 50
@@
 $EndSheet
 $Sheet
-S 2650 6550 1600 350
-U 5C46A4DA
-F0 "rk3308-acodec" 50
-F1 "rk3308-acodec.sch" 50
-$EndSheet
-$Sheet
-S 4050 950  900  1650
+S 1900 3200 900  1600
 U 5CDAE2B6
 F0 "emmc" 50
 F1 "emmc.sch" 50
+F2 "EMMC_RST" I R 2800 4300 50
+F3 "EMMC_D0" I R 2800 3300 50
+F4 "EMMC_D1" I R 2800 3400 50
+F5 "EMMC_D2" I R 2800 3500 50
+F6 "EMMC_D3" I R 2800 3600 50
+F7 "EMMC_D4" I R 2800 3700 50
+F8 "EMMC_D5" I R 2800 3800 50
+F9 "EMMC_D6" I R 2800 3900 50
+F10 "EMMC_D7" I R 2800 4000 50
+F11 "EMMC_CMD" I R 2800 4100 50
+F12 "EMMC_CLK" I R 2800 4200 50
 $EndSheet
 $Sheet
@@
 $EndSheet
 $Sheet
-S 5500 4100 1550 1200
+S 1800 6800 1550 1200
 U 5CED3BD3
 F0 "usb" 50
@@
 $EndSheet
 $Sheet
-S 5350 950  1000 700
-U 5C48B775
-F0 "pin-header" 50
-F1 "pin-header.sch" 50
+S 3750 3200 2900 2500
+U 5C87E279
+F0 "rk3308-io" 50
+F1 "rk3308-io.sch" 50
+F2 "EMMC_RST" I L 3750 4300 50
+F3 "EMMC_D0" I L 3750 3300 50
+F4 "EMMC_D1" I L 3750 3400 50
+F5 "EMMC_D2" I L 3750 3500 50
+F6 "EMMC_D3" I L 3750 3600 50
+F7 "EMMC_D4" I L 3750 3700 50
+F8 "EMMC_D5" I L 3750 3800 50
+F9 "EMMC_D6" I L 3750 3900 50
+F10 "EMMC_D7" I L 3750 4000 50
+F11 "EMMC_CMD" I L 3750 4100 50
+F12 "EMMC_CLK" I L 3750 4200 50
+F13 "WIFI_REG_ON" I R 6650 3300 50
+F14 "WIFI_WAKE_HOST" I R 6650 3400 50
+F15 "SDIO_D0" I R 6650 3500 50
+F16 "SDIO_D1" I R 6650 3600 50
+F17 "SDIO_D2" I R 6650 3700 50
+F18 "SDIO_D3" I R 6650 3800 50
+F19 "SDIO_CMD" I R 6650 3900 50
+F20 "SDIO_CLK" I R 6650 4000 50
+F21 "BT_REG_ON" I R 6650 4200 50
+F22 "HOST_WAKE_BT" I R 6650 4300 50
+F23 "BT_WAKE_HOST" I R 6650 4400 50
+F24 "UART4_CTS" I R 6650 4500 50
+F25 "UART4_RTS" I R 6650 4600 50
+F26 "UART4_RXD" I R 6650 4700 50
+F27 "UART4_TXD" I R 6650 4800 50
+F28 "PCM_SYNC" I R 6650 4900 50
+F29 "PCM_CLK" I R 6650 5000 50
+F30 "PCM_OUT" I R 6650 5100 50
+F31 "PCM_IN" I R 6650 5200 50
+F32 "CORE_DVS" I L 3750 5200 50
 $EndSheet
+Wire Wire Line
+	2800 3300 3750 3300
+Wire Wire Line
+	2800 3400 3750 3400
+Wire Wire Line
+	2800 3500 3750 3500
+Wire Wire Line
+	2800 3600 3750 3600
+Wire Wire Line
+	2800 3700 3750 3700
+Wire Wire Line
+	2800 3800 3750 3800
+Wire Wire Line
+	2800 3900 3750 3900
+Wire Wire Line
+	2800 4000 3750 4000
+Wire Wire Line
+	2800 4100 3750 4100
+Wire Wire Line
+	2800 4200 3750 4200
+Wire Wire Line
+	2800 4300 3750 4300
+Wire Wire Line
+	6650 3300 7550 3300
+Wire Wire Line
+	6650 3400 7550 3400
+Wire Wire Line
+	6650 3500 7550 3500
+Wire Wire Line
+	6650 3600 7550 3600
+Wire Wire Line
+	6650 3700 7550 3700
+Wire Wire Line
+	6650 3800 7550 3800
+Wire Wire Line
+	6650 3900 7550 3900
+Wire Wire Line
+	6650 4000 7550 4000
+Wire Wire Line
+	7550 4200 6650 4200
+Wire Wire Line
+	7550 4300 6650 4300
+Wire Wire Line
+	6650 4400 7550 4400
+Wire Wire Line
+	6650 4500 7550 4500
+Wire Wire Line
+	6650 4600 7550 4600
+Wire Wire Line
+	6650 4700 7550 4700
+Wire Wire Line
+	6650 4800 7550 4800
+Wire Wire Line
+	6650 4900 7550 4900
+Wire Wire Line
+	6650 5000 7550 5000
+Wire Wire Line
+	6650 5100 7550 5100
+Wire Wire Line
+	6650 5200 7550 5200
+Wire Wire Line
+	1900 2500 1500 2500
+Wire Wire Line
+	1500 2500 1500 5200
+Wire Wire Line
+	1500 5200 3750 5200
 $EndSCHEMATC

Commit message: wip
Parts:
- added C14: 1u, Capacitors_SMD:C_0402, symbol Device:C
- added D9: LED_GBAR_0603X2, require:LED_RGB_0603X2, symbol require:LED_GBAR_0603X2
- added H1, H2, H3, H4: MountingHole_Pad, require:PTH_MTG320_380, symbol Mechanical:MountingHole_Pad
- added J10: USB_B_Micro, Connectors_USB:USB_Micro-B_Molex_47346-0001, symbol Connector:USB_B_Micro
- added LP1, LP18, LP8, RP1, RP20: GND, require:OVAL_PIN, symbol require:OP
- added LP10: D20, require:OVAL_PIN, symbol require:OP
- added LP11: DM, require:OVAL_PIN, symbol require:OP
- added LP12: DP, require:OVAL_PIN, symbol require:OP
- added LP13: DNC, require:OVAL_PIN, symbol require:OP
- added LP14: RST, require:OVAL_PIN, symbol require:OP
- added LP15, LP16: 3V3, require:OVAL_PIN, symbol require:OP
- added LP17: 5V, require:OVAL_PIN, symbol require:OP
- added LP2: A0, require:OVAL_PIN, symbol require:OP
- added LP3: A1, require:OVAL_PIN, symbol require:OP
- added LP4: A2, require:OVAL_PIN, symbol require:OP
- added LP5: A3, require:OVAL_PIN, symbol require:OP
- added LP6: A4, require:OVAL_PIN, symbol require:OP
- added LP7: A5, require:OVAL_PIN, symbol require:OP
- added LP9: D19, require:OVAL_PIN, symbol require:OP
- added R1, R2, R322: 2.2R, Resistors_SMD:R_0402, symbol Device:R
- added R3: 30k, Resistors_SMD:R_0402, symbol Device:R
- added RP10: 9, require:OVAL_PIN, symbol require:OP
- added RP11: 10, require:OVAL_PIN, symbol require:OP
- added RP12: 11, require:OVAL_PIN, symbol require:OP
- added RP13: 12, require:OVAL_PIN, symbol require:OP
- added RP14: 13, require:OVAL_PIN, symbol require:OP
- added RP15: 14, require:OVAL_PIN, symbol require:OP
- added RP16: 15, require:OVAL_PIN, symbol require:OP
- added RP17: 16, require:OVAL_PIN, symbol require:OP
- added RP18: 17, require:OVAL_PIN, symbol require:OP
- added RP19: 18, require:OVAL_PIN, symbol require:OP
- added RP2: 1, require:OVAL_PIN, symbol require:OP
- added RP3: 2, require:OVAL_PIN, symbol require:OP
- added RP4: 3, require:OVAL_PIN, symbol require:OP
- added RP5: 4, require:OVAL_PIN, symbol require:OP
- added RP6: 5, require:OVAL_PIN, symbol require:OP
- added RP7: 6, require:OVAL_PIN, symbol require:OP
- added RP8: 7, require:OVAL_PIN, symbol require:OP
- added RP9: 8, require:OVAL_PIN, symbol require:OP
- added SW1: SW_SKSC_4PIN, require:SW_ALPS_SKSC, symbol require:SW_SKSC_4PIN
- added U2: AW2015FCR, require:AW2015FCR_QFN8L, symbol require:AW2015FCR
Connections:
- net labels added: BLUE, GND, GREEN, RED, RESET, USB_OTG_DM, USB_OTG_DP, VCC5V0_SYS, VCC_IO
- wire segments 33 -> 127
- no-connect marks 0 -> 3

Commit message: wip
Parts:
- removed H1, H2, H3, H4: MountingHole_Pad, require:PTH_MTG320_380, symbol Mechanical:MountingHole_Pad
- removed R322: 2.2R, Resistors_SMD:R_0402, symbol Device:R
- added D2, D3, D4: esd, require:ESD_SOD882, symbol Device:D_TVS
- added H1, H2: MountingHole, require:MOUNTING_HOLE_1.6mm, symbol Mechanical:MountingHole
- added H3, H4: MountingHole, require:MOUNTING_HOLE_1.6mm_NOCLEAR, symbol Mechanical:MountingHole
- SW1: footprint require:SW_ALPS_SKSC -> require:SW_ALPS_SKSCLCE010
- renumbered D9 to D1, J10 to J1
Connections:
- net labels added: USB_OTG_D_N, USB_OTG_D_P
- net labels removed: USB_OTG_DM, USB_OTG_DP
- wire segments 127 -> 125
Other:
- moved on the sheet: R1, R2

Commit message: wip
Parts:
- removed RP18: 17, require:OVAL_PIN, symbol require:OP
- removed RP19: 18, require:OVAL_PIN, symbol require:OP
- C14: footprint Capacitors_SMD:C_0402 -> require:C_0402
- R1, R2, R3: footprint Resistors_SMD:R_0402 -> require:R_0402
Connections:
- wire segments 125 -> 118
- no-connect marks 3 -> 12
Changed lines of the file:
@@
 F61 "D15" U R 6700 9100 50
 F62 "D16" U R 6700 9200 50
-F63 "D17" U R 6700 9300 50
-F64 "D18" U R 6700 9400 50
-F65 "I2C1_SCL" B R 6700 6400 50
-F66 "I2C1_SDA" B R 6700 6500 50
-F67 "POWER_SLEEP" I L 3800 5150 50
+F63 "I2C1_SCL" B R 6700 6400 50
+F64 "I2C1_SDA" B R 6700 6500 50
+F65 "POWER_SLEEP" I L 3800 5150 50
 $EndSheet
 Wire Wire Line
@@
 Wire Wire Line
 	6700 4800 7800 4800
-Wire Wire Line
-	6700 4900 7800 4900
-Wire Wire Line
-	6700 5000 7800 5000
-Wire Wire Line
-	6700 5100 7800 5100
-Wire Wire Line
-	6700 5200 7800 5200
 Wire Wire Line
 	1900 2500 1400 2500
@@
 F 0 "R1" V 2850 5900 50  0000 C CNN
 F 1 "2.2R" V 2850 5750 50  0000 C CNN
-F 2 "Resistors_SMD:R_0402" V 2680 5850 50  0001 C CNN
+F 2 "require:R_0402" V 2680 5850 50  0001 C CNN
 F 3 "~" H 2750 5850 50  0001 C CNN
 	1    2750 5850
@@
 F 0 "R2" V 2650 6000 50  0000 C CNN
 F 1 "2.2R" V 2650 5850 50  0000 C CNN
-F 2 "Resistors_SMD:R_0402" V 2680 5950 50  0001 C CNN
+F 2 "require:R_0402" V 2680 5950 50  0001 C CNN
 F 3 "~" H 2750 5950 50  0001 C CNN
 	1    2750 5950
@@
 NoConn ~ 2800 8800
 Wire Wire Line
-	6050 2400 5850 2400
-Wire Wire Line
 	5850 2400 5850 2500
 Wire Wire Line
@@
 Wire Wire Line
 	5850 2750 5850 2850
-Connection ~ 5850 2400
 Wire Wire Line
 	5250 2400 5850 2400
@@
 $Comp
 L require:OP P?
-U 1 1 5C797FDA
-P 7800 9300
-AR Path="/5C2D00B3/5C797FDA" Ref="P?"  Part="1"
-AR Path="/5C87E279/5C797FDA" Ref="P?"  Part="1"
-AR Path="/5C797FDA" Ref="RP18"  Part="1"
-F 0 "RP18" H 8050 9300 50  0000 C CNN
-F 1 "17" H 7800 9300 50  0000 C CNN
-F 2 "require:OVAL_PIN" H 7800 9250 50  0001 C CNN
-F 3 "" H 7800 9250 50  0001 C CNN
-	1    7800 9300
-	1    0    0    -1
-$EndComp
-$Comp
-L require:OP P?
-U 1 1 5C797FE1
-P 7800 9400
-AR Path="/5C2D00B3/5C797FE1" Ref="P?"  Part="1"
-AR Path="/5C87E279/5C797FE1" Ref="P?"  Part="1"
-AR Path="/5C797FE1" Ref="RP19"  Part="1"
-F 0 "RP19" H 8050 9400 50  0000 C CNN
-F 1 "18" H 7800 9400 50  0000 C CNN
-F 2 "require:OVAL_PIN" H 7800 9350 50  0001 C CNN
-F 3 "" H 7800 9350 50  0001 C CNN
-	1    7800 9400
-	1    0    0    -1
-$EndComp
-$Comp
-L require:OP P?
 U 1 1 5C797FE8
 P 7800 8300
@@
 Wire Wire Line
 	6700 9200 7600 9200
-Wire Wire Line
-	6700 9300 7600 9300
-Wire Wire Line
-	6700 9400 7600 9400
 $Comp
 L power:GND #PWR0192
@@
 F 0 "C14" H 10215 5696 50  0000 L CNN
 F 1 "1u" H 10215 5605 50  0000 L CNN
-F 2 "Capacitors_SMD:C_0402" H 10138 5500 50  0001 C CNN
+F 2 "require:C_0402" H 10138 5500 50  0001 C CNN
 F 3 "~" H 10100 5650 50  0001 C CNN
 	1    10100 5650
@@
 F 0 "R3" V 11243 5500 50  0000 C CNN
 F 1 "30k" V 11334 5500 50  0000 C CNN
-F 2 "Resistors_SMD:R_0402" V 11380 5500 50  0001 C CNN
+F 2 "require:R_0402" V 11380 5500 50  0001 C CNN
 F 3 "~" H 11450 5500 50  0001 C CNN
 	1    11450 5500
@@
 Wire Wire Line
 	2950 5650 3800 5650
+NoConn ~ 6700 4900
+NoConn ~ 6700 5000
+NoConn ~ 6700 5100
+NoConn ~ 6700 5200
+NoConn ~ 7800 4900
+NoConn ~ 7800 5000
+NoConn ~ 7800 5100
+NoConn ~ 7800 5200
+NoConn ~ 6050 2400
 $EndSCHEMATC

Commit message: wip
Parts:
- removed D2, D3: esd, require:ESD_SOD882, symbol Device:D_TVS
- removed LP7: A5, require:OVAL_PIN, symbol require:OP
- added R876, R877: 2.2R, require:R_0402, symbol Device:R
- added U1223, U878: ESD5302F, require:ESD_DFN1006_3L, symbol require:ESD5302F
- renumbered LP9 to LP10, LP10 to LP11, LP8 to LP7, LP11 to LP8, LP12 to LP9
Connections:
- wire segments 118 -> 128
Other:
- moved on the sheet: LP8, LP9
Changed lines of the file:
@@
 F35 "USB_OTG_VBUS" I L 3800 5650 50
 F36 "USB_OTG_ID" I L 3800 5750 50
-F37 "USB_HOST_DM" I L 3800 8600 50
-F38 "USB_HOST_DP" I L 3800 8700 50
+F37 "USB_HOST_DM" I L 3800 8700 50
+F38 "USB_HOST_DP" I L 3800 8600 50
 F39 "A0" I L 3800 7700 50
 F40 "A1" I L 3800 7800 50
@@
 P 2600 8300
 AR Path="/5C70CDE2/5C5E6FBC" Ref="LP?"  Part="1"
-AR Path="/5C5E6FBC" Ref="LP8"  Part="1"
-F 0 "LP8" H 2850 8300 50  0000 C CNN
+AR Path="/5C5E6FBC" Ref="LP7"  Part="1"
+F 0 "LP7" H 2850 8300 50  0000 C CNN
 F 1 "GND" H 2600 8300 50  0000 C CNN
 F 2 "require:OVAL_PIN" H 2600 8250 50  0001 C CNN
@@
 $EndComp
 Wire Wire Line
-	1650 5850 2150 5850
-Wire Wire Line
-	1650 5950 1850 5950
-Wire Wire Line
 	2900 5850 3800 5850
 Wire Wire Line
@@
 L require:OP LP?
 U 1 1 5C60EF82
-P 2600 8600
+P 1150 8700
 AR Path="/5CED3BD3/5C60EF82" Ref="LP?"  Part="1"
-AR Path="/5C60EF82" Ref="LP11"  Part="1"
-F 0 "LP11" H 2850 8600 50  0000 C CNN
-F 1 "DM" H 2600 8600 50  0000 C CNN
-F 2 "require:OVAL_PIN" H 2600 8600 50  0001 C CNN
-F 3 "" H 2600 8600 50  0001 C CNN
-	1    2600 8600
+AR Path="/5C60EF82" Ref="LP8"  Part="1"
+F 0 "LP8" H 1400 8700 50  0000 C CNN
+F 1 "DM" H 1150 8700 50  0000 C CNN
+F 2 "require:OVAL_PIN" H 1150 8700 50  0001 C CNN
+F 3 "" H 1150 8700 50  0001 C CNN
+	1    1150 8700
 	-1   0    0    1
 $EndComp
@@
 L require:OP LP?
 U 1 1 5C60EF89
-P 2600 8700
+P 1150 8600
 AR Path="/5CED3BD3/5C60EF89" Ref="LP?"  Part="1"
-AR Path="/5C60EF89" Ref="LP12"  Part="1"
-F 0 "LP12" H 2850 8700 50  0000 C CNN
-F 1 "DP" H 2600 8700 50  0000 C CNN
-F 2 "require:OVAL_PIN" H 2600 8700 50  0001 C CNN
-F 3 "" H 2600 8700 50  0001 C CNN
-	1    2600 8700
+AR Path="/5C60EF89" Ref="LP9"  Part="1"
+F 0 "LP9" H 1400 8600 50  0000 C CNN
+F 1 "DP" H 1150 8600 50  0000 C CNN
+F 2 "require:OVAL_PIN" H 1150 8600 50  0001 C CNN
+F 3 "" H 1150 8600 50  0001 C CNN
+	1    1150 8600
 	-1   0    0    1
 $EndComp
@@
 $EndComp
 $Comp
-L require:OP LP?
-U 1 1 5C62F755
-P 2600 8200
-AR Path="/5C325762/5C62F755" Ref="LP?"  Part="1"
-AR Path="/5C87E279/5C62F755" Ref="LP?"  Part="1"
-AR Path="/5C62F755" Ref="LP7"  Part="1"
-F 0 "LP7" H 2850 8200 50  0000 C CNN
-F 1 "A5" H 2600 8200 50  0000 C CNN
-F 2 "require:OVAL_PIN" H 2600 8200 50  0001 C CNN
-F 3 "" H 2600 8200 50  0001 C CNN
-	1    2600 8200
-	-1   0    0    1
-$EndComp
-$Comp
 L power:GND #PWR0215
 U 1 1 5C63ACDD
@@
 AR Path="/5C2D00B3/5C65A77B" Ref="LP?"  Part="1"
 AR Path="/5C87E279/5C65A77B" Ref="LP?"  Part="1"
-AR Path="/5C65A77B" Ref="LP9"  Part="1"
-F 0 "LP9" H 2850 8400 50  0000 C CNN
+AR Path="/5C65A77B" Ref="LP10"  Part="1"
+F 0 "LP10" H 2850 8400 50  0000 C CNN
 F 1 "D19" H 2600 8400 50  0000 C CNN
 F 2 "require:OVAL_PIN" H 2600 8350 50  0001 C CNN
@@
 AR Path="/5C2D00B3/5C671B48" Ref="LP?"  Part="1"
 AR Path="/5C87E279/5C671B48" Ref="LP?"  Part="1"
-AR Path="/5C671B48" Ref="LP10"  Part="1"
-F 0 "LP10" H 2850 8500 50  0000 C CNN
+AR Path="/5C671B48" Ref="LP11"  Part="1"
+F 0 "LP11" H 2850 8500 50  0000 C CNN
 F 1 "D20" H 2600 8500 50  0000 C CNN
 F 2 "require:OVAL_PIN" H 2600 8450 50  0001 C CNN
@@
 Wire Wire Line
 	2800 8500 3800 8500
-Wire Wire Line
-	2800 8600 3800 8600
-Wire Wire Line
-	2800 8700 3800 8700
 NoConn ~ 2800 8800
 Wire Wire Line
@@
 	1300 5150 3800 5150
 $Comp
-L Device:D_TVS D2
-U 1 1 5C6493F4
-P 1850 6300
-F 0 "D2" V 1804 6379 50  0000 L CNN
-F 1 "esd" V 1895 6379 50  0000 L CNN
-F 2 "require:ESD_SOD882" H 1850 6300 50  0001 C CNN
-F 3 "~" H 1850 6300 50  0001 C CNN
-	1    1850 6300
-	0    1    1    0
-$EndComp
-Wire Wire Line
-	1850 6150 1850 5950
-Connection ~ 1850 5950
-Wire Wire Line
-	1850 5950 2600 5950
-Wire Wire Line
-	1850 6450 1850 6650
-$Comp
-L power:GND #PWR0233
-U 1 1 5C654421
-P 1850 6650
-F 0 "#PWR0233" H 1850 6400 50  0001 C CNN
-F 1 "GND" H 1855 6477 50  0000 C CNN
-F 2 "" H 1850 6650 50  0001 C CNN
-F 3 "" H 1850 6650 50  0001 C CNN
-	1    1850 6650
-	1    0    0    -1
-$EndComp
-$Comp
-L Device:D_TVS D3
-U 1 1 5C6545E7
-P 2150 6300
-F 0 "D3" V 2104 6379 50  0000 L CNN
-F 1 "esd" V 2195 6379 50  0000 L CNN
-F 2 "require:ESD_SOD882" H 2150 6300 50  0001 C CNN
-F 3 "~" H 2150 6300 50  0001 C CNN
-	1    2150 6300
-	0    1    1    0
-$EndComp
-$Comp
 L Device:D_TVS D4
 U 1 1 5C654669
@@
 $EndComp
 Wire Wire Line
-	2150 6150 2150 5850
-Connection ~ 2150 5850
-Wire Wire Line
-	2150 5850 2600 5850
-Wire Wire Line
 	2450 6150 2450 5650
 Wire Wire Line
-	2150 6450 2150 6650
-Wire Wire Line
 	2450 6450 2450 6650
-$Comp
-L power:GND #PWR0234
-U 1 1 5C66BDDD
-P 2150 6650
-F 0 "#PWR0234" H 2150 6400 50  0001 C CNN
-F 1 "GND" H 2155 6477 50  0000 C CNN
-F 2 "" H 2150 6650 50  0001 C CNN
-F 3 "" H 2150 6650 50  0001 C CNN
-	1    2150 6650
-	1    0    0    -1
-$EndComp
 $Comp
 L power:GND #PWR0235
@@
 NoConn ~ 7800 5200
 NoConn ~ 6050 2400
+$Comp
+L require:ESD5302F U1223
+U 1 1 5C5DE8DE
+P 1900 6300
+F 0 "U1223" H 2078 6346 50  0000 L CNN
+F 1 "ESD5302F" H 2078 6255 50  0000 L CNN
+F 2 "require:ESD_DFN1006_3L" H 1900 6300 50  0001 C CNN
+F 3 "" H 1900 6300 50  0001 C CNN
+	1    1900 6300
+	1    0    0    -1
+$EndComp
+Wire Wire Line
+	1650 5950 1800 5950
+Wire Wire Line
+	1650 5850 2000 5850
+Wire Wire Line
+	1800 6000 1800 5950
+Connection ~ 1800 5950
+Wire Wire Line
+	1800 5950 2600 5950
+Wire Wire Line
+	2000 6000 2000 5850
+Connection ~ 2000 5850
+Wire Wire Line
+	2000 5850 2600 5850
+Wire Wire Line
+	1900 6600 1900 6700
+$Comp
+L power:GND #PWR0233
+U 1 1 5C5EF8BD
+P 1900 6700
+F 0 "#PWR0233" H 1900 6450 50  0001 C CNN
+F 1 "GND" H 1905 6527 50  0000 C CNN
+F 2 "" H 1900 6700 50  0001 C CNN
+F 3 "" H 1900 6700 50  0001 C CNN
+	1    1900 6700
+	1    0    0    -1
+$EndComp
+$Comp
+L Device:R R?
+U 1 1 5C5F4982
+P 2050 8600
+AR Path="/5CED3BD3/5C5F4982" Ref="R?"  Part="1"
+AR Path="/5C5F4982" Ref="R876"  Part="1"
+F 0 "R876" V 2150 8650 50  0000 C CNN
+F 1 "2.2R" V 2150 8500 50  0000 C CNN
+F 2 "require:R_0402" V 1980 8600 50  0001 C CNN
+F 3 "~" H 2050 8600 50  0001 C CNN
+	1    2050 8600
+	0    -1   -1   0
+$EndComp
+$Comp
+L Device:R R?
+U 1 1 5C5F4C59
+P 2050 8700
+AR Path="/5CED3BD3/5C5F4C59" Ref="R?"  Part="1"
+AR Path="/5C5F4C59" Ref="R877"  Part="1"
+F 0 "R877" V 2150 8750 50  0000 C CNN
+F 1 "2.2R" V 2150 8600 50  0000 C CNN
+F 2 "require:R_0402" V 1980 8700 50  0001 C CNN
+F 3 "~" H 2050 8700 50  0001 C CNN
+	1    2050 8700
+	0    -1   -1   0
+$EndComp
+Wire Wire Line
+	2200 8600 3800 8600
+Wire Wire Line
+	2200 8700 3800 8700
+$Comp
+L require:ESD5302F U878
+U 1 1 5C607C8C
+P 1250 9300
+F 0 "U878" H 1428 9346 50  0000 L CNN
+F 1 "ESD5302F" H 1428 9255 50  0000 L CNN
+F 2 "require:ESD_DFN1006_3L" H 1250 9300 50  0001 C CNN
+F 3 "" H 1250 9300 50  0001 C CNN
+	1    1250 9300
+	1    0    0    -1
+$EndComp
+Wire Wire Line
+	1350 9000 1350 8850
+Wire Wire Line
+	1350 8850 1650 8850
+Wire Wire Line
+	1150 9000 1150 8800
+Wire Wire Line
+	1150 8800 1500 8800
+Wire Wire Line
+	1250 9600 1250 9700
+$Comp
+L power:GND #PWR0234
+U 1 1 5C617F1D
+P 1250 9700
+F 0 "#PWR0234" H 1250 9450 50  0001 C CNN
+F 1 "GND" H 1255 9527 50  0000 C CNN
+F 2 "" H 1250 9700 50  0001 C CNN
+F 3 "" H 1250 9700 50  0001 C CNN
+	1    1250 9700
+	1    0    0    -1
+$EndComp
+Wire Wire Line
+	1350 8700 1650 8700
+Wire Wire Line
+	1500 8800 1500 8600
+Connection ~ 1500 8600
+Wire Wire Line
+	1500 8600 1350 8600
+Wire Wire Line
+	1500 8600 1900 8600
+Wire Wire Line
+	1650 8850 1650 8700
+Connection ~ 1650 8700
+Wire Wire Line
+	1650 8700 1900 8700
 $EndSCHEMATC
