File: hardware/require.sch (KiCad schematic (older format))
At the start: 52 parts, among them J1 USB_B_Micro, SW1 SW_SKSC_4PIN, U1223 ESD5302F, U2 AW2015FCR, U878 ESD5302F

Commit message: wip
Parts:
- added LP12: DNC, require:OVAL_PIN, symbol require:OP
- added R1323, R1326: 22R, require:R_0402, symbol Device:R
- added R323, R324: R, require:R_0402, symbol Device:R
- added U8678: ESD5302F, require:ESD_DFN1006_3L, symbol require:ESD5302F
- LP2: value A0 -> A1
- LP3: value A1 -> A2
- LP4: value A2 -> A3
- LP5: value A3 -> A4
- LP6: value A4 -> A5
- R876, R877: value 2.2R -> 22R
Connections:
- net labels added: VCC_1V8
- wire segments 128 -> 137
- no-connect marks 12 -> 13
Other:
- moved on the sheet: LP10, LP11, LP7, LP8, LP9, R876, R877, U878

Commit message: wip
Parts:
- added C25: 1u, require:C_0402, symbol Device:C
- added U8: ATECC608A-MAHDA, require:ATECC_UDFN8, symbol Security:ATECC608A-MAHDA
- D3: renamed from D4; value esd -> ESD5451N; footprint require:ESD_SOD882 -> require:ESD_DFN1006_2L
- J1: footprint Connectors_USB:USB_Micro-B_Molex_47346-0001 -> require:USB_Micro-B_Molex_47346-0001
- LP1, LP18, LP7, RP1, RP20: value GND -> G
- LP12, LP13: value DNC -> NC
- SW1: footprint require:SW_ALPS_SKSCLCE010 -> require:SW_ALPS_SKSC
- renumbered U1223 to D2, U878 to D5, U8678 to D6, R323 to R63, R324 to R64, R1326 to R66, R1323 to R67, R877 to R68, R876 to R69, R1 to R7, R2 to R8, U2 to U5
Connections:
- net labels added: +3V3, +5V
- net labels removed: VCC5V0_SYS, VCC_IO
- wire segments 137 -> 145
Other:
- moved on the sheet: D5, D6, LP10, LP11, LP12, LP13, LP14, LP15, LP16, LP17, LP18, LP8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

Commit message: wip
Parts:
- removed C14: 1u, require:C_0402, symbol Device:C
- removed D1: LED_GBAR_0603X2, require:LED_RGB_0603X2, symbol require:LED_GBAR_0603X2
- removed D3: ESD5451N, require:ESD_DFN1006_2L, symbol Device:D_TVS
- removed H1, H2: MountingHole, require:MOUNTING_HOLE_1.6mm, symbol Mechanical:MountingHole
- removed H3, H4: MountingHole, require:MOUNTING_HOLE_1.6mm_NOCLEAR, symbol Mechanical:MountingHole
- removed J1: USB_B_Micro, require:USB_Micro-B_Molex_47346-0001, symbol Connector:USB_B_Micro
- removed R3: 30k, require:R_0402, symbol Device:R
- removed SW1: SW_SKSC_4PIN, require:SW_ALPS_SKSC, symbol require:SW_SKSC_4PIN
- removed U5: AW2015FCR, require:AW2015FCR_QFN8L, symbol require:AW2015FCR
- LP17: value 5V -> NC
Connections:
- net labels added: +1V8
- net labels removed: +5V, BLUE, GREEN, RED, VCC_1V8
- wire segments 145 -> 110
- no-connect marks 13 -> 12

Commit message: wip
Parts:
- added J1: USB_B_Micro, Connectors_USB:USB_Micro-B_Molex_47346-0001, symbol Connector:USB_B_Micro
Connections:
- net GND: now also J1.5 (GND), J1.6 (Shield)
- net at D2.1, R8.1: now also J1.2 (D-)
- net at D2.2, R7.1: now also J1.3 (D+)
- new net +5V: J1.1 (VBUS)
Changed lines of the file:
@@
+	1    0    0    -1
+$EndComp
+$Comp
+L Connector:USB_B_Micro J1
+U 1 1 5C64095D
+P 1350 5850
+F 0 "J1" H 1405 6317 50  0000 C CNN
+F 1 "USB_B_Micro" H 1405 6226 50  0000 C CNN
+F 2 "Connectors_USB:USB_Micro-B_Molex_47346-0001" H 1500 5800 50  0001 C CNN
+F 3 "~" H 1500 5800 50  0001 C CNN
+	1    1350 5850
+	1    0    0    -1
+$EndComp
+Wire Wire Line
+	1250 6250 1250 6350
+Wire Wire Line
+	1250 6350 1350 6350
+Wire Wire Line
+	1350 6350 1350 6250
+Wire Wire Line
+	1250 6350 1250 6450
+Connection ~ 1250 6350
+$Comp
+L power:+5V #PWR?
+U 1 1 5C64963D
+P 1850 5550
+F 0 "#PWR?" H 1850 5400 50  0001 C CNN
+F 1 "+5V" H 1865 5723 50  0000 C CNN
+F 2 "" H 1850 5550 50  0001 C CNN
+F 3 "" H 1850 5550 50  0001 C CNN
+	1    1850 5550
+	1    0    0    -1
+$EndComp
+Wire Wire Line
+	1650 5650 1850 5650
+Wire Wire Line
+	1850 5650 1850 5550
+$Comp
+L power:GND #PWR?
+U 1 1 5C64DF40
+P 1250 6450
+F 0 "#PWR?" H 1250 6200 50  0001 C CNN
+F 1 "GND" H 1255 6277 50  0000 C CNN
+F 2 "" H 1250 6450 50  0001 C CNN
+F 3 "" H 1250 6450 50  0001 C CNN
+	1    1250 6450
 	1    0    0    -1
 $EndComp

Commit message: wip
Parts:
- removed LP12, LP17: NC, require:OVAL_PIN, symbol require:OP
- removed R66, R67: 22R, require:R_0402, symbol Device:R
- removed RP20: G, require:OVAL_PIN, symbol require:OP
- added D201: LED, LEDs:LED_0402, symbol Device:LED
- added D400: D_Schottky, Diodes_SMD:D_SOD-523, symbol Device:D_Schottky
- added LP14: NC, require:OVAL_PIN, symbol require:OP
- added LP15, RP18: G, require:OVAL_PIN, symbol require:OP
- added Q200: NPND_SOT_363, TO_SOT_Packages_SMD:SOT-363_SC-70-6, symbol require:NPND_SOT_363
- added R202: 470R, require:R_0402, symbol Device:R
- added RP19: BYP, require:OVAL_PIN, symbol require:OP
- added SW1: SW_SKSC_4PIN, require:SW_ALPS_SKSCLCE010, symbol require:SW_SKSC_4PIN
- J1: footprint Connectors_USB:USB_Micro-B_Molex_47346-0001 -> require:USB_Micro-B_Molex_47346-0001
- LP18: value G -> 5V
- renumbered LP9 to LP10, LP10 to LP11, LP11 to LP12, LP15 to LP16, LP16 to LP17, LP14 to LP8, LP8 to LP9
Connections:
- net +3V3: now also D201.2 (A), R202.1
- net +5V: now also LP18.1
- net GND: now also LP14.1, LP15.1, Q200.1, Q200.4, RP18.1; no longer LP18.1
- net rk3308-io/D19: now also D6.2, LP11.1
- net rk3308-io/D20: now also D6.1, LP12.1
- net at J1.2 (D-), R8.1: now also D2.2; no longer D2.1
- net at J1.3 (D+), R7.1: now also D2.1; no longer D2.2
- new net: D400.1 (K), RP19.1
- new net: D201.1 (K), Q200.3
- new net EMMC_D0: D400.2 (A)
- new net LED: Q200.2, Q200.5, Q200.6, R202.2
- no-connect marks 12 -> 10
Other:
- moved on the sheet: C25, LP16, LP17, LP8, U8

Commit message: wip
Parts:
- removed D400: D_Schottky, Diodes_SMD:D_SOD-523, symbol Device:D_Schottky
- added D850: ESD5302F, require:ESD_DFN1006_3L, symbol require:ESD5302F
- added H1, H2: MountingHole, require:MTG_1.8mm_2.4mm_NPL, symbol Mechanical:MountingHole
- added H3, H4: MountingHole_Pad, require:MTG_1.8mm_2.4mm_PL, symbol Mechanical:MountingHole_Pad
- added R805: 133R,1%, require:R_0402, symbol Device:R
- added R830, R831, R850: 4.7k, require:R_0402, symbol Device:R
- renumbered C25 to C830, D2 to D800, D5 to D810, D6 to D820, D201 to D840, J1 to J800, Q200 to Q840, R63 to R700, R64 to R701, R7 to R800, R8 to R801, R68 to R810, R69 to R811, R202 to R840, SW1 to SW850, U8 to U830
Connections:
- net +3V3: now also R830.1, R831.1, R850.1
- net GND: now also SW850.1, SW850.2, D850.3, H3.1, H4.1, R805.2
- net rk3308-io/I2C1_SCL: now also R830.2
- net rk3308-io/I2C1_SDA: now also R831.2
- net KEY: now reaches SW850.3
- net KEY: now also D850.1, D850.2, R850.2
- net EMMC_D0_SHORT: now reaches RP19.1
- new net rk3308-io/USB_EXTR: R805.1
- no-connect marks 10 -> 3
Other:
- moved on the sheet: D800, D840, Q840, R800, R801, R810, R811, R840, RP19, SW850

Commit message: wip
Parts:
- D800, D810, D820, D850: value ESD5302F -> PESDUC3FD5VU; footprint require:ESD_DFN1006_3L -> require:SOT-883; symbol require:ESD5302F -> require:PESDUC3FD5VU
- D840: footprint LEDs:LED_0402 -> require:LED_0402
- J800: value USB_B_Micro -> Molex 47346-0001
- Q840: value NPND_SOT_363 -> LMBT3904DW1T1G
Connections:
- net rk3308-io/D19: now also D820.1; no longer D820.2
- net rk3308-io/D20: now also D820.2; no longer D820.1
- net at J800.3 (D+), R800.1: now also D800.2; no longer D800.1
- net at J800.2 (D-), R801.1: now also D800.1; no longer D800.2
- net at LP10.1, R811.1: now also D810.1; no longer D810.2
- net at LP9.1, R810.1: now also D810.2; no longer D810.1
Changed lines of the file:
@@
 L power:GND #PWR0215
 U 1 1 5C63ACDD
-P 3000 7600
-F 0 "#PWR0215" H 3000 7350 50  0001 C CNN
-F 1 "GND" V 3005 7472 50  0000 R CNN
-F 2 "" H 3000 7600 50  0001 C CNN
-F 3 "" H 3000 7600 50  0001 C CNN
-	1    3000 7600
+P 3100 7600
+F 0 "#PWR0215" H 3100 7350 50  0001 C CNN
+F 1 "GND" V 3105 7472 50  0000 R CNN
+F 2 "" H 3100 7600 50  0001 C CNN
+F 3 "" H 3100 7600 50  0001 C CNN
+	1    3100 7600
 	0    -1   -1   0
 $EndComp
 Wire Wire Line
-	3000 7600 2800 7600
+	3100 7600 2800 7600
 $Comp
 L power:GND #PWR0216
 U 1 1 5C651787
-P 3000 8200
-F 0 "#PWR0216" H 3000 7950 50  0001 C CNN
-F 1 "GND" V 3005 8072 50  0000 R CNN
-F 2 "" H 3000 8200 50  0001 C CNN
-F 3 "" H 3000 8200 50  0001 C CNN
-	1    3000 8200
+P 3100 8200
+F 0 "#PWR0216" H 3100 7950 50  0001 C CNN
+F 1 "GND" V 3105 8072 50  0000 R CNN
+F 2 "" H 3100 8200 50  0001 C CNN
+F 3 "" H 3100 8200 50  0001 C CNN
+	1    3100 8200
 	0    -1   -1   0
 $EndComp
 Wire Wire Line
-	2800 8200 3000 8200
+	2800 8200 3100 8200
 $Comp
 L require:OP LP?
@@
 	2950 5650 3800 5650
 $Comp
-L require:ESD5302F D800
+L require:PESDUC3FD5VU D800
 U 1 1 5C5DE8DE
 P 1900 6200
 F 0 "D800" H 2000 6250 50  0000 L CNN
-F 1 "ESD5302F" H 2000 6150 50  0000 L CNN
-F 2 "require:ESD_DFN1006_3L" H 1900 6200 50  0001 C CNN
+F 1 "PESDUC3FD5VU" H 2000 6150 50  0000 L CNN
+F 2 "require:SOT-883" H 1900 6200 50  0001 C CNN
 F 3 "" H 1900 6200 50  0001 C CNN
 	1    1900 6200
@@
 $EndComp
 $Comp
-L require:ESD5302F D810
+L require:PESDUC3FD5VU D810
 U 1 1 5C607C8C
 P 1500 8950
-F 0 "D810" H 1678 8996 50  0000 L CNN
-F 1 "ESD5302F" H 1678 8905 50  0000 L CNN
-F 2 "require:ESD_DFN1006_3L" H 1500 8950 50  0001 C CNN
+F 0 "D810" H 1600 9000 50  0000 L CNN
+F 1 "PESDUC3FD5VU" H 1600 8900 50  0000 L CNN
+F 2 "require:SOT-883" H 1500 8950 50  0001 C CNN
 F 3 "" H 1500 8950 50  0001 C CNN
 	1    1500 8950
@@
 	3450 6800 3450 6850
 $Comp
-L require:ESD5302F D820
+L require:PESDUC3FD5VU D820
 U 1 1 5C621347
 P 2950 9300
-F 0 "D820" H 3128 9346 50  0000 L CNN
-F 1 "ESD5302F" H 3128 9255 50  0000 L CNN
-F 2 "require:ESD_DFN1006_3L" H 2950 9300 50  0001 C CNN
+F 0 "D820" H 3050 9350 50  0000 L CNN
+F 1 "PESDUC3FD5VU" H 3050 9250 50  0000 L CNN
+F 2 "require:SOT-883" H 2950 9300 50  0001 C CNN
 F 3 "" H 2950 9300 50  0001 C CNN
 	1    2950 9300
@@
 	2950 9450 2950 9550
 Wire Wire Line
-	1550 8800 1550 8600
-Connection ~ 1550 8600
-Wire Wire Line
-	1550 8600 1750 8600
-Wire Wire Line
-	1450 8800 1450 8500
-Connection ~ 1450 8500
-Wire Wire Line
-	1450 8500 1750 8500
-Wire Wire Line
 	1500 9100 1500 9200
-Wire Wire Line
-	1150 8500 1450 8500
-Wire Wire Line
-	1150 8600 1550 8600
 Wire Wire Line
 	1900 6350 1900 6450
@@
 P 1350 5850
 F 0 "J800" H 1405 6317 50  0000 C CNN
-F 1 "USB_B_Micro" H 1405 6226 50  0000 C CNN
+F 1 "Molex 47346-0001" H 1405 6226 50  0000 C CNN
 F 2 "require:USB_Micro-B_Molex_47346-0001" H 1500 5800 50  0001 C CNN
 F 3 "~" H 1500 5800 50  0001 C CNN
@@
 $EndComp
 Wire Wire Line
-	1650 5850 1850 5850
-Wire Wire Line
-	1950 6050 1950 5950
-Connection ~ 1950 5950
-Wire Wire Line
-	1950 5950 2350 5950
-Wire Wire Line
-	1650 5950 1950 5950
-Wire Wire Line
-	1850 6050 1850 5850
-Connection ~ 1850 5850
-Wire Wire Line
-	1850 5850 2350 5850
+	1650 5950 1850 5950
 Text Label 3000 3300 0    50   ~ 0
 EMMC_D0
@@
 $EndComp
 Wire Wire Line
-	2800 9000 2900 9000
-Wire Wire Line
-	2800 8900 3000 8900
-Wire Wire Line
-	2900 9150 2900 9000
-Connection ~ 2900 9000
-Wire Wire Line
-	2900 9000 3800 9000
-Wire Wire Line
-	3000 9150 3000 8900
-Connection ~ 3000 8900
-Wire Wire Line
-	3000 8900 3800 8900
+	2800 8900 2900 8900
 $Comp
 L require:OP P?
@@
 P 13400 5400
 F 0 "Q840" H 13678 5446 50  0000 L CNN
-F 1 "NPND_SOT_363" H 13678 5355 50  0000 L CNN
+F 1 "LMBT3904DW1T1G" H 13678 5355 50  0000 L CNN
 F 2 "TO_SOT_Packages_SMD:SOT-363_SC-70-6" H 13400 5400 50  0001 C CNN
 F 3 "" H 13400 5400 50  0001 C CNN
@@
 F 0 "D840" V 13638 4732 50  0000 R CNN
 F 1 "LED" V 13547 4732 50  0000 R CNN
-F 2 "LEDs:LED_0402" H 13600 4850 50  0001 C CNN
+F 2 "require:LED_0402" H 13600 4850 50  0001 C CNN
 F 3 "~" H 13600 4850 50  0001 C CNN
 	1    13600 4850
@@
 $EndComp
 $Comp
-L require:ESD5302F D850
+L require:PESDUC3FD5VU D850
 U 1 1 5C7834D1
 P 12150 6700
 F 0 "D850" H 12250 6750 50  0000 L CNN
-F 1 "ESD5302F" H 12250 6650 50  0000 L CNN
-F 2 "require:ESD_DFN1006_3L" H 12150 6700 50  0001 C CNN
+F 1 "PESDUC3FD5VU" H 12250 6650 50  0000 L CNN
+F 2 "require:SOT-883" H 12150 6700 50  0001 C CNN
 F 3 "" H 12150 6700 50  0001 C CNN
 	1    12150 6700
@@
 Text Label 6900 9500 0    50   ~ 0
 EMMC_D0_SHORT
+Wire Wire Line
+	1150 8600 1450 8600
+Wire Wire Line
+	1550 8800 1550 8500
+Connection ~ 1550 8500
+Wire Wire Line
+	1550 8500 1750 8500
+Wire Wire Line
+	1150 8500 1550 8500
+Wire Wire Line
+	1450 8800 1450 8600
+Connection ~ 1450 8600
+Wire Wire Line
+	1450 8600 1750 8600
+Wire Wire Line
+	2800 9000 3000 9000
+Wire Wire Line
+	2900 9150 2900 8900
+Connection ~ 2900 8900
+Wire Wire Line
+	2900 8900 3800 8900
+Wire Wire Line
+	3000 9150 3000 9000
+Connection ~ 3000 9000
+Wire Wire Line
+	3000 9000 3800 9000
+Wire Wire Line
+	1650 5850 1950 5850
+Wire Wire Line
+	1850 5950 1850 6050
+Connection ~ 1850 5950
+Wire Wire Line
+	1850 5950 2350 5950
+Wire Wire Line
+	1950 5850 1950 6050
+Connection ~ 1950 5850
+Wire Wire Line
+	1950 5850 2350 5850
 $EndSCHEMATC

Commit message: wip
Changed lines of the file:
@@
 F15 "UART_TXD" I L 7800 4700 50
 F16 "UART_RXD" I L 7800 4800 50
+F17 "LPO" I L 7800 5050 50
 $EndSheet
 $Sheet
@@
 F63 "USB_EXTR" I L 3800 6050 50
 F64 "EMMC_VSEL" I L 3800 4400 50
+F65 "RTC_CLK" I R 6700 5050 50
 $EndSheet
 Wire Wire Line
@@
 Wire Wire Line
 	1950 5850 2350 5850
+Wire Wire Line
+	6700 5050 7800 5050
 $EndSCHEMATC
