File: hardware/require.sch (KiCad schematic (older format))
At the start: 62 parts, among them J800 Molex 47346-0001, Q840 LMBT3904DW1T1G, SW850 SW_SKSC_4PIN, U830 ATECC608A-MAHDA

Commit message: wip
Parts:
- J800: footprint require:USB_Micro-B_Molex_47346-0001 -> require:USB_Micro-B_Molex-105164-0001
Connections:
- net at J800.2 (D-), R801.1: now also D800.2; no longer D800.1
- net at J800.3 (D+), R800.1: now also D800.1; no longer D800.2
Changed lines of the file:
@@
 F 0 "J800" H 1405 6317 50  0000 C CNN
 F 1 "Molex 47346-0001" H 1405 6226 50  0000 C CNN
-F 2 "require:USB_Micro-B_Molex_47346-0001" H 1500 5800 50  0001 C CNN
+F 2 "require:USB_Micro-B_Molex-105164-0001" H 1500 5800 50  0001 C CNN
 F 3 "~" H 1500 5800 50  0001 C CNN
 	1    1350 5850
@@
 	1    0    0    -1
 $EndComp
-Wire Wire Line
-	1650 5950 1850 5950
 Text Label 3000 3300 0    50   ~ 0
 EMMC_D0
@@
 	3000 9000 3800 9000
 Wire Wire Line
-	1650 5850 1950 5850
-Wire Wire Line
-	1850 5950 1850 6050
-Connection ~ 1850 5950
-Wire Wire Line
-	1850 5950 2350 5950
-Wire Wire Line
-	1950 5850 1950 6050
-Connection ~ 1950 5850
-Wire Wire Line
-	1950 5850 2350 5850
-Wire Wire Line
 	6700 5050 7800 5050
+Wire Wire Line
+	1650 5850 1850 5850
+Wire Wire Line
+	1650 5950 1950 5950
+Wire Wire Line
+	1850 6050 1850 5850
+Connection ~ 1850 5850
+Wire Wire Line
+	1850 5850 2350 5850
+Wire Wire Line
+	1950 5950 1950 6050
+Connection ~ 1950 5950
+Wire Wire Line
+	1950 5950 2350 5950
 $EndSCHEMATC

Commit message: wip
Connections:
- net KEY: now also SW850.4
- no-connect marks 3 -> 2
Changed lines of the file:
@@
 	1    0    0    -1
 $EndComp
-NoConn ~ 13000 6350
 $Comp
 L Device:R R831
@@
 	11900 6450 11650 6450
 Wire Wire Line
-	12200 6450 13000 6450
+	12200 6450 12900 6450
 Wire Wire Line
 	6700 10150 7100 10150
@@
 Wire Wire Line
 	1950 5950 2350 5950
+Wire Wire Line
+	13000 6350 12900 6350
+Wire Wire Line
+	12900 6350 12900 6450
+Connection ~ 12900 6450
+Wire Wire Line
+	12900 6450 13000 6450
 $EndSCHEMATC

Commit message: wip
Parts:
- R850: value 4.7k -> 10k
Changed lines of the file:
@@
 $EndSheet
 $Sheet
-S 7800 1600 1700 1050
+S 7800 1650 1700 1050
 U 5C2F0873
 F0 "ddr" 60
@@
 S 3800 1650 1450 1050
 U 5C325762
-F0 "rk3308-power" 50
-F1 "rk3308-power.sch" 50
+F0 "rk3308-power" 60
+F1 "rk3308-power.sch" 60
 F2 "RESET" I R 5250 2400 50
 $EndSheet
@@
 	1    0    0    -1
 $EndComp
-Wire Wire Line
-	5250 2400 5600 2400
 Text Label 5350 2400 0    50   ~ 0
 RESET
@@
 P 11900 6150
 F 0 "R850" H 11970 6196 50  0000 L CNN
-F 1 "4.7k" H 11970 6105 50  0000 L CNN
+F 1 "10k" H 11970 6105 50  0000 L CNN
 F 2 "require:R_0402" V 11830 6150 50  0001 C CNN
 F 3 "~" H 11900 6150 50  0001 C CNN
@@
 Wire Wire Line
 	12900 6450 13000 6450
+Wire Wire Line
+	5250 2400 5800 2400
 $EndSCHEMATC

Commit message: wip
Parts:
- added D400: RB521S, require:D_SOD-523, symbol Device:D_Schottky
- added R410: 2.2k, require:R_0402, symbol Device:R
- added R802: 0R, require:R_0603, symbol Device:R
- J800: value Molex 47346-0001 -> Molex 105164-0001
- LP14: value NC -> G
- Q840: footprint TO_SOT_Packages_SMD:SOT-363_SC-70-6 -> require:SOT-363_SC-70-6
- R700, R701: value R -> 51k,1%
- R800, R801: value 2.2R -> 22R
- RP19: value BYP -> U
Connections:
- net EMMC_D0: now also D400.2 (A)
- net GND: now also R410.2, R802.2; no longer J800.6 (Shield)
- net EMMC_D0_SHORT: no longer names the net of RP19.1
- net EMMC_D0_SHORT: now also D400.1 (K)
- new net SHIELD: J800.6 (Shield), R802.1
- new net rk3308-io/EMMC_VSEL: R410.1
- no-connect marks 2 -> 3
Other:
- note added: "Pin 1 is cathode"
- moved on the sheet: RP19
Changed lines of the file:
@@
 F11 "EMMC_CMD" I R 2800 4100 50
 F12 "EMMC_CLK" I R 2800 4200 50
-F13 "EMMC_VSEL" I R 2800 4400 50
-F14 "EMMC_D0_SHORT" I R 2800 4600 50
 $EndSheet
 $Sheet
@@
 F62 "D18" I R 6700 10250 50
 F63 "USB_EXTR" I L 3800 6050 50
-F64 "EMMC_VSEL" I L 3800 4400 50
+F64 "EMMC_VSEL" I L 3800 4500 50
 F65 "RTC_CLK" I R 6700 5050 50
 $EndSheet
@@
 AR Path="/5C5EE6A6" Ref="R800"  Part="1"
 F 0 "R800" V 2600 5950 50  0000 C CNN
-F 1 "2.2R" V 2600 5750 50  0000 C CNN
+F 1 "22R" V 2600 5750 50  0000 C CNN
 F 2 "require:R_0402" V 2430 5850 50  0001 C CNN
 F 3 "~" H 2500 5850 50  0001 C CNN
@@
 AR Path="/5C5EE6AD" Ref="R801"  Part="1"
 F 0 "R801" V 2400 6050 50  0000 C CNN
-F 1 "2.2R" V 2400 5850 50  0000 C CNN
+F 1 "22R" V 2400 5850 50  0000 C CNN
 F 2 "require:R_0402" V 2430 5950 50  0001 C CNN
 F 3 "~" H 2500 5950 50  0001 C CNN
@@
 P 3450 6600
 F 0 "R700" H 3520 6646 50  0000 L CNN
-F 1 "R" H 3520 6555 50  0000 L CNN
+F 1 "51k,1%" H 3520 6555 50  0000 L CNN
 F 2 "require:R_0402" V 3380 6600 50  0001 C CNN
 F 3 "~" H 3450 6600 50  0001 C CNN
@@
 P 3450 7000
 F 0 "R701" H 3520 7046 50  0000 L CNN
-F 1 "R" H 3520 6955 50  0000 L CNN
+F 1 "51k,1%" H 3520 6955 50  0000 L CNN
 F 2 "require:R_0402" V 3380 7000 50  0001 C CNN
 F 3 "~" H 3450 7000 50  0001 C CNN
@@
 P 1350 5850
 F 0 "J800" H 1405 6317 50  0000 C CNN
-F 1 "Molex 47346-0001" H 1405 6226 50  0000 C CNN
+F 1 "Molex 105164-0001" H 1405 6226 50  0000 C CNN
 F 2 "require:USB_Micro-B_Molex-105164-0001" H 1500 5800 50  0001 C CNN
 F 3 "~" H 1500 5800 50  0001 C CNN
@@
 	1    0    0    -1
 $EndComp
-Wire Wire Line
-	1250 6250 1250 6350
-Wire Wire Line
-	1250 6350 1350 6350
-Wire Wire Line
-	1350 6350 1350 6250
-Wire Wire Line
-	1250 6350 1250 6450
-Connection ~ 1250 6350
 $Comp
 L power:+5V #PWR0160
@@
 L power:GND #PWR0164
 U 1 1 5C64DF40
-P 1250 6450
-F 0 "#PWR0164" H 1250 6200 50  0001 C CNN
-F 1 "GND" H 1255 6277 50  0000 C CNN
-F 2 "" H 1250 6450 50  0001 C CNN
-F 3 "" H 1250 6450 50  0001 C CNN
-	1    1250 6450
+P 1350 6450
+F 0 "#PWR0164" H 1350 6200 50  0001 C CNN
+F 1 "GND" H 1355 6277 50  0000 C CNN
+F 2 "" H 1350 6450 50  0001 C CNN
+F 3 "" H 1350 6450 50  0001 C CNN
+	1    1350 6450
 	1    0    0    -1
 $EndComp
@@
 L require:OP RP?
 U 1 1 5C8D949C
-P 7800 9500
+P 7800 9700
 AR Path="/5C70CDE2/5C8D949C" Ref="RP?"  Part="1"
 AR Path="/5C8D949C" Ref="RP19"  Part="1"
-F 0 "RP19" H 8050 9500 50  0000 C CNN
-F 1 "BYP" H 7800 9500 50  0000 C CNN
-F 2 "require:OVAL_PIN" H 7800 9450 50  0001 C CNN
-F 3 "" H 7800 9450 50  0001 C CNN
-	1    7800 9500
+F 0 "RP19" H 8050 9700 50  0000 C CNN
+F 1 "U" H 7800 9700 50  0000 C CNN
+F 2 "require:OVAL_PIN" H 7800 9650 50  0001 C CNN
+F 3 "" H 7800 9650 50  0001 C CNN
+	1    7800 9700
 	1    0    0    -1
 $EndComp
@@
 AR Path="/5C9CA9BF" Ref="LP14"  Part="1"
 F 0 "LP14" H 2850 10100 50  0000 C CNN
-F 1 "NC" H 2600 10100 50  0000 C CNN
+F 1 "G" H 2600 10100 50  0000 C CNN
 F 2 "require:OVAL_PIN" H 2600 10050 50  0001 C CNN
 F 3 "" H 2600 10050 50  0001 C CNN
@@
 F 0 "Q840" H 13678 5446 50  0000 L CNN
 F 1 "LMBT3904DW1T1G" H 13678 5355 50  0000 L CNN
-F 2 "TO_SOT_Packages_SMD:SOT-363_SC-70-6" H 13400 5400 50  0001 C CNN
+F 2 "require:SOT-363_SC-70-6" H 13400 5400 50  0001 C CNN
 F 3 "" H 13400 5400 50  0001 C CNN
 	1    13400 5400
@@
 Wire Wire Line
 	2950 6450 2950 6550
-Wire Wire Line
-	2800 4400 3800 4400
 Connection ~ 12200 6450
 Wire Wire Line
@@
 	6700 10250 7100 10250
 Wire Wire Line
-	2800 4600 3650 4600
-Text Label 3000 4600 0    50   ~ 0
-EMMC_D0_SHORT
-Wire Wire Line
-	7600 9500 6900 9500
-Text Label 6900 9500 0    50   ~ 0
-EMMC_D0_SHORT
-Wire Wire Line
 	1150 8600 1450 8600
 Wire Wire Line
@@
 Wire Wire Line
 	5250 2400 5800 2400
+$Comp
+L Device:D_Schottky D400
+U 1 1 5C91F491
+P 7300 9700
+AR Path="/5C91F491" Ref="D400"  Part="1"
+AR Path="/5CDAE2B6/5C91F491" Ref="D?"  Part="1"
+F 0 "D400" H 7300 9484 50  0000 C CNN
+F 1 "RB521S" H 7300 9575 50  0000 C CNN
+F 2 "require:D_SOD-523" H 7300 9700 50  0001 C CNN
+F 3 "~" H 7300 9700 50  0001 C CNN
+	1    7300 9700
+	-1   0    0    1
+$EndComp
+Wire Wire Line
+	7150 9700 6800 9700
+Text Label 6800 9700 0    50   ~ 0
+EMMC_D0
+Wire Wire Line
+	7450 9700 7600 9700
+$Comp
+L Device:R R?
+U 1 1 5C946245
+P 3450 4500
+AR Path="/5CDAE2B6/5C946245" Ref="R?"  Part="1"
+AR Path="/5C946245" Ref="R410"  Part="1"
+F 0 "R410" V 3350 4500 50  0000 C CNN
+F 1 "2.2k" V 3550 4500 50  0000 C CNN
+F 2 "require:R_0402" V 3380 4500 50  0001 C CNN
+F 3 "~" H 3450 4500 50  0001 C CNN
+	1    3450 4500
+	0    1    1    0
+$EndComp
+$Comp
+L power:GND #PWR?
+U 1 1 5C94624C
+P 3200 4500
+AR Path="/5CDAE2B6/5C94624C" Ref="#PWR?"  Part="1"
+AR Path="/5C94624C" Ref="#PWR0180"  Part="1"
+F 0 "#PWR0180" H 3200 4250 50  0001 C CNN
+F 1 "GND" V 3205 4372 50  0000 R CNN
+F 2 "" H 3200 4500 50  0001 C CNN
+F 3 "" H 3200 4500 50  0001 C CNN
+	1    3200 4500
+	0    1    1    0
+$EndComp
+Wire Wire Line
+	3200 4500 3300 4500
+Wire Wire Line
+	3800 4500 3600 4500
+NoConn ~ 1650 6050
+Text Notes 7100 9900 0    50   ~ 0
+Pin 1 is cathode
+Wire Wire Line
+	1350 6250 1350 6450
+$Comp
+L Device:R R802
+U 1 1 5C9A438C
+P 1000 6550
+F 0 "R802" H 1070 6596 50  0000 L CNN
+F 1 "0R" H 1070 6505 50  0000 L CNN
+F 2 "require:R_0603" V 930 6550 50  0001 C CNN
+F 3 "~" H 1000 6550 50  0001 C CNN
+	1    1000 6550
+	1    0    0    -1
+$EndComp
+Wire Wire Line
+	1250 6250 1250 6350
+Wire Wire Line
+	1250 6350 1000 6350
+Wire Wire Line
+	1000 6350 1000 6400
+Wire Wire Line
+	1000 6700 1000 6750
+$Comp
+L power:GND #PWR0221
+U 1 1 5C9B4AD2
+P 1000 6750
+F 0 "#PWR0221" H 1000 6500 50  0001 C CNN
+F 1 "GND" H 1005 6577 50  0000 C CNN
+F 2 "" H 1000 6750 50  0001 C CNN
+F 3 "" H 1000 6750 50  0001 C CNN
+	1    1000 6750
+	1    0    0    -1
+$EndComp
+Text Label 1000 6350 0    50   ~ 0
+SHIELD
 $EndSCHEMATC

Commit message: wip
Parts:
- removed D400: RB521S, require:D_SOD-523, symbol Device:D_Schottky
- removed D850: PESDUC3FD5VU, require:SOT-883, symbol require:PESDUC3FD5VU
- removed R850: 10k, require:R_0402, symbol Device:R
- removed RP19: U, require:OVAL_PIN, symbol require:OP
- removed SW850: SW_SKSC_4PIN, require:SW_ALPS_SKSCLCE010, symbol require:SW_SKSC_4PIN
Changed lines of the file:
@@
-	1    0    0    -1
-$EndComp
-$Comp
-L require:SW_SKSC_4PIN SW850
-U 1 1 5C723DBC
-P 13400 6500
-F 0 "SW850" H 13627 6521 50  0000 L CNN
-F 1 "SW_SKSC_4PIN" H 13627 6430 50  0000 L CNN
-F 2 "require:SW_ALPS_SKSCLCE010" H 13400 6500 50  0001 C CNN
-F 3 "" H 13400 6500 50  0001 C CNN
-	1    13400 6500
 	1    0    0    -1
 $EndComp
 Text Label 3000 3300 0    50   ~ 0
 EMMC_D0
-$Comp
-L require:OP RP?
-U 1 1 5C8D949C
-P 7800 9700
-AR Path="/5C70CDE2/5C8D949C" Ref="RP?"  Part="1"
-AR Path="/5C8D949C" Ref="RP19"  Part="1"
-F 0 "RP19" H 8050 9700 50  0000 C CNN
-F 1 "U" H 7800 9700 50  0000 C CNN
-F 2 "require:OVAL_PIN" H 7800 9650 50  0001 C CNN
-F 3 "" H 7800 9650 50  0001 C CNN
-	1    7800 9700
-	1    0    0    -1
-$EndComp
 Wire Wire Line
 	2800 8900 2900 8900
@@
 Text Label 6900 10250 0    50   ~ 0
 LED
-Wire Wire Line
-	13000 6600 12900 6600
-Wire Wire Line
-	12900 6600 12900 6700
-Wire Wire Line
-	12900 6700 13000 6700
-Wire Wire Line
-	12900 6700 12900 6850
-Connection ~ 12900 6700
-$Comp
-L power:GND #PWR0222
-U 1 1 5C76E8A9
-P 12900 6850
-F 0 "#PWR0222" H 12900 6600 50  0001 C CNN
-F 1 "GND" H 12905 6677 50  0000 C CNN
-F 2 "" H 12900 6850 50  0001 C CNN
-F 3 "" H 12900 6850 50  0001 C CNN
-	1    12900 6850
-	1    0    0    -1
-$EndComp
-Text Label 11650 6450 0    50   ~ 0
-KEY
-$Comp
-L Device:R R850
-U 1 1 5C774BC5
-P 11900 6150
-F 0 "R850" H 11970 6196 50  0000 L CNN
-F 1 "10k" H 11970 6105 50  0000 L CNN
-F 2 "require:R_0402" V 11830 6150 50  0001 C CNN
-F 3 "~" H 11900 6150 50  0001 C CNN
-	1    11900 6150
-	1    0    0    -1
-$EndComp
-Wire Wire Line
-	11900 6000 11900 5900
-$Comp
-L power:+3V3 #PWR0225
-U 1 1 5C781097
-P 11900 5900
-F 0 "#PWR0225" H 11900 5750 50  0001 C CNN
-F 1 "+3V3" H 11915 6073 50  0000 C CNN
-F 2 "" H 11900 5900 50  0001 C CNN
-F 3 "" H 11900 5900 50  0001 C CNN
-	1    11900 5900
-	1    0    0    -1
-$EndComp
-$Comp
-L require:PESDUC3FD5VU D850
-U 1 1 5C7834D1
-P 12150 6700
-F 0 "D850" H 12250 6750 50  0000 L CNN
-F 1 "PESDUC3FD5VU" H 12250 6650 50  0000 L CNN
-F 2 "require:SOT-883" H 12150 6700 50  0001 C CNN
-F 3 "" H 12150 6700 50  0001 C CNN
-	1    12150 6700
-	1    0    0    -1
-$EndComp
-Wire Wire Line
-	12200 6550 12200 6450
-Wire Wire Line
-	12100 6550 12100 6450
-Wire Wire Line
-	12150 6850 12150 6950
-$Comp
-L power:GND #PWR0227
-U 1 1 5C79C1A7
-P 12150 6950
-F 0 "#PWR0227" H 12150 6700 50  0001 C CNN
-F 1 "GND" H 12155 6777 50  0000 C CNN
-F 2 "" H 12150 6950 50  0001 C CNN
-F 3 "" H 12150 6950 50  0001 C CNN
-	1    12150 6950
-	1    0    0    -1
-$EndComp
 $Comp
 L Device:R R831
@@
 Wire Wire Line
 	2950 6450 2950 6550
-Connection ~ 12200 6450
-Wire Wire Line
-	12200 6450 12100 6450
-Connection ~ 12100 6450
-Wire Wire Line
-	12100 6450 11900 6450
-Wire Wire Line
-	11900 6300 11900 6450
-Connection ~ 11900 6450
-Wire Wire Line
-	11900 6450 11650 6450
-Wire Wire Line
-	12200 6450 12900 6450
 Wire Wire Line
 	6700 10150 7100 10150
@@
 	1950 5950 2350 5950
 Wire Wire Line
-	13000 6350 12900 6350
-Wire Wire Line
-	12900 6350 12900 6450
-Connection ~ 12900 6450
-Wire Wire Line
-	12900 6450 13000 6450
-Wire Wire Line
 	5250 2400 5800 2400
 $Comp
-L Device:D_Schottky D400
-U 1 1 5C91F491
-P 7300 9700
-AR Path="/5C91F491" Ref="D400"  Part="1"
-AR Path="/5CDAE2B6/5C91F491" Ref="D?"  Part="1"
-F 0 "D400" H 7300 9484 50  0000 C CNN
-F 1 "RB521S" H 7300 9575 50  0000 C CNN
-F 2 "require:D_SOD-523" H 7300 9700 50  0001 C CNN
-F 3 "~" H 7300 9700 50  0001 C CNN
-	1    7300 9700
-	-1   0    0    1
-$EndComp
-Wire Wire Line
-	7150 9700 6800 9700
-Text Label 6800 9700 0    50   ~ 0
-EMMC_D0
-Wire Wire Line
-	7450 9700 7600 9700
-$Comp
 L Device:R R?

Commit message: wip
Parts:
- removed H1, H2: MountingHole, require:MTG_1.8mm_2.4mm_NPL, symbol Mechanical:MountingHole
Changed lines of the file:
@@
 Wire Wire Line
 	12350 2450 12350 2550
-$Comp
-L Mechanical:MountingHole H1
-U 1 1 5C71E3C7
-P 11100 1650
-F 0 "H1" H 11200 1696 50  0000 L CNN
-F 1 "MountingHole" H 11200 1605 50  0000 L CNN
-F 2 "require:MTG_1.8mm_2.4mm_NPL" H 11100 1650 50  0001 C CNN
-F 3 "~" H 11100 1650 50  0001 C CNN
-	1    11100 1650
-	1    0    0    -1
-$EndComp
-$Comp
-L Mechanical:MountingHole H2
-U 1 1 5C71E586
-P 11100 1950
-F 0 "H2" H 11200 1996 50  0000 L CNN
-F 1 "MountingHole" H 11200 1905 50  0000 L CNN
-F 2 "require:MTG_1.8mm_2.4mm_NPL" H 11100 1950 50  0001 C CNN
-F 3 "~" H 11100 1950 50  0001 C CNN
-	1    11100 1950
-	1    0    0    -1
-$EndComp
 Text Label 6900 10150 0    50   ~ 0
 KEY

Commit message: wip
Parts:
- removed D840: LED, require:LED_0402, symbol Device:LED
- removed H3, H4: MountingHole_Pad, require:MTG_1.8mm_2.4mm_PL, symbol Mechanical:MountingHole_Pad
- removed LP13: NC, require:OVAL_PIN, symbol require:OP
- removed LP6: A5, require:OVAL_PIN, symbol require:OP
- removed LP8: RST, require:OVAL_PIN, symbol require:OP
- removed Q840: LMBT3904DW1T1G, require:SOT-363_SC-70-6, symbol require:NPND_SOT_363
- removed R840: 470R, require:R_0402, symbol Device:R
- removed RP15: 14, require:OVAL_PIN, symbol require:OP
- removed RP16: 15, require:OVAL_PIN, symbol require:OP
- removed RP17: 16, require:OVAL_PIN, symbol require:OP
- LP2: value A1 -> A0
- LP3: value A2 -> A1
- LP4: value A3 -> A2
- LP5: value A4 -> A3
Connections:
- net rk3308-io/A0: now also LP2.1; no longer R700.2, R701.1
- net rk3308-io/A1: now also LP3.1; no longer LP2.1
- net rk3308-io/A2: now also LP4.1; no longer LP3.1
- net rk3308-io/A3: now also LP5.1; no longer LP4.1
- net rk3308-io/A4: now also R700.2, R701.1; no longer LP5.1
- net at J800.3 (D+), R800.1: now also D800.2; no longer D800.1
- net at J800.2 (D-), R801.1: now also D800.1; no longer D800.2

Commit message: wip
Parts:
- removed LP15, RP1: G, require:OVAL_PIN, symbol require:OP
- removed R802: 0R, require:R_0603, symbol Device:R
- added J801: Molex 105164-0001, require:USB_Micro-B_Molex-105164-0001, symbol Connector:USB_B_Micro
- added R812, R813: 22R, require:R_0402, symbol Device:R
Connections:
- net SHIELD is gone; now on net GND: J800.6 (Shield)
- net +5V: now also J801.1 (VBUS)
- net GND: now also J801.5 (GND), J801.6 (Shield)
- net at D810.1, LP10.1, R811.1: now also R812.2
- net at D810.2, LP9.1, R810.1: now also R813.2
- new net: J801.2 (D-), R813.1
- new net: J801.3 (D+), R812.1
Other:
- moved on the sheet: C830, D800, D810, D820, J800, LP1, LP10, LP11, LP12, LP14, LP16, LP17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
