File: hardware/wireless.sch (KiCad schematic (older format))
At the start: 21 parts, among them U1 ap6255, U2 AW2015FCR, Y1 Crystal_GND24, Y4 SG-3030CM

Commit message: wip
Parts:
- removed C14: 1u, Capacitors_SMD:C_0402, symbol Device:C
- removed D9: LED_GBAR_0603X2, require:LED_RGB_0603X2, symbol require:LED_GBAR_0603X2
- removed R3: 30k, Resistors_SMD:R_0402, symbol Device:R
- removed R4, R5: 22R, Resistors_SMD:R_0402, symbol Device:R
- removed U2: AW2015FCR, require:AW2015FCR_QFN8L, symbol require:AW2015FCR
Connections:
- net labels removed: I2C1_SCL, I2C1_SDA, LED1, LED2, LED3
- wire segments 133 -> 96
Changed lines of the file:
@@
 $Descr A3 16535 11693
 encoding utf-8
-Sheet 3 8
+Sheet 3 7
 Title ""
 Date ""
@@
 Wire Wire Line
 	11300 8600 11950 8600
-$Comp
-L require:AW2015FCR U2
-U 1 1 5C6107EE
-P 5700 9150
-F 0 "U2" H 5700 9565 50  0000 C CNN
-F 1 "AW2015FCR" H 5700 9474 50  0000 C CNN
-F 2 "require:AW2015FCR_QFN8L" H 5700 9150 50  0001 C CNN
-F 3 "" H 5700 9150 50  0001 C CNN
-	1    5700 9150
-	1    0    0    -1
-$EndComp
-Wire Wire Line
-	5200 9000 4350 9000
-Text Label 4800 9000 0    50   ~ 0
-I2C1_SCL
-Wire Wire Line
-	5200 9100 4700 9100
-Text Label 4800 9100 0    50   ~ 0
-I2C1_SDA
-Wire Wire Line
-	6200 9000 6550 9000
-Wire Wire Line
-	6550 9000 6550 8100
-Wire Wire Line
-	6550 8100 4700 8100
-Wire Wire Line
-	6550 8100 6550 8000
-Connection ~ 6550 8100
-$Comp
-L require:VCC_IO #PWR03
-U 1 1 5C623B98
-P 6550 8000
-F 0 "#PWR03" H 6550 7850 50  0001 C CNN
-F 1 "VCC_IO" H 6567 8173 50  0000 C CNN
-F 2 "" H 6550 8000 50  0001 C CNN
-F 3 "" H 6550 8000 50  0001 C CNN
-	1    6550 8000
-	1    0    0    -1
-$EndComp
-$Comp
-L Device:C C14
-U 1 1 5C623C9A
-P 6750 8450
-F 0 "C14" H 6865 8496 50  0000 L CNN
-F 1 "1u" H 6865 8405 50  0000 L CNN
-F 2 "Capacitors_SMD:C_0402" H 6788 8300 50  0001 C CNN
-F 3 "~" H 6750 8450 50  0001 C CNN
-	1    6750 8450
-	1    0    0    -1
-$EndComp
-Wire Wire Line
-	6750 8300 6750 8100
-Wire Wire Line
-	6750 8100 6550 8100
-Wire Wire Line
-	6750 8600 6750 8800
-$Comp
-L power:GND #PWR04
-U 1 1 5C62E12F
-P 6750 8800
-F 0 "#PWR04" H 6750 8550 50  0001 C CNN
-F 1 "GND" H 6755 8627 50  0000 C CNN
-F 2 "" H 6750 8800 50  0001 C CNN
-F 3 "" H 6750 8800 50  0001 C CNN
-	1    6750 8800
-	1    0    0    -1
-$EndComp
-$Comp
-L Device:R R5
-U 1 1 5C630056
-P 4700 8500
-F 0 "R5" V 4493 8500 50  0000 C CNN
-F 1 "22R" V 4584 8500 50  0000 C CNN
-F 2 "Resistors_SMD:R_0402" V 4630 8500 50  0001 C CNN
-F 3 "~" H 4700 8500 50  0001 C CNN
-	1    4700 8500
-	-1   0    0    1
-$EndComp
-$Comp
-L Device:R R4
-U 1 1 5C630370
-P 4350 8500
-F 0 "R4" V 4143 8500 50  0000 C CNN
-F 1 "22R" V 4234 8500 50  0000 C CNN
-F 2 "Resistors_SMD:R_0402" V 4280 8500 50  0001 C CNN
-F 3 "~" H 4350 8500 50  0001 C CNN
-	1    4350 8500
-	-1   0    0    1
-$EndComp
-Wire Wire Line
-	4700 8350 4700 8100
-Connection ~ 4700 8100
-Wire Wire Line
-	4350 8100 4350 8350
-Wire Wire Line
-	4350 8100 4700 8100
-Wire Wire Line
-	4350 8650 4350 9000
-Connection ~ 4350 9000
-Wire Wire Line
-	4350 9000 4250 9000
-Wire Wire Line
-	4700 8650 4700 9100
-Connection ~ 4700 9100
-Wire Wire Line
-	4700 9100 4250 9100
-Wire Wire Line
-	5200 9200 4350 9200
-Wire Wire Line
-	4350 9200 4350 9400
-$Comp
-L power:GND #PWR02
-U 1 1 5C656BC3
-P 4350 9400
-F 0 "#PWR02" H 4350 9150 50  0001 C CNN
-F 1 "GND" H 4355 9227 50  0000 C CNN
-F 2 "" H 4350 9400 50  0001 C CNN
-F 3 "" H 4350 9400 50  0001 C CNN
-	1    4350 9400
-	1    0    0    -1
-$EndComp
-$Comp
-L Device:R R3
-U 1 1 5C657024
-P 3950 9300
-F 0 "R3" V 3743 9300 50  0000 C CNN
-F 1 "30k" V 3834 9300 50  0000 C CNN
-F 2 "Resistors_SMD:R_0402" V 3880 9300 50  0001 C CNN
-F 3 "~" H 3950 9300 50  0001 C CNN
-	1    3950 9300
-	0    1    1    0
-$EndComp
-Wire Wire Line
-	5200 9300 4100 9300
-Wire Wire Line
-	4350 8100 3500 8100
-Wire Wire Line
-	3500 8100 3500 9300
-Wire Wire Line
-	3500 9300 3800 9300
-Connection ~ 4350 8100
-Text Label 7100 9100 0    50   ~ 0
-LED3
-Text Label 7100 9200 0    50   ~ 0
-LED2
-Text Label 7100 9300 0    50   ~ 0
-LED1
-$Comp
-L require:LED_GBAR_0603X2 D9
-U 1 1 5C9EBB75
-P 8300 8750
-F 0 "D9" H 8300 9025 50  0000 C CNN
-F 1 "LED_GBAR_0603X2" H 8300 8934 50  0000 C CNN
-F 2 "require:LED_RGB_0603X2" H 8300 8750 50  0001 C CNN
-F 3 "" H 8300 8750 50  0001 C CNN
-	1    8300 8750
-	1    0    0    -1
-$EndComp
-Wire Wire Line
-	8650 8800 8800 8800
-Wire Wire Line
-	8800 8800 8800 9300
-Wire Wire Line
-	6200 9300 8800 9300
-Wire Wire Line
-	7650 9200 7650 8700
-Wire Wire Line
-	7650 8700 7950 8700
-Wire Wire Line
-	6200 9200 7650 9200
-Wire Wire Line
-	7550 9100 7550 8300
-Wire Wire Line
-	7550 8300 9000 8300
-Wire Wire Line
-	9000 8300 9000 8700
-Wire Wire Line
-	9000 8700 8650 8700
-Wire Wire Line
-	6200 9100 7550 9100
-Wire Wire Line
-	7950 8800 7800 8800
-Wire Wire Line
-	7800 8800 7800 9200
-Wire Wire Line
-	7800 9200 8300 9200
-Wire Wire Line
-	8300 9200 8300 9100
-$Comp
-L require:VCC_IO #PWR0229
-U 1 1 5CA12DDB
-P 8300 9100
-F 0 "#PWR0229" H 8300 8950 50  0001 C CNN
-F 1 "VCC_IO" H 8317 9273 50  0000 C CNN
-F 2 "" H 8300 9100 50  0001 C CNN
-F 3 "" H 8300 9100 50  0001 C CNN
-	1    8300 9100
-	1    0    0    -1
-$EndComp
 Wire Wire Line
 	12550 5650 12550 6400

Commit message: wip
Connections:
- net labels removed: UART4_CTS, UART4_RTS, UART4_RXD, UART4_TXD
Changed lines of the file:
@@
 	1    0    0    -1
 $EndComp
-Text Label 13950 3950 0    50   ~ 0
-UART4_RTS
-Text Label 13950 4050 0    50   ~ 0
-UART4_TXD
-Text Label 13950 4150 0    50   ~ 0
-UART4_RXD
-Text Label 13950 4250 0    50   ~ 0
-UART4_CTS
-Text Label 13950 4950 0    50   ~ 0
-BT_REG_ON
 NoConn ~ 13750 4350
 NoConn ~ 13750 4450
 NoConn ~ 13750 4550
 NoConn ~ 13750 4650
-Text Label 9800 4450 0    50   ~ 0
-SDIO_CLK
-Text Label 9800 4150 0    50   ~ 0
-SDIO_D2
-Text Label 9800 4250 0    50   ~ 0
-SDIO_D3
-Text Label 9800 4350 0    50   ~ 0
-SDIO_CMD
-Text Label 9800 4550 0    50   ~ 0
-SDIO_D0
-Text Label 9800 4650 0    50   ~ 0
-SDIO_D1
 $Comp
 L power:GND #PWR0138
@@
 Wire Wire Line
 	12550 1450 10300 1450
-Text Label 10400 1450 0    50   ~ 0
-HOST_WAKE_BT
-Text Label 10400 1550 0    50   ~ 0
-BT_WAKE_HOST
 Text HLabel 10300 1550 0    50   Input ~ 0
 BT_WAKE_HOST
@@
 	1    0    0    -1
 $EndComp
-Text Label 9800 3950 0    50   ~ 0
-WIFI_REG_ON
-Text Label 9800 4050 0    50   ~ 0
-WIFI_WAKE_HOST
 Wire Wire Line
 	10150 4950 10150 4850
@@
 Wire Wire Line
 	12250 6850 13200 6850
-Text Label 12650 6400 0    50   ~ 0
-PCM_SYNC
-Text Label 12650 6550 0    50   ~ 0
-PCM_IN
-Text Label 12650 6700 0    50   ~ 0
-PCM_CLK
-Text Label 12650 6850 0    50   ~ 0
-PCM_OUT
 Wire Wire Line
 	10100 2650 9400 2650

Commit message: wip
Parts:
- C1, C2, C4, C5, C6, C7, C9: footprint Capacitors_SMD:C_0402 -> require:C_0402
- C3, C8: footprint Capacitors_SMD:C_0603 -> require:C_0603
Changed lines of the file:
@@
 F 0 "C2" H 13415 2346 50  0000 L CNN
 F 1 "C" H 13415 2255 50  0000 L CNN
-F 2 "Capacitors_SMD:C_0402" H 13338 2150 50  0001 C CNN
+F 2 "require:C_0402" H 13338 2150 50  0001 C CNN
 F 3 "~" H 13300 2300 50  0001 C CNN
 	1    13300 2300
@@
 F 0 "C1" H 14115 2346 50  0000 L CNN
 F 1 "C" H 14115 2255 50  0000 L CNN
-F 2 "Capacitors_SMD:C_0402" H 14038 2150 50  0001 C CNN
+F 2 "require:C_0402" H 14038 2150 50  0001 C CNN
 F 3 "~" H 14000 2300 50  0001 C CNN
 	1    14000 2300
@@
 F 0 "C8" H 10815 6246 50  0000 L CNN
 F 1 "4.7u" H 10815 6155 50  0000 L CNN
-F 2 "Capacitors_SMD:C_0603" H 10738 6050 50  0001 C CNN
+F 2 "require:C_0603" H 10738 6050 50  0001 C CNN
 F 3 "~" H 10700 6200 50  0001 C CNN
 	1    10700 6200
@@
 F 0 "C3" H 9515 2446 50  0000 L CNN
 F 1 "10u" H 9515 2355 50  0000 L CNN
-F 2 "Capacitors_SMD:C_0603" H 9438 2250 50  0001 C CNN
+F 2 "require:C_0603" H 9438 2250 50  0001 C CNN
 F 3 "~" H 9400 2400 50  0001 C CNN
 	1    9400 2400
@@
 F 0 "C4" H 10215 2446 50  0000 L CNN
 F 1 "0.1u" H 10215 2355 50  0000 L CNN
-F 2 "Capacitors_SMD:C_0402" H 10138 2250 50  0001 C CNN
+F 2 "require:C_0402" H 10138 2250 50  0001 C CNN
 F 3 "~" H 10100 2400 50  0001 C CNN
 	1    10100 2400
@@
 F 0 "C6" H 11215 3396 50  0000 L CNN
 F 1 "22p" H 11215 3305 50  0000 L CNN
-F 2 "Capacitors_SMD:C_0402" H 11138 3200 50  0001 C CNN
+F 2 "require:C_0402" H 11138 3200 50  0001 C CNN
 F 3 "~" H 11100 3350 50  0001 C CNN
 	1    11100 3350
@@
 F 0 "C5" H 10215 3396 50  0000 L CNN
 F 1 "22p" H 10215 3305 50  0000 L CNN
-F 2 "Capacitors_SMD:C_0402" H 10138 3200 50  0001 C CNN
+F 2 "require:C_0402" H 10138 3200 50  0001 C CNN
 F 3 "~" H 10100 3350 50  0001 C CNN
 	1    10100 3350
@@
 F 0 "C7" H 10265 5246 50  0000 L CNN
 F 1 "1u" H 10265 5155 50  0000 L CNN
-F 2 "Capacitors_SMD:C_0402" H 10188 5050 50  0001 C CNN
+F 2 "require:C_0402" H 10188 5050 50  0001 C CNN
 F 3 "~" H 10150 5200 50  0001 C CNN
 	1    10150 5200
@@
 F 0 "C9" H 12865 8996 50  0000 L CNN
 F 1 "0.1u" H 12865 8905 50  0000 L CNN
-F 2 "Capacitors_SMD:C_0402" H 12788 8800 50  0001 C CNN
+F 2 "require:C_0402" H 12788 8800 50  0001 C CNN
 F 3 "~" H 12750 8950 50  0001 C CNN
 	1    12750 8950

Commit message: wip
Parts:
- removed C9: 0.1u, require:C_0402, symbol Device:C
- removed Y4: SG-3030CM, Oscillators:Oscillator_SMD_SeikoEpson_SG3030CM, symbol Oscillator:SG-3030CM
- added U1324: SIT1532, require:SITIME_1508, symbol require:SIT1532
Connections:
- wire segments 96 -> 85
Changed lines of the file:
@@
 	12650 5650 12650 5850
-Wire Wire Line
-	11300 8600 11300 8800
-$Comp
-L power:GND #PWR0125
-U 1 1 5D11F9E0
-P 11300 8800
-F 0 "#PWR0125" H 11300 8550 50  0001 C CNN
-F 1 "GND" H 11305 8627 50  0000 C CNN
-F 2 "" H 11300 8800 50  0001 C CNN
-F 3 "" H 11300 8800 50  0001 C CNN
-	1    11300 8800
-	1    0    0    -1
-$EndComp
-Wire Wire Line
-	12550 8500 12950 8500
-Text Label 12750 8500 0    50   ~ 0
-LPO
-Wire Wire Line
-	12550 8600 12750 8600
-Wire Wire Line
-	13150 8600 13150 8500
-$Comp
-L require:VCC_IO #PWR0127
-U 1 1 5D125099
-P 13150 8500
-F 0 "#PWR0127" H 13150 8350 50  0001 C CNN
-F 1 "VCC_IO" H 13167 8673 50  0000 C CNN
-F 2 "" H 13150 8500 50  0001 C CNN
-F 3 "" H 13150 8500 50  0001 C CNN
-	1    13150 8500
-	1    0    0    -1
-$EndComp
 Wire Wire Line
 	12150 5650 12150 6050
@@
 Text Label 11200 6050 0    50   ~ 0
 LPO
-$Comp
-L Device:C C9
-U 1 1 5D14135C
-P 12750 8950
-F 0 "C9" H 12865 8996 50  0000 L CNN
-F 1 "0.1u" H 12865 8905 50  0000 L CNN
-F 2 "require:C_0402" H 12788 8800 50  0001 C CNN
-F 3 "~" H 12750 8950 50  0001 C CNN
-	1    12750 8950
-	1    0    0    -1
-$EndComp
-Wire Wire Line
-	12750 8800 12750 8600
-Connection ~ 12750 8600
-Wire Wire Line
-	12750 8600 13150 8600
-Wire Wire Line
-	12750 9100 12750 9300
-$Comp
-L power:GND #PWR0224
-U 1 1 5D1473B7
-P 12750 9300
-F 0 "#PWR0224" H 12750 9050 50  0001 C CNN
-F 1 "GND" H 12755 9127 50  0000 C CNN
-F 2 "" H 12750 9300 50  0001 C CNN
-F 3 "" H 12750 9300 50  0001 C CNN
-	1    12750 9300
-	1    0    0    -1
-$EndComp
-$Comp
-L Oscillator:SG-3030CM Y4
-U 1 1 5D151475
-P 11950 8200
-F 0 "Y4" H 11720 8246 50  0000 R CNN
-F 1 "SG-3030CM" H 11720 8155 50  0000 R CNN
-F 2 "Oscillators:Oscillator_SMD_SeikoEpson_SG3030CM" H 11950 7850 50  0001 C CNN
-F 3 "https://support.epson.biz/td/api/doc_check.php?mode=dl&lang=en&Parts=SG-3030CM" H 11850 8200 50  0001 C CNN
-	1    11950 8200
-	1    0    0    -1
-$EndComp
-Wire Wire Line
-	12550 8500 12550 8200
-Wire Wire Line
-	12550 8200 12250 8200
-Wire Wire Line
-	12050 7900 12050 7650
-Wire Wire Line
-	12050 7650 13650 7650
-Wire Wire Line
-	13650 7650 13650 8750
-Wire Wire Line
-	13650 8750 13150 8750
-Wire Wire Line
-	13150 8750 13150 8600
-Connection ~ 13150 8600
-Wire Wire Line
-	11850 7900 11850 7650
-Wire Wire Line
-	11850 7650 12050 7650
-Connection ~ 12050 7650
-Wire Wire Line
-	11950 8600 11950 8500
-Wire Wire Line
-	11300 8600 11950 8600
 Wire Wire Line
 	12550 5650 12550 6400
@@
 Wire Wire Line
 	13750 4250 14550 4250
+$Comp
+L require:SIT1532 U1324
+U 1 1 5C6D1831
+P 5550 7950
+F 0 "U1324" H 5550 8265 50  0000 C CNN
+F 1 "SIT1532" H 5550 8174 50  0000 C CNN
+F 2 "require:SITIME_1508" H 5550 7950 50  0001 C CNN
+F 3 "" H 5550 7950 50  0001 C CNN
+	1    5550 7950
+	1    0    0    -1
+$EndComp
+Wire Wire Line
+	5950 7900 6150 7900
+Wire Wire Line
+	6150 7900 6150 8000
+Wire Wire Line
+	6150 8000 5950 8000
+Wire Wire Line
+	6150 8000 6150 8100
+Connection ~ 6150 8000
+$Comp
+L power:GND #PWR0245
+U 1 1 5C6D7368
+P 6150 8100
+F 0 "#PWR0245" H 6150 7850 50  0001 C CNN
+F 1 "GND" H 6155 7927 50  0000 C CNN
+F 2 "" H 6150 8100 50  0001 C CNN
+F 3 "" H 6150 8100 50  0001 C CNN
+	1    6150 8100
+	1    0    0    -1
+$EndComp
+Wire Wire Line
+	5150 7900 4950 7900
+Wire Wire Line
+	4950 7900 4950 7800
+$Comp
+L require:VCC_IO #PWR0246
+U 1 1 5C6DA5B5
+P 4950 7800
+F 0 "#PWR0246" H 4950 7650 50  0001 C CNN
+F 1 "VCC_IO" H 4967 7973 50  0000 C CNN
+F 2 "" H 4950 7800 50  0001 C CNN
+F 3 "" H 4950 7800 50  0001 C CNN
+	1    4950 7800
+	1    0    0    -1
+$EndComp
+Wire Wire Line
+	5150 8000 4750 8000
+Text Label 4750 8000 0    50   ~ 0
+LPO
 $EndSCHEMATC

Commit message: wip
Parts:
- renumbered C5 to C905, C6 to C906, C7 to C907, C8 to C908, U1324 to U2
Connections:
- net labels added: +3V3
- net labels removed: VCC_IO
Changed lines of the file:
@@
 	10700 5850 10700 5650
 $Comp
-L Device:C C8
+L Device:C C908
 U 1 1 5D29251B
 P 10700 6200
-F 0 "C8" H 10815 6246 50  0000 L CNN
+F 0 "C908" H 10815 6246 50  0000 L CNN
 F 1 "4.7u" H 10815 6155 50  0000 L CNN
 F 2 "require:C_0603" H 10738 6050 50  0001 C CNN
@@
 	9400 2150 9400 2050
 $Comp
-L require:VCC_IO #PWR0209
-U 1 1 5CB3B3D2
-P 9400 2050
-F 0 "#PWR0209" H 9400 1900 50  0001 C CNN
-F 1 "VCC_IO" H 9417 2223 50  0000 C CNN
-F 2 "" H 9400 2050 50  0001 C CNN
-F 3 "" H 9400 2050 50  0001 C CNN
-	1    9400 2050
-	1    0    0    -1
-$EndComp
-$Comp
 L Device:C C3
 U 1 1 5CB3CB45
@@
 epson fa-128
 $Comp
-L Device:C C6
+L Device:C C906
 U 1 1 5CB62E04
 P 11100 3350
-F 0 "C6" H 11215 3396 50  0000 L CNN
+F 0 "C906" H 11215 3396 50  0000 L CNN
 F 1 "22p" H 11215 3305 50  0000 L CNN
 F 2 "require:C_0402" H 11138 3200 50  0001 C CNN
@@
 $EndComp
 $Comp
-L Device:C C5
+L Device:C C905
 U 1 1 5CB67581
 P 10100 3350
-F 0 "C5" H 10215 3396 50  0000 L CNN
+F 0 "C905" H 10215 3396 50  0000 L CNN
 F 1 "22p" H 10215 3305 50  0000 L CNN
 F 2 "require:C_0402" H 10138 3200 50  0001 C CNN
@@
 	10150 4950 10150 4850
 $Comp
-L Device:C C7
+L Device:C C907
 U 1 1 5CE549D8
 P 10150 5200
-F 0 "C7" H 10265 5246 50  0000 L CNN
+F 0 "C907" H 10265 5246 50  0000 L CNN
 F 1 "1u" H 10265 5155 50  0000 L CNN
 F 2 "require:C_0402" H 10188 5050 50  0001 C CNN
@@
 F 3 "" H 10150 5450 50  0001 C CNN
 	1    10150 5450
-	1    0    0    -1
-$EndComp
-$Comp
-L require:VCC_IO #PWR0193
-U 1 1 5CF2517A
-P 10150 4850
-F 0 "#PWR0193" H 10150 4700 50  0001 C CNN
-F 1 "VCC_IO" H 10167 5023 50  0000 C CNN
-F 2 "" H 10150 4850 50  0001 C CNN
-F 3 "" H 10150 4850 50  0001 C CNN
-	1    10150 4850
 	1    0    0    -1
 $EndComp
@@
 	13750 4250 14550 4250
 $Comp
-L require:SIT1532 U1324
+L require:SIT1532 U2
 U 1 1 5C6D1831
 P 5550 7950
-F 0 "U1324" H 5550 8265 50  0000 C CNN
+F 0 "U2" H 5550 8265 50  0000 C CNN
 F 1 "SIT1532" H 5550 8174 50  0000 C CNN
 F 2 "require:SITIME_1508" H 5550 7950 50  0001 C CNN
@@
 Wire Wire Line
 	4950 7900 4950 7800
-$Comp
-L require:VCC_IO #PWR0246
-U 1 1 5C6DA5B5
+Wire Wire Line
+	5150 8000 4750 8000
+Text Label 4750 8000 0    50   ~ 0
+LPO
+$Comp
+L power:+3V3 #PWR0193
+U 1 1 5C7EACB6
+P 9400 2050
+F 0 "#PWR0193" H 9400 1900 50  0001 C CNN
+F 1 "+3V3" H 9415 2223 50  0000 C CNN
+F 2 "" H 9400 2050 50  0001 C CNN
+F 3 "" H 9400 2050 50  0001 C CNN
+	1    9400 2050
+	1    0    0    -1
+$EndComp
+$Comp
+L power:+3V3 #PWR0209
+U 1 1 5C7EADFF
+P 10150 4850
+F 0 "#PWR0209" H 10150 4700 50  0001 C CNN
+F 1 "+3V3" H 10165 5023 50  0000 C CNN
+F 2 "" H 10150 4850 50  0001 C CNN
+F 3 "" H 10150 4850 50  0001 C CNN
+	1    10150 4850
+	1    0    0    -1
+$EndComp
+$Comp
+L power:+3V3 #PWR0222
+U 1 1 5C7EAEE6
 P 4950 7800
-F 0 "#PWR0246" H 4950 7650 50  0001 C CNN
-F 1 "VCC_IO" H 4967 7973 50  0000 C CNN
+F 0 "#PWR0222" H 4950 7650 50  0001 C CNN
+F 1 "+3V3" H 4965 7973 50  0000 C CNN
 F 2 "" H 4950 7800 50  0001 C CNN
 F 3 "" H 4950 7800 50  0001 C CNN
@@
 	1    0    0    -1
 $EndComp
-Wire Wire Line
-	5150 8000 4750 8000
-Text Label 4750 8000 0    50   ~ 0
-LPO
 $EndSCHEMATC

Commit message: wip
Other:
- note added: "From CYW43455 datasheet\nL: 0806 size, 2.2 µH, DCR=0.11Ω, ACR=1.18Ω @ 4 MHz\nCout: Ceramic, X5R, 0402, ESR <30 mΩ at 4 MHz, 4.7 µF, ±20%, 6.3V\nCin: For SR_VDDBATP5V pin, ceramic, X5R, 0603, ESR < 30 mΩ at 4 MHz, ±4.7uF ±20%, 6.3V"
Changed lines of the file:
@@
 	10100 2800 10100 3100
 Wire Wire Line
-	10100 3100 10550 3100
-Wire Wire Line
 	10100 2800 12150 2800
-Wire Wire Line
-	10850 3100 11100 3100
 Text Notes 10900 2950 0    50   ~ 0
 epson fa-128
@@
 	1    0    0    -1
 $EndComp
+Text Notes 1850 6150 0    100  ~ 0
+From CYW43455 datasheet\nL: 0806 size, 2.2 µH, DCR=0.11Ω, ACR=1.18Ω @ 4 MHz\nCout:  Ceramic, X5R, 0402, ESR <30 mΩ at 4 MHz, 4.7 µF, ±20%, 6.3V\nCin: For SR_VDDBATP5V pin, ceramic, X5R, 0603, ESR < 30 mΩ at 4 MHz, ±4.7uF ±20%, 6.3V
+Wire Wire Line
+	10100 3100 10550 3100
+Wire Wire Line
+	10850 3100 11100 3100
 $EndSCHEMATC
