File: hardware/wireless.sch (KiCad schematic (older format))
At the start: 14 parts, among them U1 ap6255, U2 SIT1532, Y1 Crystal_GND24

Commit message: wip
Parts:
- removed U2: SIT1532, require:SITIME_1508, symbol require:SIT1532
- added C550: 4.7u, require:C_0402, symbol Device:C
- added Y550: SG-3030CM, Oscillators:Oscillator_SMD_SeikoEpson_SG3030CM, symbol Oscillator:SG-3030CM
- C511: renamed from C4; value 0.1u -> 10u; footprint require:C_0402 -> require:C_0603
- L540: renamed from L2; value 3.3u -> 2.2u
- renumbered C1 to C500, C2 to C501, C3 to C510, C905 to C520, C906 to C521, C907 to C530, C908 to C540, L1 to L500, U1 to U500, Y1 to Y520
Connections:
- net +3V3: now also C550.1, Y550.1 (VIO), Y550.4 (Vcc)
- net GND: now also C550.2, Y550.2 (GND)
- net LPO: now also Y550.3 (OUT)
- net PCM_CLK: no longer names the net of U500.26 (PCM_CLK)
- net PCM_IN: no longer names the net of U500.27 (PCM_IN)
- net PCM_OUT: no longer names the net of U500.25 (PCM_OUT)
- net PCM_SYNC: no longer names the net of U500.28 (PCM_SYNC)
- no-connect marks 4 -> 8
Changed lines of the file:
@@
 $EndDescr
 $Comp
-L require-rescue:ap6255 U1
+L require-rescue:ap6255 U500
 U 1 1 5C2E29DF
 P 12550 4450
-F 0 "U1" H 12550 4500 60  0000 C CNN
+F 0 "U500" H 12550 4500 60  0000 C CNN
 F 1 "ap6255" H 12550 4400 60  0000 C CNN
 F 2 "require:AP6255_QFP_44" H 12550 4450 60  0001 C CNN
@@
 $EndComp
 $Comp
-L Device:C C2
+L Device:C C501
 U 1 1 5D28602E
 P 13300 2300
-F 0 "C2" H 13415 2346 50  0000 L CNN
+F 0 "C501" H 13415 2346 50  0000 L CNN
 F 1 "C" H 13415 2255 50  0000 L CNN
 F 2 "require:C_0402" H 13338 2150 50  0001 C CNN
@@
 	13300 1950 13500 1950
 $Comp
-L Device:L L1
+L Device:L L500
 U 1 1 5D287D6F
 P 13650 1950
-F 0 "L1" V 13840 1950 50  0000 C CNN
+F 0 "L500" V 13840 1950 50  0000 C CNN
 F 1 "L" V 13749 1950 50  0000 C CNN
 F 2 "Inductors_SMD:L_0402" H 13650 1950 50  0001 C CNN
@@
 $EndComp
 $Comp
-L Device:C C1
+L Device:C C500
 U 1 1 5D287E21
 P 14000 2300
-F 0 "C1" H 14115 2346 50  0000 L CNN
+F 0 "C500" H 14115 2346 50  0000 L CNN
 F 1 "C" H 14115 2255 50  0000 L CNN
 F 2 "require:C_0402" H 14038 2150 50  0001 C CNN
@@
 	12950 1950 13300 1950
 $Comp
-L Device:L L2
+L Device:L L540
 U 1 1 5D290030
 P 10700 5500
-F 0 "L2" H 10753 5546 50  0000 L CNN
-F 1 "3.3u" H 10753 5455 50  0000 L CNN
-F 2 "require:L_murata_2520" H 10700 5500 50  0001 C CNN
+F 0 "L540" H 10753 5546 50  0000 L CNN
+F 1 "2.2u" H 10753 5455 50  0000 L CNN
+F 2 "require:L_murata_2520" H 11150 5350 50  0000 C CNN
 F 3 "~" H 10700 5500 50  0001 C CNN
 	1    10700 5500
@@
 	10700 5850 10700 5650
 $Comp
-L Device:C C908
+L Device:C C540
 U 1 1 5D29251B
 P 10700 6200
-F 0 "C908" H 10815 6246 50  0000 L CNN
+F 0 "C540" H 10815 6246 50  0000 L CNN
 F 1 "4.7u" H 10815 6155 50  0000 L CNN
 F 2 "require:C_0603" H 10738 6050 50  0001 C CNN
@@
 	9400 2150 9400 2050
 $Comp
-L Device:C C3
+L Device:C C510
 U 1 1 5CB3CB45
 P 9400 2400
-F 0 "C3" H 9515 2446 50  0000 L CNN
+F 0 "C510" H 9515 2446 50  0000 L CNN
 F 1 "10u" H 9515 2355 50  0000 L CNN
-F 2 "require:C_0603" H 9438 2250 50  0001 C CNN
+F 2 "require:C_0603" H 9438 2250 50  0000 C CNN
 F 3 "~" H 9400 2400 50  0001 C CNN
 	1    9400 2400
@@
 $EndComp
 $Comp
-L Device:C C4
+L Device:C C511
 U 1 1 5CB3CBB9
 P 10100 2400
-F 0 "C4" H 10215 2446 50  0000 L CNN
-F 1 "0.1u" H 10215 2355 50  0000 L CNN
-F 2 "require:C_0402" H 10138 2250 50  0001 C CNN
+F 0 "C511" H 10215 2446 50  0000 L CNN
+F 1 "10u" H 10215 2355 50  0000 L CNN
+F 2 "require:C_0603" H 10138 2250 50  0000 C CNN
 F 3 "~" H 10100 2400 50  0001 C CNN
 	1    10100 2400
@@
 Connection ~ 9400 2150
 $Comp
-L Device:Crystal_GND24 Y1
+L Device:Crystal_GND24 Y520
 U 1 1 5CB46F9E
 P 10700 3100
-F 0 "Y1" H 10891 3146 50  0000 L CNN
+F 0 "Y520" H 10891 3146 50  0000 L CNN
 F 1 "Crystal_GND24" H 10891 3055 50  0000 L CNN
 F 2 "require:EPSON_FA_128" H 10700 3100 50  0001 C CNN
@@
 epson fa-128
 $Comp
-L Device:C C906
+L Device:C C521
 U 1 1 5CB62E04
 P 11100 3350
-F 0 "C906" H 11215 3396 50  0000 L CNN
+F 0 "C521" H 11215 3396 50  0000 L CNN
 F 1 "22p" H 11215 3305 50  0000 L CNN
 F 2 "require:C_0402" H 11138 3200 50  0001 C CNN
@@
 $EndComp
 $Comp
-L Device:C C905
+L Device:C C520
 U 1 1 5CB67581
 P 10100 3350
-F 0 "C905" H 10215 3396 50  0000 L CNN
+F 0 "C520" H 10215 3396 50  0000 L CNN
 F 1 "22p" H 10215 3305 50  0000 L CNN
 F 2 "require:C_0402" H 10138 3200 50  0001 C CNN
@@
 	10150 4950 10150 4850
 $Comp
-L Device:C C907
+L Device:C C530
 U 1 1 5CE549D8
 P 10150 5200
-F 0 "C907" H 10265 5246 50  0000 L CNN
+F 0 "C530" H 10265 5246 50  0000 L CNN
 F 1 "1u" H 10265 5155 50  0000 L CNN
 F 2 "require:C_0402" H 10188 5050 50  0001 C CNN
@@
 LPO
 Wire Wire Line
-	12550 5650 12550 6400
-Wire Wire Line
-	12550 6400 13200 6400
-Wire Wire Line
-	12450 5650 12450 6550
-Wire Wire Line
-	12450 6550 13200 6550
-Wire Wire Line
-	12350 5650 12350 6700
-Wire Wire Line
-	12350 6700 13200 6700
-Wire Wire Line
-	12250 5650 12250 6850
-Wire Wire Line
-	12250 6850 13200 6850
-Wire Wire Line
 	10100 2650 9400 2650
 Connection ~ 9400 2650
@@
 Wire Wire Line
 	9700 4050 11350 4050
-Text HLabel 13200 6400 2    50   Input ~ 0
-PCM_SYNC
-Text HLabel 13200 6550 2    50   Input ~ 0
-PCM_IN
-Text HLabel 13200 6700 2    50   Input ~ 0
-PCM_CLK
-Text HLabel 13200 6850 2    50   Input ~ 0
-PCM_OUT
 Text HLabel 9700 4150 0    50   Input ~ 0
 SDIO_D2
@@
 	13750 4250 14550 4250
 $Comp
-L require:SIT1532 U2
-U 1 1 5C6D1831
-P 5550 7950
-F 0 "U2" H 5550 8265 50  0000 C CNN
-F 1 "SIT1532" H 5550 8174 50  0000 C CNN
-F 2 "require:SITIME_1508" H 5550 7950 50  0001 C CNN
-F 3 "" H 5550 7950 50  0001 C CNN
-	1    5550 7950
-	1    0    0    -1
-$EndComp
-Wire Wire Line
-	5950 7900 6150 7900
-Wire Wire Line
-	6150 7900 6150 8000
-Wire Wire Line
-	6150 8000 5950 8000
-Wire Wire Line
-	6150 8000 6150 8100
-Connection ~ 6150 8000
-$Comp
-L power:GND #PWR0245
-U 1 1 5C6D7368
-P 6150 8100
-F 0 "#PWR0245" H 6150 7850 50  0001 C CNN
-F 1 "GND" H 6155 7927 50  0000 C CNN
-F 2 "" H 6150 8100 50  0001 C CNN
-F 3 "" H 6150 8100 50  0001 C CNN
-	1    6150 8100
-	1    0    0    -1
-$EndComp
-Wire Wire Line
-	5150 7900 4950 7900
-Wire Wire Line
-	4950 7900 4950 7800
-Wire Wire Line
-	5150 8000 4750 8000
-Text Label 4750 8000 0    50   ~ 0
-LPO
-$Comp
 L power:+3V3 #PWR0193
 U 1 1 5C7EACB6
@@
 	1    0    0    -1
 $EndComp
-$Comp
-L power:+3V3 #PWR0222
-U 1 1 5C7EAEE6
-P 4950 7800
-F 0 "#PWR0222" H 4950 7650 50  0001 C CNN
-F 1 "+3V3" H 4965 7973 50  0000 C CNN
-F 2 "" H 4950 7800 50  0001 C CNN
-F 3 "" H 4950 7800 50  0001 C CNN
-	1    4950 7800
-	1    0    0    -1
-$EndComp
 Text Notes 1850 6150 0    100  ~ 0
 From CYW43455 datasheet\nL: 0806 size, 2.2 µH, DCR=0.11Ω, ACR=1.18Ω @ 4 MHz\nCout:  Ceramic, X5R, 0402, ESR <30 mΩ at 4 MHz, 4.7 µF, ±20%, 6.3V\nCin: For SR_VDDBATP5V pin, ceramic, X5R, 0603, ESR < 30 mΩ at 4 MHz, ±4.7uF ±20%, 6.3V
@@
 Wire Wire Line
 	10850 3100 11100 3100
+$Comp
+L Oscillator:SG-3030CM Y550
+U 1 1 5C725C3D
+P 7400 7850
+F 0 "Y550" H 7170 7896 50  0000 R CNN
+F 1 "SG-3030CM" H 7170 7805 50  0000 R CNN
+F 2 "Oscillators:Oscillator_SMD_SeikoEpson_SG3030CM" H 7400 7500 50  0001 C CNN
+F 3 "https://support.epson.biz/td/api/doc_check.php?mode=dl&lang=en&Parts=SG-3030CM" H 7300 7850 50  0001 C CNN
+	1    7400 7850
+	1    0    0    -1
+$EndComp
+$Comp
+L power:GND #PWR0220
+U 1 1 5C729A2A
+P 7400 8250
+F 0 "#PWR0220" H 7400 8000 50  0001 C CNN
+F 1 "GND" H 7405 8077 50  0000 C CNN
+F 2 "" H 7400 8250 50  0001 C CNN
+F 3 "" H 7400 8250 50  0001 C CNN
+	1    7400 8250
+	1    0    0    -1
+$EndComp
+Wire Wire Line
+	7400 8150 7400 8250
+Wire Wire Line
+	7300 7550 7300 7400
+Wire Wire Line
+	7300 7400 7500 7400
+Wire Wire Line
+	7500 7400 7500 7550
+Wire Wire Line
+	7300 7400 6550 7400
+Connection ~ 7300 7400
+$Comp
+L Device:C C550
+U 1 1 5C730CC7
+P 6550 7750
+F 0 "C550" H 6665 7796 50  0000 L CNN
+F 1 "4.7u" H 6665 7705 50  0000 L CNN
+F 2 "require:C_0402" H 6588 7600 50  0001 C CNN
+F 3 "~" H 6550 7750 50  0001 C CNN
+	1    6550 7750
+	1    0    0    -1
+$EndComp
+Wire Wire Line
+	6550 7400 6550 7600
+Wire Wire Line
+	6550 7400 6550 7300
+Connection ~ 6550 7400
+$Comp
+L power:+3V3 #PWR0221
+U 1 1 5C7360B5
+P 6550 7300
+F 0 "#PWR0221" H 6550 7150 50  0001 C CNN
+F 1 "+3V3" H 6565 7473 50  0000 C CNN
+F 2 "" H 6550 7300 50  0001 C CNN
+F 3 "" H 6550 7300 50  0001 C CNN
+	1    6550 7300
+	1    0    0    -1
+$EndComp
+$Comp
+L power:GND #PWR0223
+U 1 1 5C73613C
+P 6550 8000
+F 0 "#PWR0223" H 6550 7750 50  0001 C CNN
+F 1 "GND" H 6555 7827 50  0000 C CNN
+F 2 "" H 6550 8000 50  0001 C CNN
+F 3 "" H 6550 8000 50  0001 C CNN
+	1    6550 8000
+	1    0    0    -1
+$EndComp
+Wire Wire Line
+	6550 7900 6550 8000
+Wire Wire Line
+	7700 7850 8100 7850
+Text Label 7900 7850 0    50   ~ 0
+LPO
+NoConn ~ 12250 5650
+NoConn ~ 12350 5650
+NoConn ~ 12450 5650
+NoConn ~ 12550 5650
 $EndSCHEMATC

Commit message: wip
Parts:
- A500: renamed from ANT1; value ANT12 -> AH104N2450D1-T
- C540: value 4.7u -> 10u
- L500: footprint Inductors_SMD:L_0402 -> require:L_0402
- U500: symbol require-rescue:ap6255 -> require:ap6255
- Y520: value Crystal_GND24 -> 37.4MHz,12pF,10ppm
Other:
- note removed: "epson fa-128"
- moved on the sheet: A500, C500, C501, C510, C511, C520, C521, C530, C540, C550, L500, L540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
