File: hardware/wireless.sch (KiCad schematic (older format))
At the start: 15 parts, among them U500 ap6255, Y520 37.4MHz,12pF,10ppm, Y550 SG-3030CM

Commit message: wip
Parts:
- removed C550: 4.7u, require:C_0402, symbol Device:C
- removed Y550: SG-3030CM, Oscillators:Oscillator_SMD_SeikoEpson_SG3030CM, symbol Oscillator:SG-3030CM
Connections:
- wire segments 79 -> 70
Changed lines of the file:
@@
 	5350 6950 5350 7350
-Wire Wire Line
-	5350 7350 4400 7350
-Text Label 4400 7350 0    50   ~ 0
-LPO
 Wire Wire Line
 	3300 3950 2600 3950
@@
 Wire Wire Line
 	4050 4400 4300 4400
-$Comp
-L Oscillator:SG-3030CM Y550
-U 1 1 5C725C3D
-P 12950 5200
-F 0 "Y550" H 12720 5246 50  0000 R CNN
-F 1 "SG-3030CM" H 12720 5155 50  0000 R CNN
-F 2 "Oscillators:Oscillator_SMD_SeikoEpson_SG3030CM" H 12950 4850 50  0001 C CNN
-F 3 "https://support.epson.biz/td/api/doc_check.php?mode=dl&lang=en&Parts=SG-3030CM" H 12850 5200 50  0001 C CNN
-	1    12950 5200
-	1    0    0    -1
-$EndComp
-$Comp
-L power:GND #PWR0220
-U 1 1 5C729A2A
-P 12950 5600
-F 0 "#PWR0220" H 12950 5350 50  0001 C CNN
-F 1 "GND" H 12955 5427 50  0000 C CNN
-F 2 "" H 12950 5600 50  0001 C CNN
-F 3 "" H 12950 5600 50  0001 C CNN
-	1    12950 5600
-	1    0    0    -1
-$EndComp
-Wire Wire Line
-	12950 5500 12950 5600
-Wire Wire Line
-	12850 4900 12850 4750
-Wire Wire Line
-	12850 4750 13050 4750
-Wire Wire Line
-	13050 4750 13050 4900
-Wire Wire Line
-	12850 4750 12100 4750
-Connection ~ 12850 4750
-$Comp
-L Device:C C550
-U 1 1 5C730CC7
-P 12100 5100
-F 0 "C550" H 12215 5146 50  0000 L CNN
-F 1 "4.7u" H 12215 5055 50  0000 L CNN
-F 2 "require:C_0402" H 12138 4950 50  0001 C CNN
-F 3 "~" H 12100 5100 50  0001 C CNN
-	1    12100 5100
-	1    0    0    -1
-$EndComp
-Wire Wire Line
-	12100 4750 12100 4950
-Wire Wire Line
-	12100 4750 12100 4650
-Connection ~ 12100 4750
-$Comp
-L power:+3V3 #PWR0221
-U 1 1 5C7360B5
-P 12100 4650
-F 0 "#PWR0221" H 12100 4500 50  0001 C CNN
-F 1 "+3V3" H 12115 4823 50  0000 C CNN
-F 2 "" H 12100 4650 50  0001 C CNN
-F 3 "" H 12100 4650 50  0001 C CNN
-	1    12100 4650
-	1    0    0    -1
-$EndComp
-$Comp
-L power:GND #PWR0223
-U 1 1 5C73613C
-P 12100 5350
-F 0 "#PWR0223" H 12100 5100 50  0001 C CNN
-F 1 "GND" H 12105 5177 50  0000 C CNN
-F 2 "" H 12100 5350 50  0001 C CNN
-F 3 "" H 12100 5350 50  0001 C CNN
-	1    12100 5350
-	1    0    0    -1
-$EndComp
-Wire Wire Line
-	12100 5250 12100 5350
-Wire Wire Line
-	13250 5200 13650 5200
-Text Label 13450 5200 0    50   ~ 0
-LPO
 NoConn ~ 5450 6950
 NoConn ~ 5550 6950
 NoConn ~ 5650 6950
 NoConn ~ 5750 6950
+Text HLabel 4850 7350 0    50   Input ~ 0
+LPO
+Wire Wire Line
+	4850 7350 5350 7350
 $EndSCHEMATC

Commit message: wip
Changed lines of the file:
@@
 Wire Wire Line
 	6050 4550 6050 3250
-Wire Wire Line
-	6250 4550 6250 4350
-Wire Wire Line
-	6250 4350 6500 4350
 $Comp
 L power:GND #PWR0142
 U 1 1 5D284F62
-P 6500 4350
-F 0 "#PWR0142" H 6500 4100 50  0001 C CNN
-F 1 "GND" V 6505 4222 50  0000 R CNN
-F 2 "" H 6500 4350 50  0001 C CNN
-F 3 "" H 6500 4350 50  0001 C CNN
-	1    6500 4350
-	0    -1   -1   0
+P 6250 4450
+F 0 "#PWR0142" H 6250 4200 50  0001 C CNN
+F 1 "GND" V 6255 4322 50  0000 R CNN
+F 2 "" H 6250 4450 50  0001 C CNN
+F 3 "" H 6250 4450 50  0001 C CNN
+	1    6250 4450
+	-1   0    0    1
 $EndComp
 $Comp
@@
 P 3900 4400
 F 0 "Y520" H 4100 4600 50  0000 L CNN
-F 1 "37.4MHz,12pF,10ppm" H 4100 4450 50  0000 L CNN
+F 1 "37.4MHz,12pF,10ppm" H 4100 4500 50  0000 L CNN
 F 2 "require:EPSON_FA_128" H 3900 4400 50  0001 C CNN
 F 3 "~" H 3900 4400 50  0001 C CNN
@@
 Wire Wire Line
 	4850 7350 5350 7350
+Wire Wire Line
+	6250 4450 6250 4550
 $EndSCHEMATC

Commit message: wip
Changed lines of the file:
@@
 F 0 "L540" H 3953 6846 50  0000 L CNN
 F 1 "2.2u" H 3953 6755 50  0000 L CNN
-F 2 "require:L_murata_2520" H 4350 6650 50  0001 C CNN
+F 2 "require:L_murata_2520" H 4350 6650 50  0000 C CNN
 F 3 "~" H 3900 6800 50  0001 C CNN
 	1    3900 6800

Commit message: wip
Parts:
- A500: footprint require:YAIYO_YUDEN_AH104N -> require:ANT_AH104N
- C520, C521: value 22p -> 15p
- L540: footprint require:L_murata_2520 -> require:L_1008
- Y520: value 37.4MHz,12pF,10ppm -> 37.4MHz,9pF,10ppm; footprint require:EPSON_FA_128 -> Crystals:Crystal_SMD_2016-4pin_2.0x1.6mm
Changed lines of the file:
@@
 F 0 "L540" H 3953 6846 50  0000 L CNN
 F 1 "2.2u" H 3953 6755 50  0000 L CNN
-F 2 "require:L_murata_2520" H 4350 6650 50  0000 C CNN
+F 2 "require:L_1008" H 3950 6650 50  0000 C CNN
 F 3 "~" H 3900 6800 50  0001 C CNN
 	1    3900 6800
@@
 P 3900 4400
 F 0 "Y520" H 4100 4600 50  0000 L CNN
-F 1 "37.4MHz,12pF,10ppm" H 4100 4500 50  0000 L CNN
-F 2 "require:EPSON_FA_128" H 3900 4400 50  0001 C CNN
+F 1 "37.4MHz,9pF,10ppm" H 4100 4500 50  0000 L CNN
+F 2 "Crystals:Crystal_SMD_2016-4pin_2.0x1.6mm" H 3900 4400 50  0001 C CNN
 F 3 "~" H 3900 4400 50  0001 C CNN
 	1    3900 4400
@@
 P 4300 4650
 F 0 "C521" H 4415 4696 50  0000 L CNN
-F 1 "22p" H 4415 4605 50  0000 L CNN
+F 1 "15p" H 4415 4605 50  0000 L CNN
 F 2 "require:C_0402" H 4338 4500 50  0001 C CNN
 F 3 "~" H 4300 4650 50  0001 C CNN
@@
 P 3300 4650
 F 0 "C520" H 3415 4696 50  0000 L CNN
-F 1 "22p" H 3415 4605 50  0000 L CNN
+F 1 "15p" H 3415 4605 50  0000 L CNN
 F 2 "require:C_0402" H 3338 4500 50  0001 C CNN
 F 3 "~" H 3300 4650 50  0001 C CNN
@@
 F 0 "A500" H 7200 3515 50  0000 C CNN
 F 1 "AH104N2450D1-T" H 7200 3424 50  0000 C CNN
-F 2 "require:YAIYO_YUDEN_AH104N" H 7200 3150 50  0001 C CNN
+F 2 "require:ANT_AH104N" H 7200 3150 50  0001 C CNN
 F 3 "" H 7200 3150 50  0001 C CNN
 	1    7200 3150

Commit message: wip
Parts:
- removed A500: AH104N2450D1-T, require:ANT_AH104N, symbol require:ANT12
Changed lines of the file:
@@
 Text Notes 6500 7150 0    50   ~ 10
 Use SDIO 2.0 (3V3)
-$Comp
-L require:ANT12 A500
-U 1 1 5CF44F61
-P 7200 3150
-F 0 "A500" H 7200 3515 50  0000 C CNN
-F 1 "AH104N2450D1-T" H 7200 3424 50  0000 C CNN
-F 2 "require:ANT_AH104N" H 7200 3150 50  0001 C CNN
-F 3 "" H 7200 3150 50  0001 C CNN
-	1    7200 3150
-	1    0    0    -1
-$EndComp
 Wire Wire Line
 	7200 3250 7200 3150

Commit message: wip
Parts:
- removed C530: 1u, require:C_0402, symbol Device:C
Changed lines of the file:
@@
 	3350 6250 3350 6150
-$Comp
-L Device:C C530
-U 1 1 5CE549D8
-P 3350 6500
-F 0 "C530" H 3465 6546 50  0000 L CNN
-F 1 "1u" H 3465 6455 50  0000 L CNN
-F 2 "require:C_0402" H 3388 6350 50  0001 C CNN
-F 3 "~" H 3350 6500 50  0001 C CNN
-	1    3350 6500
-	1    0    0    -1
-$EndComp
-Wire Wire Line
-	3350 6350 3350 6250
-Connection ~ 3350 6250
-Wire Wire Line
-	3350 6650 3350 6750
-$Comp
-L power:GND #PWR0217
-U 1 1 5CE5B30C
-P 3350 6750
-F 0 "#PWR0217" H 3350 6500 50  0001 C CNN
-F 1 "GND" H 3355 6577 50  0000 C CNN
-F 2 "" H 3350 6750 50  0001 C CNN
-F 3 "" H 3350 6750 50  0001 C CNN
-	1    3350 6750
-	1    0    0    -1
-$EndComp
 $Comp
 L power:GND #PWR0198

Commit message: wip
Parts:
- added C530: 1u, require:C_0402, symbol Device:C
Connections:
- net +3V3: now also C530.1
- net GND: now also C530.2
Changed lines of the file:
@@
 Wire Wire Line
 	6250 4450 6250 4550
+$Comp
+L Device:C C530
+U 1 1 5CD42670
+P 3350 6500
+F 0 "C530" H 3465 6546 50  0000 L CNN
+F 1 "1u" H 3465 6455 50  0000 L CNN
+F 2 "require:C_0402" H 3388 6350 50  0001 C CNN
+F 3 "~" H 3350 6500 50  0001 C CNN
+	1    3350 6500
+	1    0    0    -1
+$EndComp
+Wire Wire Line
+	3350 6350 3350 6250
+Connection ~ 3350 6250
+Wire Wire Line
+	3350 6650 3350 6750
+$Comp
+L power:GND #PWR0179
+U 1 1 5CD4524F
+P 3350 6750
+F 0 "#PWR0179" H 3350 6500 50  0001 C CNN
+F 1 "GND" H 3355 6577 50  0000 C CNN
+F 2 "" H 3350 6750 50  0001 C CNN
+F 3 "" H 3350 6750 50  0001 C CNN
+	1    3350 6750
+	1    0    0    -1
+$EndComp
 $EndSCHEMATC

Commit message: prepare gerber and drill
Parts:
- added ANT1: ANT_LA52H2450_5500_A28, require:LA52H2450_5500_A28, symbol require:ANT_LA52H2450_5500_A28
- Y520: footprint Crystals:Crystal_SMD_2016-4pin_2.0x1.6mm -> require:Crystal_SMD_2016-4pin_2.0x1.6mm
Connections:
- net GND: now also C500.1, L500.2, ANT1.2, ANT1.3
- net RFOUT: now reaches C501.1, L500.1, U500.2 (ANT)
- no-connect marks 8 -> 9
Changed lines of the file:
@@
 F 0 "Y520" H 4100 4600 50  0000 L CNN
 F 1 "37.4MHz,9pF,10ppm" H 4100 4500 50  0000 L CNN
-F 2 "Crystals:Crystal_SMD_2016-4pin_2.0x1.6mm" H 3900 4400 50  0001 C CNN
+F 2 "require:Crystal_SMD_2016-4pin_2.0x1.6mm" H 3900 4400 50  0001 C CNN
 F 3 "~" H 3900 4400 50  0001 C CNN
 	1    3900 4400
@@
 Text Notes 6500 7150 0    50   ~ 10
 Use SDIO 2.0 (3V3)
-Wire Wire Line
-	7200 3250 7200 3150
-Connection ~ 7200 3250
 Wire Wire Line
 	5850 6950 5850 7150
@@
 	1    0    0    -1
 $EndComp
+$Comp
+L power:GND #PWR0188
+U 1 1 5CDBDA48
+P 7400 3250
+F 0 "#PWR0188" H 7400 3000 50  0001 C CNN
+F 1 "GND" V 7405 3122 50  0000 R CNN
+F 2 "" H 7400 3250 50  0001 C CNN
+F 3 "" H 7400 3250 50  0001 C CNN
+	1    7400 3250
+	0    -1   -1   0
+$EndComp
+Wire Wire Line
+	7400 3250 7200 3250
+Connection ~ 7200 3250
+$Comp
+L require:ANT_LA52H2450_5500_A28 ANT1
+U 1 1 5CDC3928
+P 7700 2500
+F 0 "ANT1" H 8028 2440 50  0000 L CNN
+F 1 "ANT_LA52H2450_5500_A28" H 8028 2349 50  0000 L CNN
+F 2 "require:LA52H2450_5500_A28" H 7700 2500 50  0001 C CNN
+F 3 "" H 7700 2500 50  0001 C CNN
+	1    7700 2500
+	1    0    0    -1
+$EndComp
+NoConn ~ 7500 2750
+Wire Wire Line
+	7700 2750 7700 2850
+Wire Wire Line
+	7900 2750 7900 2850
+$Comp
+L power:GND #PWR0192
+U 1 1 5CDC7C66
+P 7700 2850
+F 0 "#PWR0192" H 7700 2600 50  0001 C CNN
+F 1 "GND" H 7705 2677 50  0000 C CNN
+F 2 "" H 7700 2850 50  0001 C CNN
+F 3 "" H 7700 2850 50  0001 C CNN
+	1    7700 2850
+	1    0    0    -1
+$EndComp
+$Comp
+L power:GND #PWR0217
+U 1 1 5CDC7CAF
+P 7900 2850
+F 0 "#PWR0217" H 7900 2600 50  0001 C CNN
+F 1 "GND" H 7905 2677 50  0000 C CNN
+F 2 "" H 7900 2850 50  0001 C CNN
+F 3 "" H 7900 2850 50  0001 C CNN
+	1    7900 2850
+	1    0    0    -1
+$EndComp
+Text Label 6200 3250 0    50   ~ 0
+RFOUT
 $EndSCHEMATC
