File: hardware/rk3308-io.sch (KiCad schematic (older format))
At the start: 27 parts, among them U1000 RK3308

Commit message: wip
Parts:
- removed DIO1: 1, require:OVAL_PIN, symbol require:OP
- removed DIO10: 10, require:OVAL_PIN, symbol require:OP
- removed DIO19: RX2, require:OVAL_PIN, symbol require:OP
- removed DIO2: 2, require:OVAL_PIN, symbol require:OP
- removed DIO20: TX2, require:OVAL_PIN, symbol require:OP
- removed DIO3: 3, require:OVAL_PIN, symbol require:OP
- removed DIO4: 4, require:OVAL_PIN, symbol require:OP
- removed DIO5: 5, require:OVAL_PIN, symbol require:OP
- removed DIO6: 6, require:OVAL_PIN, symbol require:OP
- removed DIO7: 7, require:OVAL_PIN, symbol require:OP
- removed DIO8: 8, require:OVAL_PIN, symbol require:OP
- removed DIO9: 9, require:OVAL_PIN, symbol require:OP
- removed LP2: A0, require:OVAL_PIN, symbol require:OP
- removed LP3: A1, require:OVAL_PIN, symbol require:OP
- removed LP4: A2, require:OVAL_PIN, symbol require:OP
- removed LP5: A3, require:OVAL_PIN, symbol require:OP
- removed LP6: A4, require:OVAL_PIN, symbol require:OP
- removed LP7: A5, require:OVAL_PIN, symbol require:OP
- removed RP12: 11, require:OVAL_PIN, symbol require:OP
- removed RP13: 12, require:OVAL_PIN, symbol require:OP
- removed RP14: 13, require:OVAL_PIN, symbol require:OP
- removed RP15: 14, require:OVAL_PIN, symbol require:OP
- removed RP16: 15, require:OVAL_PIN, symbol require:OP
- removed RP17: 16, require:OVAL_PIN, symbol require:OP
- removed RP18: 17, require:OVAL_PIN, symbol require:OP
- removed RP19: 18, require:OVAL_PIN, symbol require:OP
- added R4, R5: 22R, Resistors_SMD:R_0402, symbol Device:R
- added R93: 133R,1%, Resistors_SMD:R_0402, symbol Device:R
- added unit 9 of U1000
Connections:
- net labels added: D1, D10, D11, D12, D13, D14, D15, D16, D17, D18, D19, D2, D20, D3, D4, D5, D6, D7, D8, D9, GND, USB_HOST_DM, USB_HOST_DP, USB_OTG_DM, USB_OTG_DP, USB_OTG_ID, USB_OTG_VBUS, VCC_IO
- wire segments 59 -> 76
Other:
- moved on the sheet: U1000E, U1000F, U1000G

Commit message: wip
Parts:
- added R62: 2.2k, Resistors_SMD:R_0402, symbol Device:R
- renumbered R4 to R60, R5 to R61, R93 to R72
Connections:
- net labels added: POWER_SLEEP
- net labels removed: DIO10, DIO3, DIO4, DIO5, DIO6, DIO7, DIO8, DIO9, FLASH_CLK, FLASH_CMD, FLASH_D0, FLASH_D1, FLASH_D2, FLASH_D3, FLASH_D4, FLASH_D5, FLASH_D6, FLASH_D7, PWM1, PWM2, PWM3
- wire segments 76 -> 79
Other:
- moved on the sheet: R72, U1000H, U1000I, U1000J

Commit message: wip
Parts:
- R60, R61, R62, R72: footprint Resistors_SMD:R_0402 -> require:R_0402
Connections:
- net labels removed: D17, D18
- wire segments 79 -> 77
Changed lines of the file:
@@
 Wire Wire Line
 	4100 2100 4950 2100
-Wire Wire Line
-	4100 2200 4950 2200
-Wire Wire Line
-	4100 3200 4950 3200
 $Comp
 L require:RK3308 U1000
@@
 F 0 "R72" V 9500 9750 50  0000 C CNN
 F 1 "133R,1%" V 9700 9750 50  0000 C CNN
-F 2 "Resistors_SMD:R_0402" V 9530 9750 50  0001 C CNN
+F 2 "require:R_0402" V 9530 9750 50  0001 C CNN
 F 3 "~" H 9600 9750 50  0001 C CNN
 	1    9600 9750
@@
 Text HLabel 11350 6250 2    50   Input ~ 0
 D20
-Text HLabel 4950 3200 2    50   Input ~ 0
-D18
-Text HLabel 4950 2200 2    50   Input ~ 0
-D17
 Text HLabel 4950 2100 2    50   Input ~ 0
 D16
@@
 F 0 "R61" H 5850 2200 50  0000 C CNN
 F 1 "22R" H 5850 2300 50  0000 C CNN
-F 2 "Resistors_SMD:R_0402" V 5930 2250 50  0001 C CNN
+F 2 "require:R_0402" V 5930 2250 50  0001 C CNN
 F 3 "~" H 6000 2250 50  0001 C CNN
 	1    6000 2250
@@
 F 0 "R60" H 5450 2200 50  0000 C CNN
 F 1 "22R" H 5450 2300 50  0000 C CNN
-F 2 "Resistors_SMD:R_0402" V 5530 2250 50  0001 C CNN
+F 2 "require:R_0402" V 5530 2250 50  0001 C CNN
 F 3 "~" H 5600 2250 50  0001 C CNN
 	1    5600 2250
@@
 F 0 "R62" V 4350 1700 50  0000 C CNN
 F 1 "2.2k" V 4350 1900 50  0000 C CNN
-F 2 "Resistors_SMD:R_0402" V 4380 1800 50  0001 C CNN
+F 2 "require:R_0402" V 4380 1800 50  0001 C CNN
 F 3 "~" H 4450 1800 50  0001 C CNN
 	1    4450 1800

Commit message: wip
Parts:
- renumbered R61 to R1, R60 to R2
Connections:
- net labels added: +3V3
- net labels removed: POWER_SLEEP, VCC_IO
- wire segments 77 -> 76
- no-connect marks 73 -> 75
Changed lines of the file:
@@
 AR Path="/5C2D00B3/5C80A816" Ref="R?"  Part="1"
 AR Path="/5C80A816" Ref="R?"  Part="1"
-AR Path="/5C87E279/5C80A816" Ref="R61"  Part="1"
-F 0 "R61" H 5850 2200 50  0000 C CNN
+AR Path="/5C87E279/5C80A816" Ref="R1"  Part="1"
+F 0 "R1" H 5850 2200 50  0000 C CNN
 F 1 "22R" H 5850 2300 50  0000 C CNN
 F 2 "require:R_0402" V 5930 2250 50  0001 C CNN
@@
 AR Path="/5C2D00B3/5C80A81D" Ref="R?"  Part="1"
 AR Path="/5C80A81D" Ref="R?"  Part="1"
-AR Path="/5C87E279/5C80A81D" Ref="R60"  Part="1"
-F 0 "R60" H 5450 2200 50  0000 C CNN
+AR Path="/5C87E279/5C80A81D" Ref="R2"  Part="1"
+F 0 "R2" H 5450 2200 50  0000 C CNN
 F 1 "22R" H 5450 2300 50  0000 C CNN
 F 2 "require:R_0402" V 5530 2250 50  0001 C CNN
@@
 	6000 2000 6000 1900
 Connection ~ 6000 2000
-$Comp
-L require:VCC_IO #PWR0227
-U 1 1 5C812416
-P 6000 1900
-F 0 "#PWR0227" H 6000 1750 50  0001 C CNN
-F 1 "VCC_IO" H 6017 2073 50  0000 C CNN
-F 2 "" H 6000 1900 50  0001 C CNN
-F 3 "" H 6000 1900 50  0001 C CNN
-	1    6000 1900
-	1    0    0    -1
-$EndComp
 Wire Wire Line
 	5600 2400 5600 2600
@@
 	0    -1   -1   0
 $EndComp
-Text HLabel 4950 2300 2    50   Input ~ 0
-POWER_SLEEP
-Wire Wire Line
-	4950 2300 4100 2300
 NoConn ~ 4100 2400
+$Comp
+L power:+3V3 #PWR0180
+U 1 1 5C7F6AD8
+P 6000 1900
+F 0 "#PWR0180" H 6000 1750 50  0001 C CNN
+F 1 "+3V3" H 6015 2073 50  0000 C CNN
+F 2 "" H 6000 1900 50  0001 C CNN
+F 3 "" H 6000 1900 50  0001 C CNN
+	1    6000 1900
+	1    0    0    -1
+$EndComp
+NoConn ~ 4100 2200
+NoConn ~ 4100 2300
 $EndSCHEMATC

Commit message: wip
Parts:
- removed R1, R2: 22R, require:R_0402, symbol Device:R
- removed R62: 2.2k, require:R_0402, symbol Device:R
- removed R72: 133R,1%, require:R_0402, symbol Device:R
Connections:
- net USB_EXTR: now reaches U1000.C15 (USB_EXTR)
- net EMMC_VSEL: now reaches U1000.R3 (GPIO0_A4/TEST_CLKOUT_u)
- net D17: now reaches U1000.T1 (GPIO0_C1/SPDIF_TX_d)
- net D18: now reaches U1000.W3 (GPIO0_C2/SPDIF_RX_d)
- no-connect marks 75 -> 73
Changed lines of the file:
@@
 NoConn ~ 4100 3100
 NoConn ~ 4100 3300
-NoConn ~ 4100 3500
-NoConn ~ 4100 3600
 Text HLabel 4950 2700 2    50   Input ~ 0
 CORE_DVS
 Wire Wire Line
 	4100 2700 4950 2700
-Text HLabel 6600 2500 2    50   Input ~ 0
+Text HLabel 4950 2500 2    50   Input ~ 0
 I2C1_SDA
-Text HLabel 6600 2600 2    50   Input ~ 0
+Text HLabel 4950 2600 2    50   Input ~ 0
 I2C1_SCL
-Wire Wire Line
-	4100 2500 6000 2500
-Wire Wire Line
-	4100 2600 5600 2600
 $Comp
 L require:RK3308 U1000
 U 9 1 5C4EF247
 P 8300 9500
-F 0 "U1000" H 8906 10487 60  0000 C CNN
-F 1 "RK3308" H 8906 10381 60  0000 C CNN
+F 0 "U1000" H 8450 10450 60  0000 C CNN
+F 1 "RK3308" H 8450 10350 60  0000 C CNN
 F 2 "" H 8300 13750 60  0001 C CNN
 F 3 "" H 8300 13750 60  0001 C CNN
@@
 Wire Wire Line
 	9500 9300 10400 9300
-$Comp
-L Device:R R?
-U 1 1 5C4FA3AC
-P 9600 9750
-AR Path="/5CED3BD3/5C4FA3AC" Ref="R?"  Part="1"
-AR Path="/5C87E279/5C4FA3AC" Ref="R72"  Part="1"
-F 0 "R72" V 9500 9750 50  0000 C CNN
-F 1 "133R,1%" V 9700 9750 50  0000 C CNN
-F 2 "require:R_0402" V 9530 9750 50  0001 C CNN
-F 3 "~" H 9600 9750 50  0001 C CNN
-	1    9600 9750
-	-1   0    0    1
-$EndComp
-Wire Wire Line
-	9500 9400 9600 9400
-Wire Wire Line
-	9600 9400 9600 9600
-Wire Wire Line
-	9600 9900 9600 10100
-$Comp
-L power:GND #PWR0154
-U 1 1 5C61BAAB
-P 9600 10100
-F 0 "#PWR0154" H 9600 9850 50  0001 C CNN
-F 1 "GND" H 9605 9927 50  0000 C CNN
-F 2 "" H 9600 10100 50  0001 C CNN
-F 3 "" H 9600 10100 50  0001 C CNN
-	1    9600 10100
-	1    0    0    -1
-$EndComp
 Text HLabel 10400 7400 2    50   Input ~ 0
 A0
@@
 Text HLabel 11350 2750 2    50   Input ~ 0
 D2
-$Comp
-L Device:R R?
-U 1 1 5C80A816
-P 6000 2250
-AR Path="/5C2D00B3/5C80A816" Ref="R?"  Part="1"
-AR Path="/5C80A816" Ref="R?"  Part="1"
-AR Path="/5C87E279/5C80A816" Ref="R1"  Part="1"
-F 0 "R1" H 5850 2200 50  0000 C CNN
-F 1 "22R" H 5850 2300 50  0000 C CNN
-F 2 "require:R_0402" V 5930 2250 50  0001 C CNN
-F 3 "~" H 6000 2250 50  0001 C CNN
-	1    6000 2250
-	-1   0    0    1
-$EndComp
-$Comp
-L Device:R R?
-U 1 1 5C80A81D
-P 5600 2250
-AR Path="/5C2D00B3/5C80A81D" Ref="R?"  Part="1"
-AR Path="/5C80A81D" Ref="R?"  Part="1"
-AR Path="/5C87E279/5C80A81D" Ref="R2"  Part="1"
-F 0 "R2" H 5450 2200 50  0000 C CNN
-F 1 "22R" H 5450 2300 50  0000 C CNN
-F 2 "require:R_0402" V 5530 2250 50  0001 C CNN
-F 3 "~" H 5600 2250 50  0001 C CNN
-	1    5600 2250
-	-1   0    0    1
-$EndComp
-Wire Wire Line
-	5600 2100 5600 2000
-Wire Wire Line
-	5600 2000 6000 2000
-Wire Wire Line
-	6000 2000 6000 2100
-Wire Wire Line
-	6000 2000 6000 1900
-Connection ~ 6000 2000
-Wire Wire Line
-	5600 2400 5600 2600
-Connection ~ 5600 2600
-Wire Wire Line
-	5600 2600 6600 2600
-Wire Wire Line
-	6000 2400 6000 2500
-Connection ~ 6000 2500
-Wire Wire Line
-	6000 2500 6600 2500
-$Comp
-L Device:R R?
-U 1 1 5C615982
-P 4450 1800
-AR Path="/5C2D00B3/5C615982" Ref="R?"  Part="1"
-AR Path="/5C615982" Ref="R?"  Part="1"
-AR Path="/5C87E279/5C615982" Ref="R62"  Part="1"
-F 0 "R62" V 4350 1700 50  0000 C CNN
-F 1 "2.2k" V 4350 1900 50  0000 C CNN
-F 2 "require:R_0402" V 4380 1800 50  0001 C CNN
-F 3 "~" H 4450 1800 50  0001 C CNN
-	1    4450 1800
-	0    1    1    0
-$EndComp
-Wire Wire Line
-	4300 1800 4100 1800
-Wire Wire Line
-	4600 1800 4800 1800
-$Comp
-L power:GND #PWR0232
-U 1 1 5C61CEBE
-P 4800 1800
-F 0 "#PWR0232" H 4800 1550 50  0001 C CNN
-F 1 "GND" V 4805 1672 50  0000 R CNN
-F 2 "" H 4800 1800 50  0001 C CNN
-F 3 "" H 4800 1800 50  0001 C CNN
-	1    4800 1800
-	0    -1   -1   0
-$EndComp
 NoConn ~ 4100 2400
-$Comp
-L power:+3V3 #PWR0180
-U 1 1 5C7F6AD8
-P 6000 1900
-F 0 "#PWR0180" H 6000 1750 50  0001 C CNN
-F 1 "+3V3" H 6015 2073 50  0000 C CNN
-F 2 "" H 6000 1900 50  0001 C CNN
-F 3 "" H 6000 1900 50  0001 C CNN
-	1    6000 1900
-	1    0    0    -1
-$EndComp
 NoConn ~ 4100 2200
 NoConn ~ 4100 2300
+Text HLabel 4950 3500 2    50   Input ~ 0
+D17
+Wire Wire Line
+	4950 3500 4100 3500
+Text HLabel 4950 3600 2    50   Input ~ 0
+D18
+Wire Wire Line
+	4100 3600 4950 3600
+Wire Wire Line
+	4100 2500 4950 2500
+Wire Wire Line
+	4100 2600 4950 2600
+Text HLabel 10400 9400 2    50   Input ~ 0
+USB_EXTR
+Wire Wire Line
+	9500 9400 10400 9400
+Wire Wire Line
+	4100 1800 4950 1800
+Text HLabel 4950 1800 2    50   Input ~ 0
+EMMC_VSEL
 $EndSCHEMATC

Commit message: wip
Parts:
- renumbered U1000 to U100
Changed lines of the file:
@@
 $EndDescr
 $Comp
-L require:RK3308 U1000
+L require:RK3308 U100
 U 2 1 5C87ED8E
 P 2500 3700
-F 0 "U1000" H 2700 6300 60  0000 C CNN
+F 0 "U100" H 2700 6300 60  0000 C CNN
 F 1 "RK3308" H 2700 6200 60  0000 C CNN
 F 2 "" H 2500 3700 60  0001 C CNN
@@
 	4100 2100 4950 2100
 $Comp
-L require:RK3308 U1000
+L require:RK3308 U100
 U 3 1 5C8A3C28
 P 900 7000
-F 0 "U1000" H 1100 10000 60  0000 C CNN
+F 0 "U100" H 1100 10000 60  0000 C CNN
 F 1 "RK3308" H 1100 9900 60  0000 C CNN
 F 2 "" H 900 7000 60  0001 C CNN
@@
 	4100 6900 5100 6900
 $Comp
-L require:RK3308 U1000
+L require:RK3308 U100
 U 4 1 5C8B044F
 P 1900 9400
-F 0 "U1000" H 2100 11500 60  0000 C CNN
+F 0 "U100" H 2100 11500 60  0000 C CNN
 F 1 "RK3308" H 2100 11400 60  0000 C CNN
 F 2 "" H 1900 9400 60  0001 C CNN
@@
 	4100 7600 4750 7600
 $Comp
-L require:RK3308 U1000
+L require:RK3308 U100
 U 5 1 5C8BEDB2
 P 8300 2850
-F 0 "U1000" H 8500 4500 60  0000 C CNN
+F 0 "U100" H 8500 4500 60  0000 C CNN
 F 1 "RK3308" H 8500 4400 60  0000 C CNN
 F 2 "" H 8300 2850 60  0001 C CNN
@@
 NoConn ~ 10500 2450
 $Comp
-L require:RK3308 U1000
+L require:RK3308 U100
 U 6 1 5C8D1F22
 P 8300 5350
-F 0 "U1000" H 8500 7500 60  0000 C CNN
+F 0 "U100" H 8500 7500 60  0000 C CNN
 F 1 "RK3308" H 8500 7400 60  0000 C CNN
 F 2 "" H 8300 5350 60  0001 C CNN
@@
 	10500 6250 11350 6250
 $Comp
-L require:RK3308 U1000
+L require:RK3308 U100
 U 7 1 5C8F2A67
 P 8300 6650
-F 0 "U1000" H 8500 7600 60  0000 C CNN
+F 0 "U100" H 8500 7600 60  0000 C CNN
 F 1 "RK3308" H 8500 7500 60  0000 C CNN
 F 2 "" H 8300 6650 60  0001 C CNN
@@
 $EndComp
 $Comp
-L require:RK3308 U1000
+L require:RK3308 U100
 U 8 1 5D7E6903
 P 14100 3900
-F 0 "U1000" H 14500 6700 60  0000 C CNN
+F 0 "U100" H 14500 6700 60  0000 C CNN
 F 1 "RK3308" H 14500 6600 60  0000 C CNN
 F 2 "" H 14100 8150 60  0001 C CNN
@@
 P 8300 8000
 AR Path="/5C325762/5D820AC9" Ref="U?"  Part="10"
-AR Path="/5C87E279/5D820AC9" Ref="U1000"  Part="10"
-F 0 "U1000" H 8600 8900 60  0000 C CNN
+AR Path="/5C87E279/5D820AC9" Ref="U100"  Part="10"
+F 0 "U100" H 8600 8900 60  0000 C CNN
 F 1 "RK3308" H 8600 8800 60  0000 C CNN
 F 2 "" H 8300 8000 60  0001 C CNN
@@
 I2C1_SCL
 $Comp
-L require:RK3308 U1000
+L require:RK3308 U100
 U 9 1 5C4EF247
 P 8300 9500
-F 0 "U1000" H 8450 10450 60  0000 C CNN
+F 0 "U100" H 8450 10450 60  0000 C CNN
 F 1 "RK3308" H 8450 10350 60  0000 C CNN
 F 2 "" H 8300 13750 60  0001 C CNN

Commit message: wip
Connections:
- net RTC_CLK: now reaches U100.Y2 (GPIO0_C3/RTC_CLK)
- no-connect marks 73 -> 72
Changed lines of the file:
@@
 NoConn ~ 4100 1500
 NoConn ~ 4100 1700
-NoConn ~ 4100 3100
 NoConn ~ 4100 3300
 Text HLabel 4950 2700 2    50   Input ~ 0
@@
 Text HLabel 4950 1800 2    50   Input ~ 0
 EMMC_VSEL
+Wire Wire Line
+	4100 3100 4950 3100
+Text HLabel 4950 3100 2    50   Input ~ 0
+RTC_CLK
 $EndSCHEMATC

Commit message: wip
Parts:
- U100: footprint (none) -> require:RK3308_TFBGA-355
Changed lines of the file:
@@
 F 0 "U100" H 2700 6300 60  0000 C CNN
 F 1 "RK3308" H 2700 6200 60  0000 C CNN
-F 2 "" H 2500 3700 60  0001 C CNN
+F 2 "require:RK3308_TFBGA-355" H 2500 3700 60  0001 C CNN
 F 3 "" H 2500 3700 60  0001 C CNN
 	2    2500 3700
@@
 F 0 "U100" H 1100 10000 60  0000 C CNN
 F 1 "RK3308" H 1100 9900 60  0000 C CNN
-F 2 "" H 900 7000 60  0001 C CNN
+F 2 "require:RK3308_TFBGA-355" H 900 7000 60  0001 C CNN
 F 3 "" H 900 7000 60  0001 C CNN
 	3    900  7000
@@
 F 0 "U100" H 2100 11500 60  0000 C CNN
 F 1 "RK3308" H 2100 11400 60  0000 C CNN
-F 2 "" H 1900 9400 60  0001 C CNN
+F 2 "require:RK3308_TFBGA-355" H 1900 9400 60  0001 C CNN
 F 3 "" H 1900 9400 60  0001 C CNN
 	4    1900 9400
@@
 F 0 "U100" H 8500 4500 60  0000 C CNN
 F 1 "RK3308" H 8500 4400 60  0000 C CNN
-F 2 "" H 8300 2850 60  0001 C CNN
+F 2 "require:RK3308_TFBGA-355" H 8300 2850 60  0001 C CNN
 F 3 "" H 8300 2850 60  0001 C CNN
 	5    8300 2850
@@
 F 0 "U100" H 8500 7500 60  0000 C CNN
 F 1 "RK3308" H 8500 7400 60  0000 C CNN
-F 2 "" H 8300 5350 60  0001 C CNN
+F 2 "require:RK3308_TFBGA-355" H 8300 5350 60  0001 C CNN
 F 3 "" H 8300 5350 60  0001 C CNN
 	6    8300 5350
@@
 F 0 "U100" H 8500 7600 60  0000 C CNN
 F 1 "RK3308" H 8500 7500 60  0000 C CNN
-F 2 "" H 8300 6650 60  0001 C CNN
+F 2 "require:RK3308_TFBGA-355" H 8300 6650 60  0001 C CNN
 F 3 "" H 8300 6650 60  0001 C CNN
 	7    8300 6650
@@
 F 0 "U100" H 14500 6700 60  0000 C CNN
 F 1 "RK3308" H 14500 6600 60  0000 C CNN
-F 2 "" H 14100 8150 60  0001 C CNN
+F 2 "require:RK3308_TFBGA-355" H 14100 8150 60  0001 C CNN
 F 3 "" H 14100 8150 60  0001 C CNN
 	8    14100 3900
@@
 F 0 "U100" H 8600 8900 60  0000 C CNN
 F 1 "RK3308" H 8600 8800 60  0000 C CNN
-F 2 "" H 8300 8000 60  0001 C CNN
+F 2 "require:RK3308_TFBGA-355" H 8300 8000 60  0001 C CNN
 F 3 "" H 8300 8000 60  0001 C CNN
 	10   8300 8000
@@
 F 0 "U100" H 8450 10450 60  0000 C CNN
 F 1 "RK3308" H 8450 10350 60  0000 C CNN
-F 2 "" H 8300 13750 60  0001 C CNN
+F 2 "require:RK3308_TFBGA-355" H 8300 13750 60  0001 C CNN
 F 3 "" H 8300 13750 60  0001 C CNN
 	9    8300 9500
