File: hardware/rk3308-io.sch (KiCad schematic (older format))
At the start: 1 part, among them U100 RK3308

Commit message: wip
Connections:
- net D14: no longer names the net of U100.R4 (GPIO0_A5_d)
- net D15: no longer names the net of U100.T5 (GPIO0_A6_d)
- net D16: no longer names the net of U100.T4 (GPIO0_A7_d)
- net D17: no longer names the net of U100.T1 (GPIO0_C1/SPDIF_TX_d)
- net D18: no longer names the net of U100.W3 (GPIO0_C2/SPDIF_RX_d)
- net PCM_CLK: no longer names the net of U100.F18 (GPIO4_B5/I2S0_2CH_SCLK_d)
- net PCM_IN: no longer names the net of U100.H14 (GPIO4_C0/I2S0_2CH_SDI_d)
- net PCM_OUT: no longer names the net of U100.H15 (GPIO4_B7/I2S0_2CH_SDO_d)
- net PCM_SYNC: no longer names the net of U100.J15 (GPIO4_B6/I2S0_2CH_LRCK_TX_d)
- no-connect marks 72 -> 82
Changed lines of the file:
@@
 Wire Wire Line
 	4100 3000 4950 3000
-Wire Wire Line
-	4100 1900 4950 1900
-Wire Wire Line
-	4100 2000 4950 2000
-Wire Wire Line
-	4100 2100 4950 2100
 $Comp
 L require:RK3308 U100
@@
 Text HLabel 11350 4850 2    50   Input ~ 0
 BT_WAKE_HOST
-Text HLabel 11350 4950 2    50   Input ~ 0
-PCM_CLK
-Text HLabel 11350 5050 2    50   Input ~ 0
-PCM_SYNC
-Text HLabel 11350 5150 2    50   Input ~ 0
-PCM_OUT
-Text HLabel 11350 5250 2    50   Input ~ 0
-PCM_IN
 Wire Wire Line
 	10500 4850 11350 4850
-Wire Wire Line
-	10500 4950 11350 4950
-Wire Wire Line
-	10500 5050 11350 5050
-Wire Wire Line
-	10500 5150 11350 5150
-Wire Wire Line
-	10500 5250 11350 5250
 NoConn ~ 10500 5950
 NoConn ~ 10500 6050
@@
 Text HLabel 11350 6250 2    50   Input ~ 0
 D20
-Text HLabel 4950 2100 2    50   Input ~ 0
-D16
-Text HLabel 4950 2000 2    50   Input ~ 0
-D15
-Text HLabel 4950 1900 2    50   Input ~ 0
-D14
 Text HLabel 4950 3000 2    50   Input ~ 0
 D13
@@
 NoConn ~ 4100 2200
 NoConn ~ 4100 2300
-Text HLabel 4950 3500 2    50   Input ~ 0
-D17
-Wire Wire Line
-	4950 3500 4100 3500
-Text HLabel 4950 3600 2    50   Input ~ 0
-D18
-Wire Wire Line
-	4100 3600 4950 3600
 Wire Wire Line
 	4100 2500 4950 2500
@@
 Text HLabel 4950 3100 2    50   Input ~ 0
 RTC_CLK
+NoConn ~ 4100 3500
+NoConn ~ 4100 3600
+NoConn ~ 4100 3200
+NoConn ~ 10500 4950
+NoConn ~ 10500 5050
+NoConn ~ 10500 5150
+NoConn ~ 10500 5250
+NoConn ~ 4100 1900
+NoConn ~ 4100 2000
+NoConn ~ 4100 2100
 $EndSCHEMATC

Commit message: wip
Connections:
- net D1: no longer names the net of U100.W12 (GPIO3_B4/FLASH_RDY/I2C3_SDA_M1/SPI1_MOSI/UART3_RX_u)
- net D10: no longer names the net of U100.T10 (GPIO1_D1/UART1_TX/I2C0_SCL/SPI2_CSN0_u)
- net D11: no longer names the net of U100.W2 (GPIO0_B6/PWM1_d)
- net D12: no longer names the net of U100.W1 (GPIO0_B7/PWM2/I2C3_SDA_M0_d)
- net D13: no longer names the net of U100.U2 (GPIO0_C0/PWM3/I2C3_SCL_M0_d)
- net D2: no longer names the net of U100.T12 (GPIO3_B5/FLASH_CSN0/I2C3_SCL_M1/SPI1_CSN0/UART3_TX_u)
- net D3: no longer names the net of U100.U14 (GPIO2_A0/UART0_RX/SPI0_MISO_u)
- net D4: no longer names the net of U100.V16 (GPIO2_A1/UART0_TX/SPI0_MOSI_u)
- net D5: no longer names the net of U100.Y16 (GPIO2_A2/UART0_CTSN/SPI0_CLK/I2C2_SDA_u)
- net D6: no longer names the net of U100.W16 (GPIO2_A3/UART0_RTSN/SPI0_CSN0/I2C2_SCL_u)
- net D7: no longer names the net of U100.W9 (GPIO1_C6/UART1_CTSN/UART2_RX_M0/SPI2_MISO/JTAG_TCK_u)
- net D8: no longer names the net of U100.T9 (GPIO1_C7/UART1_RTSN/UART2_TX_M0/SPI2_MOSI/JTAG_TMS_u)
- net D9: no longer names the net of U100.V10 (GPIO1_D0/UART1_RX/I2C0_SDA/SPI2_CLK_u)
- no-connect marks 82 -> 94
Changed lines of the file:
@@
 	1    0    0    -1
 $EndComp
-Wire Wire Line
-	4100 2800 4950 2800
-Wire Wire Line
-	4100 2900 4950 2900
-Wire Wire Line
-	4100 3000 4950 3000
 $Comp
 L require:RK3308 U100
@@
 	1    0    0    -1
 $EndComp
-Wire Wire Line
-	4100 6600 5100 6600
-Wire Wire Line
-	4100 6700 5100 6700
-Wire Wire Line
-	4100 6800 5100 6800
-Wire Wire Line
-	4100 6900 5100 6900
 $Comp
 L require:RK3308 U100
@@
 	1    0    0    -1
 $EndComp
-Wire Wire Line
-	4100 7900 4750 7900
-Wire Wire Line
-	4100 7800 4750 7800
-Wire Wire Line
-	4100 7700 4750 7700
-Wire Wire Line
-	4100 7600 4750 7600
 $Comp
 L require:RK3308 U100
@@
 Wire Wire Line
 	10500 2550 11350 2550
-Wire Wire Line
-	10500 2650 11350 2650
-Wire Wire Line
-	10500 2750 11350 2750
 NoConn ~ 10500 2450
 $Comp
@@
 Text HLabel 11350 6250 2    50   Input ~ 0
 D20
-Text HLabel 4950 3000 2    50   Input ~ 0
-D13
-Text HLabel 4950 2900 2    50   Input ~ 0
-D12
-Text HLabel 4950 2800 2    50   Input ~ 0
-D11
-Text HLabel 5100 6900 2    50   Input ~ 0
-D10
-Text HLabel 5100 6800 2    50   Input ~ 0
-D9
-Text HLabel 5100 6700 2    50   Input ~ 0
-D8
-Text HLabel 5100 6600 2    50   Input ~ 0
-D7
-Text HLabel 4750 7900 2    50   Input ~ 0
-D6
-Text HLabel 4750 7800 2    50   Input ~ 0
-D5
-Text HLabel 4750 7700 2    50   Input ~ 0
-D4
-Text HLabel 4750 7600 2    50   Input ~ 0
-D3
-Text HLabel 11350 2650 2    50   Input ~ 0
-D1
-Text HLabel 11350 2750 2    50   Input ~ 0
-D2
 NoConn ~ 4100 2400
 NoConn ~ 4100 2200
@@
 NoConn ~ 4100 2000
 NoConn ~ 4100 2100
+NoConn ~ 4100 2800
+NoConn ~ 4100 2900
+NoConn ~ 4100 3000
+NoConn ~ 4100 6600
+NoConn ~ 4100 6700
+NoConn ~ 4100 6800
+NoConn ~ 4100 6900
+NoConn ~ 4100 7600
+NoConn ~ 4100 7700
+NoConn ~ 4100 7800
+NoConn ~ 4100 7900
+NoConn ~ 10500 2650
 $EndSCHEMATC
